File: Keyboard.kicad_pcb (KiCad board)
At the start: 2 copper layers, 50.8 x 59.5 mm, 39 parts, among them SW1 SW_Push, SW2 SW_Push, SW3 SW_Push, U1 ATmega32U2-AU, Y1 Crystal_GND24_Small

Commit message: complete rewiring
Parts:
- removed C7: 0.1u, Capacitor_SMD:C_0805_2012Metric
- removed F1: Polyfuse_Small, Fuse:Fuse_1206_3216Metric
- moved C2 15.5 mm to (78.1, 86.3), turned to 0 degrees
- moved C3 15.4 mm to (78.1, 80.0), turned to 180 degrees
- moved Y1 14.8 mm to (78.1, 83.1), turned to 90 degrees
- moved D3 11.8 mm to (103.2, 63.4), turned to 90 degrees
- moved D1 11.8 mm to (84.1, 63.4), turned to 90 degrees
- moved R7 10.4 mm to (111.8, 73.7)
- moved D4 5.91 mm to (94.5, 72.5)
- moved D2 2.76 mm to (91.4, 72.5)
- moved SW2 2.05 mm to (92.9, 72.8)
- moved R1 1.99 mm to (101.0, 82.8)
- moved SW3 1.91 mm to (107.2, 72.8)
- moved C6 1.83 mm to (98.8, 86.4)
- moved R4 1.71 mm to (82.4, 76.2)
- moved C4 1.25 mm to (82.4, 72.2)
- moved U1 0.79 mm to (90.5, 83.3)
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Connections:
- USB1 pad 11: Net-(F1-Pad2) -> +5V
- USB1 pad 2: Net-(F1-Pad2) -> +5V
Routing:
- net GND: track 277.6 -> 211.8 mm, vias 5 -> 2
- net +5V: track 306.2 -> 273.3 mm, vias 8 -> 4
- net ROW0: track 52.9 -> 31.7 mm, vias 2 -> 0
- net Net-(F1-Pad2): track 16.1 -> 0.00 mm, vias 2 -> 0
- net COL1: track 52.3 -> 43.0 mm, vias 1 -> 3
- net ROW1: track 16.8 -> 8.51 mm
- net Net-(D5-Pad4): track 10.4 -> 2.40 mm
- net Net-(D4-Pad2): track 4.42 -> 12.3 mm
- net Net-(D1-Pad2): track 3.06 -> 9.98 mm
- net Net-(D3-Pad2): track 3.09 -> 9.98 mm
- net XTAL1: track 15.9 -> 10.7 mm
- net Net-(R3-Pad1): track 11.6 -> 7.07 mm
- net Net-(R2-Pad1): track 10.9 -> 6.87 mm
- net D-: track 45.1 -> 41.1 mm
- net XTAL2: track 8.55 -> 12.0 mm
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
Commit message: Update Keyboard.kicad_pcb
Routing:
- net D+: track 38.1 -> 40.3 mm

Commit message: Update Keyboard.kicad_pcb
Parts:
- turned R2 to 270 degrees
- turned R3 to 270 degrees
Routing:
- net +5V: track 273.3 -> 287.1 mm, vias 4 -> 8
- net GND: track 211.8 -> 223.0 mm
- net Net-(R3-Pad1): track 7.07 -> 8.58 mm
- net Net-(R2-Pad1): track 6.87 -> 8.38 mm
- net Net-(D10-Pad2): track 25.0 -> 23.6 mm, vias 2 -> 0

Commit message: Update Keyboard.kicad_pcb
Routing:
- net COL0: track 45.2 -> 42.5 mm
- net +5V: track 287.1 -> 287.7 mm
- net COL1: track 43.0 -> 43.3 mm, vias 3 -> 2
Changed lines of the file:
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@@
     (thickness 1.6)
     (drawings 8)
-    (tracks 389)
+    (tracks 392)
     (zones 0)
     (modules 37)
@@
   (segment (start 68.2375 76.0625) (end 68.2375 73.79375) (width 0.381) (layer B.Cu) (net 5))
   (segment (start 83.34375 72.23125) (end 83.34375 70.64375) (width 0.381) (layer B.Cu) (net 5))
-  (segment (start 83.34375 70.64375) (end 79.375 70.64375) (width 0.381) (layer B.Cu) (net 5))
   (segment (start 79.375 70.64375) (end 76.2 73.81875) (width 0.381) (layer B.Cu) (net 5))
   (segment (start 76.2 73.81875) (end 74.6125 73.81875) (width 0.381) (layer B.Cu) (net 5))
@@
   (segment (start 93.98124 48.10001) (end 94.45625 47.625) (width 0.381) (layer B.Cu) (net 5))
   (segment (start 86.99376 48.10001) (end 93.98124 48.10001) (width 0.381) (layer B.Cu) (net 5))
+  (segment (start 83.34375 70.64375) (end 82.55 69.85) (width 0.381) (layer B.Cu) (net 5))
+  (segment (start 82.55 69.85) (end 80.16875 69.85) (width 0.381) (layer B.Cu) (net 5))
+  (segment (start 80.16875 69.85) (end 79.375 70.64375) (width 0.381) (layer B.Cu) (net 5))
   (segment (start 83.5025 52.07) (end 83.5025 54.9275) (width 0.254) (layer B.Cu) (net 6))
   (segment (start 84.1375 55.5625) (end 84.1375 61.7875) (width 0.254) (layer B.Cu) (net 6))
@@
   (segment (start 103.1875 55.5625) (end 103.1875 61.7875) (width 0.254) (layer B.Cu) (net 10))
   (segment (start 102.5525 54.9275) (end 103.1875 55.5625) (width 0.254) (layer B.Cu) (net 10))
-  (segment (start 104.13125 70.9125) (end 104.13125 70) (width 0.254) (layer F.Cu) (net 11))
-  (segment (start 104.13125 70) (end 103.1875 69.05625) (width 0.254) (layer F.Cu) (net 11))
-  (via (at 96.04375 69.05625) (size 0.8) (drill 0.4) (layers F.Cu B.Cu) (net 11))
-  (segment (start 103.1875 69.05625) (end 96.04375 69.05625) (width 0.254) (layer F.Cu) (net 11))
   (segment (start 94.488 70.868) (end 94.488 69.81825) (width 0.254) (layer B.Cu) (net 11))
   (segment (start 95.25 69.05625) (end 96.04375 69.05625) (width 0.254) (layer B.Cu) (net 11))
   (segment (start 94.488 69.81825) (end 95.25 69.05625) (width 0.254) (layer B.Cu) (net 11))
+  (segment (start 96.04375 69.05625) (end 101.6 69.05625) (width 0.254) (layer B.Cu) (net 11))
+  (segment (start 101.6 69.05625) (end 103.1875 69.05625) (width 0.254) (layer B.Cu) (net 11))
+  (via (at 103.1875 69.05625) (size 0.8) (drill 0.4) (layers F.Cu B.Cu) (net 11))
+  (segment (start 104.13125 70) (end 104.13125 70.9125) (width 0.254) (layer F.Cu) (net 11))
+  (segment (start 103.1875 69.05625) (end 104.13125 70) (width 0.254) (layer F.Cu) (net 11))
   (via (at 89.69375 76.2) (size 0.8) (drill 0.4) (layers F.Cu B.Cu) (net 12))
   (segment (start 89.6875 76.20625) (end 89.69375 76.2) (width 0.254) (layer B.Cu) (net 12))
   (segment (start 89.6875 77.68125) (end 89.6875 76.20625) (width 0.254) (layer B.Cu) (net 12))
-  (via (at 96.04375 73.025) (size 0.8) (drill 0.4) (layers F.Cu B.Cu) (net 12))
-  (segment (start 96.04375 74.6125) (end 96.04375 73.025) (width 0.254) (layer F.Cu) (net 12))
-  (segment (start 96.04375 73.025) (end 89.69375 73.025) (width 0.254) (layer B.Cu) (net 12))
-  (via (at 89.69375 73.025) (size 0.8) (drill 0.4) (layers F.Cu B.Cu) (net 12))
-  (segment (start 89.69375 73.025) (end 88.9 73.025) (width 0.254) (layer F.Cu) (net 12))
-  (segment (start 88.10625 73.81875) (end 88.10625 76.2) (width 0.254) (layer F.Cu) (net 12))
-  (segment (start 88.10625 76.2) (end 86.51875 76.2) (width 0.254) (layer F.Cu) (net 12))
+  (segment (start 96.04375 74.6125) (end 96.04375 73.81875) (width 0.254) (layer F.Cu) (net 12))
+  (segment (start 96.04375 73.81875) (end 95.25 73.025) (width 0.254) (layer F.Cu) (net 12))
+  (via (at 93.6625 73.025) (size 0.8) (drill 0.4) (layers F.Cu B.Cu) (net 12))
+  (segment (start 95.25 73.025) (end 93.6625 73.025) (width 0.254) (layer F.Cu) (net 12))
+  (via (at 90.4875 73.025) (size 0.8) (drill 0.4) (layers F.Cu B.Cu) (net 12))
+  (segment (start 93.6625 73.025) (end 90.4875 73.025) (width 0.254) (layer B.Cu) (net 12))
+  (segment (start 90.4875 73.025) (end 88.9 73.025) (width 0.254) (layer F.Cu) (net 12))
   (segment (start 88.9 73.025) (end 88.10625 73.81875) (width 0.254) (layer F.Cu) (net 12))
-  (segment (start 89.69375 76.2) (end 88.10625 76.2) (width 0.254) (layer F.Cu) (net 12))
-  (segment (start 86.51875 76.2) (end 85.725 75.40625) (width 0.254) (layer F.Cu) (net 12))
-  (via (at 85.725 74.6125) (size 0.8) (drill 0.4) (layers F.Cu B.Cu) (net 12))
-  (segment (start 85.725 75.40625) (end 85.725 74.6125) (width 0.254) (layer F.Cu) (net 12))
-  (segment (start 85.725 71.4375) (end 85.725 74.6125) (width 0.254) (layer B.Cu) (net 12))
-  (segment (start 79.375 69.85) (end 84.1375 69.85) (width 0.254) (layer B.Cu) (net 12))
-  (segment (start 84.1375 69.85) (end 85.725 71.4375) (width 0.254) (layer B.Cu) (net 12))
-  (segment (start 77.7875 68.2625) (end 79.375 69.85) (width 0.254) (layer B.Cu) (net 12))
-  (segment (start 77.7875 57.15) (end 77.7875 68.2625) (width 0.254) (layer B.Cu) (net 12))
-  (segment (start 77.1525 56.515) (end 77.7875 57.15) (width 0.254) (layer B.Cu) (net 12))
-  (segment (start 77.1525 54.61) (end 77.1525 56.515) (width 0.254) (layer B.Cu) (net 12))
+  (segment (start 88.10625 73.81875) (end 87.3125 74.6125) (width 0.254) (layer F.Cu) (net 12))
+  (segment (start 89.69375 76.2) (end 88.9 76.2) (width 0.254) (layer F.Cu) (net 12))
+  (segment (start 88.9 76.2) (end 87.3125 74.6125) (width 0.254) (layer F.Cu) (net 12))
+  (via (at 85.725 73.81875) (size 0.8) (drill 0.4) (layers F.Cu B.Cu) (net 12))
+  (segment (start 86.51875 74.6125) (end 85.725 73.81875) (width 0.254) (layer F.Cu) (net 12))
+  (segment (start 87.3125 74.6125) (end 86.51875 74.6125) (width 0.254) (layer F.Cu) (net 12))
+  (segment (start 77.1525 56.515) (end 77.1525 54.61) (width 0.254) (layer B.Cu) (net 12))
+  (segment (start 77.7875 57.15) (end 77.1525 56.515) (width 0.254) (layer B.Cu) (net 12))
+  (segment (start 77.7875 68.2625) (end 77.7875 57.15) (width 0.254) (layer B.Cu) (net 12))
+  (segment (start 78.58125 69.05625) (end 77.7875 68.2625) (width 0.254) (layer B.Cu) (net 12))
+  (segment (start 83.34375 69.05625) (end 78.58125 69.05625) (width 0.254) (layer B.Cu) (net 12))
+  (segment (start 84.93125 70.64375) (end 83.34375 69.05625) (width 0.254) (layer B.Cu) (net 12))
+  (segment (start 84.93125 73.025) (end 84.93125 70.64375) (width 0.254) (layer B.Cu) (net 12))
+  (segment (start 85.725 73.81875) (end 84.93125 73.025) (width 0.254) (layer B.Cu) (net 12))
   (segment (start 96.2025 54.61) (end 96.2025 56.515) (width 0.254) (layer B.Cu) (net 13))
   (via (at 96.8375 63.5) (size 0.8) (drill 0.4) (layers F.Cu B.Cu) (net 13))
   (segment (start 96.8375 57.15) (end 96.8375 63.5) (width 0.254) (layer B.Cu) (net 13))
   (segment (start 96.2025 56.515) (end 96.8375 57.15) (width 0.254) (layer B.Cu) (net 13))
-  (via (at 96.8375 66.675) (size 0.8) (drill 0.4) (layers F.Cu B.Cu) (net 13))
-  (segment (start 96.8375 63.5) (end 96.8375 66.675) (width 0.254) (layer F.Cu) (net 13))
-  (segment (start 110.33125 74.6125) (end 108.74375 74.6125) (width 0.254) (layer F.Cu) (net 13))
-  (segment (start 108.74375 74.6125) (end 107.15625 73.025) (width 0.254) (layer F.Cu) (net 13))
-  (segment (start 107.15625 73.025) (end 100.80625 73.025) (width 0.254) (layer F.Cu) (net 13))
   (segment (start 90.4875 77.68125) (end 90.4875 76.2) (width 0.254) (layer B.Cu) (net 13))
   (segment (start 90.4875 76.2) (end 91.28125 75.40625) (width 0.254) (layer B.Cu) (net 13))
   (segment (start 91.28125 75.40625) (end 96.8375 75.40625) (width 0.254) (layer B.Cu) (net 13))
-  (via (at 100.0125 73.025) (size 0.8) (drill 0.4) (layers F.Cu B.Cu) (net 13))
-  (segment (start 99.21875 73.025) (end 100.0125 73.025) (width 0.254) (layer B.Cu) (net 13))
   (segment (start 96.8375 75.40625) (end 99.21875 73.025) (width 0.254) (layer B.Cu) (net 13))
-  (segment (start 100.0125 73.025) (end 100.80625 73.025) (width 0.254) (layer F.Cu) (net 13))
-  (segment (start 99.21875 70.64375) (end 99.21875 73.025) (width 0.254) (layer B.Cu) (net 13))
-  (segment (start 96.8375 68.2625) (end 99.21875 70.64375) (width 0.254) (layer B.Cu) (net 13))
-  (segment (start 96.8375 66.675) (end 96.8375 68.2625) (width 0.254) (layer B.Cu) (net 13))
+  (via (at 99.21875 73.025) (size 0.8) (drill 0.4) (layers F.Cu B.Cu) (net 13))
+  (segment (start 96.8375 63.5) (end 96.8375 68.2625) (width 0.254) (layer F.Cu) (net 13))
+  (segment (start 99.21875 73.025) (end 100.409375 71.834375) (width 0.254) (layer F.Cu) (net 13))
+  (segment (start 100.409375 71.834375) (end 96.8375 68.2625) (width 0.254) (layer F.Cu) (net 13))
+  (segment (start 101.6 73.025) (end 100.409375 71.834375) (width 0.254) (layer F.Cu) (net 13))
+  (segment (start 106.3625 73.025) (end 101.6 73.025) (width 0.254) (layer F.Cu) (net 13))
+  (segment (start 107.95 74.6125) (end 106.3625 73.025) (width 0.254) (layer F.Cu) (net 13))
+  (segment (start 110.33125 74.6125) (end 107.95 74.6125) (width 0.254) (layer F.Cu) (net 13))
   (segment (start 101.01072 81.91372) (end 101.01072 80.69072) (width 0.254) (layer B.Cu) (net 14))
   (segment (start 100.457 80.137) (end 98.9965 80.137) (width 0.254) (layer B.Cu) (net 14))

Commit message: Update Keyboard.kicad_pcb
Parts:
- turned R2 to 90 degrees
- turned R3 to 90 degrees
Routing:
- net Net-(D10-Pad2): track 23.6 -> 25.1 mm, vias 0 -> 2
- net Net-(R3-Pad1): track 8.58 -> 7.66 mm, vias 0 -> 2
- net Net-(R5-Pad2): track 5.40 -> 6.23 mm
- net Net-(R2-Pad1): track 8.38 -> 7.87 mm, vias 0 -> 2
