File: Keyboard.kicad_pcb (KiCad board)
At the start: 2 copper layers, 50.8 x 59.5 mm, 37 parts, among them SW1 SW_Push, SW2 SW_Push, SW3 SW_Push, U1 ATmega32U2-AU, Y1 Crystal_GND24_Small

Commit message: sdfsdsdssdsdsssssdsds
Parts:
- D1, D2, D3, D4: footprint Diode_SMD:D_SOD-123 -> Diode_SMD:D_0805_2012Metric
- H1, H2, H3, H4: footprint MountingHole:MountingHole_2.2mm_M2_DIN965 -> MountingHole:MountingHole_2.7mm_M2.5_DIN965
- U1: footprint Package_QFP:LQFP-44_10x10mm_P0.8mm -> Package_QFP:TQFP-32_7x7mm_P0.8mm
- moved C4 21.4 mm to (98.3, 86.5), turned to 0 degrees
- moved C5 9.42 mm to (90.7, 88.9), turned to 0 degrees
- moved R1 7.69 mm to (101.8, 75.2), turned to 0 degrees
- moved R4 7.64 mm to (83.8, 83.7), turned to 270 degrees
- moved D4 7.39 mm to (101.6, 70.5)
- moved D2 4.59 mm to (87.3, 70.5)
- moved R6 3.81 mm to (92.1, 51.9)
- moved R5 3.81 mm to (88.8, 51.9)
- moved C1 3.24 mm to (97.5, 79.8), turned to 270 degrees
- moved C6 3.19 mm to (97.5, 83.5)
- moved SW1 2.53 mm to (102.8, 80.7), turned to 90 degrees
- moved U1 1.30 mm to (90.5, 82.0), turned to 90 degrees
- moved R7 0.06 mm to (111.9, 73.7)
Connections:
- D11 pad 4: Net-(D10-Pad2) -> Net-(D11-Pad4)
- D5 pad 4: Net-(D5-Pad4) -> Net-(D12-Pad2)
- R7 pad 2: Net-(D5-Pad4) -> Net-(D11-Pad4)
Routing:
- net +5V: track 287.7 -> 0.00 mm, vias 8 -> 0
- net GND: track 223.3 -> 0.00 mm, vias 2 -> 0
- net COL1: track 43.3 -> 0.00 mm, vias 2 -> 0
- net COL0: track 42.5 -> 0.00 mm, vias 4 -> 0
- net D-: track 41.4 -> 0.00 mm, vias 2 -> 0
- net D+: track 40.3 -> 0.00 mm, vias 2 -> 0
- net ROW0: track 31.7 -> 0.00 mm
- net Net-(D10-Pad2): track 25.1 -> 0.00 mm, vias 2 -> 0
- net Net-(D6-Pad2): track 21.8 -> 0.00 mm
- net RGB: track 21.7 -> 0.00 mm
- net Net-(D8-Pad2): track 17.8 -> 0.00 mm
- net Net-(D5-Pad2): track 16.1 -> 0.00 mm
- net Net-(D10-Pad4): track 16.0 -> 0.00 mm
- net Net-(D7-Pad2): track 13.2 -> 0.00 mm
- net Net-(D11-Pad2): track 13.1 -> 0.00 mm
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- added copper zone on B.Cu, net GND

Commit message: Update Keyboard.kicad_pcb
Parts:
- removed C6: 0.1u, Capacitor_SMD:C_0805_2012Metric
- moved C4 3.20 mm to (97.3, 83.5), turned to 90 degrees
- moved R7 1.84 mm to (110.0, 73.6)
- moved R4 1.18 mm to (83.8, 82.5)
- moved C1 0.29 mm to (97.3, 79.9)
Routing:
- net +5V: track 0.00 -> 260.8 mm, vias 0 -> 4
- net COL1: track 0.00 -> 56.2 mm, vias 0 -> 1
- net COL0: track 0.00 -> 49.7 mm, vias 0 -> 1
- net GND: track 0.00 -> 42.8 mm, vias 0 -> 6
- net D-: track 0.00 -> 38.6 mm, vias 0 -> 2
- net D+: track 0.00 -> 37.9 mm, vias 0 -> 2
- net Net-(D11-Pad4): track 0.00 -> 37.4 mm
- net ROW0: track 0.00 -> 37.4 mm
- net ROW1: track 0.00 -> 26.0 mm
- net RGB: track 0.00 -> 24.5 mm
- net XTAL1: track 0.00 -> 23.9 mm, vias 0 -> 2
- net Net-(D6-Pad2): track 0.00 -> 21.8 mm
- net XTAL2: track 0.00 -> 18.1 mm, vias 0 -> 2
- net Net-(D8-Pad2): track 0.00 -> 17.8 mm
- net Net-(D12-Pad2): track 0.00 -> 17.8 mm
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
Commit message: Update Keyboard.kicad_pcb
Routing:
- net GND: track 42.8 -> 41.3 mm
Changed lines of the file:
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@@
     (thickness 1.6)
     (drawings 8)
-    (tracks 302)
+    (tracks 306)
     (zones 0)
     (modules 36)
@@
   (segment (start 98.77925 78.9355) (end 99.21875 79.375) (width 0.381) (layer B.Cu) (net 2))
   (segment (start 97.2566 78.9355) (end 98.77925 78.9355) (width 0.381) (layer B.Cu) (net 2))
-  (via (at 102.39375 81.75625) (size 0.8) (drill 0.4) (layers F.Cu B.Cu) (net 2))
-  (segment (start 101.6 81.75625) (end 102.39375 81.75625) (width 0.381) (layer F.Cu) (net 2))
-  (segment (start 99.21875 79.375) (end 101.6 81.75625) (width 0.381) (layer F.Cu) (net 2))
   (via (at 95.25 87.3125) (size 0.8) (drill 0.4) (layers F.Cu B.Cu) (net 2))
-  (segment (start 93.6625 88.9) (end 95.25 87.3125) (width 0.381) (layer B.Cu) (net 2))
-  (segment (start 91.694 88.9) (end 93.6625 88.9) (width 0.381) (layer B.Cu) (net 2))
   (via (at 99.21875 86.51875) (size 0.8) (drill 0.4) (layers F.Cu B.Cu) (net 2))
   (segment (start 96.04375 86.51875) (end 99.21875 86.51875) (width 0.381) (layer F.Cu) (net 2))
@@
   (segment (start 92.075 80.16875) (end 88.10625 80.16875) (width 0.381) (layer B.Cu) (net 2))
   (segment (start 92.8605 80.95425) (end 92.075 80.16875) (width 0.381) (layer B.Cu) (net 2))
+  (via (at 101.6 81.75625) (size 0.8) (drill 0.4) (layers F.Cu B.Cu) (net 2))
+  (segment (start 99.21875 79.375) (end 101.6 81.75625) (width 0.381) (layer F.Cu) (net 2))
+  (segment (start 86.1675 43.2925) (end 86.1675 43.305) (width 0.381) (layer F.Cu) (net 2))
+  (segment (start 86.1675 43.2925) (end 86.8535 43.2925) (width 0.381) (layer B.Cu) (net 2))
+  (segment (start 87.2625 43.7015) (end 87.2625 44.2075) (width 0.381) (layer B.Cu) (net 2))
+  (segment (start 86.8535 43.2925) (end 87.2625 43.7015) (width 0.381) (layer B.Cu) (net 2))
+  (segment (start 94.8075 43.2925) (end 94.1215 43.2925) (width 0.381) (layer B.Cu) (net 2))
+  (segment (start 93.7125 43.7015) (end 93.7125 44.2075) (width 0.381) (layer B.Cu) (net 2))
+  (segment (start 94.1215 43.2925) (end 93.7125 43.7015) (width 0.381) (layer B.Cu) (net 2))
   (segment (start 77.1144 84.33435) (end 77.216 84.23275) (width 0.254) (layer B.Cu) (net 3))
   (segment (start 77.1144 86.29015) (end 77.1144 84.33435) (width 0.254) (layer B.Cu) (net 3))
@@
   (segment (start 68.25 52.4) (end 69.85 50.8) (width 0.381) (layer B.Cu) (net 5))
   (segment (start 68.25 54.7) (end 68.25 52.4) (width 0.381) (layer B.Cu) (net 5))
-  (segment (start 68.2625 56.35625) (end 68.25 56.34375) (width 0.381) (layer B.Cu) (net 5))
-  (segment (start 66.675 57.94375) (end 68.2625 56.35625) (width 0.381) (layer B.Cu) (net 5))
-  (segment (start 66.675 68.2625) (end 66.675 57.94375) (width 0.381) (layer B.Cu) (net 5))
-  (segment (start 68.25 56.34375) (end 68.25 54.7) (width 0.381) (layer B.Cu) (net 5))
-  (segment (start 68.2375 69.825) (end 66.675 68.2625) (width 0.381) (layer B.Cu) (net 5))
-  (segment (start 68.2375 76.0625) (end 68.2375 69.825) (width 0.381) (layer B.Cu) (net 5))
   (segment (start 68.2375 77.7625) (end 68.2375 76.0625) (width 0.381) (layer B.Cu) (net 5))
   (segment (start 68.2625 77.7875) (end 68.2375 77.7625) (width 0.381) (layer B.Cu) (net 5))
@@
   (segment (start 105.56875 41.4125) (end 105.70625 41.275) (width 0.381) (layer B.Cu) (net 5))
   (segment (start 105.56875 42.8625) (end 105.56875 41.4125) (width 0.381) (layer B.Cu) (net 5))
+  (segment (start 68.2375 69.825) (end 66.675 68.2625) (width 0.381) (layer B.Cu) (net 5))
+  (segment (start 68.2375 76.0625) (end 68.2375 69.825) (width 0.381) (layer B.Cu) (net 5))
+  (segment (start 66.675 68.2625) (end 66.675 57.94375) (width 0.381) (layer B.Cu) (net 5))
+  (segment (start 66.675 57.94375) (end 68.2625 56.35625) (width 0.381) (layer B.Cu) (net 5))
+  (segment (start 68.2625 54.7125) (end 68.25 54.7) (width 0.381) (layer B.Cu) (net 5))
+  (segment (start 68.2625 56.35625) (end 68.2625 54.7125) (width 0.381) (layer B.Cu) (net 5))
   (segment (start 83.5025 52.07) (end 83.5025 55.72125) (width 0.254) (layer B.Cu) (net 6))
   (segment (start 83.5025 55.72125) (end 84.1375 56.35625) (width 0.254) (layer B.Cu) (net 6))
