File: Keyboard.sch (KiCad schematic (older format))
At the start: 39 parts, among them SW1 SW_Push, SW2 SW_Push, SW3 SW_Push, U1 ATmega32U2-AU, Y1 Crystal_GND24_Small

Commit message: complete rewiring
Parts:
- removed C7: 0.1u, Capacitor_SMD:C_0805_2012Metric, symbol Device:C_Small
- removed F1: Polyfuse_Small, Fuse:Fuse_1206_3216Metric, symbol Device:Polyfuse_Small
Connections:
- net +5V: now also USB1.11 (VBUS), USB1.2 (VBUS)
Changed lines of the file:
@@
 Wire Wire Line
 	2550 3100 2550 3750
-$Comp
-L Device:Polyfuse_Small F1
-U 1 1 60B8785D
-P 2550 2900
-F 0 "F1" V 2345 2900 50  0000 C CNN
-F 1 "Polyfuse_Small" V 2650 2900 50  0000 C CNN
-F 2 "Fuse:Fuse_1206_3216Metric" H 2600 2700 50  0001 L CNN
-F 3 "~" H 2550 2900 50  0001 C CNN
-	1    2550 2900
-	0    1    1    0
-$EndComp
-Wire Wire Line
-	2450 2900 2350 2900
 Connection ~ 2350 2900
-Wire Wire Line
-	2650 2900 2750 2900
 Wire Wire Line
 	2750 2900 2750 2800
@@
 Wire Wire Line
 	3750 2200 4000 2200
-Connection ~ 4950 1950
-Wire Wire Line
-	5200 1950 4950 1950
-Wire Wire Line
-	5200 1850 5200 1950
-Connection ~ 4950 1550
-Wire Wire Line
-	5200 1550 4950 1550
-Wire Wire Line
-	5200 1650 5200 1550
-$Comp
-L Device:C_Small C7
-U 1 1 60B08D28
-P 5200 1750
-F 0 "C7" H 5292 1796 50  0000 L CNN
-F 1 "0.1u" H 5292 1705 50  0000 L CNN
-F 2 "Capacitor_SMD:C_0805_2012Metric" H 5200 1750 50  0001 C CNN
-F 3 "~" H 5200 1750 50  0001 C CNN
-	1    5200 1750
-	1    0    0    -1
-$EndComp
 Wire Wire Line
 	3350 1650 3350 2200
@@
 	1    0    0    -1
 $EndComp
+Wire Wire Line
+	2350 2900 2750 2900
 $EndSCHEMATC

Commit message: sdfsdsdssdsdsssssdsds
Parts:
- removed C6: 0.1u, Capacitor_SMD:C_0805_2012Metric, symbol Device:C_Small
- D1, D2, D3, D4: footprint Diode_SMD:D_SOD-123 -> Diode_SMD:D_0805_2012Metric
- H1, H2, H3, H4: footprint MountingHole:MountingHole_2.2mm_M2_DIN965 -> MountingHole:MountingHole_2.7mm_M2.5_DIN965
- U1: footprint Package_QFP:LQFP-44_10x10mm_P0.8mm -> Package_QFP:TQFP-32_7x7mm_P0.8mm
Connections:
- net at D5.4 (DIN): now also D12.2 (DOUT); no longer R7.2
- net at D11.4 (DIN): now also R7.2; no longer D10.2 (DOUT)
Other:
- moved on the sheet: D10, D11, D12, D5, D6, D7, D8, D9
