File: Frooastboard Walnut/KiCad Project/Frooastboard Walnut.kicad_pcb (KiCad board)
At the start: 2 copper layers, 159 parts, among them SW1 SW_Push, U1 ATmega32U4-A, Y1 Crystal_GND24_Small

Commit message: backup
Parts:
- moved C4 3.59 mm to (324.7, 91.2)
- moved C2 3.59 mm to (315.7, 91.2)
- moved C3 3.59 mm to (321.9, 91.2)
- moved R1 3.59 mm to (324.7, 94.8)
- moved SW1 3.59 mm to (329.1, 93.7)
- moved Y1 3.59 mm to (318.8, 91.2)
Connections:
- U1 pad 10: unconnected-(U1-Pad10) -> COL2
- U1 pad 11: unconnected-(U1-Pad11) -> COL3
- U1 pad 12: unconnected-(U1-Pad12) -> RGB
- U1 pad 18: unconnected-(U1-Pad18) -> ROW8
- U1 pad 19: unconnected-(U1-Pad19) -> ROW7
- U1 pad 20: unconnected-(U1-Pad20) -> ROW6
- U1 pad 21: unconnected-(U1-Pad21) -> ROW5
- U1 pad 22: unconnected-(U1-Pad22) -> ROW4
- U1 pad 25: unconnected-(U1-Pad25) -> ROW3
- U1 pad 26: unconnected-(U1-Pad26) -> ROW2
- U1 pad 27: unconnected-(U1-Pad27) -> ROW1
- U1 pad 28: unconnected-(U1-Pad28) -> ROW0
- U1 pad 29: unconnected-(U1-Pad29) -> COL4
- U1 pad 30: unconnected-(U1-Pad30) -> COL5
- U1 pad 31: unconnected-(U1-Pad31) -> COL6
- U1 pad 32: unconnected-(U1-Pad32) -> COL7
- U1 pad 8: unconnected-(U1-Pad8) -> COL0
- U1 pad 9: unconnected-(U1-Pad9) -> COL1
Routing:
- net ROW0: track 142.6 -> 336.6 mm
- net COL0: track 301.9 -> 495.0 mm, vias 2 -> 4
- net COL1: track 305.1 -> 479.5 mm, vias 2 -> 4
- net ROW2: track 147.3 -> 315.1 mm
- net ROW6: track 144.9 -> 301.3 mm
- net ROW4: track 149.7 -> 303.8 mm
- net COL2: track 307.3 -> 454.4 mm, vias 2 -> 4
- net ROW1: track 314.8 -> 174.7 mm
- net COL3: track 359.1 -> 423.7 mm, vias 2 -> 5
- net COL5: track 424.8 -> 376.5 mm, vias 2 -> 5
- net COL7: track 308.4 -> 351.2 mm, vias 2 -> 4
- net ROW7: track 138.9 -> 178.3 mm
- net ROW8: track 271.1 -> 309.1 mm, vias 0 -> 2
- net COL4: track 413.6 -> 382.7 mm, vias 2 -> 5
- net ROW5: track 122.2 -> 150.6 mm
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
Commit message: Update Frooastboard Walnut.kicad_pcb
Parts:
- R3, R4, R5, R6: moved to B.Cu
- moved R3 113.9 mm to (200.0, 22.9), turned to 90 degrees
- moved R6 111.0 mm to (194.5, 27.7), turned to 90 degrees
- moved R4 110.5 mm to (185.7, 22.9), turned to 90 degrees
- moved R5 109.8 mm to (191.3, 27.7), turned to 90 degrees
- moved D6 6.40 mm to (182.6, 26.1)
- moved C1 1.88 mm to (332.6, 77.7)
- moved USB1 0.76 mm to (192.9, 15.0)
Routing:
- net GND: track 98.2 -> 304.6 mm, vias 0 -> 2
- net D+: track 0.00 -> 182.7 mm, vias 0 -> 4
- net D-: track 0.00 -> 182.0 mm, vias 0 -> 4
- net +5V: track 45.2 -> 226.7 mm, vias 0 -> 3
- net ROW1: track 174.7 -> 266.9 mm, vias 0 -> 3
- net ROW5: track 150.6 -> 242.2 mm, vias 0 -> 4
- net ROW7: track 178.3 -> 249.1 mm, vias 0 -> 2
- net COL7: track 351.2 -> 412.3 mm
- net ROW3: track 151.3 -> 210.3 mm, vias 0 -> 3
- net COL5: track 376.5 -> 410.9 mm, vias 5 -> 6
- net COL6: track 367.9 -> 398.4 mm
- net Net-(R3-Pad1): track 0.00 -> 9.05 mm
- net Net-(R4-Pad1): track 0.00 -> 8.77 mm
- net Net-(R6-Pad2): track 0.00 -> 7.61 mm
- net Net-(R5-Pad2): track 0.00 -> 6.56 mm
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
Commit message: Finished Basic Layout
Parts:
- added H1: MountingHole, MountingHole:MountingHole_3.2mm_M3_DIN965, F.Cu at (19.1, 19.1)
- added H2: MountingHole, MountingHole:MountingHole_3.2mm_M3_DIN965, F.Cu at (376.2, 19.1)
- added H3: MountingHole, MountingHole:MountingHole_3.2mm_M3_DIN965, F.Cu at (376.2, 119.1)
- added H4: MountingHole, MountingHole:MountingHole_3.2mm_M3_DIN965, F.Cu at (19.1, 119.1)
Routing:
- net GND: track 304.6 -> 268.2 mm, vias 2 -> 1
- net +5V: track 226.7 -> 209.9 mm, vias 3 -> 2
- net Net-(R3-Pad1): track 9.05 -> 3.80 mm
- net COL2: track 454.4 -> 453.4 mm
Other:
- board outline added: 357.2 x 100 mm

Commit message: Update Frooastboard Walnut.kicad_pcb
Parts:
- moved D6 5.26 mm to (187.2, 28.6), turned to 180 degrees
- moved USB1 2.83 mm to (192.9, 17.8)
- moved R5 2.38 mm to (191.3, 30.0)
- moved R6 2.38 mm to (194.5, 30.0)
Routing:
- net GND: track 268.2 -> 297.7 mm
- net ROW1: track 266.9 -> 295.4 mm
- net +5V: track 209.9 -> 228.1 mm, vias 2 -> 3
- net Net-(R3-Pad1): track 3.80 -> 10.5 mm
- net Net-(D6-Pad2): track 0.00 -> 2.84 mm
- net D-: track 182.0 -> 179.8 mm
- net D+: track 182.7 -> 180.5 mm
- net Net-(R4-Pad1): track 8.77 -> 10.3 mm
- net Net-(R5-Pad2): track 6.56 -> 6.01 mm
- net Net-(R6-Pad2): track 7.61 -> 7.11 mm

Commit message: tqfp -> qfn
Routing:
- added copper zone on B.Cu, net GND
- added copper zone on F.Cu, net GND
Changed lines of the file:
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@@
   (segment (start 194.46875 29.13125) (end 194.46875 28.46875) (width 0.25) (layer "B.Cu") (net 102))
   (segment (start 192.63125 24.56875) (end 192.63125 25.52125) (width 0.25) (layer "B.Cu") (net 102))
+  (zone (net 1) (net_name "GND") (layers F&B.Cu) (hatch edge 0.508)
+    (connect_pads (clearance 0.508))
+    (min_thickness 0.254) (filled_areas_thickness no)
+    (fill yes (thermal_gap 0.508) (thermal_bridge_width 0.508))
+    (polygon
+      (pts
+        (xy 376.2375 119.0625)
+        (xy 19.05 119.0625)
+        (xy 19.05 19.05)
+        (xy 376.2375 19.05)
+      )
+    )
+  )
 )

Commit message: update
Parts:
- added C6: 0.1u, Capacitor_SMD:C_0805_2012Metric, B.Cu at (316.2, 83.0)
- added C7: 0.1u, Capacitor_SMD:C_0805_2012Metric, B.Cu at (329.4, 76.7)
- U1: footprint Package_QFP:TQFP-44_10x10mm_P0.8mm -> Package_DFN_QFN:QFN-44-1EP_7x7mm_P0.5mm_EP5.2x5.2mm
- moved H4 346.7 mm to (364.3, 88.1)
- moved H2 263.6 mm to (127.8, 107.2)
- moved H3 114.3 mm to (311.9, 24.6)
- moved H1 50.3 mm to (24.6, 69.1)
- moved C4 6.49 mm to (324.8, 84.7), turned to 180 degrees
- moved C5 2.36 mm to (319.8, 72.6)
- moved R2 2.31 mm to (315.8, 72.6)
Routing:
- net GND: track 297.7 -> 119.3 mm, vias 1 -> 4
- net +5V: track 228.1 -> 112.2 mm, vias 3 -> 8
- net COL5: track 410.9 -> 415.2 mm
- net RESET: track 14.0 -> 17.8 mm
- net ROW4: track 303.8 -> 306.8 mm
- net COL7: track 412.3 -> 415.2 mm
- net ROW3: track 210.3 -> 213.0 mm
- net COL6: track 398.4 -> 401.1 mm
- net UCAP: track 4.65 -> 7.38 mm
- net ROW6: track 301.3 -> 304.1 mm
- net ROW2: track 315.1 -> 317.8 mm
- net ROW7: track 249.1 -> 251.7 mm
- net ROW8: track 309.1 -> 311.6 mm
- net COL4: track 382.7 -> 385.2 mm
- net ROW1: track 295.4 -> 297.9 mm
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
Commit message: Update Frooastboard Walnut.kicad_pcb
Routing:
- net +5V: track 112.2 -> 272.8 mm, vias 8 -> 10
- net GND: track 119.3 -> 56.3 mm
