File: Frooastboard Walnut/KiCad Project/Frooastboard Walnut.kicad_pcb (KiCad board)
At the start: 2 copper layers, 357.2 x 100 mm, 169 parts, among them SW1 SW_Push, U1 ATmega32U4-A, Y1 Crystal_GND24_Small

Commit message: rename keys
Parts:
- renumbered KEY_SPECIAL5 to KEY_'1, KEY_SPECIAL1 to KEY_-1, KEY_-1 to KEY_/1, KEY_SPECIAL4 to KEY_;1, KEY_SPECIAL2 to KEY_=1, KEY_POS1 to KEY_HOME1, KEY_WIN1 to KEY_LGUI1, KEY_ALTGR1 to KEY_RALT1, KEY_SPECIAL3 to KEY_[1, KEY_<1 to KEY_\1, KEY_+1 to KEY_]1
Changed lines of the file:
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@@
     )
     (pad_to_mask_clearance 0)
+    (grid_origin 19.05 119.0625)
     (pcbplotparams
       (layerselection 0x00010fc_ffffffff)
@@
     (property "Sheetname" "")
     (attr through_hole)
-    (fp_text reference "KEY_-1" (at 0 3.175) (layer "Dwgs.User")
+    (fp_text reference "KEY_/1" (at 0 3.175) (layer "Dwgs.User")
       (effects (font (size 1 1) (thickness 0.15)))
     )
@@
     (property "Sheetname" "")
     (attr through_hole)
-    (fp_text reference "KEY_SPECIAL3" (at 0 3.175) (layer "Dwgs.User")
+    (fp_text reference "KEY_[1" (at 0 3.175) (layer "Dwgs.User")
       (effects (font (size 1 1) (thickness 0.15)))
     )
@@
     (property "Sheetname" "")
     (attr through_hole)
-    (fp_text reference "KEY_SPECIAL4" (at 0 3.175) (layer "Dwgs.User")
+    (fp_text reference "KEY_;1" (at 0 3.175) (layer "Dwgs.User")
       (effects (font (size 1 1) (thickness 0.15)))
     )
@@
     (property "Sheetname" "")
     (attr through_hole)
-    (fp_text reference "KEY_SPECIAL5" (at 0 3.175) (layer "Dwgs.User")
+    (fp_text reference "KEY_'1" (at 0 3.175) (layer "Dwgs.User")
       (effects (font (size 1 1) (thickness 0.15)))
     )
@@
     (property "Sheetname" "")
     (attr through_hole)
-    (fp_text reference "KEY_+1" (at 0 3.175) (layer "Dwgs.User")
+    (fp_text reference "KEY_]1" (at 0 3.175) (layer "Dwgs.User")
       (effects (font (size 1 1) (thickness 0.15)))
     )
@@
     (property "Sheetname" "")
     (attr through_hole)
-    (fp_text reference "KEY_WIN1" (at 0 3.175) (layer "Dwgs.User")
+    (fp_text reference "KEY_LGUI1" (at 0 3.175) (layer "Dwgs.User")
       (effects (font (size 1 1) (thickness 0.15)))
     )
@@
     (property "Sheetname" "")
     (attr through_hole)
-    (fp_text reference "KEY_POS1" (at 0 3.175) (layer "Dwgs.User")
+    (fp_text reference "KEY_HOME1" (at 0 3.175) (layer "Dwgs.User")
       (effects (font (size 1 1) (thickness 0.15)))
     )
@@
     (property "Sheetname" "")
     (attr through_hole)
-    (fp_text reference "KEY_ALTGR1" (at 0 3.175) (layer "Dwgs.User")
+    (fp_text reference "KEY_RALT1" (at 0 3.175) (layer "Dwgs.User")
       (effects (font (size 1 1) (thickness 0.15)))
     )
@@
     (property "Sheetname" "")
     (attr through_hole)
-    (fp_text reference "KEY_<1" (at 0 3.175) (layer "Dwgs.User")
+    (fp_text reference "KEY_\\1" (at 0 3.175) (layer "Dwgs.User")
       (effects (font (size 1 1) (thickness 0.15)))
     )
@@
     (property "Sheetname" "")
     (attr through_hole)
-    (fp_text reference "KEY_SPECIAL1" (at 0 3.175) (layer "Dwgs.User")
+    (fp_text reference "KEY_-1" (at 0 3.175) (layer "Dwgs.User")
       (effects (font (size 1 1) (thickness 0.15)))
     )
@@
     (property "Sheetname" "")
     (attr through_hole)
-    (fp_text reference "KEY_SPECIAL2" (at 0 3.175) (layer "Dwgs.User")
-      (effects (font (size 1 1) (thickness 0.15)))
-    )
+    (fp_text reference "KEY_=1" (at 0 3.175) (layer "Dwgs.User")
+      (effects (font (size 1 1) (thickness 0.15)))
+    )

Commit message: gerber files
Changed lines of the file:
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@@
     (grid_origin 19.05 119.0625)
     (pcbplotparams
-      (layerselection 0x00010fc_ffffffff)
+      (layerselection 0x00010f0_ffffffff)
       (disableapertmacros false)
-      (usegerberextensions false)
-      (usegerberattributes true)
-      (usegerberadvancedattributes true)
-      (creategerberjobfile true)
+      (usegerberextensions true)
+      (usegerberattributes false)
+      (usegerberadvancedattributes false)
+      (creategerberjobfile false)
       (svguseinch false)
       (svgprecision 6)
@@
       (plotinvisibletext false)
       (sketchpadsonfab false)
-      (subtractmaskfromsilk false)
+      (subtractmaskfromsilk true)
       (outputformat 1)
       (mirror false)
-      (drillshape 1)
+      (drillshape 0)
       (scaleselection 1)
-      (outputdirectory "")
+      (outputdirectory "Frooastboard Walnut-gerber/")
     )
   )
@@
     (fp_line (start 1 -0.625) (end -1 -0.625) (layer "B.Fab") (width 0.1))
     (fp_line (start -1 0.625) (end 1 0.625) (layer "B.Fab") (width 0.1))
-    (pad "1" smd roundrect (at -0.9125 0 90) (size 1.025 1.4) (layers "B.Cu" "B.Paste" "B.Mask") (roundrect_rratio 0.243902)
+    (pad "1" smd roundrect (at -0.9125 0 90) (size 1.025 1.4) (layers "B.Cu" "B.Paste" "B.Mask") (roundrect_rratio 0.243902439)
       (net 101 "D+") (pintype "passive"))
-    (pad "2" smd roundrect (at 0.9125 0 90) (size 1.025 1.4) (layers "B.Cu" "B.Paste" "B.Mask") (roundrect_rratio 0.243902)
+    (pad "2" smd roundrect (at 0.9125 0 90) (size 1.025 1.4) (layers "B.Cu" "B.Paste" "B.Mask") (roundrect_rratio 0.243902439)
       (net 102 "Net-(R6-Pad2)") (pintype "passive"))
     (model "${KICAD6_3DMODEL_DIR}/Resistor_SMD.3dshapes/R_0805_2012Metric.wrl"
@@
     (fp_line (start -3.5 2.5) (end -2.5 3.5) (layer "B.Fab") (width 0.1))
     (fp_line (start -3.5 -3.5) (end -3.5 2.5) (layer "B.Fab") (width 0.1))
-    (pad "" smd roundrect (at 1.95 0.65 180) (size 1.05 1.05) (layers "B.Paste") (roundrect_rratio 0.238095))
-    (pad "" smd roundrect (at -0.65 1.95 180) (size 1.05 1.05) (layers "B.Paste") (roundrect_rratio 0.238095))
-    (pad "" smd roundrect (at -0.65 -0.65 180) (size 1.05 1.05) (layers "B.Paste") (roundrect_rratio 0.238095))
-    (pad "" smd roundrect (at 1.95 -1.95 180) (size 1.05 1.05) (layers "B.Paste") (roundrect_rratio 0.238095))
-    (pad "" smd roundrect (at -0.65 0.65 180) (size 1.05 1.05) (layers "B.Paste") (roundrect_rratio 0.238095))
-    (pad "" smd roundrect (at 1.95 -0.65 180) (size 1.05 1.05) (layers "B.Paste") (roundrect_rratio 0.238095))
-    (pad "" smd roundrect (at 0.65 -0.65 180) (size 1.05 1.05) (layers "B.Paste") (roundrect_rratio 0.238095))
-    (pad "" smd roundrect (at -1.95 0.65 180) (size 1.05 1.05) (layers "B.Paste") (roundrect_rratio 0.238095))
-    (pad "" smd roundrect (at -1.95 -1.95 180) (size 1.05 1.05) (layers "B.Paste") (roundrect_rratio 0.238095))
-    (pad "" smd roundrect (at -1.95 -0.65 180) (size 1.05 1.05) (layers "B.Paste") (roundrect_rratio 0.238095))
-    (pad "" smd roundrect (at -1.95 1.95 180) (size 1.05 1.05) (layers "B.Paste") (roundrect_rratio 0.238095))
-    (pad "" smd roundrect (at 0.65 1.95 180) (size 1.05 1.05) (layers "B.Paste") (roundrect_rratio 0.238095))
-    (pad "" smd roundrect (at -0.65 -1.95 180) (size 1.05 1.05) (layers "B.Paste") (roundrect_rratio 0.238095))
-    (pad "" smd roundrect (at 0.65 0.65 180) (size 1.05 1.05) (layers "B.Paste") (roundrect_rratio 0.238095))
-    (pad "" smd roundrect (at 1.95 1.95 180) (size 1.05 1.05) (layers "B.Paste") (roundrect_rratio 0.238095))
-    (pad "" smd roundrect (at 0.65 -1.95 180) (size 1.05 1.05) (layers "B.Paste") (roundrect_rratio 0.238095))
+    (pad "" smd roundrect (at 1.95 0.65 180) (size 1.05 1.05) (layers "B.Paste") (roundrect_rratio 0.2380952381))
+    (pad "" smd roundrect (at -0.65 1.95 180) (size 1.05 1.05) (layers "B.Paste") (roundrect_rratio 0.2380952381))
+    (pad "" smd roundrect (at -0.65 -0.65 180) (size 1.05 1.05) (layers "B.Paste") (roundrect_rratio 0.2380952381))
+    (pad "" smd roundrect (at 1.95 -1.95 180) (size 1.05 1.05) (layers "B.Paste") (roundrect_rratio 0.2380952381))
+    (pad "" smd roundrect (at -0.65 0.65 180) (size 1.05 1.05) (layers "B.Paste") (roundrect_rratio 0.2380952381))
+    (pad "" smd roundrect (at 1.95 -0.65 180) (size 1.05 1.05) (layers "B.Paste") (roundrect_rratio 0.2380952381))
+    (pad "" smd roundrect (at 0.65 -0.65 180) (size 1.05 1.05) (layers "B.Paste") (roundrect_rratio 0.2380952381))
+    (pad "" smd roundrect (at -1.95 0.65 180) (size 1.05 1.05) (layers "B.Paste") (roundrect_rratio 0.2380952381))
+    (pad "" smd roundrect (at -1.95 -1.95 180) (size 1.05 1.05) (layers "B.Paste") (roundrect_rratio 0.2380952381))
+    (pad "" smd roundrect (at -1.95 -0.65 180) (size 1.05 1.05) (layers "B.Paste") (roundrect_rratio 0.2380952381))
+    (pad "" smd roundrect (at -1.95 1.95 180) (size 1.05 1.05) (layers "B.Paste") (roundrect_rratio 0.2380952381))
+    (pad "" smd roundrect (at 0.65 1.95 180) (size 1.05 1.05) (layers "B.Paste") (roundrect_rratio 0.2380952381))
+    (pad "" smd roundrect (at -0.65 -1.95 180) (size 1.05 1.05) (layers "B.Paste") (roundrect_rratio 0.2380952381))
+    (pad "" smd roundrect (at 0.65 0.65 180) (size 1.05 1.05) (layers "B.Paste") (roundrect_rratio 0.2380952381))
+    (pad "" smd roundrect (at 1.95 1.95 180) (size 1.05 1.05) (layers "B.Paste") (roundrect_rratio 0.2380952381))
+    (pad "" smd roundrect (at 0.65 -1.95 180) (size 1.05 1.05) (layers "B.Paste") (roundrect_rratio 0.2380952381))
     (pad "1" smd roundrect (at -3.3375 2.5 180) (size 1.075 0.25) (layers "B.Cu" "B.Paste" "B.Mask") (roundrect_rratio 0.25)
       (net 103 "unconnected-(U1-Pad1)") (pinfunction "PE6") (pintype "bidirectional"))
@@
     (fp_line (start 1 -0.625) (end -1 -0.625) (layer "B.Fab") (width 0.1))
     (fp_line (start -1 0.625) (end 1 0.625) (layer "B.Fab") (width 0.1))
-    (pad "1" smd roundrect (at -0.9125 0 90) (size 1.025 1.4) (layers "B.Cu" "B.Paste" "B.Mask") (roundrect_rratio 0.243902)
+    (pad "1" smd roundrect (at -0.9125 0 90) (size 1.025 1.4) (layers "B.Cu" "B.Paste" "B.Mask") (roundrect_rratio 0.243902439)
       (net 97 "Net-(R3-Pad1)") (pintype "passive"))
-    (pad "2" smd roundrect (at 0.9125 0 90) (size 1.025 1.4) (layers "B.Cu" "B.Paste" "B.Mask") (roundrect_rratio 0.243902)
+    (pad "2" smd roundrect (at 0.9125 0 90) (size 1.025 1.4) (layers "B.Cu" "B.Paste" "B.Mask") (roundrect_rratio 0.243902439)
       (net 1 "GND") (pintype "passive"))
     (model "${KICAD6_3DMODEL_DIR}/Resistor_SMD.3dshapes/R_0805_2012Metric.wrl"
@@
     (fp_line (start -1 -0.625) (end -1 0.625) (layer "B.Fab") (width 0.1))
     (fp_line (start 1 -0.625) (end -1 -0.625) (layer "B.Fab") (width 0.1))
-    (pad "1" smd roundrect (at -0.9125 0 90) (size 1.025 1.4) (layers "B.Cu" "B.Paste" "B.Mask") (roundrect_rratio 0.243902)
+    (pad "1" smd roundrect (at -0.9125 0 90) (size 1.025 1.4) (layers "B.Cu" "B.Paste" "B.Mask") (roundrect_rratio 0.243902439)
       (net 98 "Net-(R4-Pad1)") (pintype "passive"))
-    (pad "2" smd roundrect (at 0.9125 0 90) (size 1.025 1.4) (layers "B.Cu" "B.Paste" "B.Mask") (roundrect_rratio 0.243902)
+    (pad "2" smd roundrect (at 0.9125 0 90) (size 1.025 1.4) (layers "B.Cu" "B.Paste" "B.Mask") (roundrect_rratio 0.243902439)
       (net 1 "GND") (pintype "passive"))
     (model "${KICAD6_3DMODEL_DIR}/Resistor_SMD.3dshapes/R_0805_2012Metric.wrl"
@@
     (fp_line (start -1 -0.625) (end -1 0.625) (layer "B.Fab") (width 0.1))
     (fp_line (start -1 0.625) (end 1 0.625) (layer "B.Fab") (width 0.1))
-    (pad "1" smd roundrect (at -0.9125 0) (size 1.025 1.4) (layers "B.Cu" "B.Paste" "B.Mask") (roundrect_rratio 0.243902)
+    (pad "1" smd roundrect (at -0.9125 0) (size 1.025 1.4) (layers "B.Cu" "B.Paste" "B.Mask") (roundrect_rratio 0.243902439)
       (net 96 "HWB") (pintype "passive"))
-    (pad "2" smd roundrect (at 0.9125 0) (size 1.025 1.4) (layers "B.Cu" "B.Paste" "B.Mask") (roundrect_rratio 0.243902)
+    (pad "2" smd roundrect (at 0.9125 0) (size 1.025 1.4) (layers "B.Cu" "B.Paste" "B.Mask") (roundrect_rratio 0.243902439)
       (net 1 "GND") (pintype "passive"))
     (model "${KICAD6_3DMODEL_DIR}/Resistor_SMD.3dshapes/R_0805_2012Metric.wrl"
@@
     (fp_line (start 1 -0.625) (end -1 -0.625) (layer "B.Fab") (width 0.1))
     (fp_line (start -1 0.625) (end 1 0.625) (layer "B.Fab") (width 0.1))
-    (pad "1" smd roundrect (at -0.9125 0 90) (size 1.025 1.4) (layers "B.Cu" "B.Paste" "B.Mask") (roundrect_rratio 0.243902)
+    (pad "1" smd roundrect (at -0.9125 0 90) (size 1.025 1.4) (layers "B.Cu" "B.Paste" "B.Mask") (roundrect_rratio 0.243902439)
       (net 95 "RESET") (pintype "passive"))
-    (pad "2" smd roundrect (at 0.9125 0 90) (size 1.025 1.4) (layers "B.Cu" "B.Paste" "B.Mask") (roundrect_rratio 0.243902)
+    (pad "2" smd roundrect (at 0.9125 0 90) (size 1.025 1.4) (layers "B.Cu" "B.Paste" "B.Mask") (roundrect_rratio 0.243902439)
       (net 5 "+5V") (pintype "passive"))
     (model "${KICAD6_3DMODEL_DIR}/Resistor_SMD.3dshapes/R_0805_2012Metric.wrl"
@@
     (fp_line (start -1 0.625) (end 1 0.625) (layer "B.Fab") (width 0.1))
     (fp_line (start 1 -0.625) (end -1 -0.625) (layer "B.Fab") (width 0.1))
-    (pad "1" smd roundrect (at -0.9125 0 90) (size 1.025 1.4) (layers "B.Cu" "B.Paste" "B.Mask") (roundrect_rratio 0.243902)
+    (pad "1" smd roundrect (at -0.9125 0 90) (size 1.025 1.4) (layers "B.Cu" "B.Paste" "B.Mask") (roundrect_rratio 0.243902439)
       (net 99 "D-") (pintype "passive"))
-    (pad "2" smd roundrect (at 0.9125 0 90) (size 1.025 1.4) (layers "B.Cu" "B.Paste" "B.Mask") (roundrect_rratio 0.243902)
+    (pad "2" smd roundrect (at 0.9125 0 90) (size 1.025 1.4) (layers "B.Cu" "B.Paste" "B.Mask") (roundrect_rratio 0.243902439)
       (net 100 "Net-(R5-Pad2)") (pintype "passive"))
     (model "${KICAD6_3DMODEL_DIR}/Resistor_SMD.3dshapes/R_0805_2012Metric.wrl"

Commit message: iso ansi support
Schematic: Switches are double stacked!
Parts:
- added KEY_#2: MX-NoLED, MX_Only:MXOnly-1.5U-NoLED, F.Cu at (292.9, 50.0)
- added KEY_ENTER2: MX-NoLED, MX_Only:MXOnly-2.25U-NoLED, F.Cu at (285.8, 69.1)
- added KEY_LSHIFT2: MX-NoLED, MX_Only:MXOnly-2.25U-NoLED, F.Cu at (42.9, 88.1)
- KEY_ENTER1: footprint MX_Only:MXOnly-ISO-NoLED -> MX_Only:MXOnly-ISO-NoLED-NoStabilizers
- moved D4 3.18 mm to (42.1, 84.1)
- moved D52 1.30 mm to (300.8, 54.1), turned to -90 degrees
- moved D44 0.25 mm to (279.1, 64.9)
Routing:
- net Net-(D44-Pad2): track 3.03 -> 38.3 mm, vias 0 -> 2
- net Net-(D52-Pad2): track 3.03 -> 27.0 mm
- net COL4: track 385.2 -> 408.8 mm, vias 5 -> 6
- net COL5: track 415.2 -> 428.3 mm
- net COL0: track 495.7 -> 505.5 mm
- net Net-(D4-Pad2): track 3.03 -> 9.67 mm
- net ROW3: track 213.0 -> 216.7 mm
- net COL1: track 480.5 -> 483.7 mm
- net ROW2: track 317.8 -> 319.7 mm
- net ROW0: track 339.0 -> 341.0 mm
- net ROW6: track 304.1 -> 302.5 mm
- net ROW4: track 306.8 -> 308.3 mm
- net ROW5: track 243.7 -> 245.0 mm
