File: Frooastboard Walnut/KiCad Project/Frooastboard Walnut.kicad_sch (KiCad schematic)
At the start: 169 parts, among them SW1 SW_Push, U1 ATmega32U4-A, Y1 Crystal_GND24_Small

Commit message: iso ansi support
Schematic: Switches are double stacked!
Parts:
- added KEY_#2: MX-NoLED, MX_Only:MXOnly-1.5U-NoLED, symbol MX_Alps_Hybrid:MX-NoLED
- added KEY_ENTER2, KEY_LSHIFT2: MX-NoLED, MX_Only:MXOnly-2.25U-NoLED, symbol MX_Alps_Hybrid:MX-NoLED
- KEY_ENTER1: footprint MX_Only:MXOnly-ISO-NoLED -> MX_Only:MXOnly-ISO-NoLED-NoStabilizers
Connections:
- net COL0: now also KEY_LSHIFT2.1 (COL)
- net COL4: now also KEY_#2.1 (COL)
- net COL5: now also KEY_ENTER2.1 (COL)
- net at D52.2 (A), KEY_ENTER1.2 (ROW): now also KEY_ENTER2.2 (ROW)
- net at D4.2 (A), KEY_LSHIFT1.2 (ROW): now also KEY_LSHIFT2.2 (ROW)
- net at D44.2 (A), KEY_#1.2 (ROW): now also KEY_#2.2 (ROW)
Other:
- moved on the sheet: FID1, FID2, FID3, FID4, H1, H2, H3, H4

Commit message: rotate iso enter switch
Parts:
- KEY_ENTER1: footprint MX_Only:MXOnly-ISO-NoLED-NoStabilizers -> MX_Only:MXOnly-ISO-ROTATED-NoLED-NoStabilizers
Changed lines of the file:
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@@
       (effects (font (size 0.508 0.508)))
     )
-    (property "Footprint" "MX_Only:MXOnly-ISO-NoLED-NoStabilizers" (id 2) (at 113.665 131.445 0)
+    (property "Footprint" "MX_Only:MXOnly-ISO-ROTATED-NoLED-NoStabilizers" (id 2) (at 113.665 131.445 0)
       (effects (font (size 1.524 1.524)) hide)
     )
@@
     )
     (path "/53c8ac3c-456e-47c9-a6eb-2ee6377474f4"
-      (reference "KEY_ENTER1") (unit 1) (value "MX-NoLED") (footprint "MX_Only:MXOnly-ISO-NoLED-NoStabilizers")
+      (reference "KEY_ENTER1") (unit 1) (value "MX-NoLED") (footprint "MX_Only:MXOnly-ISO-ROTATED-NoLED-NoStabilizers")
     )
     (path "/fbda3cca-a5fe-4f20-8515-486859fc314e"

Commit message: Mounting Holes
Parts:
- removed FID1, FID2: Fiducial, Fiducial:Fiducial_1mm_Mask2mm, symbol Mechanical:Fiducial
- added H10, H11, H12, H5, H6, H7, H8, H9, H?: MountingHole, MountingHole:MountingHole_3.2mm_M3_DIN965, symbol Mechanical:MountingHole
Other:
- moved on the sheet: FID3, FID4, H1, H2, H3, H4

Commit message: annotation
Parts:
- gave numbers to parts that had none: 1
Changed lines of the file:
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@@
   (symbol (lib_id "Mechanical:MountingHole") (at 190.5 154.94 0) (unit 1)
     (in_bom yes) (on_board yes)
-    (property "Reference" "H?" (id 0) (at 193.04 153.6699 0)
+    (property "Reference" "H13" (id 0) (at 193.04 153.6699 0)
       (effects (font (size 1.27 1.27)) (justify left))
     )
@@
     )
     (path "/8ec3d026-51c1-4763-8906-c03bd74f44cf"
-      (reference "H?") (unit 1) (value "MountingHole") (footprint "MountingHole:MountingHole_3.2mm_M3_DIN965")
+      (reference "H13") (unit 1) (value "MountingHole") (footprint "MountingHole:MountingHole_3.2mm_M3_DIN965")
     )
     (path "/c8f17c30-a4f6-46fa-aabd-8086ab44b007"

Commit message: backup
Parts:
- added U?: IS31FL3737, Package_DFN_QFN:QFN-40-1EP_5x5mm_P0.4mm_EP3.8x3.8mm, symbol Driver_LED:IS31FL3737
Connections:
- new net: U?.11 (PGND), U?.4 (PGND)
- new net: U?.40 (GND), U?.41 (GND)
- no-connect marks 0 -> 1
Changed lines of the file:
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@@
   (junction (at 100.33 157.48) (diameter 0) (color 0 0 0 0)
   )
+  (no_connect (at 78.74 57.15))
   (wire (pts (xy 24.13 121.92) (xy 24.13 120.65))
     (stroke (width 0) (type default) (color 0 0 0 0))
@@
     (pin "2")
   )
+  (symbol (lib_id "Driver_LED:IS31FL3737") (at 35.56 55.88 0) (unit 1)
+    (in_bom yes) (on_board yes) (fields_autoplaced)
+    (property "Reference" "U?" (id 0) (at 42.6594 17.78 0)
+      (effects (font (size 1.27 1.27)) (justify left))
+    )
+    (property "Value" "IS31FL3737" (id 1) (at 42.6594 20.32 0)
+      (effects (font (size 1.27 1.27)) (justify left))
+    )
+    (property "Footprint" "Package_DFN_QFN:QFN-40-1EP_5x5mm_P0.4mm_EP3.8x3.8mm" (id 2) (at 35.56 55.88 0)
+      (effects (font (size 1.27 1.27)) hide)
+    )
+    (property "Datasheet" "http://www.issi.com/WW/pdf/31FL3737.pdf" (id 3) (at 35.56 55.88 0)
+      (effects (font (size 1.27 1.27)) hide)
+    )
+    (pin "1")
+    (pin "10")
+    (pin "11")
+    (pin "12")
+    (pin "13")
+    (pin "14")
+    (pin "15")
+    (pin "16")
+    (pin "17")
+    (pin "18")
+    (pin "19")
+    (pin "2")
+    (pin "20")
+    (pin "21")
+    (pin "22")
+    (pin "23")
+    (pin "24")
+    (pin "25")
+    (pin "26")
+    (pin "27")
+    (pin "28")
+    (pin "29")
+    (pin "3")
+    (pin "30")
+    (pin "31")
+    (pin "32")
+    (pin "33")
+    (pin "34")
+    (pin "35")
+    (pin "36")
+    (pin "37")
+    (pin "38")
+    (pin "39")
+    (pin "4")
+    (pin "40")
+    (pin "41")
+    (pin "5")
+    (pin "6")
+    (pin "7")
+    (pin "8")
+    (pin "9")
+  )
   (symbol (lib_id "Device:D_Small") (at 138.43 153.67 90) (unit 1)
     (in_bom yes) (on_board yes) (fields_autoplaced)
@@
       (reference "U1") (unit 1) (value "ATmega32U4-A") (footprint "Package_DFN_QFN:QFN-44-1EP_7x7mm_P0.5mm_EP5.2x5.2mm")
     )
+    (path "/9189e55c-3f50-4101-8ec0-b008b5a37edd"
+      (reference "U?") (unit 1) (value "IS31FL3737") (footprint "Package_DFN_QFN:QFN-40-1EP_5x5mm_P0.4mm_EP3.8x3.8mm")
+    )
     (path "/aab2d817-6308-4a4a-beb4-4d42d4203987"

Commit message: smd rgb led
Parts:
- added C10, C9: 0.1u, Capacitor_SMD:C_0805_2012Metric, symbol Device:C_Small
- added C8: 10u, Capacitor_SMD:C_0805_2012Metric, symbol Device:C_Small
- gave numbers to parts that had none: 1
Connections:
- net +5V: now also U2.19 (PVCC), U2.26 (PVCC), U2.31 (VCC), C10.1, C8.1, C9.1
- net GND: now also U2.36 (ADDR), U2.40 (GND), U2.41 (GND), C10.2, C8.2, C9.2
- net ROW7: now also U1.40 (PF1); no longer U1.19 (PD1)
- net ROW8: now also U1.41 (PF0); no longer U1.18 (PD0)
- net SW1: now reaches U2.1 (SW1)
- net SW9: now reaches U2.10 (SW9)
- net at U2.11 (PGND), U2.4 (PGND): now also U2.29 (AGND)
- net SW10: now reaches U2.12 (SW10)
- net SW11: now reaches U2.13 (SW11)
- net SW12: now reaches U2.14 (SW12)
- net CS1: now reaches U2.15 (CS1)
- net CS2: now reaches U2.16 (CS2)
- net CS3: now reaches U2.17 (CS3)
- net CS4: now reaches U2.18 (CS4)
- net SW2: now reaches U2.2 (SW2)
- net CS5: now reaches U2.20 (CS5)
- net CS6: now reaches U2.21 (CS6)
- net CS7: now reaches U2.22 (CS7)
- net CS8: now reaches U2.23 (CS8)
- net CS9: now reaches U2.24 (CS9)
- net CS10: now reaches U2.25 (CS10)
- net CS11: now reaches U2.27 (CS11)
- net CS12: now reaches U2.28 (CS12)
- net SW3: now reaches U2.3 (SW3)
- net SDA: now reaches U2.34 (SDA)
- net SDA: now also U1.19 (PD1)
- net SCL: now reaches U2.35 (SCL)
- net SCL: now also U1.18 (PD0)
- net SW4: now reaches U2.5 (SW4)
- net SW5: now reaches U2.6 (SW5)
- net SW6: now reaches U2.7 (SW6)
- net SW7: now reaches U2.8 (SW7)
- net SW8: now reaches U2.9 (SW8)
- no-connect marks 1 -> 0
Other:
- moved on the sheet: C1, C2, C3, C4, C5, C6, C7, D1, D10, D11, D12, D13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

Commit message: led schematic
Parts:
- added D? (x48): RGB_LED_6_Pin, symbol Frooastboard Symbols:RGB_LED_6_Pin
Connections:
- net CS1: now also D?.2 (G+), D?.2 (G+), D?.2 (G+), D?.2 (G+), D?.4 (R+), D?.4 (R+), D?.4 (R+), D?.4 (R+), D?.6 (B+), D?.6 (B+), D?.6 (B+), D?.6 (B+)
- net CS10: now also D?.2 (G+), D?.2 (G+), D?.2 (G+), D?.2 (G+), D?.4 (R+), D?.4 (R+), D?.4 (R+), D?.4 (R+), D?.6 (B+), D?.6 (B+), D?.6 (B+), D?.6 (B+)
- net CS11: now also D?.2 (G+), D?.2 (G+), D?.2 (G+), D?.2 (G+), D?.4 (R+), D?.4 (R+), D?.4 (R+), D?.4 (R+), D?.6 (B+), D?.6 (B+), D?.6 (B+), D?.6 (B+)
- net CS12: now also D?.2 (G+), D?.2 (G+), D?.2 (G+), D?.2 (G+), D?.4 (R+), D?.4 (R+), D?.4 (R+), D?.4 (R+), D?.6 (B+), D?.6 (B+), D?.6 (B+), D?.6 (B+)
- net CS2: now also D?.2 (G+), D?.2 (G+), D?.2 (G+), D?.2 (G+), D?.4 (R+), D?.4 (R+), D?.4 (R+), D?.4 (R+), D?.6 (B+), D?.6 (B+), D?.6 (B+), D?.6 (B+)
- net CS3: now also D?.2 (G+), D?.2 (G+), D?.2 (G+), D?.2 (G+), D?.4 (R+), D?.4 (R+), D?.4 (R+), D?.4 (R+), D?.6 (B+), D?.6 (B+), D?.6 (B+), D?.6 (B+)
- net CS4: now also D?.2 (G+), D?.2 (G+), D?.2 (G+), D?.2 (G+), D?.4 (R+), D?.4 (R+), D?.4 (R+), D?.4 (R+), D?.6 (B+), D?.6 (B+), D?.6 (B+), D?.6 (B+)
- net CS5: now also D?.2 (G+), D?.2 (G+), D?.2 (G+), D?.2 (G+), D?.4 (R+), D?.4 (R+), D?.4 (R+), D?.4 (R+), D?.6 (B+), D?.6 (B+), D?.6 (B+), D?.6 (B+)
- net CS6: now also D?.2 (G+), D?.2 (G+), D?.2 (G+), D?.2 (G+), D?.4 (R+), D?.4 (R+), D?.4 (R+), D?.4 (R+), D?.6 (B+), D?.6 (B+), D?.6 (B+), D?.6 (B+)
- net CS7: now also D?.2 (G+), D?.2 (G+), D?.2 (G+), D?.2 (G+), D?.4 (R+), D?.4 (R+), D?.4 (R+), D?.4 (R+), D?.6 (B+), D?.6 (B+), D?.6 (B+), D?.6 (B+)
- net CS8: now also D?.2 (G+), D?.2 (G+), D?.2 (G+), D?.2 (G+), D?.4 (R+), D?.4 (R+), D?.4 (R+), D?.4 (R+), D?.6 (B+), D?.6 (B+), D?.6 (B+), D?.6 (B+)
- net CS9: now also D?.2 (G+), D?.2 (G+), D?.2 (G+), D?.2 (G+), D?.4 (R+), D?.4 (R+), D?.4 (R+), D?.4 (R+), D?.6 (B+), D?.6 (B+), D?.6 (B+), D?.6 (B+)
- net SW1: now also D?.1 (G-), D?.1 (G-), D?.1 (G-), D?.1 (G-), D?.1 (G-), D?.1 (G-), D?.1 (G-), D?.1 (G-), D?.1 (G-), D?.1 (G-), D?.1 (G-), D?.1 (G-)
- net SW10: now also D?.1 (G-), D?.1 (G-), D?.1 (G-), D?.1 (G-), D?.1 (G-), D?.1 (G-), D?.1 (G-), D?.1 (G-), D?.1 (G-), D?.1 (G-), D?.1 (G-), D?.1 (G-)
- net SW11: now also D?.3 (R-), D?.3 (R-), D?.3 (R-), D?.3 (R-), D?.3 (R-), D?.3 (R-), D?.3 (R-), D?.3 (R-), D?.3 (R-), D?.3 (R-), D?.3 (R-), D?.3 (R-)
- net SW12: now also D?.5 (B-), D?.5 (B-), D?.5 (B-), D?.5 (B-), D?.5 (B-), D?.5 (B-), D?.5 (B-), D?.5 (B-), D?.5 (B-), D?.5 (B-), D?.5 (B-), D?.5 (B-)
- net SW2: now also D?.3 (R-), D?.3 (R-), D?.3 (R-), D?.3 (R-), D?.3 (R-), D?.3 (R-), D?.3 (R-), D?.3 (R-), D?.3 (R-), D?.3 (R-), D?.3 (R-), D?.3 (R-)
- net SW3: now also D?.5 (B-), D?.5 (B-), D?.5 (B-), D?.5 (B-), D?.5 (B-), D?.5 (B-), D?.5 (B-), D?.5 (B-), D?.5 (B-), D?.5 (B-), D?.5 (B-), D?.5 (B-)
- net SW4: now also D?.1 (G-), D?.1 (G-), D?.1 (G-), D?.1 (G-), D?.1 (G-), D?.1 (G-), D?.1 (G-), D?.1 (G-), D?.1 (G-), D?.1 (G-), D?.1 (G-), D?.1 (G-)
- net SW5: now also D?.3 (R-), D?.3 (R-), D?.3 (R-), D?.3 (R-), D?.3 (R-), D?.3 (R-), D?.3 (R-), D?.3 (R-), D?.3 (R-), D?.3 (R-), D?.3 (R-), D?.3 (R-)
- net SW6: now also D?.5 (B-), D?.5 (B-), D?.5 (B-), D?.5 (B-), D?.5 (B-), D?.5 (B-), D?.5 (B-), D?.5 (B-), D?.5 (B-), D?.5 (B-), D?.5 (B-), D?.5 (B-)
- net SW7: now also D?.1 (G-), D?.1 (G-), D?.1 (G-), D?.1 (G-), D?.1 (G-), D?.1 (G-), D?.1 (G-), D?.1 (G-), D?.1 (G-), D?.1 (G-), D?.1 (G-), D?.1 (G-)
- net SW8: now also D?.3 (R-), D?.3 (R-), D?.3 (R-), D?.3 (R-), D?.3 (R-), D?.3 (R-), D?.3 (R-), D?.3 (R-), D?.3 (R-), D?.3 (R-), D?.3 (R-), D?.3 (R-)
- net SW9: now also D?.5 (B-), D?.5 (B-), D?.5 (B-), D?.5 (B-), D?.5 (B-), D?.5 (B-), D?.5 (B-), D?.5 (B-), D?.5 (B-), D?.5 (B-), D?.5 (B-), D?.5 (B-)
Other:
- moved on the sheet: C10, C8, C9, U2
