File: Frooastboard Walnut Modular/KiCad Project/Frooastboard Walnut Modular.kicad_sch (KiCad schematic)
At the start: 90 parts, among them J1 SW Interface, J2 Conn_01x16, J3 Conn_01x06, J4 Conn_01x06, J5 Conn_01x10, J6 Conn_01x12, J7 Conn_01x04, U1 RP2040, U2 SPX3819M5-L-3-3, U3 W25Q32JVZP, U4 nRF8001, U5 IS31FL3733-QF, U6 FS312F-G, U7 FS8205, U8 IP2312, Y1 32.768kHz, Y2 16MHz, Y3 12MHz

Commit message: some new stuff
Parts:
- removed U?: nRF52810-QCxx, Package_DFN_QFN:QFN-32-1EP_5x5mm_P0.5mm_EP3.6x3.6mm, symbol MCU_Nordic:nRF52810-QCxx
- BT1: footprint (none) -> TestPoint:TestPoint_Pad_D1.5mm
- C30, C32, C36, C37: footprint (none) -> Capacitor_SMD:C_0805_2012Metric
- D1, D2: footprint (none) -> LED_SMD:LED_0805_2012Metric
- J2: footprint (none) -> Frooastboard Footprints:PinHeader_1x16_P1.27mm_Vertical
- J3, J4: footprint (none) -> Frooastboard Footprints:PinHeader_1x06_P1.27mm_Vertical
- J5: footprint (none) -> Frooastboard Footprints:PinHeader_1x10_P1.27mm_Vertical
- J6: footprint (none) -> Frooastboard Footprints:PinHeader_1x12_P1.27mm_Vertical
- J7: footprint (none) -> Frooastboard Footprints:PinHeader_1x04_P1.27mm_Vertical
- L4: footprint (none) -> Inductor_SMD:L_6.3x6.3_H3
Connections:
- net +3V3: now also R11.1; no longer R11.2
- net GND: now also R6.1, R7.1; no longer R6.2, R7.2
- net NRF_MISO: now also U1.32 (GPIO21)
- net NRF_MOSI: now also U1.37 (GPIO25)
- net NRF_RDYN: now also U1.35 (GPIO23); no longer U1.27 (GPIO16)
- net NRF_REQN: now also U1.34 (GPIO22); no longer U1.28 (GPIO17)
- net NRF_SCK: now also U1.36 (GPIO24)
- net at U1.29 (GPIO18): now also J6.9 (Pin_9)
- net at U1.30 (GPIO19): now also J6.10 (Pin_10)
- net at U1.31 (GPIO20): now also J6.11 (Pin_11)
- net at J6.7 (Pin_7): now also U1.27 (GPIO16)
- net at J6.8 (Pin_8): now also U1.28 (GPIO17)
- net IICRST: no longer names the net of U5.47 (IICRST)
- net IICRST: now also R7.2; no longer R7.1
- net RSET: no longer names the net of U5.35 (RSET)
- net RSET: now also R6.2; no longer R6.1
- net SDB: no longer names the net of U5.46 (~{SDB})
- net SDB: now also R11.2; no longer R11.1
Other:
- moved on the sheet: J6, R11, R6, R7

Commit message: asign pieces
Parts:
- R10, R12, R13, R14, R15, R16, R17, R18, R19, R20, R4, R5: footprint (none) -> Resistor_SMD:R_0805_2012Metric
- U1: footprint Sleep-Lib:RP2040-QFN-56 -> Frooastboard Footprints:RP2040-QFN-56
