File: Frooastboard Walnut Modular/KiCad Project/Frooastboard Walnut Modular.kicad_sch (KiCad schematic)
At the start: 16 parts

Commit message: update library references
Parts:
- FPC203, FPC204: footprint AFA01-SXXFCX-00:FPC-SMD_10P_P1.00_AFA01-S10FCC-00 -> AFA01-SXXFCX-00:FPC-SMD_10P-P1.00_AFA01-S10FCC-00
Changed lines of the file:
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@@
       (effects (font (size 1.27 1.27)))
     )
-    (property "Footprint" "AFA01-SXXFCX-00:FPC-SMD_10P_P1.00_AFA01-S10FCC-00" (at 118.0084 72.39 0)
+    (property "Footprint" "AFA01-SXXFCX-00:FPC-SMD_10P-P1.00_AFA01-S10FCC-00" (at 118.0084 72.39 0)
       (effects (font (size 1.27 1.27)) hide)
     )
@@
       (effects (font (size 1.27 1.27)))
     )
-    (property "Footprint" "AFA01-SXXFCX-00:FPC-SMD_10P_P1.00_AFA01-S10FCC-00" (at 153.7716 41.91 0)
-      (effects (font (size 1.27 1.27)) hide)
-    )
+    (property "Footprint" "AFA01-SXXFCX-00:FPC-SMD_10P-P1.00_AFA01-S10FCC-00" (at 153.7716 41.91 0)
+      (effects (font (size 1.27 1.27)) hide)
+    )

Commit message: some stuff
Connections:
- net F Row/fr_dn renamed F Row/fr_d-
- net F Row/fr_dp renamed F Row/fr_d+
- net Main/ce_dn renamed Main/ce_d-
- net Main/ce_dp renamed Main/ce_d+
Other:
- sheet F Row ports: added fr_d+, fr_d-; removed fr_dn, fr_dp
- sheet Main ports: added ce_d+, ce_d-; removed ce_dn, ce_dp
Changed lines of the file:
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@@
       (effects (font (size 1.27 1.27)) (justify right))
     )
-    (pin "fr_dp" bidirectional (at 60.96 34.29 0)
+    (pin "fr_d+" bidirectional (at 60.96 34.29 0)
       (effects (font (size 1.27 1.27)) (justify right))
     )
-    (pin "fr_dn" bidirectional (at 60.96 31.75 0)
+    (pin "fr_d-" bidirectional (at 60.96 31.75 0)
       (effects (font (size 1.27 1.27)) (justify right))
     )
@@
       (effects (font (size 1.27 1.27)) (justify right))
     )
-    (pin "ce_dn" bidirectional (at 116.84 199.39 0)
+    (pin "ce_d-" bidirectional (at 116.84 199.39 0)
       (effects (font (size 1.27 1.27)) (justify right))
     )
-    (pin "ce_dp" bidirectional (at 116.84 201.93 0)
+    (pin "ce_d+" bidirectional (at 116.84 201.93 0)
       (effects (font (size 1.27 1.27)) (justify right))
     )
