File: Frooastboard Walnut Modular/KiCad Project/Frooastboard Walnut Modular.kicad_pcb (KiCad board)
At the start: 2 copper layers, 428 parts, among them J1 SW Interface, J10 F Row CS, J11 F Row SW, J12 Conn_01x06_Male, J13 Conn_01x16_Male, J14 Conn_01x10_Male, J15 F Row, J16 F Row USB, J17 Numpad, J18 Conn_01x04_Male, J19 Conn_01x15_Male, J2 Conn_01x16, J20 Conn_01x06_Male, J21 Conn_01x13_Male, J3 Conn_01x06, J4 Conn_01x06, J5 Conn_01x10, J6 Conn_01x12, J7 Conn_01x04, J8 Numpad CS, J9 Numpad SW, U1 RP2040, U2 SPX3819M5-L-3-3, U3 W25Q32JVZP, U4 nRF8001, U5 IS31FL3733-QF, U6 FS312F-G, U7 FS8205, U8 IP2312, Y1 32.768kHz, Y2 16MHz, Y3 12MHz

Commit message: some backup
Parts:
- BT1: footprint TestPoint:TestPoint_Pad_D1.5mm -> TestPoint:TestPoint_2Pads_Pitch5.08mm_Drill1.3mm
- J1: footprint Connector_PinHeader_2.54mm:PinHeader_1x05_P2.54mm_Vertical -> Connector_PinHeader_1.27mm:PinHeader_1x05_P1.27mm_Vertical
- TP5: footprint TestPoint:TestPoint_Pad_D1.5mm -> Connector_PinHeader_1.27mm:PinHeader_1x02_P1.27mm_Vertical
- moved MX20 584.2 mm to (-87.3, 237.3)
- moved MX18 537.5 mm to (-87.3, 199.2)
- moved MX25 521.2 mm to (-49.2, 218.3)
- moved MX28 518.5 mm to (-68.3, 180.2)
- moved MX31 502.8 mm to (-68.3, 237.3)
- moved MX30 502.6 mm to (-68.3, 218.3)
- moved MX34 500.7 mm to (-30.2, 180.2)
- moved MX17 500.6 mm to (-87.3, 180.2)
- moved MX29 498.3 mm to (-68.3, 199.2)
- moved MX23 482.7 mm to (-49.2, 180.2)
- moved MX21 469.6 mm to (-77.8, 256.4)
- moved MX24 462.5 mm to (-49.2, 199.2)
- moved MX19 460.4 mm to (-87.3, 218.3)
- moved MX32 444.8 mm to (-49.2, 256.4)
- moved MX26 443.6 mm to (-49.2, 237.3)
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Other:
- board outline added: 57.2 x 19 mm
- copper layers 2 -> 4

Commit message: some settings
Parts:
- removed BT1: Battery_Cell, TestPoint:TestPoint_2Pads_Pitch5.08mm_Drill1.3mm
- removed C1, C2, C4: 100n, Capacitor_SMD:C_0402_1005Metric
- removed C10, C11: 12p, Capacitor_SMD:C_0402_1005Metric
- removed C12: 1.8p, Capacitor_SMD:C_0402_1005Metric
- removed C13: 1.2p, Capacitor_SMD:C_0402_1005Metric
- removed C14, C15: 22p, Capacitor_SMD:C_0805_2012Metric
- removed C16, C17, C31, C33, C37, C38, C39, C40: 10u, Capacitor_SMD:C_0805_2012Metric
- removed C18, C19, C20, C21, C22, C23, C24, C25, C26, C27, C32: 100n, Capacitor_SMD:C_0805_2012Metric
- removed C28: 0.1u, Capacitor_SMD:C_0805_2012Metric
- removed C29: 10n, Capacitor_SMD:C_0805_2012Metric
- removed C3: 1n, Capacitor_SMD:C_0402_1005Metric
- removed C30, C36: 22u, Capacitor_SMD:C_0805_2012Metric
- removed C34, C35: 10u, Capacitor_Tantalum_SMD:CP_EIA-2012-15_AVX-P
- removed C5: 33n, Capacitor_SMD:C_0402_1005Metric
- removed C6, C7: 15p, Capacitor_SMD:C_0402_1005Metric
- removed C8: 2.2n, Capacitor_SMD:C_0402_1005Metric
- removed C9: Not Mounted, Capacitor_SMD:C_0402_1005Metric
- removed D1: GREEN, LED_SMD:LED_0805_2012Metric
- removed D10, D113, D114, D115, D116, D117, D12, D122, D123, D124, D125, D126, D127, D128, D129, D13, D130, D131, D132, D133, D134, D139, D140, D141, D142, D143, D144, D145, D146, D147, D15, D152, D153, D154, D155, D156, D157, D158, D159, D16, D160, D165, D166, D167, D168, D169, D170, D171, D172, D173, D174, D175, D176, D177, D178, D18, D183, D184, D185, D186, D187, D188, D189, D19, D190, D191, D195, D196, D197, D198, D199, D20, D200, D201, D202, D203, D204, D205, D206, D207, D23, D24, D27, D28, D29, D47, D48, D49, D50, D51, D54, D55, D56, D57, D59, D6, D60, D61, D62, D63, D66, D67, D69, D8, D9: D_Small, Diode_SMD:D_0805_2012Metric
- removed D105, D107, D108, D109, D11, D110, D112, D118, D119, D120, D121, D135, D136, D137, D138, D14, D148, D149, D150, D151, D161, D162, D163, D164, D17, D179, D180, D181, D192, D194, D208, D21, D210, D211, D212, D214, D215, D216, D218, D219, D22, D220, D221, D222, D223, D228, D229, D231, D236, D237, D239, D244, D245, D247, D25, D252, D253, D255, D26, D3, D30, D31, D32, D33, D34, D35, D36, D37, D38, D39, D4, D40, D41, D42, D43, D44, D45, D46, D53, D65, D7, D71, D72, D73, D74, D75, D76, D77, D78, D79, D80, D81, D82, D83: RGB_LED_6_Pin, Frooastboard Footprints:Everlight 99-235
- removed D2: RED, LED_SMD:LED_0805_2012Metric
- removed D5: Caps Lock Indicator, LED_SMD:LED_0805_2012Metric
- removed D52: Roll Indicator, LED_SMD:LED_0805_2012Metric
- removed D58: Num Lock Indicator, LED_SMD:LED_0805_2012Metric
- removed J1: SW Interface, Connector_PinHeader_1.27mm:PinHeader_1x05_P1.27mm_Vertical
- removed J10: F Row CS, Frooastboard Footprints:PinHeader_1x16_P1.27mm_Vertical
- removed J11: F Row SW, Frooastboard Footprints:PinHeader_1x06_P1.27mm_Vertical
- removed J12, J20: Conn_01x06_Male, Frooastboard Footprints:PinHeader_1x06_P1.27mm_Vertical
- removed J13: Conn_01x16_Male, Frooastboard Footprints:PinHeader_1x16_P1.27mm_Vertical
- removed J14: Conn_01x10_Male, Frooastboard Footprints:PinHeader_1x10_P1.27mm_Vertical
- removed J15: F Row, Frooastboard Footprints:PinHeader_1x10_P1.27mm_Vertical
- removed J16: F Row USB, Frooastboard Footprints:PinHeader_1x04_P1.27mm_Vertical
- removed J17: Numpad, Frooastboard Footprints:PinHeader_1x13_P1.27mm_Vertical
- removed J18: Conn_01x04_Male, Frooastboard Footprints:PinHeader_1x04_P1.27mm_Vertical
- removed J19: Conn_01x15_Male, Frooastboard Footprints:PinHeader_1x15_P1.27mm_Vertical
- removed J2: Conn_01x16, Frooastboard Footprints:PinHeader_1x16_P1.27mm_Vertical
- removed J21: Conn_01x13_Male, Frooastboard Footprints:PinHeader_1x13_P1.27mm_Vertical
- removed J3, J4: Conn_01x06, Frooastboard Footprints:PinHeader_1x06_P1.27mm_Vertical
- removed J5: Conn_01x10, Frooastboard Footprints:PinHeader_1x10_P1.27mm_Vertical
- removed J6: Conn_01x12, Frooastboard Footprints:PinHeader_1x12_P1.27mm_Vertical
- removed J7: Conn_01x04, Frooastboard Footprints:PinHeader_1x04_P1.27mm_Vertical
- removed J8: Numpad CS, Frooastboard Footprints:PinHeader_1x16_P1.27mm_Vertical
- removed J9: Numpad SW, Frooastboard Footprints:PinHeader_1x06_P1.27mm_Vertical
- removed L1: 5.6nH, Inductor_SMD:L_0402_1005Metric
- removed L2: 8.2nH, Inductor_SMD:L_0402_1005Metric
- removed L3: 3.9nH, Inductor_SMD:L_0402_1005Metric
- removed L4: 1uH, Inductor_SMD:L_6.3x6.3_H3
- removed MX1, MX39: Escape, MX_Only:MXOnly-1U-NoLED
- removed MX10: F9, MX_Only:MXOnly-1U-NoLED
- removed MX100: Home, MX_Only:MXOnly-1U-NoLED
- removed MX101: End, MX_Only:MXOnly-1U-NoLED
- removed MX102: 7, MX_Only:MXOnly-1U-NoLED
- removed MX103: U, MX_Only:MXOnly-1U-NoLED
- removed MX104: J, MX_Only:MXOnly-1U-NoLED
- removed MX105: N, MX_Only:MXOnly-1U-NoLED
- removed MX106: Right Control, MX_Only:MXOnly-1.25U-NoLED
- removed MX107: Right, MX_Only:MXOnly-1U-NoLED
- removed MX108: Down, MX_Only:MXOnly-1U-NoLED
- removed MX109: Page Up, MX_Only:MXOnly-1U-NoLED
- removed MX11: F10, MX_Only:MXOnly-1U-NoLED
- removed MX110: Page Down, MX_Only:MXOnly-1U-NoLED
- removed MX111: Left Shift, MX_Only:MXOnly-2.25U-NoLED
- removed MX112: \, MX_Only:MXOnly-1.5U-NoLED
- removed MX113: Enter, MX_Only:MXOnly-2.25U-NoLED
- removed MX12: F11, MX_Only:MXOnly-1U-NoLED
- removed MX13: F12, MX_Only:MXOnly-1U-NoLED
- removed MX14: Print Screen, MX_Only:MXOnly-1U-NoLED
- removed MX15: Scroll Lock, MX_Only:MXOnly-1U
- removed MX16: Pause, MX_Only:MXOnly-1U-NoLED
- removed MX17: Num Lock, MX_Only:MXOnly-1U
- removed MX18: Num 7, MX_Only:MXOnly-1U-NoLED
- removed MX19: Num 4, MX_Only:MXOnly-1U-NoLED
- removed MX2: F1, MX_Only:MXOnly-1U-NoLED
- removed MX20: Num 1, MX_Only:MXOnly-1U-NoLED
- removed MX21: Num 0, MX_Only:MXOnly-2U-NoLED
- removed MX23: Multiply, MX_Only:MXOnly-1U-NoLED
- removed MX24: Num 9, MX_Only:MXOnly-1U-NoLED
- removed MX25: Num 6, MX_Only:MXOnly-1U-NoLED
- removed MX26: Num 3, MX_Only:MXOnly-1U-NoLED
- removed MX28: Divide, MX_Only:MXOnly-1U-NoLED
- removed MX29: Num 8, MX_Only:MXOnly-1U-NoLED
- removed MX3: F2, MX_Only:MXOnly-1U-NoLED
- removed MX30: Num 5, MX_Only:MXOnly-1U-NoLED
- removed MX31: Num 2, MX_Only:MXOnly-1U-NoLED
- removed MX32: Comma, MX_Only:MXOnly-1U-NoLED
- removed MX34: Minus, MX_Only:MXOnly-1U-NoLED
- removed MX35: Plus, MX_Only:MXOnly-2U-VerticalStabilizers-NoLED
- removed MX37: Enter, MX_Only:MXOnly-2U-VerticalStabilizers-NoLED
- removed MX4: F3, MX_Only:MXOnly-1U-NoLED
- removed MX40: Tab, MX_Only:MXOnly-1.5U-NoLED
- removed MX41: Caps Lock, MX_Only:MXOnly-1.75U
- removed MX42: Left Shift, MX_Only:MXOnly-1.25U-NoLED
- removed MX43: Left Control, MX_Only:MXOnly-1.25U-NoLED
- removed MX44: 8, MX_Only:MXOnly-1U-NoLED
- removed MX45: I, MX_Only:MXOnly-1U-NoLED
- removed MX46: K, MX_Only:MXOnly-1U-NoLED
- removed MX47: M, MX_Only:MXOnly-1U-NoLED
- removed MX48: 1, MX_Only:MXOnly-1U-NoLED
- removed MX49: Q, MX_Only:MXOnly-1U-NoLED
- removed MX5: F4, MX_Only:MXOnly-1U-NoLED
- removed MX50: A, MX_Only:MXOnly-1U-NoLED
- removed MX51, MX82: \, MX_Only:MXOnly-1U-NoLED
- removed MX52: Left GUI, MX_Only:MXOnly-1.25U-NoLED
- removed MX53: 9, MX_Only:MXOnly-1U-NoLED
- removed MX54: O, MX_Only:MXOnly-1U-NoLED
- removed MX55: L, MX_Only:MXOnly-1U-NoLED
- removed MX56: ,, MX_Only:MXOnly-1U-NoLED
- removed MX57: 2, MX_Only:MXOnly-1U-NoLED
- removed MX58: W, MX_Only:MXOnly-1U-NoLED
- removed MX59: S, MX_Only:MXOnly-1U-NoLED
- removed MX6: F5, MX_Only:MXOnly-1U-NoLED
- removed MX60: Z, MX_Only:MXOnly-1U-NoLED
- removed MX61: Left Alt, MX_Only:MXOnly-1.25U-NoLED
- removed MX62: 0, MX_Only:MXOnly-1U-NoLED
- removed MX63: P, MX_Only:MXOnly-1U-NoLED
- removed MX64: ;, MX_Only:MXOnly-1U-NoLED
- removed MX65: ., MX_Only:MXOnly-1U-NoLED
- removed MX66: 3, MX_Only:MXOnly-1U-NoLED
- removed MX67: E, MX_Only:MXOnly-1U-NoLED
- removed MX68: D, MX_Only:MXOnly-1U-NoLED
- removed MX69: X, MX_Only:MXOnly-1U-NoLED
- removed MX7: F6, MX_Only:MXOnly-1U-NoLED
- removed MX70: Space, MX_Only:MXOnly-6.25U-ReversedStabilizers-NoLED
- removed MX71: -, MX_Only:MXOnly-1U-NoLED
- removed MX72: [, MX_Only:MXOnly-1U-NoLED
- removed MX73: ', MX_Only:MXOnly-1U-NoLED
- removed MX74: /, MX_Only:MXOnly-1U-NoLED
- removed MX75: 4, MX_Only:MXOnly-1U-NoLED
- removed MX76: R, MX_Only:MXOnly-1U-NoLED
- removed MX77: F, MX_Only:MXOnly-1U-NoLED
- removed MX78: C, MX_Only:MXOnly-1U-NoLED
- removed MX79: Right Alt, MX_Only:MXOnly-1.25U-NoLED
- removed MX8: F7, MX_Only:MXOnly-1U-NoLED
- removed MX80: =, MX_Only:MXOnly-1U-NoLED
- removed MX81: ], MX_Only:MXOnly-1U-NoLED
- removed MX83: Right Shift, MX_Only:MXOnly-2.75U-NoLED
- removed MX84: 5, MX_Only:MXOnly-1U-NoLED
- removed MX85: T, MX_Only:MXOnly-1U-NoLED
- removed MX86: G, MX_Only:MXOnly-1U-NoLED
- removed MX87: V, MX_Only:MXOnly-1U-NoLED
- removed MX88: Function, MX_Only:MXOnly-1.25U-NoLED
- removed MX89: Backspace, MX_Only:MXOnly-2U-NoLED
- removed MX9: F8, MX_Only:MXOnly-1U-NoLED
- removed MX90: Enter, MX_Only:MXOnly-ISO-ROTATED-NoLED-NoStabilizers
- removed MX91: Insert, MX_Only:MXOnly-1U-NoLED
- removed MX92: Delete, MX_Only:MXOnly-1U-NoLED
- removed MX93: 6, MX_Only:MXOnly-1U-NoLED
- removed MX94: Y, MX_Only:MXOnly-1U-NoLED
- removed MX95: H, MX_Only:MXOnly-1U-NoLED
- removed MX96: B, MX_Only:MXOnly-1U-NoLED
- removed MX97: Menu, MX_Only:MXOnly-1.25U-NoLED
- removed MX98: Left, MX_Only:MXOnly-1U-NoLED
- removed MX99: Up, MX_Only:MXOnly-1U-NoLED
- removed R1, R8: 10k, Resistor_SMD:R_0805_2012Metric
- removed R10, R4, R5: 2k, Resistor_SMD:R_0805_2012Metric
- removed R11, R7: 100k, Resistor_SMD:R_0805_2012Metric
- removed R12: 0k5, Resistor_SMD:R_0805_2012Metric
- removed R13, R14: 1M, Resistor_SMD:R_0805_2012Metric
- removed R15, R16: 0k1, Resistor_SMD:R_0805_2012Metric
- removed R17, R20: NC, Resistor_SMD:R_0805_2012Metric
- removed R18: 51k, Resistor_SMD:R_0805_2012Metric
- removed R19, R3, R9: 1k, Resistor_SMD:R_0805_2012Metric
- removed R2: 22k, Resistor_SMD:R_0805_2012Metric
- removed R21, R22, R26, R27, R29, R30: 5k1, Resistor_SMD:R_0805_2012Metric
- removed R23, R24: 27R, Resistor_SMD:R_0805_2012Metric
- removed R25, R28, R31: 2R, Resistor_SMD:R_0805_2012Metric
- removed R6: 20k, Resistor_SMD:R_0805_2012Metric
- removed TP1: NRF_TXD, TestPoint:TestPoint_Pad_D1.5mm
- removed TP2: NRF_RXD, TestPoint:TestPoint_Pad_D1.5mm
- removed TP3: NRF_RESET, TestPoint:TestPoint_Pad_D1.5mm
- removed TP4: NRF_IREF, TestPoint:TestPoint_Pad_D1.5mm
- removed TP5: QSPI_CS, Connector_PinHeader_1.27mm:PinHeader_1x02_P1.27mm_Vertical
- removed U1: RP2040, Frooastboard Footprints:RP2040-QFN-56
- removed U2: SPX3819M5-L-3-3, Package_TO_SOT_SMD:SOT-23-5
- removed U3: W25Q32JVZP, Package_SON:WSON-8-1EP_6x5mm_P1.27mm_EP3.4x4.3mm
- removed U4: nRF8001, Package_DFN_QFN:QFN-32-1EP_5x5mm_P0.5mm_EP3.45x3.45mm
- removed U5: IS31FL3733-QF, Package_DFN_QFN:QFN-48-1EP_6x6mm_P0.4mm_EP4.2x4.2mm
- removed U6: FS312F-G, Package_TO_SOT_SMD:SOT-23-6
- removed U7: FS8205, Package_TO_SOT_SMD:SOT-23-6
- removed U8: IP2312, Package_SO:SOIC-8-1EP_3.9x4.9mm_P1.27mm_EP2.41x3.3mm
- removed USB1, USB2, USB3: HRO-TYPE-C-31-M-12, Type_C:HRO-TYPE-C-31-M-12
- removed Y1: 32.768kHz, Crystal:Crystal_SMD_EuroQuartz_EQ161-2Pin_3.2x1.5mm
- removed Y2: 16MHz, Crystal:Crystal_SMD_3225-4Pin_3.2x2.5mm
- removed Y3: 12MHz, Crystal:Crystal_SMD_3225-4Pin_3.2x2.5mm
Other:
- board outline removed

Commit message: prepare
Parts:
- added BT1: Battery_Cell, TestPoint:TestPoint_2Pads_Pitch5.08mm_Drill1.3mm, F.Cu at (430.2, 253.2)
- added C1: 100n, Capacitor_SMD:C_0402_1005Metric, F.Cu at (454.6, 279.1)
- added C10: 12p, Capacitor_SMD:C_0402_1005Metric, F.Cu at (457.5, 279.1)
- added C11: 12p, Capacitor_SMD:C_0402_1005Metric, F.Cu at (450.2, 286.5)
- added C12: 1.8p, Capacitor_SMD:C_0402_1005Metric, F.Cu at (468.2, 266.8)
- added C13: 1.2p, Capacitor_SMD:C_0402_1005Metric, F.Cu at (463.6, 273.5)
- added C14: 22p, Capacitor_SMD:C_0805_2012Metric, F.Cu at (462.9, 258.4)
- added C15: 22p, Capacitor_SMD:C_0805_2012Metric, F.Cu at (437.7, 283.7)
- added C16: 10u, Capacitor_SMD:C_0805_2012Metric, F.Cu at (442.2, 279.8)
- added C17: 10u, Capacitor_SMD:C_0805_2012Metric, F.Cu at (446.4, 276.8)
- added C18: 100n, Capacitor_SMD:C_0805_2012Metric, F.Cu at (460.8, 261.4)
- added C19: 100n, Capacitor_SMD:C_0805_2012Metric, F.Cu at (458.4, 256.8)
- added C2: 100n, Capacitor_SMD:C_0402_1005Metric, F.Cu at (459.2, 275.8)
- added C20: 100n, Capacitor_SMD:C_0805_2012Metric, F.Cu at (437.7, 280.7)
- added C21: 100n, Capacitor_SMD:C_0805_2012Metric, F.Cu at (468.2, 255.4)
- added C22: 100n, Capacitor_SMD:C_0805_2012Metric, F.Cu at (451.1, 268.5)
- added C23: 100n, Capacitor_SMD:C_0805_2012Metric, F.Cu at (451.1, 274.6)
- added C24: 100n, Capacitor_SMD:C_0805_2012Metric, F.Cu at (463.8, 252.4)
- added C25: 100n, Capacitor_SMD:C_0805_2012Metric, F.Cu at (460.2, 267.4)
- added C26: 100n, Capacitor_SMD:C_0805_2012Metric, F.Cu at (463.8, 255.4)
- added C27: 100n, Capacitor_SMD:C_0805_2012Metric, F.Cu at (442.2, 282.8)
- added C28: 0.1u, Capacitor_SMD:C_0805_2012Metric, F.Cu at (451.1, 271.5)
- added C29: 10n, Capacitor_SMD:C_0805_2012Metric, F.Cu at (433.3, 280.7)
- added C3: 1n, Capacitor_SMD:C_0402_1005Metric, F.Cu at (479.0, 257.8)
- added C30: 22u, Capacitor_SMD:C_0805_2012Metric, F.Cu at (472.7, 252.4)
- added C31: 10u, Capacitor_SMD:C_0805_2012Metric, F.Cu at (467.3, 258.4)
- added C32: 100n, Capacitor_SMD:C_0805_2012Metric, F.Cu at (455.6, 267.8)
- added C33: 10u, Capacitor_SMD:C_0805_2012Metric, F.Cu at (460.2, 264.4)
- added C34: 10u, Capacitor_Tantalum_SMD:CP_EIA-2012-15_AVX-P, F.Cu at (442.0, 276.7)
- added C35: 10u, Capacitor_Tantalum_SMD:CP_EIA-2012-15_AVX-P, F.Cu at (456.4, 261.2)
- added C36: 22u, Capacitor_SMD:C_0805_2012Metric, F.Cu at (468.2, 252.4)
- added C37: 10u, Capacitor_SMD:C_0805_2012Metric, F.Cu at (455.7, 264.7)
- added C38: 10u, Capacitor_SMD:C_0805_2012Metric, F.Cu at (484.6, 157.7)
- added C39: 10u, Capacitor_SMD:C_0805_2012Metric, F.Cu at (797.9, 45.7)
- added C4: 100n, Capacitor_SMD:C_0402_1005Metric, F.Cu at (472.6, 263.8)
- added C40: 10u, Capacitor_SMD:C_0805_2012Metric, F.Cu at (567.2, 163.7)
- added C5: 33n, Capacitor_SMD:C_0402_1005Metric, F.Cu at (454.6, 281.1)
- added C6: 15p, Capacitor_SMD:C_0402_1005Metric, F.Cu at (484.3, 251.9)
- added C7: 15p, Capacitor_SMD:C_0402_1005Metric, F.Cu at (468.2, 268.8)
- added C8: 2.2n, Capacitor_SMD:C_0402_1005Metric, F.Cu at (473.3, 261.4)
- added C9: Not Mounted, Capacitor_SMD:C_0402_1005Metric, F.Cu at (480.7, 255.4)
- added D1: GREEN, LED_SMD:LED_0805_2012Metric, F.Cu at (433.3, 283.8)
- added D10: D_Small, Diode_SMD:D_0805_2012Metric, F.Cu at (784.8, 48.4)
- added D105: RGB_LED_6_Pin, Frooastboard Footprints:Everlight 99-235, F.Cu at (579.6, 15.3)
- added D107: RGB_LED_6_Pin, Frooastboard Footprints:Everlight 99-235, F.Cu at (439.3, 151.0)
- added D108: RGB_LED_6_Pin, Frooastboard Footprints:Everlight 99-235, F.Cu at (422.4, 145.6)
- added D109: RGB_LED_6_Pin, Frooastboard Footprints:Everlight 99-235, F.Cu at (439.3, 153.7)
- added D11: RGB_LED_6_Pin, Frooastboard Footprints:Everlight 99-235, F.Cu at (752.8, 53.0)
- added D110: RGB_LED_6_Pin, Frooastboard Footprints:Everlight 99-235, F.Cu at (579.6, 12.5)
- added D112: RGB_LED_6_Pin, Frooastboard Footprints:Everlight 99-235, F.Cu at (444.9, 145.6)
- added D113: D_Small, Diode_SMD:D_0805_2012Metric, F.Cu at (506.8, 151.7)
- added D114: D_Small, Diode_SMD:D_0805_2012Metric, F.Cu at (482.5, 148.3)
- added D115: D_Small, Diode_SMD:D_0805_2012Metric, F.Cu at (484.6, 154.7)
- added D116: D_Small, Diode_SMD:D_0805_2012Metric, F.Cu at (486.9, 148.6)
- added D117: D_Small, Diode_SMD:D_0805_2012Metric, F.Cu at (489.0, 151.7)
- added D118: RGB_LED_6_Pin, Frooastboard Footprints:Everlight 99-235, F.Cu at (461.7, 156.4)
- added D119: RGB_LED_6_Pin, Frooastboard Footprints:Everlight 99-235, F.Cu at (461.7, 145.6)
- added D12: D_Small, Diode_SMD:D_0805_2012Metric, F.Cu at (784.6, 45.4)
- added D120: RGB_LED_6_Pin, Frooastboard Footprints:Everlight 99-235, F.Cu at (574.0, 12.5)
- added D121: RGB_LED_6_Pin, Frooastboard Footprints:Everlight 99-235, F.Cu at (444.9, 153.7)
- added D122: D_Small, Diode_SMD:D_0805_2012Metric, F.Cu at (524.6, 151.7)
- added D123: D_Small, Diode_SMD:D_0805_2012Metric, F.Cu at (540.3, 147.3)
- added D124: D_Small, Diode_SMD:D_0805_2012Metric, F.Cu at (512.2, 99.5)
- added D125: D_Small, Diode_SMD:D_0805_2012Metric, F.Cu at (493.5, 151.7)
- added D126: D_Small, Diode_SMD:D_0805_2012Metric, F.Cu at (529.1, 151.7)
- added D127: D_Small, Diode_SMD:D_0805_2012Metric, F.Cu at (480.1, 151.3)
- added D128: D_Small, Diode_SMD:D_0805_2012Metric, F.Cu at (480.1, 154.4)
- added D129: D_Small, Diode_SMD:D_0805_2012Metric, F.Cu at (471.2, 157.1)
- added D13: D_Small, Diode_SMD:D_0805_2012Metric, F.Cu at (789.3, 48.4)
- added D130: D_Small, Diode_SMD:D_0805_2012Metric, F.Cu at (518.1, 148.6)
- added D131: D_Small, Diode_SMD:D_0805_2012Metric, F.Cu at (472.4, 151.0)
- added D132: D_Small, Diode_SMD:D_0805_2012Metric, F.Cu at (500.3, 145.6)
- added D133: D_Small, Diode_SMD:D_0805_2012Metric, F.Cu at (540.3, 150.4)
- added D134: D_Small, Diode_SMD:D_0805_2012Metric, F.Cu at (489.0, 154.7)
- added D135: RGB_LED_6_Pin, Frooastboard Footprints:Everlight 99-235, F.Cu at (456.1, 145.6)
- added D136: RGB_LED_6_Pin, Frooastboard Footprints:Everlight 99-235, F.Cu at (444.9, 156.4)
- added D137: RGB_LED_6_Pin, Frooastboard Footprints:Everlight 99-235, F.Cu at (439.3, 156.4)
- added D138: RGB_LED_6_Pin, Frooastboard Footprints:Everlight 99-235, F.Cu at (444.9, 148.3)
- added D139: D_Small, Diode_SMD:D_0805_2012Metric, F.Cu at (509.2, 148.6)
- added D14: RGB_LED_6_Pin, Frooastboard Footprints:Everlight 99-235, F.Cu at (758.5, 55.7)
- added D140: D_Small, Diode_SMD:D_0805_2012Metric, F.Cu at (514.5, 33.4)
- added D141: D_Small, Diode_SMD:D_0805_2012Metric, F.Cu at (495.8, 145.6)
- added D142: D_Small, Diode_SMD:D_0805_2012Metric, F.Cu at (497.9, 151.7)
- added D143: D_Small, Diode_SMD:D_0805_2012Metric, F.Cu at (514.5, 36.5)
- added D144: D_Small, Diode_SMD:D_0805_2012Metric, F.Cu at (480.1, 157.4)
- added D145: D_Small, Diode_SMD:D_0805_2012Metric, F.Cu at (486.9, 145.6)
- added D146: D_Small, Diode_SMD:D_0805_2012Metric, F.Cu at (493.5, 154.7)
- added D147: D_Small, Diode_SMD:D_0805_2012Metric, F.Cu at (475.7, 157.1)
- added D148: RGB_LED_6_Pin, Frooastboard Footprints:Everlight 99-235, F.Cu at (456.1, 148.3)
- added D149: RGB_LED_6_Pin, Frooastboard Footprints:Everlight 99-235, F.Cu at (422.4, 156.4)
- added D15: D_Small, Diode_SMD:D_0805_2012Metric, F.Cu at (789.3, 51.4)
- added D150: RGB_LED_6_Pin, Frooastboard Footprints:Everlight 99-235, F.Cu at (500.3, 38.5)
- added D151: RGB_LED_6_Pin, Frooastboard Footprints:Everlight 99-235, F.Cu at (422.4, 151.0)
- added D152: D_Small, Diode_SMD:D_0805_2012Metric, F.Cu at (478.0, 148.3)
- added D153: D_Small, Diode_SMD:D_0805_2012Metric, F.Cu at (475.7, 154.0)
- added D154: D_Small, Diode_SMD:D_0805_2012Metric, F.Cu at (535.9, 148.6)
- added D155: D_Small, Diode_SMD:D_0805_2012Metric, F.Cu at (518.1, 145.6)
- added D156: D_Small, Diode_SMD:D_0805_2012Metric, F.Cu at (515.7, 154.7)
- added D157: D_Small, Diode_SMD:D_0805_2012Metric, F.Cu at (513.6, 145.6)
- added D158: D_Small, Diode_SMD:D_0805_2012Metric, F.Cu at (533.5, 154.7)
- added D159: D_Small, Diode_SMD:D_0805_2012Metric, F.Cu at (535.9, 145.6)
- added D16: D_Small, Diode_SMD:D_0805_2012Metric, F.Cu at (784.8, 51.4)
- added D160: D_Small, Diode_SMD:D_0805_2012Metric, F.Cu at (497.9, 154.7)
- added D161: RGB_LED_6_Pin, Frooastboard Footprints:Everlight 99-235, F.Cu at (433.6, 145.6)
- added D162: RGB_LED_6_Pin, Frooastboard Footprints:Everlight 99-235, F.Cu at (428.0, 153.7)
- added D163: RGB_LED_6_Pin, Frooastboard Footprints:Everlight 99-235, F.Cu at (428.0, 145.6)
- added D164: RGB_LED_6_Pin, Frooastboard Footprints:Everlight 99-235, F.Cu at (456.1, 151.0)
- added D165: D_Small, Diode_SMD:D_0805_2012Metric, F.Cu at (524.6, 154.7)
- added D166: D_Small, Diode_SMD:D_0805_2012Metric, F.Cu at (511.3, 154.7)
- added D167: D_Small, Diode_SMD:D_0805_2012Metric, F.Cu at (506.8, 154.7)
- added D168: D_Small, Diode_SMD:D_0805_2012Metric, F.Cu at (538.0, 153.4)
- added D169: D_Small, Diode_SMD:D_0805_2012Metric, F.Cu at (502.4, 154.7)
- added D17: RGB_LED_6_Pin, Frooastboard Footprints:Everlight 99-235, F.Cu at (769.7, 55.0)
- added D170: D_Small, Diode_SMD:D_0805_2012Metric, F.Cu at (495.8, 148.6)
- added D171: D_Small, Diode_SMD:D_0805_2012Metric, F.Cu at (520.2, 154.7)
- added D172: D_Small, Diode_SMD:D_0805_2012Metric, F.Cu at (543.0, 144.3)
- added D173: D_Small, Diode_SMD:D_0805_2012Metric, F.Cu at (513.6, 148.6)
- added D174: D_Small, Diode_SMD:D_0805_2012Metric, F.Cu at (547.5, 144.3)
- added D175: D_Small, Diode_SMD:D_0805_2012Metric, F.Cu at (504.7, 148.6)
- added D176: D_Small, Diode_SMD:D_0805_2012Metric, F.Cu at (529.1, 154.7)
- added D177: D_Small, Diode_SMD:D_0805_2012Metric, F.Cu at (471.2, 154.0)
- added D178: D_Small, Diode_SMD:D_0805_2012Metric, F.Cu at (512.2, 87.4)
- added D179: RGB_LED_6_Pin, Frooastboard Footprints:Everlight 99-235, F.Cu at (461.7, 151.0)
- added D18: D_Small, Diode_SMD:D_0805_2012Metric, F.Cu at (802.4, 42.7)
- added D180: RGB_LED_6_Pin, Frooastboard Footprints:Everlight 99-235, F.Cu at (467.4, 151.0)
- added D181: RGB_LED_6_Pin, Frooastboard Footprints:Everlight 99-235, F.Cu at (439.3, 148.3)
- added D183: D_Small, Diode_SMD:D_0805_2012Metric, F.Cu at (512.2, 93.5)
- added D184: D_Small, Diode_SMD:D_0805_2012Metric, F.Cu at (484.6, 151.7)
- added D185: D_Small, Diode_SMD:D_0805_2012Metric, F.Cu at (527.0, 148.6)
- added D186: D_Small, Diode_SMD:D_0805_2012Metric, F.Cu at (491.4, 145.6)
- added D187: D_Small, Diode_SMD:D_0805_2012Metric, F.Cu at (512.2, 96.5)
- added D188: D_Small, Diode_SMD:D_0805_2012Metric, F.Cu at (509.2, 145.6)
- added D189: D_Small, Diode_SMD:D_0805_2012Metric, F.Cu at (527.0, 145.6)
- added D19: D_Small, Diode_SMD:D_0805_2012Metric, F.Cu at (780.4, 54.5)
- added D190: D_Small, Diode_SMD:D_0805_2012Metric, F.Cu at (522.5, 145.6)
- added D191: D_Small, Diode_SMD:D_0805_2012Metric, F.Cu at (466.8, 157.1)
- added D192: RGB_LED_6_Pin, Frooastboard Footprints:Everlight 99-235, F.Cu at (467.4, 145.6)
- added D194: RGB_LED_6_Pin, Frooastboard Footprints:Everlight 99-235, F.Cu at (461.7, 153.7)
- added D195: D_Small, Diode_SMD:D_0805_2012Metric, F.Cu at (512.2, 90.4)
- added D196: D_Small, Diode_SMD:D_0805_2012Metric, F.Cu at (504.7, 145.6)
- added D197: D_Small, Diode_SMD:D_0805_2012Metric, F.Cu at (512.2, 84.3)
- added D198: D_Small, Diode_SMD:D_0805_2012Metric, F.Cu at (522.5, 148.6)
- added D199: D_Small, Diode_SMD:D_0805_2012Metric, F.Cu at (511.3, 151.7)
- added D2: RED, LED_SMD:LED_0805_2012Metric, F.Cu at (451.3, 264.8)
- added D20: D_Small, Diode_SMD:D_0805_2012Metric, F.Cu at (793.5, 45.4)
- added D200: D_Small, Diode_SMD:D_0805_2012Metric, F.Cu at (466.8, 154.0)
- added D201: D_Small, Diode_SMD:D_0805_2012Metric, F.Cu at (500.3, 148.6)
- added D202: D_Small, Diode_SMD:D_0805_2012Metric, F.Cu at (533.5, 151.7)
- added D203: D_Small, Diode_SMD:D_0805_2012Metric, F.Cu at (491.4, 148.6)
- added D204: D_Small, Diode_SMD:D_0805_2012Metric, F.Cu at (502.4, 151.7)
- added D205: D_Small, Diode_SMD:D_0805_2012Metric, F.Cu at (520.2, 151.7)
- added D206: D_Small, Diode_SMD:D_0805_2012Metric, F.Cu at (531.4, 148.6)
- added D207: D_Small, Diode_SMD:D_0805_2012Metric, F.Cu at (531.4, 145.6)
- added D208: RGB_LED_6_Pin, Frooastboard Footprints:Everlight 99-235, F.Cu at (461.7, 148.3)
- added D21: RGB_LED_6_Pin, Frooastboard Footprints:Everlight 99-235, F.Cu at (779.5, 42.6)
- added D210: RGB_LED_6_Pin, Frooastboard Footprints:Everlight 99-235, F.Cu at (467.4, 148.3)
- added D211: RGB_LED_6_Pin, Frooastboard Footprints:Everlight 99-235, F.Cu at (450.5, 148.3)
- added D212: RGB_LED_6_Pin, Frooastboard Footprints:Everlight 99-235, F.Cu at (444.9, 151.0)
- added D214: RGB_LED_6_Pin, Frooastboard Footprints:Everlight 99-235, F.Cu at (473.0, 145.6)
- added D215: RGB_LED_6_Pin, Frooastboard Footprints:Everlight 99-235, F.Cu at (422.4, 153.7)
- added D216: RGB_LED_6_Pin, Frooastboard Footprints:Everlight 99-235, F.Cu at (579.6, 18.0)
- added D218: RGB_LED_6_Pin, Frooastboard Footprints:Everlight 99-235, F.Cu at (450.5, 156.4)
- added D219: RGB_LED_6_Pin, Frooastboard Footprints:Everlight 99-235, F.Cu at (450.5, 151.0)
- added D22: RGB_LED_6_Pin, Frooastboard Footprints:Everlight 99-235, F.Cu at (755.5, 44.8)
- added D220: RGB_LED_6_Pin, Frooastboard Footprints:Everlight 99-235, F.Cu at (456.1, 153.7)
- added D221: RGB_LED_6_Pin, Frooastboard Footprints:Everlight 99-235, F.Cu at (428.0, 151.0)
- added D222: RGB_LED_6_Pin, Frooastboard Footprints:Everlight 99-235, F.Cu at (433.6, 148.3)
- added D223: RGB_LED_6_Pin, Frooastboard Footprints:Everlight 99-235, F.Cu at (574.0, 15.3)
- added D228: RGB_LED_6_Pin, Frooastboard Footprints:Everlight 99-235, F.Cu at (428.0, 148.3)
- added D229: RGB_LED_6_Pin, Frooastboard Footprints:Everlight 99-235, F.Cu at (433.6, 156.4)
- added D23: D_Small, Diode_SMD:D_0805_2012Metric, F.Cu at (789.0, 45.4)
- added D231: RGB_LED_6_Pin, Frooastboard Footprints:Everlight 99-235, F.Cu at (433.6, 151.0)
- added D236: RGB_LED_6_Pin, Frooastboard Footprints:Everlight 99-235, F.Cu at (422.4, 148.3)
- added D237: RGB_LED_6_Pin, Frooastboard Footprints:Everlight 99-235, F.Cu at (574.0, 18.0)
- added D239: RGB_LED_6_Pin, Frooastboard Footprints:Everlight 99-235, F.Cu at (456.1, 156.4)
- added D24: D_Small, Diode_SMD:D_0805_2012Metric, F.Cu at (784.8, 54.5)
- added D244: RGB_LED_6_Pin, Frooastboard Footprints:Everlight 99-235, F.Cu at (450.5, 153.7)
- added D245: RGB_LED_6_Pin, Frooastboard Footprints:Everlight 99-235, F.Cu at (450.5, 145.6)
- added D247: RGB_LED_6_Pin, Frooastboard Footprints:Everlight 99-235, F.Cu at (433.6, 153.7)
- added D25: RGB_LED_6_Pin, Frooastboard Footprints:Everlight 99-235, F.Cu at (775.3, 50.8)
- added D252: RGB_LED_6_Pin, Frooastboard Footprints:Everlight 99-235, F.Cu at (478.6, 145.6)
- added D253: RGB_LED_6_Pin, Frooastboard Footprints:Everlight 99-235, F.Cu at (439.3, 145.6)
- added D255: RGB_LED_6_Pin, Frooastboard Footprints:Everlight 99-235, F.Cu at (473.0, 148.3)
- added D26: RGB_LED_6_Pin, Frooastboard Footprints:Everlight 99-235, F.Cu at (775.3, 53.5)
- added D27: D_Small, Diode_SMD:D_0805_2012Metric, F.Cu at (797.9, 42.7)
- added D28: D_Small, Diode_SMD:D_0805_2012Metric, F.Cu at (793.7, 51.7)
- added D29: D_Small, Diode_SMD:D_0805_2012Metric, F.Cu at (789.3, 54.5)
- added D3: RGB_LED_6_Pin, Frooastboard Footprints:Everlight 99-235, F.Cu at (428.0, 156.4)
- added D30: RGB_LED_6_Pin, Frooastboard Footprints:Everlight 99-235, F.Cu at (755.5, 50.3)
- added D31: RGB_LED_6_Pin, Frooastboard Footprints:Everlight 99-235, F.Cu at (773.9, 48.1)
- added D32: RGB_LED_6_Pin, Frooastboard Footprints:Everlight 99-235, F.Cu at (773.9, 42.6)
- added D33: RGB_LED_6_Pin, Frooastboard Footprints:Everlight 99-235, F.Cu at (764.1, 52.3)
- added D34: RGB_LED_6_Pin, Frooastboard Footprints:Everlight 99-235, F.Cu at (785.2, 42.6)
- added D35: RGB_LED_6_Pin, Frooastboard Footprints:Everlight 99-235, F.Cu at (779.5, 45.3)
- added D36: RGB_LED_6_Pin, Frooastboard Footprints:Everlight 99-235, F.Cu at (758.5, 53.0)
- added D37: RGB_LED_6_Pin, Frooastboard Footprints:Everlight 99-235, F.Cu at (764.1, 55.0)
- added D38: RGB_LED_6_Pin, Frooastboard Footprints:Everlight 99-235, F.Cu at (773.9, 45.3)
- added D39: RGB_LED_6_Pin, Frooastboard Footprints:Everlight 99-235, F.Cu at (790.8, 42.6)
- added D4: RGB_LED_6_Pin, Frooastboard Footprints:Everlight 99-235, F.Cu at (755.5, 47.5)
- added D40: RGB_LED_6_Pin, Frooastboard Footprints:Everlight 99-235, F.Cu at (747.2, 54.5)
- added D41: RGB_LED_6_Pin, Frooastboard Footprints:Everlight 99-235, F.Cu at (779.5, 48.1)
- added D42: RGB_LED_6_Pin, Frooastboard Footprints:Everlight 99-235, F.Cu at (752.8, 55.7)
- added D43: RGB_LED_6_Pin, Frooastboard Footprints:Everlight 99-235, F.Cu at (422.4, 245.0)
- added D44: RGB_LED_6_Pin, Frooastboard Footprints:Everlight 99-235, F.Cu at (456.1, 246.1)
- added D45: RGB_LED_6_Pin, Frooastboard Footprints:Everlight 99-235, F.Cu at (443.2, 194.3)
- added D46: RGB_LED_6_Pin, Frooastboard Footprints:Everlight 99-235, F.Cu at (439.3, 244.0)
- added D47: D_Small, Diode_SMD:D_0805_2012Metric, F.Cu at (562.7, 163.7)
- added D48: D_Small, Diode_SMD:D_0805_2012Metric, F.Cu at (562.7, 166.8)
- added D49: D_Small, Diode_SMD:D_0805_2012Metric, F.Cu at (515.4, 210.2)
- added D5: Caps Lock Indicator, LED_SMD:LED_0805_2012Metric, F.Cu at (515.7, 151.7)
- added D50: D_Small, Diode_SMD:D_0805_2012Metric, F.Cu at (480.8, 244.5)
- added D51: D_Small, Diode_SMD:D_0805_2012Metric, F.Cu at (510.9, 207.2)
- added D52: Roll Indicator, LED_SMD:LED_0805_2012Metric, F.Cu at (774.8, 56.2)
- added D53: RGB_LED_6_Pin, Frooastboard Footprints:Everlight 99-235, F.Cu at (448.9, 197.0)
- added D54: D_Small, Diode_SMD:D_0805_2012Metric, F.Cu at (542.5, 183.9)
- added D55: D_Small, Diode_SMD:D_0805_2012Metric, F.Cu at (467.5, 244.5)
- added D56: D_Small, Diode_SMD:D_0805_2012Metric, F.Cu at (463.0, 244.5)
- added D57: D_Small, Diode_SMD:D_0805_2012Metric, F.Cu at (476.4, 244.5)
- added D58: Num Lock Indicator, LED_SMD:LED_0805_2012Metric, F.Cu at (485.3, 244.5)
- added D59: D_Small, Diode_SMD:D_0805_2012Metric, F.Cu at (524.3, 204.1)
- added D6: D_Small, Diode_SMD:D_0805_2012Metric, F.Cu at (793.7, 48.7)
- added D60: D_Small, Diode_SMD:D_0805_2012Metric, F.Cu at (510.9, 213.3)
- added D61: D_Small, Diode_SMD:D_0805_2012Metric, F.Cu at (515.4, 207.2)
- added D62: D_Small, Diode_SMD:D_0805_2012Metric, F.Cu at (515.4, 204.1)
- added D63: D_Small, Diode_SMD:D_0805_2012Metric, F.Cu at (471.9, 244.5)
- added D65: RGB_LED_6_Pin, Frooastboard Footprints:Everlight 99-235, F.Cu at (433.6, 244.0)
- added D66: D_Small, Diode_SMD:D_0805_2012Metric, F.Cu at (519.8, 204.1)
- added D67: D_Small, Diode_SMD:D_0805_2012Metric, F.Cu at (510.9, 204.1)
- added D69: D_Small, Diode_SMD:D_0805_2012Metric, F.Cu at (510.9, 210.2)
- added D7: RGB_LED_6_Pin, Frooastboard Footprints:Everlight 99-235, F.Cu at (769.7, 52.3)
- added D71: RGB_LED_6_Pin, Frooastboard Footprints:Everlight 99-235, F.Cu at (448.9, 194.3)
- added D72: RGB_LED_6_Pin, Frooastboard Footprints:Everlight 99-235, F.Cu at (448.9, 199.7)
- added D73: RGB_LED_6_Pin, Frooastboard Footprints:Everlight 99-235, F.Cu at (454.5, 197.0)
- added D74: RGB_LED_6_Pin, Frooastboard Footprints:Everlight 99-235, F.Cu at (446.7, 243.4)
- added D75: RGB_LED_6_Pin, Frooastboard Footprints:Everlight 99-235, F.Cu at (454.5, 199.7)
- added D76: RGB_LED_6_Pin, Frooastboard Footprints:Everlight 99-235, F.Cu at (444.9, 246.1)
- added D77: RGB_LED_6_Pin, Frooastboard Footprints:Everlight 99-235, F.Cu at (443.2, 199.7)
- added D78: RGB_LED_6_Pin, Frooastboard Footprints:Everlight 99-235, F.Cu at (450.5, 246.1)
- added D79: RGB_LED_6_Pin, Frooastboard Footprints:Everlight 99-235, F.Cu at (458.0, 243.4)
- added D8: D_Small, Diode_SMD:D_0805_2012Metric, F.Cu at (780.4, 50.8)
- added D80: RGB_LED_6_Pin, Frooastboard Footprints:Everlight 99-235, F.Cu at (428.0, 244.0)
- added D81: RGB_LED_6_Pin, Frooastboard Footprints:Everlight 99-235, F.Cu at (454.5, 194.3)
- added D82: RGB_LED_6_Pin, Frooastboard Footprints:Everlight 99-235, F.Cu at (452.4, 243.4)
- added D83: RGB_LED_6_Pin, Frooastboard Footprints:Everlight 99-235, F.Cu at (443.2, 197.0)
- added D9: D_Small, Diode_SMD:D_0805_2012Metric, F.Cu at (843.5, 2.25)
- added J1: SW Interface, Connector_PinHeader_1.27mm:PinHeader_1x05_P1.27mm_Vertical, F.Cu at (438.5, 266.5)
- added J10: F Row CS, Frooastboard Footprints:PinHeader_1x16_P1.27mm_Vertical, F.Cu at (506.1, 23.9)
- added J11: F Row SW, Frooastboard Footprints:PinHeader_1x06_P1.27mm_Vertical, F.Cu at (510.2, 23.9)
- added J12: Conn_01x06_Male, Frooastboard Footprints:PinHeader_1x06_P1.27mm_Vertical, F.Cu at (746.5, 45.0)
- added J13: Conn_01x16_Male, Frooastboard Footprints:PinHeader_1x16_P1.27mm_Vertical, F.Cu at (742.3, -17.8)
- added J14: Conn_01x10_Male, Frooastboard Footprints:PinHeader_1x10_P1.27mm_Vertical, F.Cu at (742.3, 45.0)
- added J15: F Row, Frooastboard Footprints:PinHeader_1x10_P1.27mm_Vertical, F.Cu at (499.5, 23.9)
- added J16: F Row USB, Frooastboard Footprints:PinHeader_1x04_P1.27mm_Vertical, F.Cu at (510.2, 33.6)
- added J17: Numpad, Frooastboard Footprints:PinHeader_1x13_P1.27mm_Vertical, F.Cu at (495.4, 23.9)
- added J18: Conn_01x04_Male, Frooastboard Footprints:PinHeader_1x04_P1.27mm_Vertical, F.Cu at (750.6, 45.0)
- added J19: Conn_01x15_Male, Frooastboard Footprints:PinHeader_1x15_P1.27mm_Vertical, F.Cu at (421.7, 224.0)
- added J2: Conn_01x16, Frooastboard Footprints:PinHeader_1x16_P1.27mm_Vertical, F.Cu at (421.7, 252.6)
- added J20: Conn_01x06_Male, Frooastboard Footprints:PinHeader_1x06_P1.27mm_Vertical, F.Cu at (453.1, 184.7)
- added J21: Conn_01x13_Male, Frooastboard Footprints:PinHeader_1x13_P1.27mm_Vertical, F.Cu at (506.6, 204.3)
- added J3: Conn_01x06, Frooastboard Footprints:PinHeader_1x06_P1.27mm_Vertical, F.Cu at (439.7, 252.6)
- added J4: Conn_01x06, Frooastboard Footprints:PinHeader_1x06_P1.27mm_Vertical, F.Cu at (425.8, 269.9)
- added J5: Conn_01x10, Frooastboard Footprints:PinHeader_1x10_P1.27mm_Vertical, F.Cu at (421.7, 275.0)
- added J6: Conn_01x12, Frooastboard Footprints:PinHeader_1x12_P1.27mm_Vertical, F.Cu at (425.8, 252.6)
- added J7: Conn_01x04, Frooastboard Footprints:PinHeader_1x04_P1.27mm_Vertical, F.Cu at (443.8, 252.6)
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
Commit message: backup
Parts:
- moved C10 472.2 mm to (67.5, 12.9)
- moved C2 471.0 mm to (71.4, 8.40)
- moved C1 466.6 mm to (69.0, 16.5)
- moved C5 466.3 mm to (73.4, 12.5)
- moved R24 464.5 mm to (43.1, 87.0)
- moved C11 463.1 mm to (73.2, 17.6)
- moved C6 461.0 mm to (79.3, 31.7)
- moved C7 460.8 mm to (78.7, 22.5)
- moved C9 460.4 mm to (82.8, 23.8)
- moved R2 459.5 mm to (70.5, 23.0)
- moved C12 457.7 mm to (83.9, 18.3)
- moved R1 457.6 mm to (65.3, 20.7)
- moved C13 456.7 mm to (78.6, 27.8)
- moved C4 456.6 mm to (88.6, 16.9)
- moved C3 456.2 mm to (85.4, 27.2)
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Other:
- board outline added: 52.7 x 21.2 mm

Commit message: antenna
Parts:
- REF**: moved to B.Cu
- moved L3 50.2 mm to (50.9, 45.8), turned to -90 degrees
- moved L1 48.2 mm to (49.9, 42.9), turned to 90 degrees
- moved L2 48.2 mm to (50.9, 43.9), turned to -90 degrees
- moved C12 44.1 mm to (50.9, 47.6), turned to -90 degrees
- moved C3 42.5 mm to (51.4, 52.8)
- moved C4 40.2 mm to (61.9, 46.9)
- moved C10 39.7 mm to (63.3, 52.4), turned to 90 degrees
- moved C11 39.1 mm to (54.6, 52.0), turned to -90 degrees
- moved C9 38.4 mm to (47.9, 39.9), turned to 90 degrees
- moved C8 38.3 mm to (51.2, 39.7), turned to 90 degrees
- moved C13 35.2 mm to (50.9, 49.5), turned to -90 degrees
- moved C5 33.0 mm to (61.9, 43.5)
- moved R2 30.1 mm to (54.8, 48.7), turned to -90 degrees
- moved C2 30.0 mm to (60.5, 36.4)
- moved Y1 27.6 mm to (66.2, 44.2), turned to 90 degrees
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Routing:
- net /ANT: track 0.00 -> 3.73 mm
Other:
- board outline removed

Commit message: do some stuff (probably redo that)
Parts:
- moved TP3 27.5 mm to (52.6, 37.7)
- moved C3 13.6 mm to (61.6, 43.9), turned to 90 degrees
- moved C6 10.6 mm to (59.8, 39.8), turned to 180 degrees
- moved C10 9.66 mm to (54.1, 49.3), turned to -90 degrees
- moved C1 6.16 mm to (62.7, 43.9), turned to 90 degrees
- moved C7 6.15 mm to (60.1, 42.4), turned to 0 degrees
- moved C11 6.14 mm to (58.6, 47.4), turned to 90 degrees
- moved R2 5.73 mm to (60.1, 46.6), turned to 90 degrees
- moved Y2 5.37 mm to (56.4, 47.6), turned to -90 degrees
- moved Y1 5.17 mm to (62.3, 40.8), turned to -90 degrees
- moved R1 4.89 mm to (49.6, 38.6), turned to 180 degrees
- moved C2 3.77 mm to (57.4, 38.5)
- moved C4 3.12 mm to (60.1, 44.4)
- moved C9 2.31 mm to (49.9, 41.0)
- moved C5 1.83 mm to (60.1, 43.4)
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Connections:
- L1 pad 1: ANT2 -> ANT1
- L2 pad 1: ANT2 -> ANT1
- L2 pad 2: ANT1 -> ANT2
- L3 pad 1: ANT1 -> ANT2
Routing:
- net GND: track 0.00 -> 55.7 mm, vias 0 -> 8
- net +3V3: track 0.00 -> 43.2 mm, vias 0 -> 4
- net NRF_IREF: track 0.00 -> 11.1 mm, vias 0 -> 2
- net XC2: track 0.00 -> 7.14 mm, vias 0 -> 2
- net XL1: track 0.00 -> 7.12 mm
- net XL2: track 0.00 -> 6.56 mm
- net NRF_RESET: track 0.00 -> 6.54 mm, vias 0 -> 2
- net XC1: track 0.00 -> 5.20 mm
- net VDD_PA: track 0.00 -> 4.79 mm
- net ANT2: track 0.00 -> 3.75 mm
- net ANT1: track 0.00 -> 3.51 mm
- net DEC1: track 0.00 -> 2.38 mm
- net DEC2: track 0.00 -> 2.17 mm
- net NRF_TXD: track 0.00 -> 1.39 mm, vias 0 -> 1
- net Net-(C12-Pad1): track 0.00 -> 0.92 mm
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
Commit message: mmmhhh rp2040
Parts:
- removed C27: 100n, Capacitor_SMD:C_0805_2012Metric
- moved R11 153.1 mm to (25.2, 66.8)
- moved C33 147.9 mm to (21.2, 72.7)
- moved C35 146.6 mm to (18.6, 67.8)
- moved R6 131.7 mm to (27.6, 73.9)
- moved C28 124.7 mm to (35.2, 77.0)
- moved C34 122.0 mm to (28.7, 79.5)
- moved R7 117.9 mm to (37.2, 67.7)
- moved R5 97.4 mm to (75.5, 56.2), turned to 90 degrees
- moved C19 96.2 mm to (71.0, 60.0), turned to -90 degrees
- moved R4 91.5 mm to (73.6, 56.2), turned to 90 degrees
- moved C21 86.0 mm to (90.8, 55.5)
- moved C18 85.9 mm to (83.2, 58.0), turned to 90 degrees
- moved R9 84.3 mm to (75.5, 66.0), turned to 180 degrees
- moved R3 82.4 mm to (95.1, 64.3), turned to 90 degrees
- moved C14 78.3 mm to (94.3, 67.8)
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Connections:
- net Net-(J7-Pad3) renamed /DP
- net Net-(J7-Pad4) renamed /DN
- R9 pad 1: QSPI_CS -> /QSPI_CS_TP
- TP5 pad 2: QSPI_CS -> /QSPI_CS_TP
Routing:
- net GND: track 55.7 -> 18.7 mm, vias 8 -> 2
- net +3V3: track 43.2 -> 9.95 mm, vias 4 -> 3
- net +1V1: track 0.00 -> 18.8 mm, vias 0 -> 2
- net Net-(J6-Pad1): track 0.00 -> 15.7 mm, vias 0 -> 1
- net XTAL1: track 0.00 -> 14.3 mm
- net RP_D-: track 0.00 -> 13.1 mm, vias 0 -> 2
- net Net-(J6-Pad2): track 0.00 -> 13.1 mm, vias 0 -> 1
- net Net-(J6-Pad5): track 0.00 -> 12.5 mm, vias 0 -> 1
- net RP_D+: track 0.00 -> 12.2 mm, vias 0 -> 2
- net Net-(J6-Pad3): track 0.00 -> 12.0 mm, vias 0 -> 1
- net Net-(J6-Pad6): track 0.00 -> 11.5 mm, vias 0 -> 1
- net Net-(J6-Pad4): track 0.00 -> 11.2 mm, vias 0 -> 1
- net /DP: track 0.00 -> 11.1 mm
- net /DN: track 0.00 -> 11.1 mm
- net NRF_IREF: track 11.1 -> 0.00 mm, vias 2 -> 0
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- added copper zone on In1.Cu, net +3V3
- added copper zone on In2.Cu, net GND

Commit message: Update Frooastboard Walnut Modular.kicad_pcb
Parts:
- moved TP5 51.7 mm to (67.2, 66.3)
- moved C25 30.0 mm to (82.2, 64.9), turned to 0 degrees
- moved J1 30.0 mm to (85.6, 72.6), turned to 180 degrees
- moved C24 20.5 mm to (88.6, 68.5), turned to -90 degrees
- moved C23 19.9 mm to (90.5, 69.3), turned to -90 degrees
Routing:
- net Net-(J5-Pad6): track 0.00 -> 20.1 mm, vias 0 -> 1
- net Net-(J5-Pad5): track 0.00 -> 19.5 mm, vias 0 -> 1
- net Net-(J5-Pad10): track 0.00 -> 19.4 mm, vias 0 -> 1
- net Net-(J5-Pad8): track 0.00 -> 18.7 mm, vias 0 -> 2
- net Net-(J5-Pad4): track 0.00 -> 18.7 mm, vias 0 -> 1
- net Net-(J5-Pad9): track 0.94 -> 18.9 mm, vias 1 -> 2
- net Net-(J5-Pad3): track 0.00 -> 17.9 mm, vias 0 -> 1
- net Net-(J5-Pad2): track 0.00 -> 17.4 mm, vias 0 -> 1
- net Net-(J5-Pad7): track 0.00 -> 17.2 mm, vias 0 -> 2
- net Net-(J5-Pad1): track 0.00 -> 15.9 mm, vias 0 -> 1
- net GND: track 18.7 -> 30.7 mm
- net +3V3: track 9.95 -> 21.3 mm, vias 3 -> 5
- net Net-(J6-Pad7): track 5.35 -> 14.2 mm
- net Net-(J6-Pad8): track 5.61 -> 13.2 mm
- net RP_D+: track 12.2 -> 12.9 mm
