File: Frooastboard Walnut Modular/KiCad Project/Frooastboard Walnut Modular.kicad_pcb (KiCad board)
At the start: 4 copper layers, 379 parts, among them J1 SW Interface, J10 F Row CS, J11 F Row SW, J12 Conn_01x06_Male, J13 Conn_01x16_Male, J14 Conn_01x10_Male, J15 F Row, J16 F Row USB, J17 Numpad, J18 Conn_01x04_Male, J19 Conn_01x15_Male, J2 Conn_01x16, J20 Conn_01x06_Male, J21 Conn_01x13_Male, J3 Conn_01x06, J4 Conn_01x06, J5 Conn_01x10, J6 Conn_01x12, J7 Conn_01x04, J8 Numpad CS, J9 Numpad SW, U1 RP2040, U3 W25Q32JVZP, U5 IS31FL3733-QF, Y3 12MHz

Commit message: change some stuff maybe finally get started
Parts:
- removed C18, C19, C20, C21, C22, C23, C24, C25, C26: 100n, Capacitor_SMD:C_0805_2012Metric
- removed C28: 0.1u, Capacitor_SMD:C_0805_2012Metric
- removed C33: 10u, Capacitor_SMD:C_0805_2012Metric
- removed C34, C35: 10u, Capacitor_Tantalum_SMD:CP_EIA-2012-15_AVX-P
- removed R11: 100k, Resistor_SMD:R_0805_2012Metric
- removed R23, R24: 27R, Resistor_SMD:R_0805_2012Metric
- removed TP5: QSPI_CS, Connector_PinHeader_1.27mm:PinHeader_1x02_P1.27mm_Vertical
- removed U5: IS31FL3733-QF, Package_DFN_QFN:QFN-48-1EP_6x6mm_P0.4mm_EP4.2x4.2mm
- removed Y3: 12MHz, Crystal:Crystal_SMD_3225-4Pin_3.2x2.5mm
- added C1: 0.1u, Capacitor_SMD:C_0402_1005Metric, F.Cu at (145.0, 86.6)
- added C10: 100n, Capacitor_SMD:C_0402_1005Metric, F.Cu at (159.9, 26.7)
- added C11: 100n, Capacitor_SMD:C_0402_1005Metric, F.Cu at (159.9, 28.7)
- added C12: 100n, Capacitor_SMD:C_0402_1005Metric, F.Cu at (159.9, 30.7)
- added C13: 100n, Capacitor_SMD:C_0402_1005Metric, F.Cu at (159.9, 32.7)
- added C2: 10u, Capacitor_SMD:C_0402_1005Metric, F.Cu at (145.0, 88.5)
- added C3: 10u, Capacitor_Tantalum_SMD:CP_EIA-2012-15_AVX-P, F.Cu at (144.9, 91.4)
- added C4: 10u, Capacitor_Tantalum_SMD:CP_EIA-2012-15_AVX-P, F.Cu at (144.9, 94.2)
- added C5: 22p, Capacitor_SMD:C_0402_1005Metric, F.Cu at (160.4, 55.6)
- added C6: 22p, Capacitor_SMD:C_0402_1005Metric, F.Cu at (160.4, 57.6)
- added C7: 10u, Capacitor_SMD:C_0402_1005Metric, F.Cu at (157.0, 32.7)
- added C8: 100n, Capacitor_SMD:C_0402_1005Metric, F.Cu at (157.0, 34.6)
- added C9: 100n, Capacitor_SMD:C_0402_1005Metric, F.Cu at (159.9, 24.8)
- added M1: Frooastboard_MM2040, Frooastboard Footprints:MM2040, F.Cu at (0.25, 0.25)
- added M2: Frooastboard_MM2040, Frooastboard Footprints:MM2040, F.Cu at (0.25, 3.75)
- added R1: 100k, Resistor_SMD:R_0402_1005Metric, F.Cu at (167.9, 89.1)
- added R10: 1k, Resistor_SMD:R_0402_1005Metric, F.Cu at (57.4, 36.1)
- added R2: 100k, Resistor_SMD:R_0402_1005Metric, F.Cu at (167.9, 91.1)
- added TP1: QSPI_CS, Connector_PinHeader_1.00mm:PinHeader_1x02_P1.00mm_Vertical, F.Cu at (65.5, 34.1)
- added U2: RP2040, Frooastboard Footprints:RP2040-QFN-56, F.Cu at (40.5, 36.2)
- added Y1: 12MHz, Crystal:Crystal_SMD_3225-4Pin_3.2x2.5mm, F.Cu at (156.2, 56.5)
- C14: value 22p -> 100n; footprint Capacitor_SMD:C_0805_2012Metric -> Capacitor_SMD:C_0402_1005Metric
- C15: value 22p -> 10u; footprint Capacitor_SMD:C_0805_2012Metric -> Capacitor_SMD:C_0402_1005Metric
- C16, C17: value 10u -> 100n; footprint Capacitor_SMD:C_0805_2012Metric -> Capacitor_SMD:C_0402_1005Metric
- J1: value SW Interface -> Conn_01x16; footprint Connector_PinHeader_1.27mm:PinHeader_1x05_P1.27mm_Vertical -> Frooastboard Footprints:PinHeader_1x16_P1.27mm_Vertical
- J10, J13, J8: footprint Frooastboard Footprints:PinHeader_1x16_P1.27mm_Vertical -> Connector_PinHeader_1.27mm:PinHeader_1x16_P1.27mm_Vertical
- J11, J12, J20, J9: footprint Frooastboard Footprints:PinHeader_1x06_P1.27mm_Vertical -> Connector_PinHeader_1.27mm:PinHeader_1x06_P1.27mm_Vertical
- J14, J15: footprint Frooastboard Footprints:PinHeader_1x10_P1.27mm_Vertical -> Connector_PinHeader_1.27mm:PinHeader_1x10_P1.27mm_Vertical
- J16, J18, J7: footprint Frooastboard Footprints:PinHeader_1x04_P1.27mm_Vertical -> Connector_PinHeader_1.27mm:PinHeader_1x04_P1.27mm_Vertical
- J17, J21: footprint Frooastboard Footprints:PinHeader_1x13_P1.27mm_Vertical -> Connector_PinHeader_1.27mm:PinHeader_1x13_P1.27mm_Vertical
- J19: footprint Frooastboard Footprints:PinHeader_1x15_P1.27mm_Vertical -> Connector_PinHeader_1.27mm:PinHeader_1x15_P1.27mm_Vertical
- J2: value Conn_01x16 -> Conn_01x06; footprint Frooastboard Footprints:PinHeader_1x16_P1.27mm_Vertical -> Frooastboard Footprints:PinHeader_1x06_P1.27mm_Vertical
- J4: value Conn_01x06 -> Conn_01x10; footprint Frooastboard Footprints:PinHeader_1x06_P1.27mm_Vertical -> Frooastboard Footprints:PinHeader_1x10_P1.27mm_Vertical
- J5: value Conn_01x10 -> Conn_01x12; footprint Frooastboard Footprints:PinHeader_1x10_P1.27mm_Vertical -> Frooastboard Footprints:PinHeader_1x12_P1.27mm_Vertical
- J6: value Conn_01x12 -> SW Interface; footprint Frooastboard Footprints:PinHeader_1x12_P1.27mm_Vertical -> Connector_PinHeader_1.27mm:PinHeader_1x05_P1.27mm_Vertical
- R3: value 1k -> 20k; footprint Resistor_SMD:R_0805_2012Metric -> Resistor_SMD:R_0402_1005Metric
- R4: value 2k -> 10k; footprint Resistor_SMD:R_0805_2012Metric -> Resistor_SMD:R_0402_1005Metric
- R5: footprint Resistor_SMD:R_0805_2012Metric -> Resistor_SMD:R_0402_1005Metric
- R6: value 20k -> 2k; footprint Resistor_SMD:R_0805_2012Metric -> Resistor_SMD:R_0402_1005Metric
- R7: value 100k -> 1k; footprint Resistor_SMD:R_0805_2012Metric -> Resistor_SMD:R_0402_1005Metric
- R8: value 10k -> 27R; footprint Resistor_SMD:R_0805_2012Metric -> Resistor_SMD:R_0402_1005Metric
- R9: value 1k -> 27R; footprint Resistor_SMD:R_0805_2012Metric -> Resistor_SMD:R_0402_1005Metric
- U1: value RP2040 -> IS31FL3733-QF; footprint Frooastboard Footprints:RP2040-QFN-56 -> Package_DFN_QFN:QFN-48-1EP_6x6mm_P0.4mm_EP4.2x4.2mm
- moved MX4 382.5 mm to (554.2, 274.6)
- moved MX1 359.1 mm to (554.2, 214.0)
- moved MX12 347.5 mm to (594.6, 274.6)
- moved MX3 339.5 mm to (554.2, 254.4)
- moved MX7 339.5 mm to (574.4, 254.4)
- moved D9 333.2 mm to (627.2, 255.6)
- moved MX13 328.4 mm to (614.8, 214.0)
- moved MX2 327.4 mm to (554.2, 234.2)
- moved MX11 325.4 mm to (594.6, 254.4)
- moved MX14 315.4 mm to (614.8, 234.2)
- moved MX8 315.3 mm to (574.4, 274.6)
- moved MX16 306.3 mm to (614.8, 274.6)
- moved MX5 300.0 mm to (574.4, 214.0)
- moved MX15 298.5 mm to (614.8, 254.4)
- moved R26 288.7 mm to (635.4, 205.4)
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Connections:
- C14 pad 2: XTAL1 -> +3V3
- C15 pad 1: GND -> +1V1
- C15 pad 2: Net-(C15-Pad2) -> GND
- C17 pad 1: +3V3 -> +1V1
- J1 pad 1: GND -> Net-(J1-Pin_1)
- J1 pad 2: +3V3 -> Net-(J1-Pin_2)
- J1 pad 3: RP_RESET -> Net-(J1-Pin_3)
- J1 pad 4: SWDIO -> Net-(J1-Pin_4)
- J1 pad 5: SWCLK -> Net-(J1-Pin_5)
- J2 pad 1: Net-(J2-Pad1) -> Net-(J2-Pin_1)
- J2 pad 2: Net-(J2-Pad2) -> Net-(J2-Pin_2)
- J2 pad 3: Net-(J2-Pad3) -> Net-(J2-Pin_3)
- J2 pad 4: Net-(J2-Pad4) -> Net-(J2-Pin_4)
- J2 pad 5: Net-(J2-Pad5) -> Net-(J2-Pin_5)
- J2 pad 6: Net-(J2-Pad6) -> Net-(J2-Pin_6)
- J3 pad 1: Net-(J3-Pad1) -> Net-(J3-Pin_1)
- J3 pad 2: Net-(J3-Pad2) -> Net-(J3-Pin_2)
- J3 pad 3: Net-(J3-Pad3) -> Net-(J3-Pin_3)
- J3 pad 4: Net-(J3-Pad4) -> Net-(J3-Pin_4)
- J3 pad 5: Net-(J3-Pad5) -> Net-(J3-Pin_5)
- J3 pad 6: Net-(J3-Pad6) -> Net-(J3-Pin_6)
- J5 pad 1: Net-(J5-Pad1) -> Net-(J5-Pin_1)
- J5 pad 10: Net-(J5-Pad10) -> Net-(J5-Pin_10)
- J5 pad 2: Net-(J5-Pad2) -> Net-(J5-Pin_2)
- J5 pad 3: Net-(J5-Pad3) -> Net-(J5-Pin_3)
- J5 pad 4: Net-(J5-Pad4) -> Net-(J5-Pin_4)
- J5 pad 5: Net-(J5-Pad5) -> Net-(J5-Pin_5)
- J5 pad 6: Net-(J5-Pad6) -> Net-(J5-Pin_6)
- J5 pad 7: Net-(J5-Pad7) -> Net-(J5-Pin_7)
- J5 pad 8: Net-(J5-Pad8) -> Net-(J5-Pin_8)
- J5 pad 9: Net-(J5-Pad9) -> Net-(J5-Pin_9)
- J6 pad 1: Net-(J6-Pad1) -> GND
- J6 pad 2: Net-(J6-Pad2) -> +3V3
- J6 pad 3: Net-(J6-Pad3) -> RP_RESET
- J6 pad 4: Net-(J6-Pad4) -> SWDIO
- J6 pad 5: Net-(J6-Pad5) -> SWCLK
- J7 pad 3: /DP -> /MM2040/DP
- J7 pad 4: /DN -> /MM2040/DN
- R3 pad 1: XTAL2 -> GND
- R3 pad 2: Net-(C15-Pad2) -> Net-(U1-RSET)
- R4 pad 1: SDA -> +3V3
- R4 pad 2: +3V3 -> RP_RESET
- R5 pad 1: SCL -> SDA
- R6 pad 1: GND -> SCL
- R6 pad 2: Net-(R6-Pad2) -> +3V3
- R7 pad 1: GND -> XTAL2
- R8 pad 1: +3V3 -> RP_D+
- R8 pad 2: RP_RESET -> /MM2040/DP
- R9 pad 1: /QSPI_CS_TP -> RP_D-
- R9 pad 2: QSPI_CS -> /MM2040/DN
- U1 pad 1: +3V3 -> unconnected-(U1-NC-Pad1)
- U1 pad 10: +3V3 -> Net-(J3-Pin_2)
- U1 pad 11: Net-(J5-Pad9) -> Net-(J3-Pin_3)
- U1 pad 12: Net-(J5-Pad10) -> GND
- U1 pad 13: Net-(J6-Pad1) -> Net-(J3-Pin_4)
- U1 pad 14: Net-(J6-Pad2) -> Net-(J3-Pin_5)
- U1 pad 15: Net-(J6-Pad3) -> Net-(J3-Pin_6)
- U1 pad 16: Net-(J6-Pad4) -> Net-(J1-Pin_1)
- U1 pad 17: Net-(J6-Pad5) -> Net-(J1-Pin_2)
- U1 pad 18: Net-(J6-Pad6) -> Net-(J1-Pin_3)
- U1 pad 19: GND -> Net-(J1-Pin_4)
- U1 pad 2: Net-(J5-Pad1) -> Net-(J2-Pin_1)
- U1 pad 20: XTAL1 -> +3V3
- U1 pad 21: XTAL2 -> Net-(J1-Pin_5)
- U1 pad 22: +3V3 -> Net-(J1-Pin_6)
- U1 pad 23: +1V1 -> Net-(J1-Pin_7)
- U1 pad 24: SWCLK -> Net-(J1-Pin_8)
- U1 pad 25: SWDIO -> Net-(J1-Pin_9)
- U1 pad 26: RP_RESET -> Net-(J1-Pin_10)
- U1 pad 27: Net-(J6-Pad7) -> Net-(J1-Pin_11)
- U1 pad 28: Net-(J6-Pad8) -> Net-(J1-Pin_12)
- U1 pad 29: Net-(J6-Pad9) -> +3V3
- U1 pad 3: Net-(J5-Pad2) -> Net-(J2-Pin_2)
- U1 pad 30: Net-(J6-Pad10) -> Net-(J1-Pin_13)
- U1 pad 31: Net-(J6-Pad11) -> Net-(J1-Pin_14)
- U1 pad 32: NRF_MISO -> Net-(J1-Pin_15)
- U1 pad 33: +3V3 -> Net-(J1-Pin_16)
- U1 pad 34: NRF_REQN -> GND
- U1 pad 35: NRF_RDYN -> Net-(U1-RSET)
- U1 pad 36: NRF_SCK -> unconnected-(U1-NC-Pad36)
- U1 pad 37: NRF_MOSI -> +3V3
- U1 pad 38: BATTERY_VOLTAGE -> +3V3
- U1 pad 39: unconnected-(U1-Pad39) -> +3V3
- U1 pad 4: Net-(J5-Pad3) -> Net-(J2-Pin_3)
- U1 pad 40: SDA -> unconnected-(U1-SYNC-Pad40)
- U1 pad 41: SCL -> SDA
- U1 pad 42: +3V3 -> SCL
- U1 pad 43: +3V3 -> GND
- U1 pad 44: +3V3 -> GND
- U1 pad 45: +1V1 -> unconnected-(U1-~{INTB}-Pad45)
- U1 pad 46: RP_D- -> Net-(U1-~{SDB})
- U1 pad 47: RP_D+ -> Net-(U1-IICRST)
- U1 pad 48: +3V3 -> GND
- U1 pad 49: +3V3 -> GND
- U1 pad 5: Net-(J5-Pad4) -> GND
- U1 pad 6: Net-(J5-Pad5) -> Net-(J2-Pin_4)
- U1 pad 7: Net-(J5-Pad6) -> Net-(J2-Pin_5)
- U1 pad 8: Net-(J5-Pad7) -> Net-(J2-Pin_6)
- U1 pad 9: Net-(J5-Pad8) -> Net-(J3-Pin_1)
Routing:
- net GND: track 105.5 -> 0.00 mm, vias 14 -> 0
- net +3V3: track 96.1 -> 0.00 mm, vias 16 -> 0
- net RP_RESET: track 49.1 -> 0.00 mm, vias 4 -> 0
- net SCL: track 48.1 -> 0.00 mm, vias 3 -> 0
- net SDA: track 45.6 -> 0.00 mm, vias 3 -> 0
- net SWDIO: track 44.1 -> 0.00 mm, vias 2 -> 0
- net SWCLK: track 39.1 -> 0.00 mm, vias 2 -> 0
- net Net-(J4-Pin_6): track 28.0 -> 0.00 mm, vias 2 -> 0
- net Net-(J4-Pin_5): track 23.6 -> 0.00 mm, vias 2 -> 0
- net Net-(J2-Pad14): track 21.0 -> 0.00 mm, vias 1 -> 0
- net Net-(J4-Pin_4): track 20.7 -> 0.00 mm, vias 2 -> 0
- net Net-(J5-Pad6): track 20.1 -> 0.00 mm, vias 1 -> 0
- net Net-(J5-Pad5): track 19.5 -> 0.00 mm, vias 1 -> 0
- net Net-(J5-Pad10): track 19.4 -> 0.00 mm, vias 1 -> 0
- net Net-(J5-Pad9): track 19.1 -> 0.00 mm, vias 2 -> 0
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- added copper zone on In2.Cu, net +3V3
- added copper zone on In1.Cu, net GND
- removed copper zone on In1.Cu, net +3V3
- removed copper zone on In2.Cu, net GND

Commit message: some errors and board outline
Parts:
- J7: footprint Connector_PinHeader_1.27mm:PinHeader_1x04_P1.27mm_Vertical -> Frooastboard Footprints:PinHeader_1x04_P1.27mm_Vertical
- moved J4 37.5 mm to (19.6, 55.9), turned to 90 degrees
- moved J1 36.3 mm to (148.1, 100.6), turned to 90 degrees
- moved J5 35.5 mm to (47.8, 55.9), turned to 90 degrees
- moved J7 33.9 mm to (82.7, 48.3), turned to 90 degrees
- moved R8 27.1 mm to (85.2, 45.6), turned to -90 degrees
- moved R9 25.2 mm to (86.5, 45.6), turned to -90 degrees
- moved U2 15.7 mm to (39.4, 51.8), turned to 90 degrees
- moved TP1 9.94 mm to (55.6, 33.3)
- moved C14 9.54 mm to (48.7, 38.4), turned to 180 degrees
- moved R10 2.59 mm to (54.9, 36.6), turned to -90 degrees
- moved U3 1.05 mm to (51.1, 35.1), turned to 180 degrees
Routing:
- net Net-(J4-Pin_1): track 0.00 -> 16.4 mm
- net Net-(J5-Pin_2): track 0.00 -> 9.89 mm
- net Net-(J5-Pin_1): track 0.00 -> 9.37 mm
- net +3V3: track 0.00 -> 7.03 mm, vias 0 -> 1
- net QSPI_SD3: track 0.00 -> 3.88 mm
- net QSPI_CLK: track 0.00 -> 3.65 mm
- net QSPI_SD0: track 0.00 -> 2.77 mm
- net QSPI_CS: track 0.00 -> 2.64 mm
- net QSPI_SD1: track 0.00 -> 2.49 mm
- net QSPI_SD2: track 0.00 -> 2.37 mm
- net GND: track 0.00 -> 2.28 mm
Other:
- board outline added: 43.4 x 25.7 mm

Commit message: some more stuff changed
Parts:
- added U4: LM317_SOT-223, Package_TO_SOT_SMD:SOT-223-3_TabPin2, F.Cu at (93.2, 59.0)
Connections:
- J5 pad 12: unconnected-(J5-Pin_12-Pad12) -> Net-(J5-Pin_12)
- U2 pad 32: unconnected-(U2-GPIO21-Pad32) -> Net-(J5-Pin_12)
Routing:
- net Net-(J4-Pin_2): track 0.00 -> 21.7 mm
- net Net-(J4-Pin_4): track 0.00 -> 21.1 mm, vias 0 -> 1
- net Net-(J4-Pin_3): track 0.00 -> 20.1 mm
- net Net-(J4-Pin_6): track 0.00 -> 18.7 mm, vias 0 -> 1
- net Net-(J4-Pin_5): track 0.00 -> 18.4 mm, vias 0 -> 1
- net Net-(J4-Pin_7): track 0.00 -> 16.9 mm, vias 0 -> 1
- net Net-(J4-Pin_9): track 0.00 -> 16.2 mm, vias 0 -> 2
- net Net-(J4-Pin_10): track 0.00 -> 16.0 mm, vias 0 -> 2
- net Net-(J4-Pin_8): track 0.00 -> 15.7 mm, vias 0 -> 1
- net Net-(J5-Pin_1): track 9.37 -> 1.23 mm
- net Net-(J4-Pin_1): track 16.4 -> 22.7 mm
- net Net-(J5-Pin_2): track 9.89 -> 5.11 mm
- net +3V3: track 7.03 -> 11.7 mm, vias 1 -> 2
- net QSPI_SD3: track 3.88 -> 0.00 mm
- net QSPI_CLK: track 3.65 -> 0.00 mm
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
Commit message: some more progress
Parts:
- removed U4: LM317_SOT-223, Package_TO_SOT_SMD:SOT-223-3_TabPin2
- added U5: LM317L_SOT-89, Package_TO_SOT_SMD:SOT-89-3, F.Cu at (57.3, 49.6)
- TP1: footprint Connector_PinHeader_1.00mm:PinHeader_1x02_P1.00mm_Vertical -> Connector_PinHeader_1.27mm:PinHeader_1x02_P1.27mm_Vertical
- moved R6 118.1 mm to (38.3, 46.4), turned to 90 degrees
- moved R5 116.4 mm to (40.6, 46.4), turned to 90 degrees
- moved R7 114.8 mm to (49.4, 48.8)
- moved C5 111.8 mm to (48.6, 53.2), turned to 180 degrees
- moved C6 109.5 mm to (51.3, 48.8), turned to 180 degrees
- moved Y1 107.2 mm to (49.2, 51.0)
- moved C10 84.0 mm to (79.2, 49.8)
- moved C11 84.0 mm to (79.2, 51.7)
- moved C12 84.0 mm to (79.2, 53.7)
- moved C13 84.0 mm to (79.2, 55.7)
- moved C9 84.0 mm to (79.2, 47.8)
- moved C15 84.0 mm to (92.1, 51.0)
- moved C16 84.0 mm to (92.1, 52.9)
- moved C17 84.0 mm to (92.1, 54.9)
- moved C7 84.0 mm to (76.3, 55.7)
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Routing:
- net GND: track 3.85 -> 27.1 mm, vias 0 -> 2
- net QSPI_CS: track 0.00 -> 21.8 mm
- net QSPI_SD1: track 0.00 -> 17.9 mm
- net QSPI_SD2: track 0.00 -> 15.1 mm
- net /MM2040/DN: track 0.00 -> 12.2 mm, vias 0 -> 1
- net /MM2040/DP: track 0.00 -> 11.2 mm, vias 0 -> 1
- net +5V: track 0.00 -> 10.7 mm
- net QSPI_SD3: track 0.00 -> 9.82 mm
- net QSPI_CLK: track 0.00 -> 8.68 mm
- net QSPI_SD0: track 0.00 -> 8.09 mm
- net /MM2040/QSPI_CS_TP: track 0.00 -> 7.23 mm
- net RP_D+: track 0.00 -> 5.52 mm, vias 0 -> 3
- net +1V1: track 0.00 -> 5.33 mm
- net RP_D-: track 0.00 -> 5.12 mm, vias 0 -> 3
- net +3V3: track 11.7 -> 13.6 mm
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Other:
- board size 43.4 x 25.7 mm -> 45.7 x 25.7 mm

Commit message: Main Module placement
Parts:
- moved C3 69.0 mm to (114.9, 29.3)
- moved C4 69.0 mm to (114.9, 32.1)
- moved U1 69.0 mm to (122.1, 28.5)
- moved C1 69.0 mm to (115.0, 24.4)
- moved C2 69.0 mm to (115.0, 26.4)
- moved J1 69.0 mm to (118.1, 38.4)
- moved J2 69.0 mm to (155.2, 32.7)
- moved J3 69.0 mm to (159.4, 32.7)
- moved R1 69.0 mm to (137.8, 26.9)
- moved R3 69.0 mm to (137.8, 31.3)
- moved R2 69.0 mm to (137.8, 28.9)
- moved U5 0.78 mm to (56.6, 49.9)
- moved Y1 0.52 mm to (48.7, 51.0)
Routing:
- net Net-(J5-Pin_1): track 1.23 -> 7.88 mm
- net Net-(J5-Pin_2): track 5.11 -> 8.92 mm

Commit message: import mm2040
Parts:
- removed C1: 0.1u, Capacitor_SMD:C_0402_1005Metric
- removed C10, C11, C12, C13, C14, C16, C17, C8, C9: 100n, Capacitor_SMD:C_0402_1005Metric
- removed C15, C2, C7: 10u, Capacitor_SMD:C_0402_1005Metric
- removed C3, C4: 10u, Capacitor_Tantalum_SMD:CP_EIA-2012-15_AVX-P
- removed C5, C6: 22p, Capacitor_SMD:C_0402_1005Metric
- removed J1: Conn_01x16, Frooastboard Footprints:PinHeader_1x16_P1.27mm_Vertical
- removed J2, J3: Conn_01x06, Frooastboard Footprints:PinHeader_1x06_P1.27mm_Vertical
- removed J4: Conn_01x10, Frooastboard Footprints:PinHeader_1x10_P1.27mm_Vertical
- removed J5: Conn_01x12, Frooastboard Footprints:PinHeader_1x12_P1.27mm_Vertical
- removed J6: SW Interface, Connector_PinHeader_1.27mm:PinHeader_1x05_P1.27mm_Vertical
- removed J7: Conn_01x04, Frooastboard Footprints:PinHeader_1x04_P1.27mm_Vertical
- removed R1, R2: 100k, Resistor_SMD:R_0402_1005Metric
- removed R10, R7: 1k, Resistor_SMD:R_0402_1005Metric
- removed R3: 20k, Resistor_SMD:R_0402_1005Metric
- removed R4: 10k, Resistor_SMD:R_0402_1005Metric
- removed R5, R6: 2k, Resistor_SMD:R_0402_1005Metric
- removed R8, R9: 27R, Resistor_SMD:R_0402_1005Metric
- removed REF**: 1U, Frooastboard Footprints:Footprint Holes
- removed TP1: QSPI_CS, Connector_PinHeader_1.27mm:PinHeader_1x02_P1.27mm_Vertical
- removed U1: IS31FL3733-QF, Package_DFN_QFN:QFN-48-1EP_6x6mm_P0.4mm_EP4.2x4.2mm
- removed U2: RP2040, Frooastboard Footprints:RP2040-QFN-56
- removed U3: W25Q32JVZP, Package_SON:WSON-8-1EP_6x5mm_P1.27mm_EP3.4x4.3mm
- removed U5: LM317L_SOT-89, Package_TO_SOT_SMD:SOT-89-3
- removed Y1: 12MHz, Crystal:Crystal_SMD_3225-4Pin_3.2x2.5mm
- moved MX83 570.3 mm to (37.9, -8.21)
- moved R21 549.8 mm to (213.0, -140.7)
- moved R22 549.8 mm to (213.0, -137.8)
- moved R25 549.8 mm to (213.0, -134.8)
- moved J16 548.1 mm to (212.8, -131.7)
- moved C40 499.8 mm to (255.6, -118.4)
- moved J20 494.8 mm to (246.9, -118.3)
- moved R29 494.8 mm to (251.2, -118.5)
- moved R30 494.8 mm to (251.2, -115.5)
- moved R31 494.8 mm to (251.2, -112.6)
- moved USB3 492.8 mm to (239.5, -111.0)
- moved D105 490.9 mm to (205.3, -177.5)
- moved D107 490.9 mm to (205.3, -174.8)
- moved D108 490.9 mm to (205.3, -172.1)
- moved D109 490.9 mm to (205.3, -169.4)
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Routing:
- net GND: track 27.1 -> 0.00 mm, vias 2 -> 0
- net Net-(J4-Pin_1): track 21.8 -> 0.00 mm
- net QSPI_CS: track 21.8 -> 0.00 mm
- net Net-(J4-Pin_2): track 20.6 -> 0.00 mm
- net Net-(J4-Pin_4): track 20.4 -> 0.00 mm, vias 1 -> 0
- net Net-(J4-Pin_3): track 20.1 -> 0.00 mm
- net Net-(J4-Pin_5): track 19.8 -> 0.00 mm, vias 1 -> 0
- net Net-(J4-Pin_6): track 18.6 -> 0.00 mm, vias 1 -> 0
- net Net-(J4-Pin_7): track 17.9 -> 0.00 mm, vias 1 -> 0
- net QSPI_SD1: track 17.9 -> 0.00 mm
- net Net-(J4-Pin_8): track 17.0 -> 0.00 mm, vias 1 -> 0
- net Net-(J4-Pin_9): track 16.7 -> 0.00 mm, vias 1 -> 0
- net QSPI_SD2: track 15.1 -> 0.00 mm
- net Net-(J4-Pin_10): track 15.0 -> 0.00 mm, vias 2 -> 0
- net +3V3: track 13.6 -> 0.00 mm, vias 2 -> 0
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- removed copper zone on In2.Cu, net +3V3
- removed copper zone on In1.Cu, net GND
Other:
- board outline removed

Commit message: some stuff and caps lock
Parts:
- added MX22: Caps Lock, MX_Only:MXOnly-1U-NoLED, F.Cu at (9.53, -47.6)
- moved MX42 238.0 mm to (11.9, -28.6)
- moved MX43 237.2 mm to (11.9, -9.53)
- moved D125 225.9 mm to (191.4, 206.1)
- moved D140 225.9 mm to (195.8, 206.1)
- moved D155 225.9 mm to (200.3, 206.1)
- moved D170 225.9 mm to (204.7, 206.1)
- moved D185 225.9 mm to (209.2, 206.1)
- moved D199 225.9 mm to (213.6, 206.1)
- moved MX107 225.9 mm to (139.8, 15.1)
- moved MX12 225.9 mm to (282.0, 188.6)
- moved MX16 225.9 mm to (302.2, 188.6)
- moved MX17 225.9 mm to (241.6, 15.1)
- moved MX24 225.9 mm to (261.8, 15.1)
- moved MX30 225.9 mm to (282.0, 15.1)
- moved MX4 225.9 mm to (241.6, 188.6)
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
Commit message: stuff
Parts:
- M2: moved to B.Cu
- moved MX92 275.0 mm to (304.8, -66.7)
- moved MX109 197.7 mm to (295.3, -66.7)
- moved M2 127.8 mm to (224.8, 30.8), turned to 180 degrees
- moved M1 123.9 mm to (392.9, -39.3)
- moved J19 18.2 mm to (289.3, 96.8)
- moved MX91 5.97 mm to (304.8, -85.7)
- moved J14 4.59 mm to (314.4, 186.5)
- turned MX112 to 180 degrees
