File: Frooastboard Walnut Modular/KiCad Project/Frooastboard Walnut Modular.kicad_pcb (KiCad board)
At the start: 4 copper layers, 392 parts, among them J10 F Row CS, J11 F Row SW, J12 Conn_01x06_Male, J13 Conn_01x16_Male, J14 Conn_01x10_Male, J15 F Row, J16 F Row USB, J17 Numpad, J18 Conn_01x04_Male, J19 Conn_01x15_Pin, J20 Conn_01x06_Male, J21 Conn_01x13_Male, J8 Numpad CS, J9 Numpad SW, M1 Frooastboard_MM2040, M2 Frooastboard_MM2040

Commit message: update reference multi leds
Parts:
- removed J10: F Row CS, Connector_PinHeader_1.27mm:PinHeader_1x16_P1.27mm_Vertical
- removed J11: F Row SW, Connector_PinHeader_1.27mm:PinHeader_1x06_P1.27mm_Vertical
- removed J12, J20: Conn_01x06_Male, Connector_PinHeader_1.27mm:PinHeader_1x06_P1.27mm_Vertical
- removed J13: Conn_01x16_Male, Connector_PinHeader_1.27mm:PinHeader_1x16_P1.27mm_Vertical
- removed J14: Conn_01x10_Male, Connector_PinHeader_1.27mm:PinHeader_1x10_P1.27mm_Vertical
- removed J15: F Row, Connector_PinHeader_1.27mm:PinHeader_1x10_P1.27mm_Vertical
- removed J16: F Row USB, Connector_PinHeader_1.27mm:PinHeader_1x04_P1.27mm_Vertical
- removed J17: Numpad, Connector_PinHeader_1.27mm:PinHeader_1x13_P1.27mm_Vertical
- removed J18: Conn_01x04_Male, Connector_PinHeader_1.27mm:PinHeader_1x04_P1.27mm_Vertical
- removed J19: Conn_01x15_Pin, Connector_PinHeader_1.27mm:PinHeader_1x15_P1.27mm_Vertical
- removed J21: Conn_01x13_Male, Connector_PinHeader_1.27mm:PinHeader_1x13_P1.27mm_Vertical
- removed J8: Numpad CS, Connector_PinHeader_1.27mm:PinHeader_1x16_P1.27mm_Vertical
- removed J9: Numpad SW, Connector_PinHeader_1.27mm:PinHeader_1x06_P1.27mm_Vertical
- added FPC201: AFA01-S06FCC-00, AFA01-SXXFCX-00:FPC-SMD_6P-P1.00_AFA01-S06FCC-00, F.Cu at (54.7, 37.5)
- added FPC202: AFA01-S06FCC-00, AFA01-SXXFCX-00:FPC-SMD_6P-P1.00_AFA01-S06FCC-00, F.Cu at (54.7, 44.9)
- added FPC203: AFA01-S10FCC-00, AFA01-SXXFCX-00:FPC-SMD_10P_P1.00_AFA01-S10FCC-00, F.Cu at (33.4, 85.7)
- added FPC204: AFA01-S10FCC-00, AFA01-SXXFCX-00:FPC-SMD_10P_P1.00_AFA01-S10FCC-00, F.Cu at (33.4, 93.2)
- added FPC205: AFA01-S06FCC-00, AFA01-SXXFCX-00:FPC-SMD_6P-P1.00_AFA01-S06FCC-00, F.Cu at (54.7, 52.3)
- added FPC206: AFA01-S06FCC-00, AFA01-SXXFCX-00:FPC-SMD_6P-P1.00_AFA01-S06FCC-00, F.Cu at (54.7, 59.6)
- added FPC207: AFA01-S16FCA-00, AFA01-SXXFCX-00:FPC-SMD_16P-P1.00_AFA01-S16FCC-00, F.Cu at (36.3, 40.1)
- added FPC208: AFA01-S16FCA-00, AFA01-SXXFCX-00:FPC-SMD_16P-P1.00_AFA01-S16FCC-00, F.Cu at (36.3, 48.2)
- added FPC209: AFA01-S16FCA-00, AFA01-SXXFCX-00:FPC-SMD_16P-P1.00_AFA01-S16FCC-00, F.Cu at (36.3, 56.2)
- added FPC210: AFA01-S16FCA-00, AFA01-SXXFCX-00:FPC-SMD_16P-P1.00_AFA01-S16FCC-00, F.Cu at (36.3, 64.3)
- added FPC211: AFA01-S06FCC-00, AFA01-SXXFCX-00:FPC-SMD_6P-P1.00_AFA01-S06FCC-00, F.Cu at (54.7, 67.0)
- added FPC212: AFA01-S06FCC-00, AFA01-SXXFCX-00:FPC-SMD_6P-P1.00_AFA01-S06FCC-00, F.Cu at (54.7, 74.4)
- added FPC213: AFA01-S06FCC-00, AFA01-SXXFCX-00:FPC-SMD_6P-P1.00_AFA01-S06FCC-00, F.Cu at (54.7, 81.8)
- added FPC214: AFA01-S06FCC-00, AFA01-SXXFCX-00:FPC-SMD_6P-P1.00_AFA01-S06FCC-00, F.Cu at (54.7, 89.1)
- added FPC215: AFA01-S16FCA-00, AFA01-SXXFCX-00:FPC-SMD_16P-P1.00_AFA01-S16FCC-00, F.Cu at (36.3, 72.4)
- added FPC216: AFA01-S16FCA-00, AFA01-SXXFCX-00:FPC-SMD_16P-P1.00_AFA01-S16FCC-00, F.Cu at (36.3, 80.4)
- added JP1: SolderJumper_2_Open, Jumper:SolderJumper-2_P1.3mm_Open_RoundedPad1.0x1.5mm, F.Cu at (65.5, 36.7)
- added JP2: SolderJumper_2_Open, Jumper:SolderJumper-2_P1.3mm_Open_RoundedPad1.0x1.5mm, F.Cu at (65.5, 40.2)
- added JP201: SolderJumper_2_Open, Jumper:SolderJumper-2_P1.3mm_Open_RoundedPad1.0x1.5mm, F.Cu at (3.32, 50.5)
- added JP202: SolderJumper_2_Open, Jumper:SolderJumper-2_P1.3mm_Open_RoundedPad1.0x1.5mm, F.Cu at (3.32, 54.0)
- added JP203: SolderJumper_2_Open, Jumper:SolderJumper-2_P1.3mm_Open_RoundedPad1.0x1.5mm, F.Cu at (3.32, 57.6)
- added JP204: SolderJumper_2_Bridged, Jumper:SolderJumper-2_P1.3mm_Bridged_RoundedPad1.0x1.5mm, F.Cu at (3.32, 61.1)
- added JP205: SolderJumper_2_Bridged, Jumper:SolderJumper-2_P1.3mm_Bridged_RoundedPad1.0x1.5mm, F.Cu at (3.32, 64.7)
- added JP206: SolderJumper_2_Bridged, Jumper:SolderJumper-2_P1.3mm_Bridged_RoundedPad1.0x1.5mm, F.Cu at (3.32, 68.2)
- added JP3: SolderJumper_2_Open, Jumper:SolderJumper-2_P1.3mm_Open_RoundedPad1.0x1.5mm, F.Cu at (65.5, 43.8)
- added JP4: SolderJumper_2_Open, Jumper:SolderJumper-2_P1.3mm_Open_RoundedPad1.0x1.5mm, F.Cu at (69.8, 36.7)
- added JP5: SolderJumper_2_Open, Jumper:SolderJumper-2_P1.3mm_Open_RoundedPad1.0x1.5mm, F.Cu at (69.8, 40.2)
- added JP6: SolderJumper_2_Open, Jumper:SolderJumper-2_P1.3mm_Open_RoundedPad1.0x1.5mm, F.Cu at (69.8, 43.8)
- added JP7: SolderJumper_2_Bridged, Jumper:SolderJumper-2_P1.3mm_Bridged_RoundedPad1.0x1.5mm, F.Cu at (74.2, 36.7)
- added JP8: SolderJumper_2_Bridged, Jumper:SolderJumper-2_P1.3mm_Bridged_RoundedPad1.0x1.5mm, F.Cu at (74.2, 40.2)
- added JP9: SolderJumper_2_Bridged, Jumper:SolderJumper-2_P1.3mm_Bridged_RoundedPad1.0x1.5mm, F.Cu at (74.2, 43.8)
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- renumbered D38 to D29_1, D93 to D29_2, D110 to D34_1, D70 to D34_2, D1 to D34_3, D119 to D35_1, D86 to D35_2, D2 to D35_3, D136 to D36_1, D90 to D36_2, D64 to D36_3, D149 to D37_1, D94 to D37_2, D68 to D37_3, D162 to D38_1, D98 to D38_2, D84 to D38_3, D180 to D39_1, D102 to D39_2, D85 to D39_3, M2 to M1, M1 to M2
Connections:
- net ROW11 renamed /Main/ce_row11
- net SW10 renamed /Main/ce_sw10
- net SW11 renamed /Main/ce_sw11
- net SW12 renamed /Main/ce_sw12
- C38 pad 2: GND -> /Main/GND
- C39 pad 2: GND -> /F Row/GND
- C40 pad 2: GND -> /Numpad/GND
- D10 pad 1: ROW10 -> /F Row/fr_row11
- D100 pad 1: SW4 -> /Numpad/np_sw1
- D100 pad 2: CS11 -> /Numpad/np_cs6
- D100 pad 3: SW5 -> /Numpad/np_sw2
- D100 pad 4: CS11 -> /Numpad/np_cs6
- D100 pad 5: SW6 -> /Numpad/np_sw3
- D100 pad 6: CS11 -> /Numpad/np_cs6
- D101 pad 1: SW4 -> /Numpad/np_sw1
- D101 pad 2: CS12 -> /Numpad/np_cs7
- D101 pad 3: SW5 -> /Numpad/np_sw2
- D101 pad 4: CS12 -> /Numpad/np_cs7
- D101 pad 5: SW6 -> /Numpad/np_sw3
- D101 pad 6: CS12 -> /Numpad/np_cs7
- D103 pad 1: SW4 -> /Numpad/np_sw1
- D103 pad 2: CS7 -> /Numpad/np_cs2
- D103 pad 3: SW5 -> /Numpad/np_sw2
- D103 pad 4: CS7 -> /Numpad/np_cs2
- D103 pad 5: SW6 -> /Numpad/np_sw3
- D103 pad 6: CS7 -> /Numpad/np_cs2
- D104 pad 1: SW4 -> /Numpad/np_sw1
- D104 pad 2: CS8 -> /Numpad/np_cs3
- D104 pad 3: SW5 -> /Numpad/np_sw2
- D104 pad 4: CS8 -> /Numpad/np_cs3
- D104 pad 5: SW6 -> /Numpad/np_sw3
- D104 pad 6: CS8 -> /Numpad/np_cs3
- D105 pad 2: CS1 -> /Main/ce_cs1
- D105 pad 4: CS1 -> /Main/ce_cs1
- D105 pad 6: CS1 -> /Main/ce_cs1
- D106 pad 1: SW4 -> /Numpad/np_sw1
- D106 pad 2: CS9 -> /Numpad/np_cs4
- D106 pad 3: SW5 -> /Numpad/np_sw2
- D106 pad 4: CS9 -> /Numpad/np_cs4
- D106 pad 5: SW6 -> /Numpad/np_sw3
- D106 pad 6: CS9 -> /Numpad/np_cs4
- D107 pad 1: SW4 -> /Main/ce_sw4
- D107 pad 2: CS1 -> /Main/ce_cs1
- D107 pad 3: SW5 -> /Main/ce_sw5
- D107 pad 4: CS1 -> /Main/ce_cs1
- D107 pad 5: SW6 -> /Main/ce_sw6
- D107 pad 6: CS1 -> /Main/ce_cs1
- D108 pad 1: SW1 -> /Main/ce_sw1
- D108 pad 2: CS1 -> /Main/ce_cs1
- D108 pad 3: SW2 -> /Main/ce_sw2
- D108 pad 4: CS1 -> /Main/ce_cs1
- D108 pad 5: SW3 -> /Main/ce_sw3
- D108 pad 6: CS1 -> /Main/ce_cs1
- D109 pad 2: CS2 -> /Main/ce_cs2
- D109 pad 4: CS2 -> /Main/ce_cs2
- D109 pad 6: CS2 -> /Main/ce_cs2
- D11 pad 1: SW4 -> /F Row/fr_sw4
- D11 pad 2: CS4 -> /F Row/fr_cs4
- D11 pad 3: SW5 -> /F Row/fr_sw5
- D11 pad 4: CS4 -> /F Row/fr_cs4
- D11 pad 5: SW6 -> /F Row/fr_sw6
- D11 pad 6: CS4 -> /F Row/fr_cs4
- D111 pad 1: SW4 -> /Numpad/np_sw1
- D111 pad 2: CS6 -> /Numpad/np_cs1
- D111 pad 3: SW5 -> /Numpad/np_sw2
- D111 pad 4: CS6 -> /Numpad/np_cs1
- D111 pad 5: SW6 -> /Numpad/np_sw3
- D111 pad 6: CS6 -> /Numpad/np_cs1
- D112 pad 1: SW1 -> /Main/ce_sw1
- D112 pad 2: Net-(D112-B+) -> /Main/ce_cs2
- D112 pad 3: SW2 -> /Main/ce_sw2
- D112 pad 4: Net-(D112-B+) -> /Main/ce_cs2
- D112 pad 5: SW3 -> /Main/ce_sw3
- D112 pad 6: Net-(D112-B+) -> /Main/ce_cs2
- D113 pad 1: ROW0 -> /Main/ce_row0
- D114 pad 1: ROW2 -> /Main/ce_row2
- D115 pad 1: ROW4 -> /Main/ce_row4
- D116 pad 1: ROW6 -> /Main/ce_row6
- D117 pad 1: ROW8 -> /Main/ce_row8
- D118 pad 2: CS3 -> /Main/ce_cs3
- D118 pad 4: CS3 -> /Main/ce_cs3
- D118 pad 6: CS3 -> /Main/ce_cs3
- D12 pad 1: ROW9 -> /F Row/fr_row10
- D120 pad 1: SW4 -> /Main/ce_sw4
- D120 pad 2: Net-(D120-B+) -> /Main/ce_cs3
- D120 pad 3: SW5 -> /Main/ce_sw5
- D120 pad 4: Net-(D120-B+) -> /Main/ce_cs3
- D120 pad 5: SW6 -> /Main/ce_sw6
- D120 pad 6: Net-(D120-B+) -> /Main/ce_cs3
- D121 pad 1: SW1 -> /Main/ce_sw1
- D121 pad 2: Net-(D120-B+) -> /Main/ce_cs3
- D121 pad 3: SW2 -> /Main/ce_sw2
- D121 pad 4: Net-(D120-B+) -> /Main/ce_cs3
- D121 pad 5: SW3 -> /Main/ce_sw3
- D121 pad 6: Net-(D120-B+) -> /Main/ce_cs3
- D122 pad 1: ROW1 -> /Main/ce_row1
- D123 pad 1: ROW3 -> /Main/ce_row3
- D124 pad 1: ROW5 -> /Main/ce_row5
- D125 pad 1: ROW7 -> /Main/ce_row7
- D126 pad 1: ROW0 -> /Main/ce_row0
- D127 pad 1: ROW2 -> /Main/ce_row2
- D128 pad 1: ROW4 -> /Main/ce_row4
- D129 pad 1: ROW6 -> /Main/ce_row6
- D13 pad 1: ROW10 -> /F Row/fr_row11
- D130 pad 1: ROW8 -> /Main/ce_row8
- D131 pad 1: ROW1 -> /Main/ce_row1
- D132 pad 1: ROW3 -> /Main/ce_row3
- D133 pad 1: ROW5 -> /Main/ce_row5
- D134 pad 1: ROW7 -> /Main/ce_row7
- D135 pad 2: CS4 -> /Main/ce_cs4
- D135 pad 4: CS4 -> /Main/ce_cs4
- D135 pad 6: CS4 -> /Main/ce_cs4
- D137 pad 1: SW4 -> /Main/ce_sw4
- D137 pad 2: Net-(D137-B+) -> /Main/ce_cs4
- D137 pad 3: SW5 -> /Main/ce_sw5
- D137 pad 4: Net-(D137-B+) -> /Main/ce_cs4
- D137 pad 5: SW6 -> /Main/ce_sw6
- D137 pad 6: Net-(D137-B+) -> /Main/ce_cs4
- D138 pad 1: SW1 -> /Main/ce_sw1
- D138 pad 2: Net-(D137-B+) -> /Main/ce_cs4
- D138 pad 3: SW2 -> /Main/ce_sw2
- D138 pad 4: Net-(D137-B+) -> /Main/ce_cs4
- D138 pad 5: SW3 -> /Main/ce_sw3
- D138 pad 6: Net-(D137-B+) -> /Main/ce_cs4
- D139 pad 1: ROW0 -> /Main/ce_row0
- D14 pad 1: SW4 -> /F Row/fr_sw4
- D14 pad 2: CS5 -> /F Row/fr_cs5
- D14 pad 3: SW5 -> /F Row/fr_sw5
- D14 pad 4: CS5 -> /F Row/fr_cs5
- D14 pad 5: SW6 -> /F Row/fr_sw6
- D14 pad 6: CS5 -> /F Row/fr_cs5
- D140 pad 1: ROW2 -> /Main/ce_row2
- D141 pad 1: ROW4 -> /Main/ce_row4
- D142 pad 1: ROW6 -> /Main/ce_row6
- D143 pad 1: ROW8 -> /Main/ce_row8
- D144 pad 1: ROW1 -> /Main/ce_row1
- D145 pad 1: ROW3 -> /Main/ce_row3
- D146 pad 1: ROW5 -> /Main/ce_row5
- D147 pad 1: ROW7 -> /Main/ce_row7
- D148 pad 2: CS5 -> /Main/ce_cs5
- D148 pad 4: CS5 -> /Main/ce_cs5
- D148 pad 6: CS5 -> /Main/ce_cs5
- D15 pad 1: ROW9 -> /F Row/fr_row10
- D150 pad 1: SW4 -> /Main/ce_sw4
- D150 pad 2: Net-(D150-B+) -> /Main/ce_cs5
- D150 pad 3: SW5 -> /Main/ce_sw5
- D150 pad 4: Net-(D150-B+) -> /Main/ce_cs5
- D150 pad 5: SW6 -> /Main/ce_sw6
- D150 pad 6: Net-(D150-B+) -> /Main/ce_cs5
- D151 pad 1: SW1 -> /Main/ce_sw1
- D151 pad 2: Net-(D150-B+) -> /Main/ce_cs5
- D151 pad 3: SW2 -> /Main/ce_sw2
- D151 pad 4: Net-(D150-B+) -> /Main/ce_cs5
- D151 pad 5: SW3 -> /Main/ce_sw3
- D151 pad 6: Net-(D150-B+) -> /Main/ce_cs5
- D152 pad 1: ROW0 -> /Main/ce_row0
- D153 pad 1: ROW2 -> /Main/ce_row2
- D154 pad 1: ROW4 -> /Main/ce_row4
- D155 pad 1: ROW6 -> /Main/ce_row6
- D156 pad 1: ROW8 -> /Main/ce_row8
- D157 pad 1: ROW1 -> /Main/ce_row1
- D158 pad 1: ROW3 -> /Main/ce_row3
- D159 pad 1: ROW5 -> /Main/ce_row5
- D16 pad 1: ROW10 -> /F Row/fr_row11
- D160 pad 1: ROW7 -> /Main/ce_row7
- D161 pad 2: CS6 -> /Main/ce_cs6
- D161 pad 4: CS6 -> /Main/ce_cs6
- D161 pad 6: CS6 -> /Main/ce_cs6
- D163 pad 1: SW4 -> /Main/ce_sw4
- D163 pad 2: Net-(D163-B+) -> /Main/ce_cs6
- D163 pad 3: SW5 -> /Main/ce_sw5
- D163 pad 4: Net-(D163-B+) -> /Main/ce_cs6
- D163 pad 5: SW6 -> /Main/ce_sw6
- D163 pad 6: Net-(D163-B+) -> /Main/ce_cs6
- D164 pad 1: SW1 -> /Main/ce_sw1
- D164 pad 2: Net-(D163-B+) -> /Main/ce_cs6
- D164 pad 3: SW2 -> /Main/ce_sw2
- D164 pad 4: Net-(D163-B+) -> /Main/ce_cs6
- D164 pad 5: SW3 -> /Main/ce_sw3
- D164 pad 6: Net-(D163-B+) -> /Main/ce_cs6
- D165 pad 1: ROW0 -> /Main/ce_row0
- D166 pad 1: ROW2 -> /Main/ce_row2
- D167 pad 1: ROW4 -> /Main/ce_row4
- D168 pad 1: ROW6 -> /Main/ce_row6
- D169 pad 1: ROW8 -> /Main/ce_row8
- D17 pad 1: SW4 -> /F Row/fr_sw4
- D17 pad 2: CS6 -> /F Row/fr_cs6
- D17 pad 3: SW5 -> /F Row/fr_sw5
- D17 pad 4: CS6 -> /F Row/fr_cs6
- D17 pad 5: SW6 -> /F Row/fr_sw6
- D17 pad 6: CS6 -> /F Row/fr_cs6
- D170 pad 1: ROW1 -> /Main/ce_row1
- D171 pad 1: ROW3 -> /Main/ce_row3
- D172 pad 1: ROW5 -> /Main/ce_row5
- D173 pad 1: ROW7 -> /Main/ce_row7
- D174 pad 1: ROW0 -> /Main/ce_row0
- D175 pad 1: ROW2 -> /Main/ce_row2
- D176 pad 1: ROW4 -> /Main/ce_row4
- D177 pad 1: ROW6 -> /Main/ce_row6
- D178 pad 1: ROW8 -> /Main/ce_row8
- D179 pad 2: CS7 -> /Main/ce_cs7
- D179 pad 4: CS7 -> /Main/ce_cs7
- D179 pad 6: CS7 -> /Main/ce_cs7
- D18 pad 1: ROW9 -> /F Row/fr_row10
- D181 pad 1: SW4 -> /Main/ce_sw4
- D181 pad 2: Net-(D181-B+) -> /Main/ce_cs7
- D181 pad 3: SW5 -> /Main/ce_sw5
- D181 pad 4: Net-(D181-B+) -> /Main/ce_cs7
- D181 pad 5: SW6 -> /Main/ce_sw6
- D181 pad 6: Net-(D181-B+) -> /Main/ce_cs7
- D183 pad 1: ROW1 -> /Main/ce_row1
- D184 pad 1: ROW3 -> /Main/ce_row3
- D185 pad 1: ROW5 -> /Main/ce_row5
- D186 pad 1: ROW7 -> /Main/ce_row7
- D187 pad 1: ROW0 -> /Main/ce_row0
- D188 pad 1: ROW2 -> /Main/ce_row2
- D189 pad 1: ROW4 -> /Main/ce_row4
- D19 pad 1: ROW10 -> /F Row/fr_row11
- D190 pad 1: ROW6 -> /Main/ce_row6
- D191 pad 1: ROW8 -> /Main/ce_row8
- D192 pad 2: CS8 -> /Main/ce_cs8
- D192 pad 4: CS8 -> /Main/ce_cs8
- D192 pad 6: CS8 -> /Main/ce_cs8
- D194 pad 1: SW4 -> /Main/ce_sw4
- D194 pad 2: CS8 -> /Main/ce_cs8
- D194 pad 3: SW5 -> /Main/ce_sw5
- D194 pad 4: CS8 -> /Main/ce_cs8
- D194 pad 5: SW6 -> /Main/ce_sw6
- D194 pad 6: CS8 -> /Main/ce_cs8
- D195 pad 1: ROW1 -> /Main/ce_row1
- D196 pad 1: ROW3 -> /Main/ce_row3
- D197 pad 1: ROW5 -> /Main/ce_row5
- D198 pad 1: ROW7 -> /Main/ce_row7
- D199 pad 1: ROW0 -> /Main/ce_row0
- D20 pad 1: ROW9 -> /F Row/fr_row10
- D200 pad 1: ROW2 -> /Main/ce_row2
- D201 pad 1: ROW4 -> /Main/ce_row4
- D202 pad 1: ROW6 -> /Main/ce_row6
- D203 pad 1: ROW8 -> /Main/ce_row8
- D204 pad 1: ROW1 -> /Main/ce_row1
- D205 pad 1: ROW3 -> /Main/ce_row3
- D206 pad 1: ROW5 -> /Main/ce_row5
- D207 pad 1: ROW7 -> /Main/ce_row7
- D208 pad 2: CS9 -> /Main/ce_cs9
- D208 pad 4: CS9 -> /Main/ce_cs9
- D208 pad 6: CS9 -> /Main/ce_cs9
- D21 pad 1: SW4 -> /F Row/fr_sw4
- D21 pad 2: CS7 -> /F Row/fr_cs7
- D21 pad 3: SW5 -> /F Row/fr_sw5
- D21 pad 4: CS7 -> /F Row/fr_cs7
- D21 pad 5: SW6 -> /F Row/fr_sw6
- D21 pad 6: CS7 -> /F Row/fr_cs7
- D210 pad 1: SW4 -> /Main/ce_sw4
- D210 pad 2: CS9 -> /Main/ce_cs9
- D210 pad 3: SW5 -> /Main/ce_sw5
- D210 pad 4: CS9 -> /Main/ce_cs9
- D210 pad 5: SW6 -> /Main/ce_sw6
- D210 pad 6: CS9 -> /Main/ce_cs9
- D211 pad 1: SW1 -> /Main/ce_sw1
- D211 pad 2: CS9 -> /Main/ce_cs9
- D211 pad 3: SW2 -> /Main/ce_sw2
- D211 pad 4: CS9 -> /Main/ce_cs9
- D211 pad 5: SW3 -> /Main/ce_sw3
- D211 pad 6: CS9 -> /Main/ce_cs9
- D212 pad 2: CS10 -> /Main/ce_cs10
- D212 pad 4: CS10 -> /Main/ce_cs10
- D212 pad 6: CS10 -> /Main/ce_cs10
- D214 pad 1: SW4 -> /Main/ce_sw4
- D214 pad 2: CS10 -> /Main/ce_cs10
- D214 pad 3: SW5 -> /Main/ce_sw5
- D214 pad 4: CS10 -> /Main/ce_cs10
- D214 pad 5: SW6 -> /Main/ce_sw6
- D214 pad 6: CS10 -> /Main/ce_cs10
- D215 pad 1: SW1 -> /Main/ce_sw1
- D215 pad 2: CS10 -> /Main/ce_cs10
- D215 pad 3: SW2 -> /Main/ce_sw2
- D215 pad 4: CS10 -> /Main/ce_cs10
- D215 pad 5: SW3 -> /Main/ce_sw3
- D215 pad 6: CS10 -> /Main/ce_cs10
- D216 pad 2: CS11 -> /Main/ce_cs11
- D216 pad 4: CS11 -> /Main/ce_cs11
- D216 pad 6: CS11 -> /Main/ce_cs11
- D218 pad 1: SW4 -> /Main/ce_sw4
- D218 pad 2: CS11 -> /Main/ce_cs11
- D218 pad 3: SW5 -> /Main/ce_sw5
- D218 pad 4: CS11 -> /Main/ce_cs11
- D218 pad 5: SW6 -> /Main/ce_sw6
- D218 pad 6: CS11 -> /Main/ce_cs11
- D219 pad 1: SW1 -> /Main/ce_sw1
- D219 pad 2: CS11 -> /Main/ce_cs11
- D219 pad 3: SW2 -> /Main/ce_sw2
- D219 pad 4: CS11 -> /Main/ce_cs11
- D219 pad 5: SW3 -> /Main/ce_sw3
- D219 pad 6: CS11 -> /Main/ce_cs11
- D22 pad 1: SW1 -> /F Row/fr_sw1
- D22 pad 2: CS7 -> /F Row/fr_cs7
- D22 pad 3: SW2 -> /F Row/fr_sw2
- D22 pad 4: CS7 -> /F Row/fr_cs7
- D22 pad 5: SW3 -> /F Row/fr_sw3
- D22 pad 6: CS7 -> /F Row/fr_cs7
- D220 pad 2: CS12 -> /Main/ce_cs12
- D220 pad 4: CS12 -> /Main/ce_cs12
- D220 pad 6: CS12 -> /Main/ce_cs12
- D221 pad 1: SW7 -> /Main/ce_sw7
- D221 pad 2: CS12 -> /Main/ce_cs12
- D221 pad 3: SW8 -> /Main/ce_sw8
- D221 pad 4: CS12 -> /Main/ce_cs12
- D221 pad 5: SW9 -> /Main/ce_sw9
- D221 pad 6: CS12 -> /Main/ce_cs12
- D222 pad 1: SW4 -> /Main/ce_sw4
- D222 pad 2: CS12 -> /Main/ce_cs12
- D222 pad 3: SW5 -> /Main/ce_sw5
- D222 pad 4: CS12 -> /Main/ce_cs12
- D222 pad 5: SW6 -> /Main/ce_sw6
- D222 pad 6: CS12 -> /Main/ce_cs12
- D223 pad 1: SW1 -> /Main/ce_sw1
- D223 pad 2: CS12 -> /Main/ce_cs12
- D223 pad 3: SW2 -> /Main/ce_sw2
- D223 pad 4: CS12 -> /Main/ce_cs12
- D223 pad 5: SW3 -> /Main/ce_sw3
- D223 pad 6: CS12 -> /Main/ce_cs12
- D228 pad 2: CS13 -> /Main/ce_cs13
- D228 pad 4: CS13 -> /Main/ce_cs13
- D228 pad 6: CS13 -> /Main/ce_cs13
- D229 pad 1: SW7 -> /Main/ce_sw7
- D229 pad 2: CS13 -> /Main/ce_cs13
- D229 pad 3: SW8 -> /Main/ce_sw8
- D229 pad 4: CS13 -> /Main/ce_cs13
- D229 pad 5: SW9 -> /Main/ce_sw9
- D229 pad 6: CS13 -> /Main/ce_cs13
- D23 pad 1: ROW10 -> /F Row/fr_row11
- D231 pad 1: SW1 -> /Main/ce_sw1
- D231 pad 2: CS13 -> /Main/ce_cs13
- D231 pad 3: SW2 -> /Main/ce_sw2
- D231 pad 4: CS13 -> /Main/ce_cs13
- D231 pad 5: SW3 -> /Main/ce_sw3
- D231 pad 6: CS13 -> /Main/ce_cs13
- D236 pad 2: CS14 -> /Main/ce_cs14
- D236 pad 4: CS14 -> /Main/ce_cs14
- D236 pad 6: CS14 -> /Main/ce_cs14
- D237 pad 1: SW7 -> /Main/ce_sw7
- D237 pad 2: CS14 -> /Main/ce_cs14
- D237 pad 3: SW8 -> /Main/ce_sw8
- D237 pad 4: CS14 -> /Main/ce_cs14
- D237 pad 5: SW9 -> /Main/ce_sw9
- D237 pad 6: CS14 -> /Main/ce_cs14
- D239 pad 1: SW1 -> /Main/ce_sw1
- D239 pad 2: CS14 -> /Main/ce_cs14
- D239 pad 3: SW2 -> /Main/ce_sw2
- D239 pad 4: CS14 -> /Main/ce_cs14
- D239 pad 5: SW3 -> /Main/ce_sw3
- D239 pad 6: CS14 -> /Main/ce_cs14
- D24 pad 1: ROW9 -> /F Row/fr_row10
- D244 pad 2: CS15 -> /Main/ce_cs15
- D244 pad 4: CS15 -> /Main/ce_cs15
- D244 pad 6: CS15 -> /Main/ce_cs15
- D245 pad 1: SW7 -> /Main/ce_sw7
- D245 pad 2: CS15 -> /Main/ce_cs15
- D245 pad 3: SW8 -> /Main/ce_sw8
- D245 pad 4: CS15 -> /Main/ce_cs15
- D245 pad 5: SW9 -> /Main/ce_sw9
- D245 pad 6: CS15 -> /Main/ce_cs15
- D247 pad 1: SW1 -> /Main/ce_sw1
- D247 pad 2: CS15 -> /Main/ce_cs15
- D247 pad 3: SW2 -> /Main/ce_sw2
- D247 pad 4: CS15 -> /Main/ce_cs15
- D247 pad 5: SW3 -> /Main/ce_sw3
- D247 pad 6: CS15 -> /Main/ce_cs15
- D25 pad 1: SW4 -> /F Row/fr_sw4
- D25 pad 2: CS8 -> /F Row/fr_cs8
- D25 pad 3: SW5 -> /F Row/fr_sw5
- D25 pad 4: CS8 -> /F Row/fr_cs8
- D25 pad 5: SW6 -> /F Row/fr_sw6
- D25 pad 6: CS8 -> /F Row/fr_cs8
- D252 pad 2: CS16 -> /Main/ce_cs16
- D252 pad 4: CS16 -> /Main/ce_cs16
- D252 pad 6: CS16 -> /Main/ce_cs16
- D253 pad 1: SW7 -> /Main/ce_sw7
- D253 pad 2: CS16 -> /Main/ce_cs16
- D253 pad 3: SW8 -> /Main/ce_sw8
- D253 pad 4: CS16 -> /Main/ce_cs16
- D253 pad 5: SW9 -> /Main/ce_sw9
- D253 pad 6: CS16 -> /Main/ce_cs16
- D255 pad 1: SW1 -> /Main/ce_sw1
- D255 pad 2: CS16 -> /Main/ce_cs16
- D255 pad 3: SW2 -> /Main/ce_sw2
- D255 pad 4: CS16 -> /Main/ce_cs16
- D255 pad 5: SW3 -> /Main/ce_sw3
- D255 pad 6: CS16 -> /Main/ce_cs16
- D26 pad 1: SW1 -> /F Row/fr_sw1
- D26 pad 2: CS8 -> /F Row/fr_cs8
- D26 pad 3: SW2 -> /F Row/fr_sw2
- D26 pad 4: CS8 -> /F Row/fr_cs8
- D26 pad 5: SW3 -> /F Row/fr_sw3
- D26 pad 6: CS8 -> /F Row/fr_cs8
- D27 pad 1: ROW10 -> /F Row/fr_row11
- D28 pad 1: ROW9 -> /F Row/fr_row10
- D29 pad 1: ROW10 -> /F Row/fr_row11
- D29_1 pad 1: SW4 -> Net-(D29_1-G-)
- D29_1 pad 2: CS13 -> /F Row/fr_cs13
- D29_1 pad 3: SW5 -> Net-(D29_1-R-)
- D29_1 pad 4: CS13 -> /F Row/fr_cs13
- D29_1 pad 5: SW6 -> Net-(D29_1-B-)
- D29_1 pad 6: CS13 -> /F Row/fr_cs13
- D29_2 pad 1: SW4 -> Net-(D29_2-G-)
- D29_2 pad 2: CS13 -> /F Row/fr_cs13
- D29_2 pad 3: SW5 -> Net-(D29_2-R-)
- D29_2 pad 4: CS13 -> /F Row/fr_cs13
- D29_2 pad 5: SW6 -> Net-(D29_2-B-)
- D29_2 pad 6: CS13 -> /F Row/fr_cs13
- D3 pad 1: SW1 -> /Main/ce_sw1
- D3 pad 2: CS8 -> /Main/ce_cs8
- D3 pad 3: SW2 -> /Main/ce_sw2
- D3 pad 4: CS8 -> /Main/ce_cs8
- D3 pad 5: SW3 -> /Main/ce_sw3
- D3 pad 6: CS8 -> /Main/ce_cs8
- D30 pad 1: SW4 -> /F Row/fr_sw4
- D30 pad 2: CS9 -> /F Row/fr_cs9
- D30 pad 3: SW5 -> /F Row/fr_sw5
- D30 pad 4: CS9 -> /F Row/fr_cs9
- D30 pad 5: SW6 -> /F Row/fr_sw6
- D30 pad 6: CS9 -> /F Row/fr_cs9
- D31 pad 1: SW1 -> /F Row/fr_sw1
- D31 pad 2: CS9 -> /F Row/fr_cs9
- D31 pad 3: SW2 -> /F Row/fr_sw2
- D31 pad 4: CS9 -> /F Row/fr_cs9
- D31 pad 5: SW3 -> /F Row/fr_sw3
- D31 pad 6: CS9 -> /F Row/fr_cs9
- D32 pad 1: SW4 -> /F Row/fr_sw4
- D32 pad 2: CS10 -> /F Row/fr_cs10
- D32 pad 3: SW5 -> /F Row/fr_sw5
- D32 pad 4: CS10 -> /F Row/fr_cs10
- D32 pad 5: SW6 -> /F Row/fr_sw6
- D32 pad 6: CS10 -> /F Row/fr_cs10
- D33 pad 1: SW1 -> /F Row/fr_sw1
- D33 pad 2: CS10 -> /F Row/fr_cs10
- D33 pad 3: SW2 -> /F Row/fr_sw2
- D33 pad 4: CS10 -> /F Row/fr_cs10
- D33 pad 5: SW3 -> /F Row/fr_sw3
- D33 pad 6: CS10 -> /F Row/fr_cs10
- D34 pad 1: SW4 -> /F Row/fr_sw4
- D34 pad 2: CS11 -> /F Row/fr_cs11
- D34 pad 3: SW5 -> /F Row/fr_sw5
- D34 pad 4: CS11 -> /F Row/fr_cs11
- D34 pad 5: SW6 -> /F Row/fr_sw6
- D34 pad 6: CS11 -> /F Row/fr_cs11
- D34_1 pad 2: CS2 -> /Main/ce_cs2
- D34_1 pad 4: CS2 -> /Main/ce_cs2
- D34_1 pad 6: CS2 -> /Main/ce_cs2
- D34_2 pad 2: CS2 -> /Main/ce_cs2
- D34_2 pad 4: CS2 -> /Main/ce_cs2
- D34_2 pad 6: CS2 -> /Main/ce_cs2
- D34_3 pad 2: CS2 -> /Main/ce_cs2
- D34_3 pad 4: CS2 -> /Main/ce_cs2
- D34_3 pad 6: CS2 -> /Main/ce_cs2
- D35 pad 1: SW1 -> /F Row/fr_sw1
- D35 pad 2: CS11 -> /F Row/fr_cs11
- D35 pad 3: SW2 -> /F Row/fr_sw2
- D35 pad 4: CS11 -> /F Row/fr_cs11
- D35 pad 5: SW3 -> /F Row/fr_sw3
- D35 pad 6: CS11 -> /F Row/fr_cs11
- D35_1 pad 2: CS3 -> /Main/ce_cs3
- D35_1 pad 4: CS3 -> /Main/ce_cs3
- D35_1 pad 6: CS3 -> /Main/ce_cs3
- D35_2 pad 2: CS3 -> /Main/ce_cs3
- D35_2 pad 4: CS3 -> /Main/ce_cs3
- D35_2 pad 6: CS3 -> /Main/ce_cs3
- D35_3 pad 2: CS3 -> /Main/ce_cs3
- D35_3 pad 4: CS3 -> /Main/ce_cs3
- D35_3 pad 6: CS3 -> /Main/ce_cs3
- D36 pad 1: SW4 -> /F Row/fr_sw4
- D36 pad 2: CS12 -> /F Row/fr_cs12
- D36 pad 3: SW5 -> /F Row/fr_sw5
- D36 pad 4: CS12 -> /F Row/fr_cs12
- D36 pad 5: SW6 -> /F Row/fr_sw6
- D36 pad 6: CS12 -> /F Row/fr_cs12
- D36_1 pad 2: CS4 -> /Main/ce_cs4
- D36_1 pad 4: CS4 -> /Main/ce_cs4
- D36_1 pad 6: CS4 -> /Main/ce_cs4
- D36_2 pad 2: CS4 -> /Main/ce_cs4
- D36_2 pad 4: CS4 -> /Main/ce_cs4
- D36_2 pad 6: CS4 -> /Main/ce_cs4
- D36_3 pad 2: CS4 -> /Main/ce_cs4
- D36_3 pad 4: CS4 -> /Main/ce_cs4
- D36_3 pad 6: CS4 -> /Main/ce_cs4
- D37 pad 1: SW1 -> /F Row/fr_sw1
- D37 pad 2: CS12 -> /F Row/fr_cs12
- D37 pad 3: SW2 -> /F Row/fr_sw2
- D37 pad 4: CS12 -> /F Row/fr_cs12
- D37 pad 5: SW3 -> /F Row/fr_sw3
- D37 pad 6: CS12 -> /F Row/fr_cs12
- D37_1 pad 2: CS5 -> /Main/ce_cs5
- D37_1 pad 4: CS5 -> /Main/ce_cs5
- D37_1 pad 6: CS5 -> /Main/ce_cs5
- D37_2 pad 2: CS5 -> /Main/ce_cs5
- D37_2 pad 4: CS5 -> /Main/ce_cs5
- D37_2 pad 6: CS5 -> /Main/ce_cs5
- D37_3 pad 2: CS5 -> /Main/ce_cs5
- D37_3 pad 4: CS5 -> /Main/ce_cs5
- D37_3 pad 6: CS5 -> /Main/ce_cs5
- D38_1 pad 2: CS6 -> /Main/ce_cs6
- D38_1 pad 4: CS6 -> /Main/ce_cs6
- D38_1 pad 6: CS6 -> /Main/ce_cs6
- D38_2 pad 2: CS6 -> /Main/ce_cs6
- D38_2 pad 4: CS6 -> /Main/ce_cs6
- D38_2 pad 6: CS6 -> /Main/ce_cs6
- D38_3 pad 2: CS6 -> /Main/ce_cs6
- D38_3 pad 4: CS6 -> /Main/ce_cs6
- D38_3 pad 6: CS6 -> /Main/ce_cs6
- D39 pad 1: SW1 -> /F Row/fr_sw1
- D39 pad 2: CS13 -> /F Row/fr_cs13
- D39 pad 3: SW2 -> /F Row/fr_sw2
- D39 pad 4: CS13 -> /F Row/fr_cs13
- D39 pad 5: SW3 -> /F Row/fr_sw3
- D39 pad 6: CS13 -> /F Row/fr_cs13
- D39_1 pad 2: CS7 -> /Main/ce_cs7
- D39_1 pad 4: CS7 -> /Main/ce_cs7
- D39_1 pad 6: CS7 -> /Main/ce_cs7
- D39_2 pad 2: CS7 -> /Main/ce_cs7
- D39_2 pad 4: CS7 -> /Main/ce_cs7
- D39_2 pad 6: CS7 -> /Main/ce_cs7
- D39_3 pad 2: CS7 -> /Main/ce_cs7
- D39_3 pad 4: CS7 -> /Main/ce_cs7
- D39_3 pad 6: CS7 -> /Main/ce_cs7
- D4 pad 1: SW4 -> /F Row/fr_sw4
- D4 pad 2: CS1 -> /F Row/fr_cs1
- D4 pad 3: SW5 -> /F Row/fr_sw5
- D4 pad 4: CS1 -> /F Row/fr_cs1
- D4 pad 5: SW6 -> /F Row/fr_sw6
- D4 pad 6: CS1 -> /F Row/fr_cs1
- D40 pad 1: SW1 -> /F Row/fr_sw1
- D40 pad 2: CS14 -> /F Row/fr_cs14
- D40 pad 3: SW2 -> /F Row/fr_sw2
- D40 pad 4: CS14 -> /F Row/fr_cs14
- D40 pad 5: SW3 -> /F Row/fr_sw3
- D40 pad 6: CS14 -> /F Row/fr_cs14
- D41 pad 1: SW1 -> /F Row/fr_sw1
- D41 pad 2: CS15 -> /F Row/fr_cs15
- D41 pad 3: SW2 -> /F Row/fr_sw2
- D41 pad 4: CS15 -> /F Row/fr_cs15
- D41 pad 5: SW3 -> /F Row/fr_sw3
- D41 pad 6: CS15 -> /F Row/fr_cs15
- D42 pad 1: SW1 -> /F Row/fr_sw1
- D42 pad 2: CS16 -> /F Row/fr_cs16
- D42 pad 3: SW2 -> /F Row/fr_sw2
- D42 pad 4: CS16 -> /F Row/fr_cs16
- D42 pad 5: SW3 -> /F Row/fr_sw3
- D42 pad 6: CS16 -> /F Row/fr_cs16
- D43 pad 1: SW7 -> /Numpad/np_sw7
- D43 pad 2: CS1 -> /Numpad/np_cs1
- D43 pad 3: SW8 -> /Numpad/np_sw8
- D43 pad 4: CS1 -> /Numpad/np_cs1
- D43 pad 5: SW9 -> /Numpad/np_sw9
- D43 pad 6: CS1 -> /Numpad/np_cs1
- D44 pad 1: SW7 -> /Numpad/np_sw7
- D44 pad 2: CS2 -> /Numpad/np_cs2
- D44 pad 3: SW8 -> /Numpad/np_sw8
- D44 pad 4: CS2 -> /Numpad/np_cs2
- D44 pad 5: SW9 -> /Numpad/np_sw9
- D44 pad 6: CS2 -> /Numpad/np_cs2
- D45 pad 1: SW7 -> /Numpad/np_sw7
- D45 pad 2: CS3 -> /Numpad/np_cs3
- D45 pad 3: SW8 -> /Numpad/np_sw8
- D45 pad 4: CS3 -> /Numpad/np_cs3
- D45 pad 5: SW9 -> /Numpad/np_sw9
- D45 pad 6: CS3 -> /Numpad/np_cs3
- D46 pad 1: SW7 -> /Numpad/np_sw7
- D46 pad 2: CS4 -> /Numpad/np_cs4
- D46 pad 3: SW8 -> /Numpad/np_sw8
- D46 pad 4: CS4 -> /Numpad/np_cs4
- D46 pad 5: SW9 -> /Numpad/np_sw9
- D46 pad 6: CS4 -> /Numpad/np_cs4
- D47 pad 1: ROW0 -> /Numpad/np_row0
- D48 pad 1: ROW2 -> /Numpad/np_row2
- D49 pad 1: ROW4 -> /Numpad/np_row4
- D5 pad 1: SW4 -> /Main/ce_sw4
- D5 pad 2: CS2 -> /Main/ce_cs2
- D50 pad 1: ROW6 -> /Numpad/np_row6
- D51 pad 1: ROW8 -> /Numpad/np_row8
- D52 pad 1: SW5 -> /F Row/fr_sw5
- D52 pad 2: CS2 -> /F Row/fr_cs2
- D53 pad 1: SW7 -> /Numpad/np_sw7
- D53 pad 2: CS5 -> /Numpad/np_cs5
- D53 pad 3: SW8 -> /Numpad/np_sw8
- D53 pad 4: CS5 -> /Numpad/np_cs5
- D53 pad 5: SW9 -> /Numpad/np_sw9
- D53 pad 6: CS5 -> /Numpad/np_cs5
- D54 pad 1: ROW1 -> /Numpad/np_row1
- D55 pad 1: ROW3 -> /Numpad/np_row3
- D56 pad 1: ROW5 -> /Numpad/np_row5
- D57 pad 1: ROW7 -> /Numpad/np_row7
- D58 pad 1: SW6 -> /Numpad/np_sw6
- D58 pad 2: CS2 -> /Numpad/np_cs2
- D59 pad 1: ROW0 -> /Numpad/np_row0
- D6 pad 1: ROW9 -> /F Row/fr_row10
- D60 pad 1: ROW2 -> /Numpad/np_row2
- D61 pad 1: ROW4 -> /Numpad/np_row4
- D62 pad 1: ROW6 -> /Numpad/np_row6
- D63 pad 1: ROW8 -> /Numpad/np_row8
- D65 pad 1: SW7 -> /Numpad/np_sw7
- D65 pad 2: CS6 -> /Numpad/np_cs6
- D65 pad 3: SW8 -> /Numpad/np_sw8
- D65 pad 4: CS6 -> /Numpad/np_cs6
- D65 pad 5: SW9 -> /Numpad/np_sw9
- D65 pad 6: CS6 -> /Numpad/np_cs6
- D66 pad 1: ROW1 -> /Numpad/np_row1
- D67 pad 1: ROW3 -> /Numpad/np_row3
- D69 pad 1: ROW7 -> /Numpad/np_row7
- D7 pad 1: SW4 -> /F Row/fr_sw4
- D7 pad 2: CS3 -> /F Row/fr_cs3
- D7 pad 3: SW5 -> /F Row/fr_sw5
- D7 pad 4: CS3 -> /F Row/fr_cs3
- D7 pad 5: SW6 -> /F Row/fr_sw6
- D7 pad 6: CS3 -> /F Row/fr_cs3
- D71 pad 1: SW7 -> /Numpad/np_sw7
- D71 pad 2: CS7 -> /Numpad/np_cs7
- D71 pad 3: SW8 -> /Numpad/np_sw8
- D71 pad 4: CS7 -> /Numpad/np_cs7
- D71 pad 5: SW9 -> /Numpad/np_sw9
- D71 pad 6: CS7 -> /Numpad/np_cs7
- D72 pad 1: SW7 -> /Numpad/np_sw7
- D72 pad 2: CS8 -> /Numpad/np_cs8
- D72 pad 3: SW8 -> /Numpad/np_sw8
- D72 pad 4: CS8 -> /Numpad/np_cs8
- D72 pad 5: SW9 -> /Numpad/np_sw9
- D72 pad 6: CS8 -> /Numpad/np_cs8
- D73 pad 1: SW7 -> /Numpad/np_sw7
- D73 pad 2: CS9 -> /Numpad/np_cs9
- D73 pad 3: SW8 -> /Numpad/np_sw8
- D73 pad 4: CS9 -> /Numpad/np_cs9
- D73 pad 5: SW9 -> /Numpad/np_sw9
- D73 pad 6: CS9 -> /Numpad/np_cs9
- D74 pad 1: SW7 -> /Numpad/np_sw7
- D74 pad 2: CS10 -> /Numpad/np_cs10
- D74 pad 3: SW8 -> /Numpad/np_sw8
- D74 pad 4: CS10 -> /Numpad/np_cs10
- D74 pad 5: SW9 -> /Numpad/np_sw9
- D74 pad 6: CS10 -> /Numpad/np_cs10
- D75 pad 1: SW7 -> /Numpad/np_sw7
- D75 pad 2: CS11 -> /Numpad/np_cs11
- D75 pad 3: SW8 -> /Numpad/np_sw8
- D75 pad 4: CS11 -> /Numpad/np_cs11
- D75 pad 5: SW9 -> /Numpad/np_sw9
- D75 pad 6: CS11 -> /Numpad/np_cs11
- D76 pad 1: SW4 -> /Numpad/np_sw4
- D76 pad 2: CS13 -> /Numpad/np_cs13
- D76 pad 3: SW5 -> /Numpad/np_sw5
- D76 pad 4: CS13 -> /Numpad/np_cs13
- D76 pad 5: SW6 -> /Numpad/np_sw6
- D76 pad 6: CS13 -> /Numpad/np_cs13
- D77 pad 1: SW4 -> /Numpad/np_sw4
- D77 pad 2: CS14 -> /Numpad/np_cs14
- D77 pad 3: SW5 -> /Numpad/np_sw5
- D77 pad 4: CS14 -> /Numpad/np_cs14
- D77 pad 5: SW6 -> /Numpad/np_sw6
- D77 pad 6: CS14 -> /Numpad/np_cs14
- D78 pad 1: SW4 -> /Numpad/np_sw4
- D78 pad 2: CS15 -> /Numpad/np_cs15
- D78 pad 3: SW5 -> /Numpad/np_sw5
- D78 pad 4: CS15 -> /Numpad/np_cs15
- D78 pad 5: SW6 -> /Numpad/np_sw6
- D78 pad 6: CS15 -> /Numpad/np_cs15
- D79 pad 1: SW4 -> /Numpad/np_sw4
- D79 pad 2: CS16 -> /Numpad/np_cs16
- D79 pad 3: SW5 -> /Numpad/np_sw5
- D79 pad 4: CS16 -> /Numpad/np_cs16
- D79 pad 5: SW6 -> /Numpad/np_sw6
- D79 pad 6: CS16 -> /Numpad/np_cs16
- D8 pad 1: ROW10 -> /F Row/fr_row11
- D80 pad 1: SW4 -> /Numpad/np_sw4
- D80 pad 2: CS13 -> /Numpad/np_cs13
- D80 pad 3: SW5 -> /Numpad/np_sw5
- D80 pad 4: CS13 -> /Numpad/np_cs13
- D80 pad 5: SW6 -> /Numpad/np_sw6
- D80 pad 6: CS13 -> /Numpad/np_cs13
- D81 pad 1: SW4 -> /Numpad/np_sw4
- D81 pad 2: CS14 -> /Numpad/np_cs14
- D81 pad 3: SW5 -> /Numpad/np_sw5
- D81 pad 4: CS14 -> /Numpad/np_cs14
- D81 pad 5: SW6 -> /Numpad/np_sw6
- D81 pad 6: CS14 -> /Numpad/np_cs14
- D82 pad 1: SW4 -> /Numpad/np_sw4
- D82 pad 2: CS15 -> /Numpad/np_cs15
- D82 pad 3: SW5 -> /Numpad/np_sw5
- D82 pad 4: CS15 -> /Numpad/np_cs15
- D82 pad 5: SW6 -> /Numpad/np_sw6
- D82 pad 6: CS15 -> /Numpad/np_cs15
- D83 pad 1: SW4 -> /Numpad/np_sw4
- D83 pad 2: CS16 -> /Numpad/np_cs16
- D83 pad 3: SW5 -> /Numpad/np_sw5
- D83 pad 4: CS16 -> /Numpad/np_cs16
- D83 pad 5: SW6 -> /Numpad/np_sw6
- D83 pad 6: CS16 -> /Numpad/np_cs16
- D9 pad 1: ROW9 -> /F Row/fr_row10
- D91 pad 1: ROW5 -> /Numpad/np_row5
- D92 pad 1: ROW9 -> /Numpad/np_row9
- D99 pad 1: SW4 -> /Numpad/np_sw1
- D99 pad 2: CS10 -> /Numpad/np_cs5
- D99 pad 3: SW5 -> /Numpad/np_sw2
- D99 pad 4: CS10 -> /Numpad/np_cs5
- D99 pad 5: SW6 -> /Numpad/np_sw3
- D99 pad 6: CS10 -> /Numpad/np_cs5
- M1 pad 1: GND -> /Main/GND
- M1 pad 12: COL0 -> /Main/ce_col0
- M1 pad 13: COL1 -> /Main/ce_col1
- M1 pad 14: COL2 -> /Main/ce_col2
- M1 pad 15: COL3 -> /Main/ce_col3
- M1 pad 16: COL4 -> /Main/ce_col4
- M1 pad 17: COL5 -> /Main/ce_col5
- M1 pad 18: COL6 -> /Main/ce_col6
- M1 pad 19: COL7 -> /Main/ce_col7
- M1 pad 2: +3V3 -> /Main/+3.3V
- M1 pad 20: COL8 -> /Main/ce_col8
- M1 pad 21: COL9 -> /Main/ce_col9
- M1 pad 22: ROW0 -> /Main/ce_row0
- M1 pad 23: ROW1 -> /Main/ce_row1
- M1 pad 24: ROW2 -> /Main/ce_row2
- M1 pad 25: ROW3 -> /Main/ce_row3
- M1 pad 26: ROW4 -> /Main/ce_row4
- M1 pad 27: ROW5 -> /Main/ce_row5
- M1 pad 28: ROW6 -> /Main/ce_row6
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
Commit message: idk some updates
Parts:
- FPC201, FPC202, FPC203, FPC204, FPC205, FPC206, FPC207, FPC208, FPC209, FPC210, FPC211, FPC212, FPC213, FPC214, FPC215, FPC216: moved to B.Cu
- moved FPC214 404.3 mm to (439.0, -36.6), turned to 90 degrees
- moved FPC215 401.0 mm to (407.5, -79.2)
- moved FPC216 399.2 mm to (418.7, -34.1), turned to -90 degrees
- moved JP204 379.8 mm to (342.2, -110.3)
- moved JP205 379.8 mm to (342.2, -106.8)
- moved JP206 379.8 mm to (342.2, -103.2)
- moved FPC213 359.9 mm to (372.6, -87.0), turned to 90 degrees
- moved FPC211 322.9 mm to (328.7, -103.9), turned to -90 degrees
- moved FPC209 321.2 mm to (327.2, -79.9), turned to 90 degrees
- moved JP201 320.5 mm to (280.8, -109.9)
- moved JP202 320.5 mm to (280.8, -106.4)
- moved JP203 320.5 mm to (280.8, -102.8)
- moved FPC210 308.9 mm to (327.4, -38.9), turned to 90 degrees
- moved FPC212 304.2 mm to (327.5, -60.2), turned to -90 degrees
- moved JP7 277.5 mm to (340.3, -42.0)
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
Commit message: Update Frooastboard Walnut Modular.kicad_pcb
Parts:
- FPC203, FPC204: footprint AFA01-SXXFCX-00:FPC-SMD_10P_P1.00_AFA01-S10FCC-00 -> AFA01-SXXFCX-00:FPC-SMD_10P-P1.00_AFA01-S10FCC-00
- MX35: footprint MX_Only:MXOnly-2U-ReversedVerticalStabilizers-NoLED -> MX_Only:MXOnly-2U-NoLED
- moved FPC214 56.4 mm to (392.7, -4.50)
- moved FPC216 28.5 mm to (392.7, -22.6), turned to 90 degrees
- moved FPC207 22.2 mm to (49.2, -108.1), turned to 180 degrees
- moved FPC208 21.4 mm to (48.4, -75.7), turned to 0 degrees
- moved FPC215 18.9 mm to (404.8, -60.5), turned to 180 degrees
- moved FPC206 15.6 mm to (74.1, -75.7)
- moved FPC204 8.50 mm to (97.1, -75.7)
- moved FPC202 5.01 mm to (119.7, -75.7)
- moved FPC213 2.49 mm to (374.0, -89.0)
- turned MX148 to 90 degrees
- turned MX28 to 180 degrees
- turned MX35 to -90 degrees

Commit message: update leds and diodes
Parts:
- removed D5: Caps Lock Indicator, LED_SMD:LED_0805_2012Metric
- removed D52: Roll Indicator, LED_SMD:LED_0805_2012Metric
- removed D58: Num Lock Indicator, LED_SMD:LED_0805_2012Metric
- MX35: footprint MX_Only:MXOnly-2U-NoLED -> MX_Only:MXOnly-2U-ReversedVerticalStabilizers-NoLED
- moved D6 275.9 mm to (14.7, -117.5), turned to 90 degrees
- moved D8 248.4 mm to (52.8, -117.5), turned to 90 degrees
- moved D9 236.8 mm to (71.8, -117.5), turned to 90 degrees
- moved D10 226.3 mm to (90.9, -117.5), turned to 90 degrees
- moved D12 217.0 mm to (109.9, -117.5), turned to 90 degrees
- moved D126 211.9 mm to (33.7, -88.9), turned to 90 degrees
- moved D113 207.2 mm to (14.7, -88.9), turned to 90 degrees
- moved D54 205.1 mm to (405.2, -88.9), turned to 90 degrees
- moved D13 204.3 mm to (138.5, -117.5), turned to 90 degrees
- moved D66 203.7 mm to (424.3, -88.9), turned to 90 degrees
- moved D29 198.9 mm to (343.3, -117.5), turned to 90 degrees
- moved D139 197.6 mm to (52.8, -88.9), turned to 90 degrees
- moved D114 193.8 mm to (19.4, -69.8), turned to 90 degrees
- moved D55 193.7 mm to (405.2, -69.8), turned to 90 degrees
- moved D28 187.5 mm to (324.2, -117.5), turned to 90 degrees
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Connections:
- net /F Row/D+ renamed /F Row/fr_dp
- net /F Row/D- renamed /F Row/fr_dn
- M1 pad 10: (no net) -> unconnected-(M1-GND-Pad10)
- M1 pad 11: (no net) -> unconnected-(M1-RESET-Pad11)
- M2 pad 10: (no net) -> unconnected-(M2-GND-Pad10)
- M2 pad 11: (no net) -> unconnected-(M2-RESET-Pad11)

Commit message: flip footprint to back for clearence
Parts:
- C38, C39, C40, D10, D100, D101, D103, D104, D105, D106, D107, D108, D109, D11, D111, D112, D113, D114, D115, D116, D117, D118, D12, D120, D121, D122, D123, D124, D125, D126, D127, D128, D129, D13, D130, D131, D132, D133, D134, D135, D137, D138, D139, D14, D140, D141, D142, D143, D144, D145, D146, D147, D148, D15, D150, D151, D152, D153, D154, D155, D156, D157, D158, D159, D16, D160, D161, D163, D164, D165, D166, D167, D168, D169, D17, D170, D171, D172, D173, D174, D175, D176, D177, D178, D179, D18, D181, D183, D184, D185, D186, D187, D188, D189, D19, D190, D191, D192, D194, D195, D196, D197, D198, D199, D20, D200, D201, D202, D203, D204, D205, D206, D207, D208, D21, D210, D211, D212, D214, D215, D216, D218, D219, D22, D220, D221, D222, D223, D228, D229, D23, D231, D236, D237, D239, D24, D244, D245, D247, D25, D252, D253, D255, D26, D27, D28, D29, D29_1, D29_2, D3, D30, D31, D32, D33, D34, D34_1, D34_2, D34_3, D35, D35_1, D35_2, D35_3, D36, D36_1, D36_2, D36_3, D37, D37_1, D37_2, D37_3, D38_1, D38_2, D38_3, D39, D39_1, D39_2, D39_3, D4, D40, D41, D42, D43, D44, D45, D46, D47, D48, D49, D50, D51, D53, D54, D55, D56, D57, D59, D6, D60, D61, D62, D63, D65, D66, D67, D69, D7, D71, D72, D73, D74, D75, D76, D77, D78, D79, D8, D80, D81, D82, D83, D87, D88, D89, D9, D91, D92, D99, JP1, JP2, JP201, JP202, JP203, JP204, JP205, JP206, JP3, JP4, JP5, JP6, JP7, JP8, JP9, R21, R22, R25, R26, R27, R28, R29, R30, R31: moved to B.Cu
- MX35: footprint MX_Only:MXOnly-2U-ReversedVerticalStabilizers-NoLED -> MX_Only:MXOnly-2U-NoLED
- moved JP4 5.56 mm to (299.5, -39.3)
- moved JP6 5.56 mm to (299.5, -44.8)
- moved JP1 5.56 mm to (282.2, -58.3), turned to 0 degrees
- moved JP3 5.56 mm to (282.2, -52.8), turned to 0 degrees
- moved JP7 5.56 mm to (342.1, -35.7)
- moved JP9 5.56 mm to (342.1, -41.3)
- moved JP201 5.56 mm to (281.0, -106.0)
- moved JP203 5.56 mm to (281.0, -111.5)
- moved JP204 5.56 mm to (342.9, -106.0)
- moved JP206 5.56 mm to (342.9, -111.5)
- moved JP5 0.29 mm to (299.5, -42.1)
- moved JP2 0.15 mm to (282.2, -55.6), turned to 0 degrees
- turned D100 to 90 degrees
- turned D101 to 90 degrees
- turned D103 to 90 degrees
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
Commit message: update to 2 layer pcb
Other:
- copper layers 4 -> 2
Changed lines of the file:
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@@
   (layers
     (0 "F.Cu" signal)
-    (1 "In1.Cu" signal)
-    (2 "In2.Cu" signal)
     (31 "B.Cu" signal)
     (32 "B.Adhes" user "B.Adhesive")
@@
       (layer "F.Mask" (type "Top Solder Mask") (color "Black") (thickness 0.01))
       (layer "F.Cu" (type "copper") (thickness 0.035))
-      (layer "dielectric 1" (type "prepreg") (thickness 0.2104) (material "FR4") (epsilon_r 4.5) (loss_tangent 0.02))
-      (layer "In1.Cu" (type "copper") (thickness 0.0152))
-      (layer "dielectric 2" (type "core") (thickness 1.065) (material "FR4") (epsilon_r 4.5) (loss_tangent 0.02))
-      (layer "In2.Cu" (type "copper") (thickness 0.0152))
-      (layer "dielectric 3" (type "prepreg") (thickness 0.2104) (material "FR4") (epsilon_r 4.5) (loss_tangent 0.02))
+      (layer "dielectric 1" (type "core") (thickness 1.5162) (material "FR4") (epsilon_r 4.5) (loss_tangent 0.02))
       (layer "B.Cu" (type "copper") (thickness 0.035))
       (layer "B.Mask" (type "Bottom Solder Mask") (color "Black") (thickness 0.01))

Commit message: some stuff
Parts:
- MX147: value MX-LED -> Scroll Lock
- turned D91 to 0 degrees
Connections:
- net /F Row/fr_dn renamed /F Row/fr_d-
- net /F Row/fr_dp renamed /F Row/fr_d+
- net /Main/ce_dn renamed /Main/ce_d-
- net /Main/ce_dp renamed /Main/ce_d+
- net /Numpad/np_dn renamed /Numpad/np_d-
- net /Numpad/np_dp renamed /Numpad/np_d+
- D10 pad 1: /F Row/fr_row11 -> /F Row/fr_row10
- D13 pad 1: /F Row/fr_row11 -> /F Row/fr_row10
- D16 pad 1: /F Row/fr_row11 -> /F Row/fr_row10
- D18 pad 1: /F Row/fr_row10 -> /F Row/fr_row11
- D20 pad 1: /F Row/fr_row10 -> /F Row/fr_row11
- D24 pad 1: /F Row/fr_row10 -> /F Row/fr_row11
- D28 pad 1: /F Row/fr_row10 -> /F Row/fr_row11
- D8 pad 1: /F Row/fr_row11 -> /F Row/fr_row10
- FPC201 pad 7: (no net) -> /F Row/GND
- FPC201 pad 8: (no net) -> /F Row/GND
- FPC202 pad 7: (no net) -> /Main/GND
- FPC202 pad 8: (no net) -> /Main/GND
- FPC203 pad 11: (no net) -> /F Row/GND
- FPC203 pad 12: (no net) -> /F Row/GND
- FPC204 pad 11: (no net) -> /Main/GND
- FPC204 pad 12: (no net) -> /Main/GND
- FPC205 pad 7: (no net) -> /F Row/GND
- FPC205 pad 8: (no net) -> /F Row/GND
- FPC206 pad 7: (no net) -> /Main/GND
- FPC206 pad 8: (no net) -> /Main/GND
- FPC207 pad 17: (no net) -> /F Row/GND
- FPC207 pad 18: (no net) -> /F Row/GND
- FPC208 pad 17: (no net) -> /Main/GND
- FPC208 pad 18: (no net) -> /Main/GND
- FPC209 pad 17: (no net) -> /Main/GND
- FPC209 pad 18: (no net) -> /Main/GND
- FPC210 pad 17: (no net) -> /Main/GND
- FPC210 pad 18: (no net) -> /Main/GND
- FPC211 pad 7: (no net) -> /Main/GND
- FPC211 pad 8: (no net) -> /Main/GND
- FPC212 pad 7: (no net) -> /Main/GND
- FPC212 pad 8: (no net) -> /Main/GND
- FPC213 pad 7: (no net) -> /Numpad/GND
- FPC213 pad 8: (no net) -> /Numpad/GND
- FPC214 pad 7: (no net) -> /Numpad/GND
- FPC214 pad 8: (no net) -> /Numpad/GND
- FPC215 pad 17: (no net) -> /Numpad/GND
- FPC215 pad 18: (no net) -> /Numpad/GND
- FPC216 pad 17: (no net) -> /Numpad/GND
- FPC216 pad 18: (no net) -> /Numpad/GND
- MX10 pad 1: /F Row/fr_col4 -> /F Row/fr_col1
- MX11 pad 1: /F Row/fr_col5 -> /F Row/fr_col2
- MX12 pad 1: /F Row/fr_col5 -> /F Row/fr_col3
- MX13 pad 1: /F Row/fr_col6 -> /F Row/fr_col4
- MX14 pad 1: /F Row/fr_col6 -> /F Row/fr_col5
- MX147 pad 1: /F Row/fr_col7 -> /F Row/fr_col6
- MX2 pad 1: /F Row/fr_col0 -> /F Row/fr_col1
- MX3 pad 1: /F Row/fr_col1 -> /F Row/fr_col2
- MX4 pad 1: /F Row/fr_col1 -> /F Row/fr_col3
- MX5 pad 1: /F Row/fr_col2 -> /F Row/fr_col4
- MX6 pad 1: /F Row/fr_col2 -> /F Row/fr_col5
- MX7 pad 1: /F Row/fr_col3 -> /F Row/fr_col6
- MX8 pad 1: /F Row/fr_col3 -> /F Row/fr_col7
- MX9 pad 1: /F Row/fr_col4 -> /F Row/fr_col0
Routing:
- net /F Row/fr_row11: track 0.00 -> 270.9 mm
- net /Numpad/np_col8: track 0.00 -> 212.1 mm, vias 0 -> 2
- net /Main/ce_col3: track 0.00 -> 201.2 mm
- net /F Row/fr_row10: track 0.00 -> 197.1 mm, vias 0 -> 4
- net /Main/ce_d-: track 0.00 -> 169.3 mm
- net /Main/ce_d+: track 0.00 -> 167.2 mm
- net /Numpad/np_col9: track 0.00 -> 141.8 mm
- net /Main/ce_row0: track 0.00 -> 140.0 mm, vias 0 -> 2
- net /Main/ce_col2: track 0.00 -> 138.8 mm
- net /Main/ce_col1: track 0.00 -> 134.7 mm
- net /Main/ce_col0: track 0.00 -> 130.2 mm
- net /Main/ce_row4: track 0.00 -> 115.6 mm, vias 0 -> 2
- net /F Row/GND: track 0.00 -> 102.9 mm
- net /F Row/fr_col0: track 0.00 -> 93.8 mm, vias 0 -> 1
- net /Main/ce_col4: track 0.00 -> 90.3 mm
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