File: Frooastboard Walnut Modular/KiCad Project/Frooastboard Walnut Modular.kicad_pcb (KiCad board)
At the start: 2 copper layers, 406 parts, among them M1 Frooastboard_MM2040, M2 Frooastboard_MM2040

Commit message: fix errors
Parts:
- MX32: value Comma -> Dot
Connections:
- D87 pad 1: /Main/ce_row11 -> /Main/ce_col9
- D88 pad 1: /Main/ce_row11 -> /Main/ce_col9
- D89 pad 1: /Main/ce_row11 -> /Main/ce_col9
Changed lines of the file:
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@@
         (effects (font (size 1 1) (thickness 0.15)))
     )
-    (fp_text value "Comma" (at 0 -7.9375) (layer "Dwgs.User")
+    (fp_text value "Dot" (at 0 -7.9375) (layer "Dwgs.User")
         (effects (font (size 1 1) (thickness 0.15)))
     )
@@
       (stroke (width 0.1) (type solid)) (layer "B.Fab"))
     (pad "1" smd roundrect (at -0.9375 0 180) (size 0.975 1.4) (layers "B.Cu" "B.Paste" "B.Mask") (roundrect_rratio 0.25)
-      (net 207 "/Main/ce_row11") (pinfunction "K") (pintype "passive"))
+      (net 262 "/Main/ce_col9") (pinfunction "K") (pintype "passive"))
     (pad "2" smd roundrect (at 0.9375 0 180) (size 0.975 1.4) (layers "B.Cu" "B.Paste" "B.Mask") (roundrect_rratio 0.25)
       (net 27 "Net-(D89-A)") (pinfunction "A") (pintype "passive"))
@@
     (fp_arc (start 0.5748 5.9436) (mid 1.281907 6.236493) (end 1.5748 6.9436)
       (stroke (width 0.1) (type default)) (layer "B.Fab"))
-    (fp_arc (start 1.633379 12.428379) (mid 1.589998 12.363508) (end 1.5748 12.286957)
+    (fp_arc (start 1.633379 12.428379) (mid 1.589986 12.363508) (end 1.5748 12.286957)
       (stroke (width 0.1) (type default)) (layer "B.Fab"))
     (fp_arc (start 2.704307 13.499307) (mid 2.921095 13.823724) (end 2.9972 14.206414)
@@
     (fp_arc (start 3.1972 26.7462) (mid 3.055779 26.687621) (end 2.9972 26.5462)
       (stroke (width 0.1) (type default)) (layer "B.Fab"))
-    (fp_arc (start 14.059693 1.281907) (mid 13.735253 1.498635) (end 13.352586 1.5748)
+    (fp_arc (start 14.059693 1.281907) (mid 13.735253 1.498646) (end 13.352586 1.5748)
       (stroke (width 0.1) (type default)) (layer "B.Fab"))
-    (fp_arc (start 15.283022 0.058578) (mid 15.347893 0.015186) (end 15.424443 0)
+    (fp_arc (start 15.283022 0.058578) (mid 15.347893 0.015197) (end 15.424443 0)
       (stroke (width 0.1) (type default)) (layer "B.Fab"))
-    (fp_arc (start 15.333786 26.7462) (mid 15.716457 26.822343) (end 16.040893 27.039093)
+    (fp_arc (start 15.333786 26.7462) (mid 15.716468 26.822331) (end 16.040893 27.039093)
       (stroke (width 0.1) (type default)) (layer "B.Fab"))
     (fp_arc (start 17.380243 28.2956) (mid 17.303717 28.280348) (end 17.238822 28.237022)
       (stroke (width 0.1) (type default)) (layer "B.Fab"))
-    (fp_arc (start 26.637957 0) (mid 26.714487 0.015237) (end 26.779378 0.058578)
+    (fp_arc (start 26.637957 0) (mid 26.714493 0.015231) (end 26.779378 0.058578)
       (stroke (width 0.1) (type default)) (layer "B.Fab"))
-    (fp_arc (start 27.795378 28.237022) (mid 27.730507 28.280414) (end 27.653957 28.2956)
+    (fp_arc (start 27.795378 28.237022) (mid 27.730507 28.280403) (end 27.653957 28.2956)
       (stroke (width 0.1) (type default)) (layer "B.Fab"))
     (fp_arc (start 28.709814 1.5748) (mid 28.327123 1.498699) (end 28.002707 1.281907)
       (stroke (width 0.1) (type default)) (layer "B.Fab"))
-    (fp_arc (start 29.171107 26.861293) (mid 29.495547 26.644565) (end 29.878214 26.5684)
+    (fp_arc (start 29.171107 26.861293) (mid 29.495547 26.644554) (end 29.878214 26.5684)
       (stroke (width 0.1) (type default)) (layer "B.Fab"))
-    (fp_arc (start 41.1734 18.448214) (mid 41.249522 18.065533) (end 41.466293 17.741107)
+    (fp_arc (start 41.1734 18.448214) (mid 41.249516 18.065528) (end 41.466293 17.741107)
       (stroke (width 0.1) (type default)) (layer "B.Fab"))
     (fp_arc (start 41.1734 26.3684) (mid 41.114821 26.509821) (end 40.9734 26.5684)
       (stroke (width 0.1) (type default)) (layer "B.Fab"))
-    (fp_arc (start 43.0276 4.884614) (mid 43.103743 4.501943) (end 43.320493 4.177507)
+    (fp_arc (start 43.0276 4.884614) (mid 43.103731 4.501932) (end 43.320493 4.177507)
       (stroke (width 0.1) (type default)) (layer "B.Fab"))
     (fp_arc (start 43.0276 15.972693) (mid 42.989542 16.164036) (end 42.881154 16.326246)
@@
     (fp_arc (start 44.3516 1.5748) (mid 44.493021 1.633379) (end 44.5516 1.7748)
       (stroke (width 0.1) (type default)) (layer "B.Fab"))
-    (fp_arc (start 44.5516 2.863557) (mid 44.536363 2.940087) (end 44.493022 3.004978)
+    (fp_arc (start 44.5516 2.863557) (mid 44.536369 2.940093) (end 44.493022 3.004978)
       (stroke (width 0.1) (type default)) (layer "B.Fab"))
     (fp_circle (center 7.747 11.7856) (end 8.747 11.7856)
@@
     (fp_arc (start 0.5748 5.9436) (mid 1.281907 6.236493) (end 1.5748 6.9436)
       (stroke (width 0.1) (type default)) (layer "B.Fab"))
-    (fp_arc (start 1.633379 12.428379) (mid 1.589998 12.363508) (end 1.5748 12.286957)
+    (fp_arc (start 1.633379 12.428379) (mid 1.589986 12.363508) (end 1.5748 12.286957)
       (stroke (width 0.1) (type default)) (layer "B.Fab"))
     (fp_arc (start 2.704307 13.499307) (mid 2.921095 13.823724) (end 2.9972 14.206414)
@@
     (fp_arc (start 3.1972 26.7462) (mid 3.055779 26.687621) (end 2.9972 26.5462)
       (stroke (width 0.1) (type default)) (layer "B.Fab"))
-    (fp_arc (start 14.059693 1.281907) (mid 13.735253 1.498635) (end 13.352586 1.5748)
+    (fp_arc (start 14.059693 1.281907) (mid 13.735253 1.498646) (end 13.352586 1.5748)
       (stroke (width 0.1) (type default)) (layer "B.Fab"))
-    (fp_arc (start 15.283022 0.058578) (mid 15.347893 0.015186) (end 15.424443 0)
+    (fp_arc (start 15.283022 0.058578) (mid 15.347893 0.015197) (end 15.424443 0)
       (stroke (width 0.1) (type default)) (layer "B.Fab"))
-    (fp_arc (start 15.333786 26.7462) (mid 15.716457 26.822343) (end 16.040893 27.039093)
+    (fp_arc (start 15.333786 26.7462) (mid 15.716468 26.822331) (end 16.040893 27.039093)
       (stroke (width 0.1) (type default)) (layer "B.Fab"))
     (fp_arc (start 17.380243 28.2956) (mid 17.303717 28.280348) (end 17.238822 28.237022)
       (stroke (width 0.1) (type default)) (layer "B.Fab"))
-    (fp_arc (start 26.637957 0) (mid 26.714487 0.015237) (end 26.779378 0.058578)
+    (fp_arc (start 26.637957 0) (mid 26.714493 0.015231) (end 26.779378 0.058578)
       (stroke (width 0.1) (type default)) (layer "B.Fab"))
-    (fp_arc (start 27.795378 28.237022) (mid 27.730507 28.280414) (end 27.653957 28.2956)
+    (fp_arc (start 27.795378 28.237022) (mid 27.730507 28.280403) (end 27.653957 28.2956)
       (stroke (width 0.1) (type default)) (layer "B.Fab"))
     (fp_arc (start 28.709814 1.5748) (mid 28.327123 1.498699) (end 28.002707 1.281907)
       (stroke (width 0.1) (type default)) (layer "B.Fab"))
-    (fp_arc (start 29.171107 26.861293) (mid 29.495547 26.644565) (end 29.878214 26.5684)
+    (fp_arc (start 29.171107 26.861293) (mid 29.495547 26.644554) (end 29.878214 26.5684)
       (stroke (width 0.1) (type default)) (layer "B.Fab"))
-    (fp_arc (start 41.1734 18.448214) (mid 41.249522 18.065533) (end 41.466293 17.741107)
+    (fp_arc (start 41.1734 18.448214) (mid 41.249516 18.065528) (end 41.466293 17.741107)
       (stroke (width 0.1) (type default)) (layer "B.Fab"))
     (fp_arc (start 41.1734 26.3684) (mid 41.114821 26.509821) (end 40.9734 26.5684)
       (stroke (width 0.1) (type default)) (layer "B.Fab"))
-    (fp_arc (start 43.0276 4.884614) (mid 43.103743 4.501943) (end 43.320493 4.177507)
+    (fp_arc (start 43.0276 4.884614) (mid 43.103731 4.501932) (end 43.320493 4.177507)
       (stroke (width 0.1) (type default)) (layer "B.Fab"))
     (fp_arc (start 43.0276 15.972693) (mid 42.989542 16.164036) (end 42.881154 16.326246)
@@
     (fp_arc (start 44.3516 1.5748) (mid 44.493021 1.633379) (end 44.5516 1.7748)
       (stroke (width 0.1) (type default)) (layer "B.Fab"))
-    (fp_arc (start 44.5516 2.863557) (mid 44.536363 2.940087) (end 44.493022 3.004978)
+    (fp_arc (start 44.5516 2.863557) (mid 44.536369 2.940093) (end 44.493022 3.004978)
       (stroke (width 0.1) (type default)) (layer "B.Fab"))
     (fp_circle (center 7.747 11.7856) (end 8.747 11.7856)
@@
       (stroke (width 0.1) (type solid)) (layer "B.Fab"))
     (pad "1" smd roundrect (at -0.9375 0 90) (size 0.975 1.4) (layers "B.Cu" "B.Paste" "B.Mask") (roundrect_rratio 0.25)
-      (net 207 "/Main/ce_row11") (pinfunction "K") (pintype "passive"))
+      (net 262 "/Main/ce_col9") (pinfunction "K") (pintype "passive"))
     (pad "2" smd roundrect (at 0.9375 0 90) (size 0.975 1.4) (layers "B.Cu" "B.Paste" "B.Mask") (roundrect_rratio 0.25)
       (net 29 "Net-(D87-A)") (pinfunction "A") (pintype "passive"))
@@
       (stroke (width 0.1) (type solid)) (layer "B.Fab"))
     (pad "1" smd roundrect (at -0.9375 0 90) (size 0.975 1.4) (layers "B.Cu" "B.Paste" "B.Mask") (roundrect_rratio 0.25)
-      (net 207 "/Main/ce_row11") (pinfunction "K") (pintype "passive"))
+      (net 262 "/Main/ce_col9") (pinfunction "K") (pintype "passive"))
     (pad "2" smd roundrect (at 0.9375 0 90) (size 0.975 1.4) (layers "B.Cu" "B.Paste" "B.Mask") (roundrect_rratio 0.25)
       (net 28 "Net-(D88-A)") (pinfunction "A") (pintype "passive"))
