File: Frooastboard Walnut Modular/KiCad Project/MM2040.kicad_sch (KiCad schematic)
At the start: 39 parts, among them J1 SW Interface, J2 Conn_01x16, J3 Conn_01x06, J4 Conn_01x06, J5 Conn_01x10, J6 Conn_01x12, J7 Conn_01x04, U1 RP2040, U3 W25Q32JVZP, U5 IS31FL3733-QF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

Commit message: some errors and board outline
Parts:
- J7: footprint Connector_PinHeader_1.27mm:PinHeader_1x04_P1.27mm_Vertical -> Frooastboard Footprints:PinHeader_1x04_P1.27mm_Vertical
Changed lines of the file:
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@@
       (effects (font (size 1.27 1.27)) (justify left))
     )
-    (property "Footprint" "Connector_PinHeader_1.27mm:PinHeader_1x04_P1.27mm_Vertical" (at 213.36 130.81 0)
+    (property "Footprint" "Frooastboard Footprints:PinHeader_1x04_P1.27mm_Vertical" (at 213.36 130.81 0)
       (effects (font (size 1.27 1.27)) hide)
     )

Commit message: some more stuff changed
Parts:
- added U4: LM317_SOT-223, Package_TO_SOT_SMD:SOT-223-3_TabPin2, symbol Regulator_Linear:LM317_SOT-223
Connections:
- net +3V3: now also U4.2 (VO)
- net +5V: now also U4.3 (VI)
- net GND: now also U4.1 (ADJ)
- net at J6.12 (Pin_12): now also U1.32 (GPIO21)
Changed lines of the file:
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@@
+    (stroke (width 0) (type default))
+  )
+  (wire (pts (xy 280.67 36.83) (xy 280.67 39.37))
     (stroke (width 0) (type default))
   )
@@
     (stroke (width 0) (type default))
   )
+  (wire (pts (xy 109.22 90.17) (xy 111.76 90.17))
+    (stroke (width 0) (type default))
+  )
   (wire (pts (xy 208.28 128.27) (xy 205.74 128.27))
     (stroke (width 0) (type default))
@@
     (stroke (width 0) (type default))
   )
+  (wire (pts (xy 280.67 39.37) (xy 283.21 39.37))
+    (stroke (width 0) (type default))
+  )
   (wire (pts (xy 66.04 48.26) (xy 68.58 48.26))
     (stroke (width 0) (type default))
@@
     (stroke (width 0) (type default))
   )
+  (wire (pts (xy 290.83 46.99) (xy 290.83 49.53))
+    (stroke (width 0) (type default))
+  )
   (wire (pts (xy 66.04 91.44) (xy 68.58 91.44))
     (stroke (width 0) (type default))
@@
     (stroke (width 0) (type default))
   )
+  (wire (pts (xy 300.99 39.37) (xy 300.99 36.83))
+    (stroke (width 0) (type default))
+  )
   (wire (pts (xy 57.15 204.47) (xy 54.61 204.47))
     (stroke (width 0) (type default))
@@
   )
   (wire (pts (xy 83.82 26.67) (xy 83.82 29.21))
+    (stroke (width 0) (type default))
+  )
+  (wire (pts (xy 298.45 39.37) (xy 300.99 39.37))
     (stroke (width 0) (type default))
   )
@@
         (path "/e63e39d7-6ac0-4ffd-8aa3-1841a4541b55/eba7bed6-3b4a-4b7a-b4a2-784017f24fe8"
           (reference "C11") (unit 1)
+        )
+      )
+    )
+  )
+  (symbol (lib_id "power:GND") (at 290.83 49.53 0) (unit 1)
+    (in_bom yes) (on_board yes) (dnp no) (fields_autoplaced)
+    (property "Reference" "#PWR0132" (at 290.83 55.88 0)
+      (effects (font (size 1.27 1.27)) hide)
+    )
+    (property "Value" "GND" (at 290.83 54.61 0)
+      (effects (font (size 1.27 1.27)))
+    )
+    (property "Footprint" "" (at 290.83 49.53 0)
+      (effects (font (size 1.27 1.27)) hide)
+    )
+    (property "Datasheet" "" (at 290.83 49.53 0)
+      (effects (font (size 1.27 1.27)) hide)
+    )
+    (pin "1")
+    (instances
+      (project "Frooastboard Walnut Modular"
+        (path "/e63e39d7-6ac0-4ffd-8aa3-1841a4541b55"
+          (reference "#PWR0132") (unit 1)
+        )
+        (path "/e63e39d7-6ac0-4ffd-8aa3-1841a4541b55/eba7bed6-3b4a-4b7a-b4a2-784017f24fe8"
+          (reference "#PWR030") (unit 1)
         )
       )
@@
     )
   )
+  (symbol (lib_id "Regulator_Linear:LM317_SOT-223") (at 290.83 39.37 0) (unit 1)
+    (in_bom yes) (on_board yes) (dnp no) (fields_autoplaced)
+    (property "Reference" "U4" (at 290.83 33.02 0)
+      (effects (font (size 1.27 1.27)))
+    )
+    (property "Value" "LM317_SOT-223" (at 290.83 35.56 0)
+      (effects (font (size 1.27 1.27)))
+    )
+    (property "Footprint" "Package_TO_SOT_SMD:SOT-223-3_TabPin2" (at 290.83 33.02 0)
+      (effects (font (size 1.27 1.27) italic) hide)
+    )
+    (property "Datasheet" "http://www.ti.com/lit/ds/symlink/lm317.pdf" (at 290.83 39.37 0)
+      (effects (font (size 1.27 1.27)) hide)
+    )
+    (pin "1")
+    (pin "2")
+    (pin "3")
+    (instances
+      (project "Frooastboard Walnut Modular"
+        (path "/e63e39d7-6ac0-4ffd-8aa3-1841a4541b55/eba7bed6-3b4a-4b7a-b4a2-784017f24fe8"
+          (reference "U4") (unit 1)
+        )
+      )
+    )
+  )
   (symbol (lib_id "power:+3.3V") (at 83.82 24.13 0) (unit 1)
     (in_bom yes) (on_board yes) (dnp no) (fields_autoplaced)
@@
     )
   )
+  (symbol (lib_id "power:+5V") (at 280.67 36.83 0) (unit 1)
+    (in_bom yes) (on_board yes) (dnp no) (fields_autoplaced)
+    (property "Reference" "#PWR0146" (at 280.67 40.64 0)
+      (effects (font (size 1.27 1.27)) hide)
+    )
+    (property "Value" "+5V" (at 280.67 31.75 0)
+      (effects (font (size 1.27 1.27)))
+    )
+    (property "Footprint" "" (at 280.67 36.83 0)
+      (effects (font (size 1.27 1.27)) hide)
+    )
+    (property "Datasheet" "" (at 280.67 36.83 0)
+      (effects (font (size 1.27 1.27)) hide)
+    )
+    (pin "1")
+    (instances
+      (project "Frooastboard Walnut Modular"
+        (path "/e63e39d7-6ac0-4ffd-8aa3-1841a4541b55"
+          (reference "#PWR0146") (unit 1)
+        )
+        (path "/e63e39d7-6ac0-4ffd-8aa3-1841a4541b55/eba7bed6-3b4a-4b7a-b4a2-784017f24fe8"
+          (reference "#PWR029") (unit 1)
+        )
+      )
+    )
+  )
   (symbol (lib_id "Connector:TestPoint_2Pole") (at 189.23 39.37 0) (unit 1)
     (in_bom yes) (on_board yes) (dnp no) (fields_autoplaced)
@@
         )
       )
+    )
+  )
+  (symbol (lib_id "power:+3.3V") (at 300.99 36.83 0) (unit 1)
+    (in_bom yes) (on_board yes) (dnp no) (fields_autoplaced)
+    (property "Reference" "#PWR0133" (at 300.99 40.64 0)
+      (effects (font (size 1.27 1.27)) hide)
+    )
+    (property "Value" "+3.3V" (at 300.99 31.75 0)
+      (effects (font (size 1.27 1.27)))
+    )
+    (property "Footprint" "" (at 300.99 36.83 0)
+      (effects (font (size 1.27 1.27)) hide)
+    )
+    (property "Datasheet" "" (at 300.99 36.83 0)
+      (effects (font (size 1.27 1.27)) hide)
+    )
+    (pin "1")
+    (instances
+      (project "Frooastboard Walnut Modular"
+        (path "/e63e39d7-6ac0-4ffd-8aa3-1841a4541b55"
+          (reference "#PWR0133") (unit 1)
+        )
+        (path "/e63e39d7-6ac0-4ffd-8aa3-1841a4541b55/eba7bed6-3b4a-4b7a-b4a2-784017f24fe8"
+          (reference "#PWR028") (unit 1)
+        )
+      )

Commit message: some more progress
Parts:
- removed U4: LM317_SOT-223, Package_TO_SOT_SMD:SOT-223-3_TabPin2, symbol Regulator_Linear:LM317_SOT-223
- added U5: LM317L_SOT-89, Package_TO_SOT_SMD:SOT-89-3, symbol Regulator_Linear:LM317L_SOT-89
- TP5: footprint Connector_PinHeader_1.00mm:PinHeader_1x02_P1.00mm_Vertical -> Connector_PinHeader_1.27mm:PinHeader_1x02_P1.27mm_Vertical
Connections:
- net +3V3: now also U5.2 (VO)
- net +5V: now also U5.3 (VI)
- net GND: now also U5.1 (ADJ)
Changed lines of the file:
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@@
+    )
+  )
+  (symbol (lib_id "Regulator_Linear:LM317L_SOT-89") (at 290.83 39.37 0) (unit 1)
+    (in_bom yes) (on_board yes) (dnp no) (fields_autoplaced)
+    (property "Reference" "U5" (at 290.83 33.02 0)
+      (effects (font (size 1.27 1.27)))
+    )
+    (property "Value" "LM317L_SOT-89" (at 290.83 35.56 0)
+      (effects (font (size 1.27 1.27)))
+    )
+    (property "Footprint" "Package_TO_SOT_SMD:SOT-89-3" (at 290.83 33.02 0)
+      (effects (font (size 1.27 1.27) italic) hide)
+    )
+    (property "Datasheet" "http://www.ti.com/lit/ds/symlink/lm317l.pdf" (at 290.83 39.37 0)
+      (effects (font (size 1.27 1.27)) hide)
+    )
+    (pin "1")
+    (pin "2")
+    (pin "3")
+    (instances
+      (project "Frooastboard Walnut Modular"
+        (path "/e63e39d7-6ac0-4ffd-8aa3-1841a4541b55/eba7bed6-3b4a-4b7a-b4a2-784017f24fe8"
+          (reference "U5") (unit 1)
+        )
+      )
     )
   )
@@
         (path "/e63e39d7-6ac0-4ffd-8aa3-1841a4541b55/eba7bed6-3b4a-4b7a-b4a2-784017f24fe8"
           (reference "R2") (unit 1)
-        )
-      )
-    )
-  )
-  (symbol (lib_id "Regulator_Linear:LM317_SOT-223") (at 290.83 39.37 0) (unit 1)
-    (in_bom yes) (on_board yes) (dnp no) (fields_autoplaced)
-    (property "Reference" "U4" (at 290.83 33.02 0)
-      (effects (font (size 1.27 1.27)))
-    )
-    (property "Value" "LM317_SOT-223" (at 290.83 35.56 0)
-      (effects (font (size 1.27 1.27)))
-    )
-    (property "Footprint" "Package_TO_SOT_SMD:SOT-223-3_TabPin2" (at 290.83 33.02 0)
-      (effects (font (size 1.27 1.27) italic) hide)
-    )
-    (property "Datasheet" "http://www.ti.com/lit/ds/symlink/lm317.pdf" (at 290.83 39.37 0)
-      (effects (font (size 1.27 1.27)) hide)
-    )
-    (pin "1")
-    (pin "2")
-    (pin "3")
-    (instances
-      (project "Frooastboard Walnut Modular"
-        (path "/e63e39d7-6ac0-4ffd-8aa3-1841a4541b55/eba7bed6-3b4a-4b7a-b4a2-784017f24fe8"
-          (reference "U4") (unit 1)
         )
       )
@@
       (effects (font (size 1.27 1.27)))
     )
-    (property "Footprint" "Connector_PinHeader_1.00mm:PinHeader_1x02_P1.00mm_Vertical" (at 189.23 39.37 0)
-      (effects (font (size 1.27 1.27)) hide)
-    )
+    (property "Footprint" "Connector_PinHeader_1.27mm:PinHeader_1x02_P1.27mm_Vertical" (at 189.23 39.37 0)
+      (effects (font (size 1.27 1.27)) hide)
+    )
