File: Frooastboard Walnut Modular/KiCad Project/F Row.kicad_sch (KiCad schematic)
At the start: 64 parts, among them J12 Conn_01x06_Male, J13 Conn_01x16_Male, J14 Conn_01x10_Male, J18 Conn_01x04_Male

Commit message: do some stuff
Parts:
- MX1: value MX-NoLED -> Escape
- MX10: value MX-NoLED -> F9
- MX11: value MX-NoLED -> F10
- MX12: value MX-NoLED -> F11
- MX13: value MX-NoLED -> F12
- MX14: value MX-NoLED -> Print Screen
- MX15: value MX-NoLED -> Scroll Lock
- MX16: value MX-NoLED -> Pause
- MX2: value MX-NoLED -> F1
- MX3: value MX-NoLED -> F2
- MX4: value MX-NoLED -> F3
- MX5: value MX-NoLED -> F4
- MX6: value MX-NoLED -> F5
- MX7: value MX-NoLED -> F6
- MX8: value MX-NoLED -> F7
- MX9: value MX-NoLED -> F8
Changed lines of the file:
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@@
       (effects (font (size 1.524 1.524)))
     )
-    (property "Value" "MX-NoLED" (id 1) (at 96.1356 172.72 0)
+    (property "Value" "F2" (id 1) (at 96.1356 172.72 0)
       (effects (font (size 0.508 0.508)))
     )
@@
       (effects (font (size 1.524 1.524)))
     )
-    (property "Value" "MX-NoLED" (id 1) (at 162.1756 175.26 0)
+    (property "Value" "F9" (id 1) (at 162.1756 175.26 0)
       (effects (font (size 0.508 0.508)))
     )
@@
       (effects (font (size 1.524 1.524)))
     )
-    (property "Value" "MX-NoLED" (id 1) (at 105.0256 175.26 0)
+    (property "Value" "F3" (id 1) (at 105.0256 175.26 0)
       (effects (font (size 0.508 0.508)))
     )
@@
       (effects (font (size 1.524 1.524)))
     )
-    (property "Value" "MX-NoLED" (id 1) (at 115.1856 172.72 0)
+    (property "Value" "F4" (id 1) (at 115.1856 172.72 0)
       (effects (font (size 0.508 0.508)))
     )
@@
       (effects (font (size 1.524 1.524)))
     )
-    (property "Value" "MX-NoLED" (id 1) (at 219.3256 175.26 0)
+    (property "Value" "Pause" (id 1) (at 219.3256 175.26 0)
       (effects (font (size 0.508 0.508)))
     )
@@
       (effects (font (size 1.524 1.524)))
     )
-    (property "Value" "MX-NoLED" (id 1) (at 200.2756 175.26 0)
+    (property "Value" "Print Screen" (id 1) (at 200.2756 175.26 0)
       (effects (font (size 0.508 0.508)))
     )
@@
       (effects (font (size 1.524 1.524)))
     )
-    (property "Value" "MX-NoLED" (id 1) (at 134.2356 172.72 0)
+    (property "Value" "F6" (id 1) (at 134.2356 172.72 0)
       (effects (font (size 0.508 0.508)))
     )
@@
       (effects (font (size 1.524 1.524)))
     )
-    (property "Value" "MX-NoLED" (id 1) (at 124.0756 175.26 0)
+    (property "Value" "F5" (id 1) (at 124.0756 175.26 0)
       (effects (font (size 0.508 0.508)))
     )
@@
       (effects (font (size 1.524 1.524)))
     )
-    (property "Value" "MX-NoLED" (id 1) (at 85.9756 175.26 0)
+    (property "Value" "F1" (id 1) (at 85.9756 175.26 0)
       (effects (font (size 0.508 0.508)))
     )
@@
       (effects (font (size 1.524 1.524)))
     )
-    (property "Value" "MX-NoLED" (id 1) (at 77.0856 172.72 0)
+    (property "Value" "Escape" (id 1) (at 77.0856 172.72 0)
       (effects (font (size 0.508 0.508)))
     )
@@
       (effects (font (size 1.524 1.524)))
     )
-    (property "Value" "MX-NoLED" (id 1) (at 181.2256 175.26 0)
+    (property "Value" "F11" (id 1) (at 181.2256 175.26 0)
       (effects (font (size 0.508 0.508)))
     )
@@
       (effects (font (size 1.524 1.524)))
     )
-    (property "Value" "MX-NoLED" (id 1) (at 153.2856 172.72 0)
+    (property "Value" "F8" (id 1) (at 153.2856 172.72 0)
       (effects (font (size 0.508 0.508)))
     )
@@
       (effects (font (size 1.524 1.524)))
     )
-    (property "Value" "MX-NoLED" (id 1) (at 210.4356 172.72 0)
+    (property "Value" "Scroll Lock" (id 1) (at 210.4356 172.72 0)
       (effects (font (size 0.508 0.508)))
     )
@@
       (effects (font (size 1.524 1.524)))
     )
-    (property "Value" "MX-NoLED" (id 1) (at 172.3356 172.72 0)
+    (property "Value" "F10" (id 1) (at 172.3356 172.72 0)
       (effects (font (size 0.508 0.508)))
     )
@@
       (effects (font (size 1.524 1.524)))
     )
-    (property "Value" "MX-NoLED" (id 1) (at 191.3856 172.72 0)
+    (property "Value" "F12" (id 1) (at 191.3856 172.72 0)
       (effects (font (size 0.508 0.508)))
     )
@@
       (effects (font (size 1.524 1.524)))
     )
-    (property "Value" "MX-NoLED" (id 1) (at 143.1256 175.26 0)
-      (effects (font (size 0.508 0.508)))
-    )
+    (property "Value" "F7" (id 1) (at 143.1256 175.26 0)
+      (effects (font (size 0.508 0.508)))
+    )

Commit message: some new stuff
Parts:
- removed D5: RGB_LED_6_Pin, Frooastboard Footprints:Everlight 99-235, symbol Frooastboard Symbols:RGB_LED_6_Pin
- added D52: Roll Indicator, LED_SMD:LED_0805_2012Metric, symbol Device:LED
- C39: footprint (none) -> Capacitor_SMD:C_0805_2012Metric
- D10, D12, D13, D15, D16, D18, D19, D20, D23, D24, D27, D28, D29, D6, D8, D9: footprint (none) -> Diode_SMD:D_0805_2012Metric
- J12: footprint (none) -> Frooastboard Footprints:PinHeader_1x06_P1.27mm_Vertical
- J13: footprint (none) -> Frooastboard Footprints:PinHeader_1x16_P1.27mm_Vertical
- J14: footprint (none) -> Frooastboard Footprints:PinHeader_1x10_P1.27mm_Vertical
- J18: footprint (none) -> Frooastboard Footprints:PinHeader_1x04_P1.27mm_Vertical
Connections:
- net CS2: now also D52.2 (A)
- net SW5: now also D52.1 (K)

Commit message: asign pieces
Parts:
- MX1, MX10, MX11, MX12, MX13, MX14, MX16, MX2, MX3, MX4, MX5, MX6, MX7, MX8, MX9: footprint (none) -> MX_Only:MXOnly-1U-NoLED
- MX15: footprint (none) -> MX_Only:MXOnly-1U
- R28: footprint (none) -> Resistor_SMD:R_0805_2012Metric
Changed lines of the file:
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@@
       (effects (font (size 0.508 0.508)))
     )
-    (property "Footprint" "" (id 2) (at 79.375 178.435 0)
+    (property "Footprint" "MX_Only:MXOnly-1U-NoLED" (id 2) (at 79.375 178.435 0)
       (effects (font (size 1.524 1.524)) hide)
     )
@@
       (effects (font (size 0.508 0.508)))
     )
-    (property "Footprint" "" (id 2) (at 145.415 180.975 0)
+    (property "Footprint" "MX_Only:MXOnly-1U-NoLED" (id 2) (at 145.415 180.975 0)
       (effects (font (size 1.524 1.524)) hide)
     )
@@
       (effects (font (size 0.508 0.508)))
     )
-    (property "Footprint" "" (id 2) (at 88.265 180.975 0)
+    (property "Footprint" "MX_Only:MXOnly-1U-NoLED" (id 2) (at 88.265 180.975 0)
       (effects (font (size 1.524 1.524)) hide)
     )
@@
       (effects (font (size 0.508 0.508)))
     )
-    (property "Footprint" "" (id 2) (at 98.425 178.435 0)
+    (property "Footprint" "MX_Only:MXOnly-1U-NoLED" (id 2) (at 98.425 178.435 0)
       (effects (font (size 1.524 1.524)) hide)
     )
@@
       (effects (font (size 0.508 0.508)))
     )
-    (property "Footprint" "" (id 2) (at 202.565 180.975 0)
+    (property "Footprint" "MX_Only:MXOnly-1U-NoLED" (id 2) (at 202.565 180.975 0)
       (effects (font (size 1.524 1.524)) hide)
     )
@@
       (effects (font (size 0.508 0.508)))
     )
-    (property "Footprint" "" (id 2) (at 183.515 180.975 0)
+    (property "Footprint" "MX_Only:MXOnly-1U-NoLED" (id 2) (at 183.515 180.975 0)
       (effects (font (size 1.524 1.524)) hide)
     )
@@
       (effects (font (size 0.508 0.508)))
     )
-    (property "Footprint" "" (id 2) (at 117.475 178.435 0)
+    (property "Footprint" "MX_Only:MXOnly-1U-NoLED" (id 2) (at 117.475 178.435 0)
       (effects (font (size 1.524 1.524)) hide)
     )
@@
       (effects (font (size 0.508 0.508)))
     )
-    (property "Footprint" "" (id 2) (at 107.315 180.975 0)
+    (property "Footprint" "MX_Only:MXOnly-1U-NoLED" (id 2) (at 107.315 180.975 0)
       (effects (font (size 1.524 1.524)) hide)
     )
@@
       (effects (font (size 0.508 0.508)))
     )
-    (property "Footprint" "" (id 2) (at 69.215 180.975 0)
+    (property "Footprint" "MX_Only:MXOnly-1U-NoLED" (id 2) (at 69.215 180.975 0)
       (effects (font (size 1.524 1.524)) hide)
     )
@@
       (effects (font (size 0.508 0.508)))
     )
-    (property "Footprint" "" (id 2) (at 60.325 178.435 0)
+    (property "Footprint" "MX_Only:MXOnly-1U-NoLED" (id 2) (at 60.325 178.435 0)
       (effects (font (size 1.524 1.524)) hide)
     )
@@
       (effects (font (size 0.508 0.508)))
     )
-    (property "Footprint" "" (id 2) (at 164.465 180.975 0)
+    (property "Footprint" "MX_Only:MXOnly-1U-NoLED" (id 2) (at 164.465 180.975 0)
       (effects (font (size 1.524 1.524)) hide)
     )
@@
       (effects (font (size 0.508 0.508)))
     )
-    (property "Footprint" "" (id 2) (at 136.525 178.435 0)
+    (property "Footprint" "MX_Only:MXOnly-1U-NoLED" (id 2) (at 136.525 178.435 0)
       (effects (font (size 1.524 1.524)) hide)
     )
@@
       (effects (font (size 0.508 0.508)))
     )
-    (property "Footprint" "" (id 2) (at 193.675 178.435 0)
+    (property "Footprint" "MX_Only:MXOnly-1U" (id 2) (at 193.675 178.435 0)
       (effects (font (size 1.524 1.524)) hide)
     )
@@
       (effects (font (size 1.27 1.27)) (justify left))
     )
-    (property "Footprint" "" (id 2) (at 367.792 116.84 90)
+    (property "Footprint" "Resistor_SMD:R_0805_2012Metric" (id 2) (at 367.792 116.84 90)
       (effects (font (size 1.27 1.27)) hide)
     )
@@
       (effects (font (size 0.508 0.508)))
     )
-    (property "Footprint" "" (id 2) (at 155.575 178.435 0)
+    (property "Footprint" "MX_Only:MXOnly-1U-NoLED" (id 2) (at 155.575 178.435 0)
       (effects (font (size 1.524 1.524)) hide)
     )
@@
       (effects (font (size 0.508 0.508)))
     )
-    (property "Footprint" "" (id 2) (at 174.625 178.435 0)
+    (property "Footprint" "MX_Only:MXOnly-1U-NoLED" (id 2) (at 174.625 178.435 0)
       (effects (font (size 1.524 1.524)) hide)
     )
@@
       (effects (font (size 0.508 0.508)))
     )
-    (property "Footprint" "" (id 2) (at 126.365 180.975 0)
-      (effects (font (size 1.524 1.524)) hide)
-    )
+    (property "Footprint" "MX_Only:MXOnly-1U-NoLED" (id 2) (at 126.365 180.975 0)
+      (effects (font (size 1.524 1.524)) hide)
+    )

Commit message: change some stuff maybe finally get started
Parts:
- J12: footprint Frooastboard Footprints:PinHeader_1x06_P1.27mm_Vertical -> Connector_PinHeader_1.27mm:PinHeader_1x06_P1.27mm_Vertical
- J13: footprint Frooastboard Footprints:PinHeader_1x16_P1.27mm_Vertical -> Connector_PinHeader_1.27mm:PinHeader_1x16_P1.27mm_Vertical
- J14: footprint Frooastboard Footprints:PinHeader_1x10_P1.27mm_Vertical -> Connector_PinHeader_1.27mm:PinHeader_1x10_P1.27mm_Vertical
- J18: footprint Frooastboard Footprints:PinHeader_1x04_P1.27mm_Vertical -> Connector_PinHeader_1.27mm:PinHeader_1x04_P1.27mm_Vertical

Commit message: fix some issues
Parts:
- removed MX15: Scroll Lock, MX_Only:MXOnly-1U, symbol MX_Alps_Hybrid:MX-NoLED
- added MX131: Escape, MX_Only:MXOnly-1U-NoLED, symbol MX_Alps_Hybrid:MX-NoLED
- added MX132: F1, MX_Only:MXOnly-1U-NoLED, symbol MX_Alps_Hybrid:MX-NoLED
- added MX133: F2, MX_Only:MXOnly-1U-NoLED, symbol MX_Alps_Hybrid:MX-NoLED
- added MX134: F3, MX_Only:MXOnly-1U-NoLED, symbol MX_Alps_Hybrid:MX-NoLED
- added MX135: F4, MX_Only:MXOnly-1U-NoLED, symbol MX_Alps_Hybrid:MX-NoLED
- added MX136: F5, MX_Only:MXOnly-1U-NoLED, symbol MX_Alps_Hybrid:MX-NoLED
- added MX137: F6, MX_Only:MXOnly-1U-NoLED, symbol MX_Alps_Hybrid:MX-NoLED
- added MX138: F7, MX_Only:MXOnly-1U-NoLED, symbol MX_Alps_Hybrid:MX-NoLED
- added MX139: F8, MX_Only:MXOnly-1U-NoLED, symbol MX_Alps_Hybrid:MX-NoLED
- added MX140: F9, MX_Only:MXOnly-1U-NoLED, symbol MX_Alps_Hybrid:MX-NoLED
- added MX141: F10, MX_Only:MXOnly-1U-NoLED, symbol MX_Alps_Hybrid:MX-NoLED
- added MX142: F11, MX_Only:MXOnly-1U-NoLED, symbol MX_Alps_Hybrid:MX-NoLED
- added MX143: F12, MX_Only:MXOnly-1U-NoLED, symbol MX_Alps_Hybrid:MX-NoLED
- added MX144: Print Screen, MX_Only:MXOnly-1U-NoLED, symbol MX_Alps_Hybrid:MX-NoLED
- added MX146: Pause, MX_Only:MXOnly-1U-NoLED, symbol MX_Alps_Hybrid:MX-NoLED
- added MX147, MX15: MX-LED, MX_Only:MXOnly-1U, symbol MX_Alps_Hybrid:MX-LED
- added USB4: HRO-TYPE-C-31-M-12, Type_C:HRO-TYPE-C-31-M-12, symbol Type-C:HRO-TYPE-C-31-M-12
- J12: symbol Connector:Conn_01x06_Male -> Connector:Conn_01x06_Pin
- J13: symbol Connector:Conn_01x16_Male -> Connector:Conn_01x16_Pin
- J14: symbol Connector:Conn_01x10_Male -> Connector:Conn_01x10_Pin
- J18: symbol Connector:Conn_01x04_Male -> Connector:Conn_01x04_Pin
Connections:
- net +5V: now also USB4.11 (VBUS), USB4.2 (VBUS)
- net COL0: now also MX131.1 (COL), MX132.1 (COL)
- net COL1: now also MX133.1 (COL), MX134.1 (COL)
- net COL2: now also MX135.1 (COL), MX136.1 (COL)
- net COL3: now also MX137.1 (COL), MX138.1 (COL)
- net COL4: now also MX139.1 (COL), MX140.1 (COL)
- net COL5: now also MX141.1 (COL), MX142.1 (COL)
- net COL6: now also MX143.1 (COL), MX144.1 (COL)
- net COL7: now also MX146.1 (COL), MX147.1 (COL), MX15.1 (COL)
- net CS12: now also D36.2 (G+), D36.4 (R+), D36.6 (B+), D37.2 (G+), D37.4 (R+), D37.6 (B+)
- net CS2: now also MX147.3 (LED), MX15.3 (LED)
- net D+: now also USB4.6 (DP1), USB4.8 (DP2)
- net D-: now also USB4.5 (DN2), USB4.7 (DN1)
- net GND: now also USB4.1 (GND), USB4.12 (GND), USB4.13 (SHIELD)
- net SW5: now also MX147.4 (LEDGND), MX15.4 (LEDGND)
- net at D8.2 (A), MX2.2 (ROW): now also MX132.2 (ROW)
- net at D29.2 (A), MX16.2 (ROW): now also MX146.2 (ROW)
- net at D9.2 (A), MX3.2 (ROW): now also MX133.2 (ROW)
- net at D20.2 (A), MX11.2 (ROW): now also MX141.2 (ROW)
- net at D10.2 (A), MX4.2 (ROW): now also MX134.2 (ROW)
- net at D19.2 (A), MX10.2 (ROW): now also MX140.2 (ROW)
- net at D13.2 (A), MX6.2 (ROW): now also MX136.2 (ROW)
- net at D16.2 (A), MX8.2 (ROW): now also MX138.2 (ROW)
- net at D28.2 (A): now also MX147.2 (ROW), MX15.2 (ROW)
- net at D23.2 (A), MX12.2 (ROW): now also MX142.2 (ROW)
- net at R27.1, USB2.10 (CC2): now also USB4.10 (CC2)
- net at USB2.3 (SBU2): now also USB4.3 (SBU2)
- net at R26.1, USB2.4 (CC1): now also USB4.4 (CC1)
- net at USB2.9 (SBU1): now also USB4.9 (SBU1)
- net at D12.2 (A), MX5.2 (ROW): now also MX135.2 (ROW)
- net at D24.2 (A), MX13.2 (ROW): now also MX143.2 (ROW)
- net at D27.2 (A), MX14.2 (ROW): now also MX144.2 (ROW)
- net at D15.2 (A), MX7.2 (ROW): now also MX137.2 (ROW)
- net at D6.2 (A), MX1.2 (ROW): now also MX131.2 (ROW)
- net at D18.2 (A), MX9.2 (ROW): now also MX139.2 (ROW)

Commit message: updates or something like that
Parts:
- added D93: RGB_LED_6_Pin, Frooastboard Footprints:Everlight 99-235, symbol Frooastboard Symbols:RGB_LED_6_Pin
Connections:
- net CS13: now also D93.2 (G+), D93.4 (R+), D93.6 (B+)
- net SW4: now also D93.1 (G-)
- net SW5: now also D93.3 (R-)
- net SW6: now also D93.5 (B-)
Changed lines of the file:
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@@
   (junction (at 109.22 176.53) (diameter 0) (color 0 0 0 0)
   )
+  (junction (at 311.15 44.45) (diameter 0) (color 0 0 0 0)
+  )
   (junction (at 41.91 45.72) (diameter 0) (color 0 0 0 0)
   )
@@
   (junction (at 339.09 110.49) (diameter 0) (color 0 0 0 0)
   )
+  (junction (at 316.23 44.45) (diameter 0) (color 0 0 0 0)
+  )
   (junction (at 354.33 69.85) (diameter 0) (color 0 0 0 0)
   )
@@
   (junction (at 166.37 67.31) (diameter 0) (color 0 0 0 0)
   )
+  (junction (at 308.61 44.45) (diameter 0) (color 0 0 0 0)
+  )
   (junction (at 120.65 49.53) (diameter 0) (color 0 0 0 0)
   )
@@
   (junction (at 173.99 45.72) (diameter 0) (color 0 0 0 0)
   )
+  (junction (at 303.53 44.45) (diameter 0) (color 0 0 0 0)
+  )
   (junction (at 336.55 107.95) (diameter 0) (color 0 0 0 0)
   )
@@
   (junction (at 190.5 67.31) (diameter 0) (color 0 0 0 0)
   )
+  (junction (at 313.69 44.45) (diameter 0) (color 0 0 0 0)
+  )
   (junction (at 262.89 52.07) (diameter 0) (color 0 0 0 0)
   )
@@
   )
   (junction (at 93.98 181.61) (diameter 0) (color 0 0 0 0)
+  )
+  (junction (at 306.07 44.45) (diameter 0) (color 0 0 0 0)
   )
   (junction (at 308.61 69.85) (diameter 0) (color 0 0 0 0)
@@
         )
       )
+    )
+  )
+  (symbol (lib_id "Frooastboard Symbols:RGB_LED_6_Pin") (at 309.88 36.83 0) (unit 1)
+    (in_bom yes) (on_board yes) (dnp no)
+    (property "Reference" "D93" (at 316.23 35.56 0)
+      (effects (font (size 1.27 1.27)) (justify left))
+    )
+    (property "Value" "RGB_LED_6_Pin" (at 318.77 40.005 0)
+      (effects (font (size 1.27 1.27)) (justify left))
+    )
+    (property "Footprint" "Frooastboard Footprints:Everlight 99-235" (at 336.55 40.005 0)
+      (effects (font (size 1.27 1.27)) hide)
+    )
+    (property "Datasheet" "" (at 336.55 40.005 0)
+      (effects (font (size 1.27 1.27)) hide)
+    )
+    (pin "1")
+    (pin "2")
+    (pin "3")
+    (pin "4")
+    (pin "5")
+    (pin "6")
+    (instances
+      (project "Frooastboard Walnut Modular"
+        (path "/e63e39d7-6ac0-4ffd-8aa3-1841a4541b55/26642831-2675-418c-b9f8-1fa8a8351387"
+          (reference "D93") (unit 1)
+        )
+      )
