File: Frooastboard Modular/Kicad Project/Frooastboard Modular.kicad_pcb (KiCad board)
At the start: 4 copper layers, 45.7 x 25.7 mm, 41 parts, among them J1 Conn_01x16, J2 Conn_01x06, J3 Conn_01x06, J4 Conn_01x10, J5 Conn_01x12, J6 SW Interface, J7 Conn_01x04, U1 IS31FL3733-QF, U2 RP2040, U3 W25Q32JVZP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

Commit message: basic left side
Parts:
- R10: footprint Resistor_SMD:R_0402_1005Metric -> Resistor_SMD:R_0805_2012Metric
- moved U3 0.13 mm to (46.4, 62.0)
- moved R10 0.11 mm to (44.0, 58.2)
- moved J7 0.05 mm to (40.7, 58.4)
Routing:
- net Net-(J4-Pin_1): track 0.00 -> 25.3 mm, vias 0 -> 1
- net QSPI_CS: track 0.00 -> 24.6 mm
- net Net-(J4-Pin_3): track 0.00 -> 23.1 mm, vias 0 -> 1
- net Net-(J4-Pin_2): track 0.00 -> 23.0 mm, vias 0 -> 1
- net Net-(J4-Pin_5): track 0.00 -> 21.8 mm, vias 0 -> 1
- net Net-(J4-Pin_4): track 0.00 -> 21.6 mm, vias 0 -> 1
- net Net-(J4-Pin_7): track 0.00 -> 21.0 mm, vias 0 -> 1
- net Net-(J4-Pin_6): track 0.00 -> 19.8 mm, vias 0 -> 1
- net QSPI_SD1: track 0.00 -> 19.3 mm
- net Net-(J4-Pin_8): track 0.00 -> 17.8 mm
- net Net-(J4-Pin_9): track 0.00 -> 17.5 mm
- net Net-(J4-Pin_10): track 0.00 -> 16.7 mm
- net QSPI_SD2: track 0.00 -> 16.2 mm, vias 0 -> 2
- net QSPI_SD0: track 0.00 -> 9.26 mm
- net GND: track 0.00 -> 8.16 mm, vias 0 -> 1
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Other:
- board size 45.7 x 25.7 mm -> 44.6 x 25.7 mm

Commit message: backup before differential
Connections:
- J7 pad 2: GND -> /DN
- J7 pad 4: /DN -> GND
- R8 pad 1: RP_D+ -> RP_D-
- R8 pad 2: /DP -> /DN
- R9 pad 1: RP_D- -> RP_D+
- R9 pad 2: /DN -> /DP
Routing:
- net QSPI_SD3: track 0.00 -> 10.8 mm
- net QSPI_CLK: track 0.00 -> 9.95 mm
Changed lines of the file:
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@@
       (stroke (width 0.1) (type solid)) (layer "F.Fab"))
     (pad "1" smd roundrect (at -0.51 0) (size 0.54 0.64) (layers "F.Cu" "F.Paste" "F.Mask") (roundrect_rratio 0.25)
-      (net 69 "RP_D-") (pintype "passive"))
+      (net 68 "RP_D+") (pintype "passive"))
     (pad "2" smd roundrect (at 0.51 0) (size 0.54 0.64) (layers "F.Cu" "F.Paste" "F.Mask") (roundrect_rratio 0.25)
-      (net 61 "/DN") (pintype "passive"))
+      (net 60 "/DP") (pintype "passive"))
     (model "${KICAD6_3DMODEL_DIR}/Resistor_SMD.3dshapes/R_0402_1005Metric.wrl"
       (offset (xyz 0 0 0))
@@
       (stroke (width 0.1) (type solid)) (layer "F.Fab"))
     (pad "1" smd roundrect (at -0.51 0) (size 0.54 0.64) (layers "F.Cu" "F.Paste" "F.Mask") (roundrect_rratio 0.25)
-      (net 68 "RP_D+") (pintype "passive"))
+      (net 69 "RP_D-") (pintype "passive"))
     (pad "2" smd roundrect (at 0.51 0) (size 0.54 0.64) (layers "F.Cu" "F.Paste" "F.Mask") (roundrect_rratio 0.25)
-      (net 60 "/DP") (pintype "passive"))
+      (net 61 "/DN") (pintype "passive"))
     (model "${KICAD6_3DMODEL_DIR}/Resistor_SMD.3dshapes/R_0402_1005Metric.wrl"
       (offset (xyz 0 0 0))
@@
       (net 59 "+5V") (pinfunction "Pin_1") (pintype "passive"))
     (pad "2" thru_hole roundrect (at 0 1.27) (size 1.825 1) (drill 0.65 (offset 0.5875 0)) (property pad_prop_castellated) (layers "*.Cu" "*.Mask") (roundrect_rratio 0.1)
-      (net 1 "GND") (pinfunction "Pin_2") (pintype "passive"))
+      (net 61 "/DN") (pinfunction "Pin_2") (pintype "passive"))
     (pad "3" thru_hole roundrect (at 0 2.54) (size 1.825 1) (drill 0.65 (offset 0.5875 0)) (property pad_prop_castellated) (layers "*.Cu" "*.Mask") (roundrect_rratio 0.1)
       (net 60 "/DP") (pinfunction "Pin_3") (pintype "passive"))
     (pad "4" thru_hole roundrect (at 0 3.81) (size 1.825 1) (drill 0.65 (offset 0.5875 0)) (property pad_prop_castellated) (layers "*.Cu" "*.Mask") (roundrect_rratio 0.1)
-      (net 61 "/DN") (pinfunction "Pin_4") (pintype "passive"))
+      (net 1 "GND") (pinfunction "Pin_4") (pintype "passive"))
     (model "${KICAD6_3DMODEL_DIR}/Connector_PinHeader_1.27mm.3dshapes/PinHeader_1x04_P1.27mm_Vertical.wrl"
       (offset (xyz 0 0 0))
@@
   (segment (start 43.9039 59.8729) (end 43.9039 58.4073) (width 0.2032) (layer "F.Cu") (net 71))
   (segment (start 57.9568 66.0721) (end 54.112619 66.0721) (width 0.2032) (layer "F.Cu") (net 71))
+  (segment (start 50.0396 62.983826) (end 50.0396 63.5254) (width 0.2032) (layer "F.Cu") (net 82))
+  (segment (start 50.166601 63.652401) (end 50.0396 63.5254) (width 0.2032) (layer "F.Cu") (net 82))
+  (segment (start 54.02779 63.652402) (end 50.166601 63.652401) (width 0.2032) (layer "F.Cu") (net 82))
+  (segment (start 49.738087 62.682313) (end 50.0396 62.983826) (width 0.2032) (layer "F.Cu") (net 82))
+  (segment (start 49.738087 62.682313) (end 49.738087 61.853887) (width 0.2032) (layer "F.Cu") (net 82))
+  (segment (start 54.447488 64.0721) (end 54.02779 63.652402) (width 0.2032) (layer "F.Cu") (net 82))
+  (segment (start 57.9568 64.0721) (end 54.447488 64.0721) (width 0.2032) (layer "F.Cu") (net 82))
+  (segment (start 49.2252 61.341) (end 49.1058 61.341) (width 0.2032) (layer "F.Cu") (net 82))
+  (segment (start 49.738087 61.853887) (end 49.2252 61.341) (width 0.2032) (layer "F.Cu") (net 82))
+  (segment (start 49.1998 62.611) (end 49.1058 62.611) (width 0.2032) (layer "F.Cu") (net 83))
+  (segment (start 49.7094 63.6778) (end 49.7094 63.1206) (width 0.2032) (layer "F.Cu") (net 83))
+  (segment (start 50.014201 63.982601) (end 49.7094 63.6778) (width 0.2032) (layer "F.Cu") (net 83))
+  (segment (start 53.891016 63.982602) (end 50.014201 63.982601) (width 0.2032) (layer "F.Cu") (net 83))
+  (segment (start 57.9568 64.4721) (end 54.380514 64.4721) (width 0.2032) (layer "F.Cu") (net 83))
+  (segment (start 54.380514 64.4721) (end 53.891016 63.982602) (width 0.2032) (layer "F.Cu") (net 83))
+  (segment (start 49.7094 63.1206) (end 49.1998 62.611) (width 0.2032) (layer "F.Cu") (net 83))
   (segment (start 49.657001 64.312801) (end 53.754242 64.312802) (width 0.2032) (layer "F.Cu") (net 84))
   (segment (start 49.1058 63.881) (end 49.2252 63.881) (width 0.2032) (layer "F.Cu") (net 84))

Commit message: Update Frooastboard Modular.kicad_pcb
Parts:
- moved R8 0.85 mm to (52.0, 61.8), turned to 180 degrees
- moved R9 0.19 mm to (52.0, 62.8), turned to 180 degrees
Routing:
- net /DN: track 0.00 -> 12.0 mm, vias 0 -> 1
- net /DP: track 0.00 -> 12.0 mm, vias 0 -> 1
- net RP_D-: track 0.00 -> 5.88 mm
- net RP_D+: track 0.00 -> 5.55 mm
Changed lines of the file:
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@@
   )
   (footprint "Resistor_SMD:R_0402_1005Metric" (layer "F.Cu")
-    (at 51.9664 62.9412)
+    (at 52.0172 62.7546 180)
     (descr "Resistor SMD 0402 (1005 Metric), square (rectangular) end terminal, IPC_7351 nominal, (Body size source: IPC-SM-782 page 72, https://www.pcb-3d.com/wordpress/wp-content/uploads/ipc-sm-782a_amendment_1_and_2.pdf), generated with kicad-footprint-generator")
     (tags "resistor")
@@
     (fp_line (start 0.525 0.27) (end -0.525 0.27)
       (stroke (width 0.1) (type solid)) (layer "F.Fab"))
-    (pad "1" smd roundrect (at -0.51 0) (size 0.54 0.64) (layers "F.Cu" "F.Paste" "F.Mask") (roundrect_rratio 0.25)
+    (pad "1" smd roundrect (at -0.51 0 180) (size 0.54 0.64) (layers "F.Cu" "F.Paste" "F.Mask") (roundrect_rratio 0.25)
       (net 68 "RP_D+") (pintype "passive"))
-    (pad "2" smd roundrect (at 0.51 0) (size 0.54 0.64) (layers "F.Cu" "F.Paste" "F.Mask") (roundrect_rratio 0.25)
+    (pad "2" smd roundrect (at 0.51 0 180) (size 0.54 0.64) (layers "F.Cu" "F.Paste" "F.Mask") (roundrect_rratio 0.25)
       (net 60 "/DP") (pintype "passive"))
     (model "${KICAD6_3DMODEL_DIR}/Resistor_SMD.3dshapes/R_0402_1005Metric.wrl"
@@
   )
   (footprint "Resistor_SMD:R_0402_1005Metric" (layer "F.Cu")
-    (at 51.9664 60.9512)
+    (at 52.0172 61.7982 180)
     (descr "Resistor SMD 0402 (1005 Metric), square (rectangular) end terminal, IPC_7351 nominal, (Body size source: IPC-SM-782 page 72, https://www.pcb-3d.com/wordpress/wp-content/uploads/ipc-sm-782a_amendment_1_and_2.pdf), generated with kicad-footprint-generator")
     (tags "resistor")
@@
     (fp_line (start 0.525 0.27) (end -0.525 0.27)
       (stroke (width 0.1) (type solid)) (layer "F.Fab"))
-    (pad "1" smd roundrect (at -0.51 0) (size 0.54 0.64) (layers "F.Cu" "F.Paste" "F.Mask") (roundrect_rratio 0.25)
+    (pad "1" smd roundrect (at -0.51 0 180) (size 0.54 0.64) (layers "F.Cu" "F.Paste" "F.Mask") (roundrect_rratio 0.25)
       (net 69 "RP_D-") (pintype "passive"))
-    (pad "2" smd roundrect (at 0.51 0) (size 0.54 0.64) (layers "F.Cu" "F.Paste" "F.Mask") (roundrect_rratio 0.25)
+    (pad "2" smd roundrect (at 0.51 0 180) (size 0.54 0.64) (layers "F.Cu" "F.Paste" "F.Mask") (roundrect_rratio 0.25)
       (net 61 "/DN") (pintype "passive"))
     (model "${KICAD6_3DMODEL_DIR}/Resistor_SMD.3dshapes/R_0402_1005Metric.wrl"
@@
   (segment (start 53.086 67.51503) (end 54.66537 69.0944) (width 0.2032) (layer "F.Cu") (net 43))
   (segment (start 62.5275 69.0944) (end 63.1943 68.4276) (width 0.2032) (layer "F.Cu") (net 43))
+  (segment (start 51.204 62.5014) (end 51.4572 62.7546) (width 0.2) (layer "F.Cu") (net 60))
+  (segment (start 50.331634 62.164966) (end 50.543767 62.164966) (width 0.2) (layer "F.Cu") (net 60))
+  (segment (start 50.543767 62.164966) (end 50.880201 62.5014) (width 0.2) (layer "F.Cu") (net 60))
+  (segment (start 51.4572 62.7546) (end 51.5072 62.7546) (width 0.2) (layer "F.Cu") (net 60))
+  (segment (start 50.880201 62.5014) (end 51.204 62.5014) (width 0.2) (layer "F.Cu") (net 60))
+  (via (at 50.331634 62.164966) (size 0.42) (drill 0.25) (layers "F.Cu" "B.Cu") (net 60))
+  (segment (start 42.469551 60.4992) (end 48.878001 60.4992) (width 0.2) (layer "B.Cu") (net 60))
+  (segment (start 48.878001 60.4992) (end 50.331634 61.952833) (width 0.2) (layer "B.Cu") (net 60))
+  (segment (start 42.059551 60.9092) (end 42.469551 60.4992) (width 0.2) (layer "B.Cu") (net 60))
+  (segment (start 50.331634 61.952833) (end 50.331634 62.164966) (width 0.2) (layer "B.Cu") (net 60))
+  (segment (start 40.6908 60.9092) (end 42.059551 60.9092) (width 0.2) (layer "B.Cu") (net 60))
+  (segment (start 51.066599 62.0514) (end 51.204 62.0514) (width 0.2) (layer "F.Cu") (net 61))
+  (segment (start 50.861966 61.846767) (end 51.066599 62.0514) (width 0.2) (layer "F.Cu") (net 61))
+  (segment (start 50.861966 61.634634) (end 50.861966 61.846767) (width 0.2) (layer "F.Cu") (net 61))
+  (segment (start 51.4572 61.7982) (end 51.5072 61.7982) (width 0.2) (layer "F.Cu") (net 61))
+  (segment (start 51.204 62.0514) (end 51.4572 61.7982) (width 0.2) (layer "F.Cu") (net 61))
+  (via (at 50.861966 61.634634) (size 0.42) (drill 0.25) (layers "F.Cu" "B.Cu") (net 61))
+  (segment (start 40.6908 59.6392) (end 42.059551 59.6392) (width 0.2) (layer "B.Cu") (net 61))
+  (segment (start 50.649833 61.634634) (end 50.861966 61.634634) (width 0.2) (layer "B.Cu") (net 61))
+  (segment (start 42.469551 60.0492) (end 49.064399 60.0492) (width 0.2) (layer "B.Cu") (net 61))
+  (segment (start 42.059551 59.6392) (end 42.469551 60.0492) (width 0.2) (layer "B.Cu") (net 61))
+  (segment (start 49.064399 60.0492) (end 50.649833 61.634634) (width 0.2) (layer "B.Cu") (net 61))
+  (segment (start 57.9275 62.5014) (end 57.9568 62.4721) (width 0.2) (layer "F.Cu") (net 68))
+  (segment (start 53.007201 62.7546) (end 53.260401 62.5014) (width 0.2) (layer "F.Cu") (net 68))
+  (segment (start 53.260401 62.5014) (end 57.9275 62.5014) (width 0.2) (layer "F.Cu") (net 68))
+  (segment (start 52.5272 62.7546) (end 53.007201 62.7546) (width 0.2) (layer "F.Cu") (net 68))
+  (segment (start 52.847203 61.7982) (end 52.5272 61.7982) (width 0.2) (layer "F.Cu") (net 69))
+  (segment (start 57.9361 62.0514) (end 57.9568 62.0721) (width 0.2) (layer "F.Cu") (net 69))
+  (segment (start 54.626848 61.7724) (end 54.905848 62.0514) (width 0.2) (layer "F.Cu") (net 69))
+  (segment (start 54.905848 62.0514) (end 57.9361 62.0514) (width 0.2) (layer "F.Cu") (net 69))
+  (segment (start 52.5272 61.7982) (end 53.007201 61.7982) (width 0.2) (layer "F.Cu") (net 69))
+  (segment (start 53.033001 61.7724) (end 54.626848 61.7724) (width 0.2) (layer "F.Cu") (net 69))
+  (segment (start 53.007201 61.7982) (end 53.033001 61.7724) (width 0.2) (layer "F.Cu") (net 69))
   (segment (start 42.4194 63.1684) (end 42.4194 59.7394) (width 0.2032) (layer "F.Cu") (net 70))
   (segment (start 41.5648 64.8716) (end 41.5648 64.023) (width 0.2032) (layer "F.Cu") (net 70))

Commit message: basically done
Parts:
- moved R8 0.46 mm to (51.6, 61.8)
- moved R9 0.46 mm to (51.6, 62.8)
Changed lines of the file:
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@@
   )
   (footprint "Resistor_SMD:R_0402_1005Metric" (layer "F.Cu")
-    (at 52.0172 62.7546 180)
+    (at 51.56 62.7546 180)
     (descr "Resistor SMD 0402 (1005 Metric), square (rectangular) end terminal, IPC_7351 nominal, (Body size source: IPC-SM-782 page 72, https://www.pcb-3d.com/wordpress/wp-content/uploads/ipc-sm-782a_amendment_1_and_2.pdf), generated with kicad-footprint-generator")
     (tags "resistor")
@@
   )
   (footprint "Resistor_SMD:R_0402_1005Metric" (layer "F.Cu")
-    (at 52.0172 61.7982 180)
+    (at 51.56 61.7982 180)
     (descr "Resistor SMD 0402 (1005 Metric), square (rectangular) end terminal, IPC_7351 nominal, (Body size source: IPC-SM-782 page 72, https://www.pcb-3d.com/wordpress/wp-content/uploads/ipc-sm-782a_amendment_1_and_2.pdf), generated with kicad-footprint-generator")
     (tags "resistor")
@@
   (segment (start 53.086 67.51503) (end 54.66537 69.0944) (width 0.2032) (layer "F.Cu") (net 43))
   (segment (start 62.5275 69.0944) (end 63.1943 68.4276) (width 0.2032) (layer "F.Cu") (net 43))
-  (segment (start 51.204 62.5014) (end 51.4572 62.7546) (width 0.2) (layer "F.Cu") (net 60))
-  (segment (start 50.331634 62.164966) (end 50.543767 62.164966) (width 0.2) (layer "F.Cu") (net 60))
-  (segment (start 50.543767 62.164966) (end 50.880201 62.5014) (width 0.2) (layer "F.Cu") (net 60))
-  (segment (start 51.4572 62.7546) (end 51.5072 62.7546) (width 0.2) (layer "F.Cu") (net 60))
-  (segment (start 50.880201 62.5014) (end 51.204 62.5014) (width 0.2) (layer "F.Cu") (net 60))
-  (via (at 50.331634 62.164966) (size 0.42) (drill 0.25) (layers "F.Cu" "B.Cu") (net 60))
-  (segment (start 42.469551 60.4992) (end 48.878001 60.4992) (width 0.2) (layer "B.Cu") (net 60))
-  (segment (start 48.878001 60.4992) (end 50.331634 61.952833) (width 0.2) (layer "B.Cu") (net 60))
+  (segment (start 50.275084 62.7546) (end 51.05 62.7546) (width 0.2) (layer "F.Cu") (net 60))
+  (segment (start 49.899834 60.869566) (end 50.066687 61.036419) (width 0.2) (layer "F.Cu") (net 60))
+  (segment (start 50.066687 62.546203) (end 50.275084 62.7546) (width 0.2) (layer "F.Cu") (net 60))
+  (segment (start 50.066687 61.036419) (end 50.066687 62.546203) (width 0.2) (layer "F.Cu") (net 60))
+  (via (at 49.899834 60.869566) (size 0.42) (drill 0.25) (layers "F.Cu" "B.Cu") (net 60))
+  (segment (start 49.741601 60.4992) (end 49.899834 60.657433) (width 0.2) (layer "B.Cu") (net 60))
+  (segment (start 49.899834 60.657433) (end 49.899834 60.869566) (width 0.2) (layer "B.Cu") (net 60))
   (segment (start 42.059551 60.9092) (end 42.469551 60.4992) (width 0.2) (layer "B.Cu") (net 60))
-  (segment (start 50.331634 61.952833) (end 50.331634 62.164966) (width 0.2) (layer "B.Cu") (net 60))
   (segment (start 40.6908 60.9092) (end 42.059551 60.9092) (width 0.2) (layer "B.Cu") (net 60))
-  (segment (start 51.066599 62.0514) (end 51.204 62.0514) (width 0.2) (layer "F.Cu") (net 61))
-  (segment (start 50.861966 61.846767) (end 51.066599 62.0514) (width 0.2) (layer "F.Cu") (net 61))
-  (segment (start 50.861966 61.634634) (end 50.861966 61.846767) (width 0.2) (layer "F.Cu") (net 61))
-  (segment (start 51.4572 61.7982) (end 51.5072 61.7982) (width 0.2) (layer "F.Cu") (net 61))
-  (segment (start 51.204 62.0514) (end 51.4572 61.7982) (width 0.2) (layer "F.Cu") (net 61))
-  (via (at 50.861966 61.634634) (size 0.42) (drill 0.25) (layers "F.Cu" "B.Cu") (net 61))
+  (segment (start 42.469551 60.4992) (end 49.741601 60.4992) (width 0.2) (layer "B.Cu") (net 60))
+  (segment (start 50.485599 60.394667) (end 50.485599 61.661599) (width 0.2) (layer "F.Cu") (net 61))
+  (segment (start 50.6222 61.7982) (end 51.05 61.7982) (width 0.2) (layer "F.Cu") (net 61))
+  (segment (start 50.430166 60.339234) (end 50.485599 60.394667) (width 0.2) (layer "F.Cu") (net 61))
+  (segment (start 50.485599 61.661599) (end 50.6222 61.7982) (width 0.2) (layer "F.Cu") (net 61))
+  (via (at 50.430166 60.339234) (size 0.42) (drill 0.25) (layers "F.Cu" "B.Cu") (net 61))
   (segment (start 40.6908 59.6392) (end 42.059551 59.6392) (width 0.2) (layer "B.Cu") (net 61))
-  (segment (start 50.649833 61.634634) (end 50.861966 61.634634) (width 0.2) (layer "B.Cu") (net 61))
-  (segment (start 42.469551 60.0492) (end 49.064399 60.0492) (width 0.2) (layer "B.Cu") (net 61))
   (segment (start 42.059551 59.6392) (end 42.469551 60.0492) (width 0.2) (layer "B.Cu") (net 61))
-  (segment (start 49.064399 60.0492) (end 50.649833 61.634634) (width 0.2) (layer "B.Cu") (net 61))
-  (segment (start 57.9275 62.5014) (end 57.9568 62.4721) (width 0.2) (layer "F.Cu") (net 68))
-  (segment (start 53.007201 62.7546) (end 53.260401 62.5014) (width 0.2) (layer "F.Cu") (net 68))
-  (segment (start 53.260401 62.5014) (end 57.9275 62.5014) (width 0.2) (layer "F.Cu") (net 68))
-  (segment (start 52.5272 62.7546) (end 53.007201 62.7546) (width 0.2) (layer "F.Cu") (net 68))
-  (segment (start 52.847203 61.7982) (end 52.5272 61.7982) (width 0.2) (layer "F.Cu") (net 69))
-  (segment (start 57.9361 62.0514) (end 57.9568 62.0721) (width 0.2) (layer "F.Cu") (net 69))
-  (segment (start 54.626848 61.7724) (end 54.905848 62.0514) (width 0.2) (layer "F.Cu") (net 69))
-  (segment (start 54.905848 62.0514) (end 57.9361 62.0514) (width 0.2) (layer "F.Cu") (net 69))
-  (segment (start 52.5272 61.7982) (end 53.007201 61.7982) (width 0.2) (layer "F.Cu") (net 69))
-  (segment (start 53.033001 61.7724) (end 54.626848 61.7724) (width 0.2) (layer "F.Cu") (net 69))
-  (segment (start 53.007201 61.7982) (end 53.033001 61.7724) (width 0.2) (layer "F.Cu") (net 69))
+  (segment (start 42.469551 60.0492) (end 49.927999 60.0492) (width 0.2) (layer "B.Cu") (net 61))
+  (segment (start 50.218033 60.339234) (end 50.430166 60.339234) (width 0.2) (layer "B.Cu") (net 61))
+  (segment (start 49.927999 60.0492) (end 50.218033 60.339234) (width 0.2) (layer "B.Cu") (net 61))
+  (segment (start 52.8439 62.4721) (end 52.5614 62.7546) (width 0.2) (layer "F.Cu") (net 68))
+  (segment (start 52.5614 62.7546) (end 52.07 62.7546) (width 0.2) (layer "F.Cu") (net 68))
+  (segment (start 57.9568 62.4721) (end 52.8439 62.4721) (width 0.2) (layer "F.Cu") (net 68))
+  (segment (start 52.8273 62.0721) (end 52.5534 61.7982) (width 0.2) (layer "F.Cu") (net 69))
+  (segment (start 52.5534 61.7982) (end 52.07 61.7982) (width 0.2) (layer "F.Cu") (net 69))
+  (segment (start 57.9568 62.0721) (end 52.8273 62.0721) (width 0.2) (layer "F.Cu") (net 69))
   (segment (start 42.4194 63.1684) (end 42.4194 59.7394) (width 0.2032) (layer "F.Cu") (net 70))
   (segment (start 41.5648 64.8716) (end 41.5648 64.023) (width 0.2032) (layer "F.Cu") (net 70))

Commit message: more stuff little weird
Parts:
- moved C14 61.7 mm to (46.5, 65.3)
- moved C15 60.5 mm to (51.9, 63.7), turned to 180 degrees
- moved C16 57.3 mm to (54.2, 60.8), turned to 90 degrees
- moved C7 52.1 mm to (53.1, 61.1), turned to 90 degrees
- moved C12 3.98 mm to (104.6, 53.7)
- moved C13 3.98 mm to (104.6, 55.7)
- moved C8 3.98 mm to (101.7, 57.7)
- moved C10 3.98 mm to (104.6, 49.8)
- moved C11 3.98 mm to (104.6, 51.8)
- moved C9 3.98 mm to (104.6, 47.8)
- moved C17 3.59 mm to (111.0, 57.6)
- moved U2 2.60 mm to (58.8, 63.5)
- moved R5 0.72 mm to (62.8, 58.0)
- moved R6 0.20 mm to (62.3, 57.0)
Routing:
- net +5V: track 0.00 -> 22.9 mm
- net +3V3: track 0.00 -> 22.1 mm, vias 0 -> 4
- net +1V1: track 0.00 -> 17.2 mm, vias 0 -> 2
- net SDA: track 0.00 -> 10.4 mm, vias 0 -> 2
- net GND: track 8.16 -> 18.3 mm, vias 1 -> 4
- net SCL: track 0.00 -> 8.75 mm
- net Net-(J4-Pin_4): track 21.6 -> 19.0 mm
- net Net-(J4-Pin_8): track 17.8 -> 15.2 mm
- net Net-(J4-Pin_6): track 19.8 -> 17.2 mm
- net Net-(J4-Pin_10): track 16.7 -> 14.1 mm
- net Net-(J4-Pin_1): track 25.3 -> 22.7 mm
- net Net-(J4-Pin_9): track 17.5 -> 14.9 mm
- net Net-(J4-Pin_7): track 21.0 -> 18.4 mm
- net Net-(J4-Pin_5): track 21.8 -> 19.2 mm
- net Net-(J4-Pin_2): track 23.0 -> 20.4 mm
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