File: Frooastboard Modular/Kicad Project/Frooastboard Modular.kicad_pcb (KiCad board)
At the start: 4 copper layers, 44.6 x 25.7 mm, 41 parts, among them J1 Conn_01x16, J2 Conn_01x06, J3 Conn_01x06, J4 Conn_01x10, J5 Conn_01x12, J6 SW Interface, J7 Conn_01x04, U1 IS31FL3733-QF, U2 RP2040, U3 W25Q32JVZP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

Commit message: some more stuff
Parts:
- moved C9 45.5 mm to (63.9, 68.1)
- moved C8 39.0 mm to (63.9, 67.1)
Routing:
- net Net-(J5-Pin_2): track 0.00 -> 12.6 mm, vias 0 -> 1
- net Net-(J5-Pin_1): track 0.00 -> 11.0 mm, vias 0 -> 1
- net +3V3: track 22.1 -> 29.2 mm, vias 4 -> 6
- net GND: track 18.3 -> 20.6 mm, vias 4 -> 5
Changed lines of the file:
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@@
   )
   (footprint "Capacitor_SMD:C_0402_1005Metric" (layer "F.Cu")
-    (at 104.5946 47.8222)
+    (at 63.8836 68.0974)
     (descr "Capacitor SMD 0402 (1005 Metric), square (rectangular) end terminal, IPC_7351 nominal, (Body size source: IPC-SM-782 page 76, https://www.pcb-3d.com/wordpress/wp-content/uploads/ipc-sm-782a_amendment_1_and_2.pdf), generated with kicad-footprint-generator")
     (tags "capacitor")
@@
   )
   (footprint "Capacitor_SMD:C_0402_1005Metric" (layer "F.Cu")
-    (at 101.7246 57.6722)
+    (at 63.8836 67.1322)
     (descr "Capacitor SMD 0402 (1005 Metric), square (rectangular) end terminal, IPC_7351 nominal, (Body size source: IPC-SM-782 page 76, https://www.pcb-3d.com/wordpress/wp-content/uploads/ipc-sm-782a_amendment_1_and_2.pdf), generated with kicad-footprint-generator")
     (tags "capacitor")
@@
   (segment (start 45.9792 62.4026) (end 46.4058 61.976) (width 0.381) (layer "F.Cu") (net 1))
   (segment (start 45.9792 65.3034) (end 45.9792 62.4026) (width 0.381) (layer "F.Cu") (net 1))
+  (segment (start 64.3636 68.0974) (end 64.3636 67.1322) (width 0.381) (layer "F.Cu") (net 1))
   (segment (start 46.4058 61.976) (end 46.4058 63.3476) (width 0.381) (layer "F.Cu") (net 1))
   (segment (start 50.6222 63.7286) (end 50.5206 63.627) (width 0.381) (layer "F.Cu") (net 1))
   (segment (start 45.9792 65.3034) (end 44.6024 65.3034) (width 0.381) (layer "F.Cu") (net 1))
   (segment (start 44.6024 65.3034) (end 44.2468 64.9478) (width 0.381) (layer "F.Cu") (net 1))
+  (segment (start 64.3636 68.0974) (end 64.8462 68.0974) (width 0.381) (layer "F.Cu") (net 1))
   (segment (start 46.4058 63.3476) (end 45.8724 63.881) (width 0.381) (layer "F.Cu") (net 1))
+  (segment (start 64.8462 68.0974) (end 65.4558 67.4878) (width 0.381) (layer "F.Cu") (net 1))
   (segment (start 43.7058 63.881) (end 43.7058 64.4068) (width 0.381) (layer "F.Cu") (net 1))
   (segment (start 43.7058 64.4068) (end 44.2468 64.9478) (width 0.381) (layer "F.Cu") (net 1))
@@
   (segment (start 45.9538 65.278) (end 45.9792 65.3034) (width 0.381) (layer "F.Cu") (net 1))
   (via (at 55.2958 59.8678) (size 0.8) (drill 0.5) (layers "F.Cu" "B.Cu") (net 1))
+  (via (at 65.4558 67.4878) (size 0.8) (drill 0.5) (layers "F.Cu" "B.Cu") (net 1))
   (via (at 44.2468 64.9478) (size 0.8) (drill 0.5) (layers "F.Cu" "B.Cu") (net 1))
   (via (at 48.7426 59.182) (size 0.8) (drill 0.5) (layers "F.Cu" "B.Cu") (net 1))
@@
   (segment (start 54.1528 63.0428) (end 54.5592 63.0428) (width 0.381) (layer "F.Cu") (net 2))
   (segment (start 63.3242 57.5056) (end 62.8162 56.9976) (width 0.381) (layer "F.Cu") (net 2))
+  (segment (start 60.421979 65.8114) (end 60.4266 65.8114) (width 0.254) (layer "F.Cu") (net 2))
+  (segment (start 62.2554 67.6402) (end 62.2808 67.6148) (width 0.381) (layer "F.Cu") (net 2))
   (segment (start 55.3537 61.2721) (end 55.3537 60.8721) (width 0.254) (layer "F.Cu") (net 2))
   (segment (start 63.3242 57.9882) (end 62.7502 58.5622) (width 0.254) (layer "F.Cu") (net 2))
@@
   (segment (start 49.1058 60.071) (end 50.0634 60.071) (width 0.3556) (layer "F.Cu") (net 2))
   (segment (start 48.8442 60.071) (end 48.4106 60.5046) (width 0.3556) (layer "F.Cu") (net 2))
+  (segment (start 59.7912 66.442179) (end 60.421979 65.8114) (width 0.254) (layer "F.Cu") (net 2))
+  (segment (start 59.7912 66.9096) (end 59.7912 66.442179) (width 0.254) (layer "F.Cu") (net 2))
   (segment (start 47.538 65.3034) (end 46.9392 65.3034) (width 0.3556) (layer "F.Cu") (net 2))
+  (segment (start 62.7126 68.0974) (end 63.4036 68.0974) (width 0.381) (layer "F.Cu") (net 2))
   (segment (start 51.054 61.0616) (end 52.5526 61.0616) (width 0.3556) (layer "F.Cu") (net 2))
   (segment (start 63.3242 57.9882) (end 63.3242 57.5056) (width 0.381) (layer "F.Cu") (net 2))
   (segment (start 49.1058 60.071) (end 48.8442 60.071) (width 0.3556) (layer "F.Cu") (net 2))
   (segment (start 50.0634 60.071) (end 50.546 60.5536) (width 0.3556) (layer "F.Cu") (net 2))
+  (segment (start 63.4036 67.6148) (end 63.4036 67.1322) (width 0.381) (layer "F.Cu") (net 2))
   (segment (start 54.0512 62.9412) (end 54.1528 63.0428) (width 0.381) (layer "F.Cu") (net 2))
   (segment (start 56.1912 60.0346) (end 56.1912 60.7886) (width 0.254) (layer "F.Cu") (net 2))
@@
   (segment (start 62.7502 58.5622) (end 59.949094 58.5622) (width 0.254) (layer "F.Cu") (net 2))
   (segment (start 48.4106 64.4308) (end 47.9498 64.8916) (width 0.3556) (layer "F.Cu") (net 2))
+  (segment (start 62.2554 67.6402) (end 62.7126 68.0974) (width 0.381) (layer "F.Cu") (net 2))
   (segment (start 56.2747 60.8721) (end 55.3537 60.8721) (width 0.381) (layer "F.Cu") (net 2))
   (segment (start 56.6674 61.2648) (end 56.2747 60.8721) (width 0.381) (layer "F.Cu") (net 2))
+  (segment (start 63.4036 68.0974) (end 63.4036 67.6148) (width 0.381) (layer "F.Cu") (net 2))
   (segment (start 47.9498 64.8916) (end 47.538 65.3034) (width 0.3556) (layer "F.Cu") (net 2))
+  (via (at 60.4266 65.8114) (size 0.8) (drill 0.5) (layers "F.Cu" "B.Cu") (net 2))
   (via (at 54.0512 62.9412) (size 0.8) (drill 0.5) (layers "F.Cu" "B.Cu") (net 2))
+  (via (at 62.2554 67.6402) (size 0.8) (drill 0.5) (layers "F.Cu" "B.Cu") (net 2))
   (via (at 47.9498 64.8916) (size 0.8) (drill 0.5) (layers "F.Cu" "B.Cu") (net 2))
   (via (at 56.6674 61.2648) (size 0.8) (drill 0.5) (layers "F.Cu" "B.Cu") (net 2))
   (via (at 50.546 60.5536) (size 0.8) (drill 0.5) (layers "F.Cu" "B.Cu") (net 2))
+  (segment (start 61.7728 65.8114) (end 60.4266 65.8114) (width 0.381) (layer "B.Cu") (net 2))
+  (segment (start 62.2554 66.294) (end 61.7728 65.8114) (width 0.381) (layer "B.Cu") (net 2))
+  (segment (start 62.2554 67.6402) (end 62.2554 66.294) (width 0.381) (layer "B.Cu") (net 2))
   (segment (start 54.245 61.2342) (end 54.483 61.4722) (width 0.254) (layer "F.Cu") (net 5))
   (segment (start 55.821121 61.6721) (end 56.0452 61.896179) (width 0.254) (layer "F.Cu") (net 5))
@@
   (via (at 53.2892 63.627) (size 0.8) (drill 0.5) (layers "F.Cu" "B.Cu") (net 5))
   (via (at 61.1124 63.4238) (size 0.8) (drill 0.5) (layers "F.Cu" "B.Cu") (net 5))
+  (segment (start 56.1806 63.6482) (end 56.6365 64.1041) (width 0.254) (layer "B.Cu") (net 5))
   (segment (start 53.2892 63.627) (end 53.3104 63.6482) (width 0.254) (layer "B.Cu") (net 5))
-  (segment (start 56.7902 63.6482) (end 57.2461 64.1041) (width 0.254) (layer "B.Cu") (net 5))
-  (segment (start 60.4321 64.1041) (end 61.1124 63.4238) (width 0.254) (layer "B.Cu") (net 5))
-  (segment (start 57.2461 64.1041) (end 60.4321 64.1041) (width 0.254) (layer "B.Cu") (net 5))
-  (segment (start 53.3104 63.6482) (end 56.7902 63.6482) (width 0.254) (layer "B.Cu") (net 5))
+  (segment (start 61.1124 64.008) (end 61.1124 63.4238) (width 0.254) (layer "B.Cu") (net 5))
+  (segment (start 61.0163 64.1041) (end 61.1124 64.008) (width 0.254) (layer "B.Cu") (net 5))
+  (segment (start 56.6365 64.1041) (end 61.0163 64.1041) (width 0.254) (layer "B.Cu") (net 5))
+  (segment (start 53.3104 63.6482) (end 56.1806 63.6482) (width 0.254) (layer "B.Cu") (net 5))
   (segment (start 56.5912 66.9096) (end 56.5912 66.0523) (width 0.2032) (layer "F.Cu") (net 34))
   (segment (start 56.5912 66.0523) (end 56.5789 66.04) (width 0.2032) (layer "F.Cu") (net 34))
@@
   (segment (start 53.086 67.51503) (end 54.66537 69.0944) (width 0.2032) (layer "F.Cu") (net 43))
   (segment (start 59.9244 69.0944) (end 60.5912 68.4276) (width 0.2032) (layer "F.Cu") (net 43))
+  (segment (start 60.9912 68.662) (end 61.214 68.8848) (width 0.2032) (layer "F.Cu") (net 44))
+  (segment (start 60.9912 68.662) (end 60.9912 66.9096) (width 0.2032) (layer "F.Cu") (net 44))
+  (via (at 61.214 68.8848) (size 0.42) (drill 0.25) (layers "F.Cu" "B.Cu") (net 44))
+  (segment (start 61.4236 69.0944) (end 61.214 68.8848) (width 0.2032) (layer "In2.Cu") (net 44))
+  (segment (start 65.62903 69.0944) (end 61.4236 69.0944) (width 0.2032) (layer "In2.Cu") (net 44))
+  (segment (start 67.54043 67.183) (end 65.62903 69.0944) (width 0.2032) (layer "In2.Cu") (net 44))
+  (segment (start 68.5292 67.3608) (end 68.3514 67.183) (width 0.2032) (layer "In2.Cu") (net 44))
+  (segment (start 68.5292 68.0212) (end 68.5292 67.3608) (width 0.2032) (layer "In2.Cu") (net 44))
+  (segment (start 68.3514 67.183) (end 67.54043 67.183) (width 0.2032) (layer "In2.Cu") (net 44))
+  (segment (start 61.3912 67.9952) (end 61.8236 68.4276) (width 0.2032) (layer "F.Cu") (net 45))
+  (segment (start 69.7484 67.9704) (end 69.7992 68.0212) (width 0.2032) (layer "F.Cu") (net 45))
+  (segment (start 61.3912 66.9096) (end 61.3912 67.9952) (width 0.2032) (layer "F.Cu") (net 45))
+  (via (at 61.8236 68.4276) (size 0.42) (drill 0.25) (layers "F.Cu" "B.Cu") (net 45))
+  (segment (start 65.3224 68.7642) (end 62.1602 68.7642) (width 0.2032) (layer "In2.Cu") (net 45))
+  (segment (start 67.794 66.2926) (end 65.3224 68.7642) (width 0.2032) (layer "In2.Cu") (net 45))
+  (segment (start 69.7992 68.0212) (end 69.7992 66.421) (width 0.2032) (layer "In2.Cu") (net 45))
+  (segment (start 69.6708 66.2926) (end 67.794 66.2926) (width 0.2032) (layer "In2.Cu") (net 45))
+  (segment (start 69.7992 66.421) (end 69.6708 66.2926) (width 0.2032) (layer "In2.Cu") (net 45))
+  (segment (start 62.1602 68.7642) (end 61.8236 68.4276) (width 0.2032) (layer "In2.Cu") (net 45))
   (segment (start 45.4914 60.0964) (end 48.514 60.0964) (width 0.381) (layer "B.Cu") (net 59))
   (segment (start 60.8076 61.954914) (end 60.8076 62.2554) (width 0.381) (layer "B.Cu") (net 59))

Commit message: some more stuff
Parts:
- moved C5 9.54 mm to (66.2, 64.8), turned to 90 degrees
- moved R7 5.86 mm to (65.8, 63.4)
- moved R4 5.66 mm to (85.0, 61.8), turned to -90 degrees
- moved Y1 2.56 mm to (68.8, 63.5)
- moved C6 2.52 mm to (71.4, 62.7), turned to 90 degrees
Routing:
- net Net-(J5-Pin_12): track 0.00 -> 28.1 mm, vias 0 -> 1
- net Net-(J5-Pin_11): track 0.00 -> 26.1 mm, vias 0 -> 1
- net Net-(J5-Pin_10): track 0.00 -> 25.9 mm, vias 0 -> 3
- net Net-(J5-Pin_9): track 0.00 -> 23.3 mm, vias 0 -> 1
- net Net-(J5-Pin_8): track 0.00 -> 21.3 mm, vias 0 -> 1
- net Net-(J5-Pin_7): track 0.00 -> 20.2 mm, vias 0 -> 1
- net Net-(J5-Pin_6): track 0.00 -> 14.9 mm, vias 0 -> 1
- net Net-(J5-Pin_5): track 0.00 -> 13.8 mm
- net Net-(J5-Pin_4): track 0.00 -> 12.0 mm, vias 0 -> 1
- net Net-(J5-Pin_3): track 0.00 -> 10.4 mm
- net GND: track 20.6 -> 29.0 mm
- net XTAL1: track 0.00 -> 5.71 mm
- net Net-(C6-Pad2): track 0.00 -> 5.64 mm
- net +3V3: track 29.2 -> 26.5 mm, vias 6 -> 7
- net XTAL2: track 0.00 -> 2.65 mm

Commit message: Update Frooastboard Modular.kicad_pcb
Routing:
- net +5V: track 22.9 -> 37.0 mm
- net RP_RESET: track 0.00 -> 5.95 mm, vias 0 -> 1
- net SWCLK: track 0.00 -> 4.93 mm, vias 0 -> 1
- net SWDIO: track 0.00 -> 3.09 mm, vias 0 -> 1
Changed lines of the file:
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@@
   (segment (start 62.7447 66.0721) (end 63.1952 66.5226) (width 0.2032) (layer "F.Cu") (net 46))
   (segment (start 67.54 66.2926) (end 70.382 66.2926) (width 0.2032) (layer "F.Cu") (net 46))
-  (segment (start 63.4492 65.9638) (end 63.1575 65.6721) (width 0.2032) (layer "F.Cu") (net 47))
-  (segment (start 63.1575 65.6721) (end 62.2287 65.6721) (width 0.2032) (layer "F.Cu") (net 47))
+  (segment (start 63.103374 65.9638) (end 63.4492 65.9638) (width 0.2032) (layer "F.Cu") (net 47))
+  (segment (start 62.2287 65.6721) (end 62.811674 65.6721) (width 0.2032) (layer "F.Cu") (net 47))
+  (segment (start 62.811674 65.6721) (end 63.103374 65.9638) (width 0.2032) (layer "F.Cu") (net 47))
   (via (at 63.4492 65.9638) (size 0.42) (drill 0.25) (layers "F.Cu" "B.Cu") (net 47))
   (segment (start 72.3392 66.4464) (end 72.1854 66.2926) (width 0.2032) (layer "B.Cu") (net 47))
   (segment (start 72.3392 68.0212) (end 72.3392 66.4464) (width 0.2032) (layer "B.Cu") (net 47))
-  (segment (start 72.1854 66.2926) (end 63.778 66.2926) (width 0.2032) (layer "B.Cu") (net 47))
-  (segment (start 63.778 66.2926) (end 63.4492 65.9638) (width 0.2032) (layer "B.Cu") (net 47))
+  (segment (start 63.4492 65.9638) (end 64.0094 65.9638) (width 0.2032) (layer "B.Cu") (net 47))
+  (segment (start 64.0094 65.9638) (end 64.3382 66.2926) (width 0.2032) (layer "B.Cu") (net 47))
+  (segment (start 72.1854 66.2926) (end 64.3382 66.2926) (width 0.2032) (layer "B.Cu") (net 47))
   (segment (start 63.544652 65.2721) (end 64.464952 66.1924) (width 0.2032) (layer "F.Cu") (net 48))
   (segment (start 62.2287 65.2721) (end 63.544652 65.2721) (width 0.2032) (layer "F.Cu") (net 48))
@@
   (segment (start 73.4046 65.9624) (end 73.6092 66.167) (width 0.2032) (layer "F.Cu") (net 48))
   (segment (start 64.464952 66.1924) (end 67.173227 66.1924) (width 0.2032) (layer "F.Cu") (net 48))
-  (segment (start 64.5922 65.5066) (end 63.9577 64.8721) (width 0.2032) (layer "F.Cu") (net 49))
-  (segment (start 63.9577 64.8721) (end 62.2287 64.8721) (width 0.2032) (layer "F.Cu") (net 49))
+  (segment (start 63.611626 64.8721) (end 62.2287 64.8721) (width 0.2032) (layer "F.Cu") (net 49))
+  (segment (start 64.5922 65.5066) (end 64.246126 65.5066) (width 0.2032) (layer "F.Cu") (net 49))
+  (segment (start 64.246126 65.5066) (end 63.611626 64.8721) (width 0.2032) (layer "F.Cu") (net 49))
   (via (at 64.5922 65.5066) (size 0.42) (drill 0.25) (layers "F.Cu" "B.Cu") (net 49))
   (segment (start 74.446 65.9624) (end 74.8792 66.3956) (width 0.2032) (layer "B.Cu") (net 49))
@@
   (segment (start 76.476206 60.6806) (end 71.374 60.6806) (width 0.2032) (layer "In1.Cu") (net 55))
   (segment (start 69.2912 60.6806) (end 68.199 59.5884) (width 0.2032) (layer "In1.Cu") (net 55))
+  (segment (start 62.2287 61.6721) (end 60.9863 61.6721) (width 0.2032) (layer "F.Cu") (net 56))
+  (segment (start 60.9863 61.6721) (end 60.9854 61.6712) (width 0.2032) (layer "F.Cu") (net 56))
+  (via (at 60.9854 61.6712) (size 0.42) (drill 0.25) (layers "F.Cu" "B.Cu") (net 56))
+  (segment (start 62.7634 61.3642) (end 62.4564 61.6712) (width 0.2032) (layer "B.Cu") (net 56))
+  (segment (start 62.7634 61.3642) (end 65.1996 61.3642) (width 0.2032) (layer "B.Cu") (net 56))
+  (segment (start 65.1996 61.3642) (end 65.4558 61.6204) (width 0.2032) (layer "B.Cu") (net 56))
+  (segment (start 62.4564 61.6712) (end 60.9854 61.6712) (width 0.2032) (layer "B.Cu") (net 56))
+  (segment (start 63.5 61.9252) (end 63.0428 61.9252) (width 0.2032) (layer "F.Cu") (net 57))
+  (segment (start 63.0428 61.9252) (end 62.8959 62.0721) (width 0.2032) (layer "F.Cu") (net 57))
+  (segment (start 62.8959 62.0721) (end 62.2287 62.0721) (width 0.2032) (layer "F.Cu") (net 57))
+  (via (at 63.5 61.9252) (size 0.42) (drill 0.25) (layers "F.Cu" "B.Cu") (net 57))
+  (segment (start 63.5 61.9252) (end 63.7308 61.6944) (width 0.2032) (layer "B.Cu") (net 57))
+  (segment (start 63.7308 61.6944) (end 65.062826 61.6944) (width 0.2032) (layer "B.Cu") (net 57))
+  (segment (start 65.062826 61.6944) (end 65.133413 61.764987) (width 0.2032) (layer "B.Cu") (net 57))
+  (segment (start 62.2287 62.4721) (end 61.2021 62.4721) (width 0.2032) (layer "F.Cu") (net 58))
+  (segment (start 61.2021 62.4721) (end 61.1886 62.4586) (width 0.2032) (layer "F.Cu") (net 58))
+  (via (at 61.1886 62.4586) (size 0.42) (drill 0.25) (layers "F.Cu" "B.Cu") (net 58))
+  (segment (start 61.2118 62.4818) (end 63.730552 62.4818) (width 0.2032) (layer "B.Cu") (net 58))
+  (segment (start 61.1886 62.4586) (end 61.2118 62.4818) (width 0.2032) (layer "B.Cu") (net 58))
+  (segment (start 63.730552 62.4818) (end 64.187752 62.0246) (width 0.2032) (layer "B.Cu") (net 58))
+  (segment (start 64.187752 62.0246) (end 64.8716 62.0246) (width 0.2032) (layer "B.Cu") (net 58))
+  (segment (start 65.7098 60.6044) (end 65.7098 61.2648) (width 0.381) (layer "B.Cu") (net 59))
+  (segment (start 58.382575 61.5801) (end 58.469275 61.4934) (width 0.381) (layer "B.Cu") (net 59))
+  (segment (start 68.1885 61.7833) (end 68.7324 61.2394) (width 0.381) (layer "B.Cu") (net 59))
+  (segment (start 40.6908 58.3692) (end 43.7642 58.3692) (width 0.381) (layer "B.Cu") (net 59))
   (segment (start 45.4914 60.0964) (end 48.514 60.0964) (width 0.381) (layer "B.Cu") (net 59))
-  (segment (start 60.8076 61.954914) (end 60.8076 62.2554) (width 0.381) (layer "B.Cu") (net 59))
+  (segment (start 56.9468 60.452) (end 57.4379 60.9431) (width 0.381) (layer "B.Cu") (net 59))
+  (segment (start 65.7098 61.2648) (end 66.2283 61.7833) (width 0.381) (layer "B.Cu") (net 59))
+  (segment (start 60.2742 61.0616) (end 60.2742 59.9948) (width 0.381) (layer "B.Cu") (net 59))
+  (segment (start 57.847825 61.5801) (end 58.382575 61.5801) (width 0.381) (layer "B.Cu") (net 59))
+  (segment (start 57.4379 60.9431) (end 57.4379 61.170175) (width 0.381) (layer "B.Cu") (net 59))
+  (segment (start 58.469275 61.4934) (end 59.8424 61.4934) (width 0.381) (layer "B.Cu") (net 59))
+  (segment (start 55.122404 61.387396) (end 56.0578 60.452) (width 0.381) (layer "B.Cu") (net 59))
+  (segment (start 66.2283 61.7833) (end 68.1885 61.7833) (width 0.381) (layer "B.Cu") (net 59))
+  (segment (start 56.0578 60.452) (end 56.9468 60.452) (width 0.381) (layer "B.Cu") (net 59))
+  (segment (start 61.2902 58.9788) (end 64.0842 58.9788) (width 0.381) (layer "B.Cu") (net 59))
+  (segment (start 49.804996 61.387396) (end 55.122404 61.387396) (width 0.381) (layer "B.Cu") (net 59))
+  (segment (start 64.0842 58.9788) (end 65.7098 60.6044) (width 0.381) (layer "B.Cu") (net 59))
+  (segment (start 68.7324 61.2394) (end 71.9836 61.2394) (width 0.381) (layer "B.Cu") (net 59))
+  (segment (start 48.514 60.0964) (end 49.804996 61.387396) (width 0.381) (layer "B.Cu") (net 59))
+  (segment (start 60.2742 59.9948) (end 61.2902 58.9788) (width 0.381) (layer "B.Cu") (net 59))
+  (segment (start 59.8424 61.4934) (end 60.2742 61.0616) (width 0.381) (layer "B.Cu") (net 59))
   (segment (start 43.7642 58.3692) (end 45.4914 60.0964) (width 0.381) (layer "B.Cu") (net 59))
-  (segment (start 40.6908 58.3692) (end 43.7642 58.3692) (width 0.381) (layer "B.Cu") (net 59))
-  (segment (start 58.382575 61.5801) (end 58.469275 61.4934) (width 0.381) (layer "B.Cu") (net 59))
-  (segment (start 55.122404 61.387396) (end 56.0578 60.452) (width 0.381) (layer "B.Cu") (net 59))
-  (segment (start 49.804996 61.387396) (end 55.122404 61.387396) (width 0.381) (layer "B.Cu") (net 59))
-  (segment (start 56.9468 60.452) (end 57.4379 60.9431) (width 0.381) (layer "B.Cu") (net 59))
-  (segment (start 48.514 60.0964) (end 49.804996 61.387396) (width 0.381) (layer "B.Cu") (net 59))
-  (segment (start 60.346086 61.4934) (end 60.8076 61.954914) (width 0.381) (layer "B.Cu") (net 59))
   (segment (start 57.4379 61.170175) (end 57.847825 61.5801) (width 0.381) (layer "B.Cu") (net 59))
-  (segment (start 57.4379 60.9431) (end 57.4379 61.170175) (width 0.381) (layer "B.Cu") (net 59))
-  (segment (start 56.0578 60.452) (end 56.9468 60.452) (width 0.381) (layer "B.Cu") (net 59))
-  (segment (start 57.847825 61.5801) (end 58.382575 61.5801) (width 0.381) (layer "B.Cu") (net 59))
-  (segment (start 58.469275 61.4934) (end 60.346086 61.4934) (width 0.381) (layer "B.Cu") (net 59))
   (segment (start 51.021704 62.782896) (end 51.05 62.7546) (width 0.2) (layer "F.Cu") (net 60))
   (segment (start 50.270645 62.782896) (end 51.021704 62.782896) (width 0.2) (layer "F.Cu") (net 60))
