File: Frooastboard Modular/Kicad Project/Frooastboard Modular.kicad_pcb (KiCad board)
At the start: 4 copper layers, 44.6 x 25.7 mm, 41 parts, among them J1 Conn_01x16, J2 Conn_01x06, J3 Conn_01x06, J4 Conn_01x10, J5 Conn_01x12, J6 SW Interface, J7 Conn_01x04, U1 IS31FL3733-QF, U2 RP2040, U3 W25Q32JVZP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

Commit message: Update Frooastboard Modular.kicad_pcb
Parts:
- moved C8 1.18 mm to (64.8, 67.9)
- moved C9 1.18 mm to (64.8, 68.8)
Routing:
- net Net-(J5-Pin_12): track 28.1 -> 8.99 mm, vias 1 -> 0
- net Net-(J5-Pin_7): track 20.2 -> 1.67 mm
- net Net-(J5-Pin_11): track 26.1 -> 7.63 mm, vias 1 -> 0
- net Net-(J5-Pin_10): track 25.9 -> 7.96 mm, vias 3 -> 2
- net Net-(J5-Pin_9): track 23.3 -> 5.78 mm, vias 1 -> 0
- net Net-(J5-Pin_8): track 21.3 -> 4.26 mm, vias 1 -> 0
- net +3V3: track 26.5 -> 30.6 mm
- net GND: track 29.0 -> 32.8 mm, vias 5 -> 4
- net QSPI_SD2: track 14.6 -> 16.4 mm
- net QSPI_CLK: track 8.93 -> 10.7 mm
- net Net-(J5-Pin_3): track 10.4 -> 11.3 mm
- net Net-(J5-Pin_5): track 13.8 -> 14.4 mm
- added copper zone on In2.Cu, net +3V3
- added copper zone on In1.Cu, net GND
Other:
- outline, holes or cut-outs redrawn

Commit message: Update Frooastboard Modular.kicad_pcb
Parts:
- moved C17 47.5 mm to (63.9, 62.7)
- moved C10 43.3 mm to (63.9, 64.6), turned to 180 degrees
- moved C11 42.1 mm to (64.8, 65.5)
- moved C8 0.91 mm to (63.9, 67.9)
- moved C9 0.91 mm to (63.9, 68.8)
Routing:
- net GND: track 32.8 -> 36.4 mm, vias 4 -> 6
- net Net-(J5-Pin_4): track 12.4 -> 13.9 mm
- net +1V1: track 17.2 -> 18.4 mm
- net Net-(J5-Pin_6): track 15.3 -> 16.0 mm
- net Net-(J5-Pin_5): track 14.4 -> 15.0 mm

Commit message: Update Frooastboard Modular.kicad_pcb
Parts:
- moved C13 33.9 mm to (71.4, 62.7), turned to -90 degrees
- moved C12 29.0 mm to (77.8, 65.0), turned to -90 degrees
- moved R4 4.95 mm to (80.1, 62.0)
- moved U4 3.03 mm to (74.5, 63.9), turned to 180 degrees
- moved C6 1.88 mm to (71.4, 64.6)
- moved Y1 0.31 mm to (68.8, 63.8)
- moved C5 0.27 mm to (66.1, 65.1)
- moved R7 0.23 mm to (65.8, 63.7)
- moved C11 0.13 mm to (64.6, 65.5), turned to 180 degrees
Routing:
- net +3V3: track 30.4 -> 74.0 mm, vias 7 -> 10
- net SWDIO: track 3.09 -> 24.5 mm
- net Net-(J5-Pin_12): track 8.99 -> 28.0 mm, vias 0 -> 1
- net RP_RESET: track 5.95 -> 24.6 mm
- net Net-(J5-Pin_11): track 7.63 -> 25.9 mm, vias 0 -> 1
- net SWCLK: track 4.93 -> 23.2 mm
- net Net-(J5-Pin_10): track 7.96 -> 25.7 mm, vias 2 -> 3
- net GND: track 36.4 -> 50.0 mm
- net +5V: track 37.0 -> 28.8 mm, vias 0 -> 1
- net Net-(J5-Pin_8): track 4.26 -> 0.00 mm
- net Net-(J5-Pin_7): track 1.67 -> 0.00 mm, vias 1 -> 0
- net Net-(C6-Pad2): track 5.64 -> 6.17 mm

Commit message: Update Frooastboard Modular.kicad_pcb
Routing:
- net Net-(J5-Pin_8): track 0.00 -> 19.3 mm, vias 0 -> 1
- net Net-(J5-Pin_7): track 0.00 -> 18.0 mm, vias 0 -> 1
- net Net-(J5-Pin_9): track 5.78 -> 22.0 mm, vias 0 -> 1
- net +5V: track 28.8 -> 41.3 mm
- net Net-(J5-Pin_10): track 25.7 -> 28.7 mm
- net +3V3: track 74.0 -> 76.7 mm

Commit message: Update Frooastboard Modular.kicad_pcb
Routing:
- net +3V3: track 76.7 -> 84.3 mm
- net SCL: track 8.75 -> 14.5 mm
- net SDA: track 10.4 -> 16.1 mm
Changed lines of the file:
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@@
     (property "ki_keywords" "R resistor")
     (attr smd)
-    (fp_text reference "R4" (at 0 -1.17 90) (layer "F.SilkS")
+    (fp_text reference "R4" (at 0 1.0668 90) (layer "F.SilkS")
         (effects (font (size 1 1) (thickness 0.15)))
     )
@@
   (segment (start 54.5592 63.0428) (end 54.744 63.2276) (width 0.381) (layer "F.Cu") (net 2))
   (segment (start 63.4036 68.834) (end 62.611 68.834) (width 0.381) (layer "F.Cu") (net 2))
+  (segment (start 62.7233 56.0324) (end 62.7253 56.0304) (width 0.381) (layer "F.Cu") (net 2))
   (segment (start 54.1528 63.0428) (end 54.5592 63.0428) (width 0.381) (layer "F.Cu") (net 2))
   (segment (start 63.3242 57.5056) (end 62.8162 56.9976) (width 0.381) (layer "F.Cu") (net 2))
@@
   (segment (start 49.1058 60.071) (end 50.0634 60.071) (width 0.3556) (layer "F.Cu") (net 2))
   (segment (start 48.8442 60.071) (end 48.4106 60.5046) (width 0.3556) (layer "F.Cu") (net 2))
+  (segment (start 62.8162 56.9976) (end 62.7233 56.9047) (width 0.381) (layer "F.Cu") (net 2))
   (segment (start 64.3584 64.7648) (end 65.1256 65.532) (width 0.381) (layer "F.Cu") (net 2))
   (segment (start 82.1396 61.464) (end 82.1436 61.468) (width 0.381) (layer "F.Cu") (net 2))
@@
   (segment (start 64.6886 63.2766) (end 64.9986 62.9666) (width 0.254) (layer "F.Cu") (net 2))
   (segment (start 73.025 62.5602) (end 72.4356 62.5602) (width 0.381) (layer "F.Cu") (net 2))
+  (segment (start 62.7233 56.9047) (end 62.7233 56.0324) (width 0.381) (layer "F.Cu") (net 2))
   (segment (start 47.9498 64.8916) (end 47.538 65.3034) (width 0.3556) (layer "F.Cu") (net 2))
   (segment (start 73.025 63.4746) (end 73.025 63.8608) (width 0.381) (layer "F.Cu") (net 2))
   (segment (start 80.0862 61.464) (end 82.1396 61.464) (width 0.381) (layer "F.Cu") (net 2))
   (segment (start 77.8496 64.4666) (end 77.851 64.4652) (width 0.381) (layer "F.Cu") (net 2))
+  (segment (start 62.7253 56.0304) (end 62.7253 49.4919) (width 0.381) (layer "F.Cu") (net 2))
   (via (at 73.025 62.5602) (size 0.8) (drill 0.5) (layers "F.Cu" "B.Cu") (net 2))
   (via (at 64.0334 57.9882) (size 0.8) (drill 0.5) (layers "F.Cu" "B.Cu") (net 2))
@@
   (segment (start 56.9912 60.0346) (end 56.9912 60.4661) (width 0.2032) (layer "F.Cu") (net 65))
   (segment (start 56.9912 60.4661) (end 57.2258 60.7007) (width 0.2032) (layer "F.Cu") (net 65))
-  (segment (start 62.3042 55.3232) (end 62.3062 55.3212) (width 0.2032) (layer "F.Cu") (net 65))
   (segment (start 62.3042 57.9882) (end 62.3042 55.3232) (width 0.2032) (layer "F.Cu") (net 65))
   (segment (start 57.2258 60.7007) (end 57.4597 60.9346) (width 0.2032) (layer "F.Cu") (net 65))
   (segment (start 59.8018 58.2066) (end 62.0858 58.2066) (width 0.2032) (layer "F.Cu") (net 65))
+  (segment (start 62.3042 55.3232) (end 62.3062 55.3212) (width 0.2032) (layer "F.Cu") (net 65))
+  (segment (start 62.3062 55.3212) (end 62.3062 49.6316) (width 0.2032) (layer "F.Cu") (net 65))
   (segment (start 59.1058 58.9026) (end 59.8018 58.2066) (width 0.2032) (layer "F.Cu") (net 65))
   (segment (start 62.0858 58.2066) (end 62.3042 57.9882) (width 0.2032) (layer "F.Cu") (net 65))
@@
   (segment (start 59.1058 58.9026) (end 58.1152 59.8932) (width 0.2032) (layer "B.Cu") (net 65))
   (segment (start 56.5912 60.0346) (end 56.5912 59.5399) (width 0.2032) (layer "F.Cu") (net 66))
+  (segment (start 61.6052 57.8764) (end 59.3446 57.8764) (width 0.2032) (layer "F.Cu") (net 66))
+  (segment (start 61.974 49.7606) (end 61.976 49.7586) (width 0.2032) (layer "F.Cu") (net 66))
+  (segment (start 61.974 56.8198) (end 61.974 49.7606) (width 0.2032) (layer "F.Cu") (net 66))
   (segment (start 61.7962 56.9976) (end 61.974 56.8198) (width 0.2032) (layer "F.Cu") (net 66))
-  (segment (start 61.974 56.8198) (end 61.974 55.4736) (width 0.2032) (layer "F.Cu") (net 66))
-  (segment (start 61.6052 57.8764) (end 59.3446 57.8764) (width 0.2032) (layer "F.Cu") (net 66))
   (segment (start 61.7962 56.9976) (end 61.7962 57.6854) (width 0.2032) (layer "F.Cu") (net 66))
   (segment (start 56.7626 59.3685) (end 57.8525 59.3685) (width 0.2032) (layer "F.Cu") (net 66))

Commit message: Update Frooastboard Modular.kicad_pcb
Routing:
- net Net-(J4-Pin_5): track 19.3 -> 17.5 mm
- net Net-(J4-Pin_3): track 21.2 -> 19.5 mm
- net Net-(J4-Pin_1): track 23.3 -> 21.8 mm
Other:
- board size 44.6 x 25.7 mm -> 44.6 x 24 mm

Commit message: some updates
Parts:
- added J8: Conn_01x08, Frooastboard Footprints:PinHeader_1x08_P1.27mm_Vertical, F.Cu at (53.7, 42.8)
- J1: value Conn_01x16 -> Conn_01x08; footprint Frooastboard Footprints:PinHeader_1x16_P1.27mm_Vertical -> Frooastboard Footprints:PinHeader_1x08_P1.27mm_Vertical
- moved C3 128.0 mm to (56.5, 44.3), turned to 90 degrees
- moved J1 126.9 mm to (42.1, 43.8)
- moved C1 126.4 mm to (62.3, 42.2)
- moved C2 122.4 mm to (66.4, 44.3)
- moved C4 122.3 mm to (61.4, 51.7)
- moved R3 119.6 mm to (56.8, 49.0), turned to -90 degrees
- moved U1 116.8 mm to (61.2, 46.7), turned to 180 degrees
- moved R1 109.7 mm to (66.2, 49.7)
- moved R2 109.5 mm to (67.0, 47.7)
- moved J3 103.9 mm to (76.1, 43.0), turned to -90 degrees
- moved J2 102.5 mm to (80.3, 50.4), turned to 180 degrees
Connections:
- U1 pad 16: Net-(J1-Pin_1) -> Net-(J8-Pin_1)
- U1 pad 17: Net-(J1-Pin_2) -> Net-(J8-Pin_2)
- U1 pad 18: Net-(J1-Pin_3) -> Net-(J8-Pin_3)
- U1 pad 19: Net-(J1-Pin_4) -> Net-(J8-Pin_4)
- U1 pad 21: Net-(J1-Pin_5) -> Net-(J8-Pin_5)
- U1 pad 22: Net-(J1-Pin_6) -> Net-(J8-Pin_6)
- U1 pad 23: Net-(J1-Pin_7) -> Net-(J8-Pin_7)
- U1 pad 24: Net-(J1-Pin_8) -> Net-(J8-Pin_8)
- U1 pad 25: Net-(J1-Pin_9) -> Net-(J1-Pin_1)
- U1 pad 26: Net-(J1-Pin_10) -> Net-(J1-Pin_2)
- U1 pad 27: Net-(J1-Pin_11) -> Net-(J1-Pin_3)
- U1 pad 28: Net-(J1-Pin_12) -> Net-(J1-Pin_4)
- U1 pad 30: Net-(J1-Pin_13) -> Net-(J1-Pin_5)
- U1 pad 31: Net-(J1-Pin_14) -> Net-(J1-Pin_6)
- U1 pad 32: Net-(J1-Pin_15) -> Net-(J1-Pin_7)
- U1 pad 33: Net-(J1-Pin_16) -> Net-(J1-Pin_8)
Routing:
- net GND: track 50.0 -> 93.6 mm, vias 6 -> 8
- net +3V3: track 84.3 -> 102.0 mm, vias 10 -> 12
- net Net-(J8-Pin_4): track 0.00 -> 4.20 mm
- net SDA: track 16.1 -> 19.9 mm, vias 2 -> 3
- net Net-(U1-~{SDB}): track 0.00 -> 3.52 mm, vias 0 -> 1
- net Net-(U1-IICRST): track 0.00 -> 3.40 mm, vias 0 -> 1
- net Net-(J8-Pin_5): track 0.00 -> 3.01 mm
- net Net-(J5-Pin_10): track 28.7 -> 26.3 mm
- net Net-(J8-Pin_6): track 0.00 -> 2.20 mm
- net Net-(U1-RSET): track 0.00 -> 2.04 mm
- net Net-(J8-Pin_7): track 0.00 -> 1.40 mm
- net QSPI_CS: track 22.5 -> 21.6 mm
- net SCL: track 14.5 -> 15.1 mm
Other:
- board size 44.6 x 24 mm -> 44.6 x 28.3 mm

Commit message: before moving stuff
Parts:
- added J9: Conn_01x04, Frooastboard Footprints:PinHeader_1x04_P1.27mm_Vertical, F.Cu at (86.8, 62.5)
Connections:
- U2 pad 38: unconnected-(U2-GPIO26/ADC0-Pad38) -> GPIO_1
- U2 pad 39: unconnected-(U2-GPIO27/ADC1-Pad39) -> GPIO_2
Routing:
- net SCL: track 15.1 -> 17.4 mm, vias 0 -> 2
- net SDA: track 19.9 -> 18.8 mm, vias 3 -> 2
