File: Frooastboard Modular/Kicad Project/Frooastboard Modular.kicad_pcb (KiCad board)
At the start: 4 copper layers, 44.6 x 28.3 mm, 43 parts, among them J1 Conn_01x08, J2 Conn_01x06, J3 Conn_01x06, J4 Conn_01x10, J5 Conn_01x12, J6 SW Interface, J7 Conn_01x04, J8 Conn_01x08, J9 Conn_01x04, U1 IS31FL3733-QF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

Commit message: some stuff
Parts:
- added REF**: Fiducial_1mm_Mask2mm, Fiducial:Fiducial_1mm_Mask2mm, F.Cu at (80.9, 57.5)
- added REF**: Fiducial_1mm_Mask2mm, Fiducial:Fiducial_1mm_Mask2mm, F.Cu at (43.4, 55.2)
Connections:
- net Net-(J1-Pin_1) renamed /CS9
- net Net-(J1-Pin_2) renamed /CS10
- net Net-(J1-Pin_3) renamed /CS11
- net Net-(J1-Pin_4) renamed /CS12
- net Net-(J1-Pin_5) renamed /CS13
- net Net-(J1-Pin_6) renamed /CS14
- net Net-(J1-Pin_7) renamed /CS15
- net Net-(J1-Pin_8) renamed /CS16
- net Net-(J2-Pin_1) renamed /SW1
- net Net-(J2-Pin_2) renamed /SW2
- net Net-(J2-Pin_3) renamed /SW3
- net Net-(J2-Pin_4) renamed /SW4
- net Net-(J2-Pin_5) renamed /SW5
- net Net-(J2-Pin_6) renamed /SW6
- net Net-(J3-Pin_1) renamed /SW7
- net Net-(J3-Pin_2) renamed /SW8
- net Net-(J3-Pin_3) renamed /SW9
- net Net-(J3-Pin_4) renamed /SW10
- net Net-(J3-Pin_5) renamed /SW11
- net Net-(J3-Pin_6) renamed /SW12
- net Net-(J8-Pin_1) renamed /CS1
- net Net-(J8-Pin_2) renamed /CS2
- net Net-(J8-Pin_3) renamed /CS3
- net Net-(J8-Pin_4) renamed /CS4
- net Net-(J8-Pin_5) renamed /CS5
- net Net-(J8-Pin_6) renamed /CS6
- net Net-(J8-Pin_7) renamed /CS7
- net Net-(J8-Pin_8) renamed /CS8

Commit message: do some stuff
Parts:
- added J10: Conn_01x02, Frooastboard Footprints:PinHeader_1x02_P1.27mm_Vertical, F.Cu at (73.7, 49.0)
- J9: value Conn_01x04 -> Conn_01x05; footprint Frooastboard Footprints:PinHeader_1x04_P1.27mm_Vertical -> Frooastboard Footprints:PinHeader_1x05_P1.27mm_Vertical
- moved REF** 1.17 mm to (80.9, 56.3)
Routing:
- net GND: track 99.0 -> 116.3 mm, vias 14 -> 15
- net +3V3: track 102.3 -> 114.1 mm
- net +5V: track 41.4 -> 51.4 mm
- net /SW1: track 17.3 -> 19.2 mm
- net /SW3: track 16.5 -> 17.8 mm, vias 0 -> 1
- net /SW2: track 16.9 -> 18.2 mm, vias 0 -> 1
Other:
- outline, holes or cut-outs redrawn

Commit message: remove lockfile
Other:
- board text added: "JLCJLCJLCJLC"
Changed lines of the file:
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@@
       (plot_on_all_layers_selection 0x0000000_00000000)
       (disableapertmacros false)
-      (usegerberextensions false)
-      (usegerberattributes true)
-      (usegerberadvancedattributes true)
-      (creategerberjobfile true)
+      (usegerberextensions true)
+      (usegerberattributes false)
+      (usegerberadvancedattributes false)
+      (creategerberjobfile false)
       (dashed_line_dash_ratio 12.000000)
       (dashed_line_gap_ratio 3.000000)
@@
       (psa4output false)
       (plotreference true)
-      (plotvalue true)
+      (plotvalue false)
       (plotinvisibletext false)
       (sketchpadsonfab false)
-      (subtractmaskfromsilk false)
+      (subtractmaskfromsilk true)
       (outputformat 1)
       (mirror false)
-      (drillshape 1)
+      (drillshape 0)
       (scaleselection 1)
       (outputdirectory "")
@@
     (fp_line (start 1 0.625) (end -1 0.625)
       (stroke (width 0.1) (type solid)) (layer "F.Fab"))
-    (pad "1" smd roundrect (at -0.9125 0) (size 1.025 1.4) (layers "F.Cu" "F.Paste" "F.Mask") (roundrect_rratio 0.243902)
+    (pad "1" smd roundrect (at -0.9125 0) (size 1.025 1.4) (layers "F.Cu" "F.Paste" "F.Mask") (roundrect_rratio 0.243902439)
       (net 62 "/QSPI_CS_TP") (pintype "passive"))
-    (pad "2" smd roundrect (at 0.9125 0) (size 1.025 1.4) (layers "F.Cu" "F.Paste" "F.Mask") (roundrect_rratio 0.243902)
+    (pad "2" smd roundrect (at 0.9125 0) (size 1.025 1.4) (layers "F.Cu" "F.Paste" "F.Mask") (roundrect_rratio 0.243902439)
       (net 63 "QSPI_CS") (pintype "passive"))
     (model "${KICAD6_3DMODEL_DIR}/Resistor_SMD.3dshapes/R_0805_2012Metric.wrl"
@@
     (fp_line (start 3 3) (end -3 3)
       (stroke (width 0.1) (type solid)) (layer "F.Fab"))
-    (pad "" smd roundrect (at -1.4 -1.4 180) (size 1.13 1.13) (layers "F.Paste") (roundrect_rratio 0.221239))
-    (pad "" smd roundrect (at -1.4 0 180) (size 1.13 1.13) (layers "F.Paste") (roundrect_rratio 0.221239))
-    (pad "" smd roundrect (at -1.4 1.4 180) (size 1.13 1.13) (layers "F.Paste") (roundrect_rratio 0.221239))
-    (pad "" smd roundrect (at 0 -1.4 180) (size 1.13 1.13) (layers "F.Paste") (roundrect_rratio 0.221239))
-    (pad "" smd roundrect (at 0 0 180) (size 1.13 1.13) (layers "F.Paste") (roundrect_rratio 0.221239))
-    (pad "" smd roundrect (at 0 1.4 180) (size 1.13 1.13) (layers "F.Paste") (roundrect_rratio 0.221239))
-    (pad "" smd roundrect (at 1.4 -1.4 180) (size 1.13 1.13) (layers "F.Paste") (roundrect_rratio 0.221239))
-    (pad "" smd roundrect (at 1.4 0 180) (size 1.13 1.13) (layers "F.Paste") (roundrect_rratio 0.221239))
-    (pad "" smd roundrect (at 1.4 1.4 180) (size 1.13 1.13) (layers "F.Paste") (roundrect_rratio 0.221239))
+    (pad "" smd roundrect (at -1.4 -1.4 180) (size 1.13 1.13) (layers "F.Paste") (roundrect_rratio 0.2212389381))
+    (pad "" smd roundrect (at -1.4 0 180) (size 1.13 1.13) (layers "F.Paste") (roundrect_rratio 0.2212389381))
+    (pad "" smd roundrect (at -1.4 1.4 180) (size 1.13 1.13) (layers "F.Paste") (roundrect_rratio 0.2212389381))
+    (pad "" smd roundrect (at 0 -1.4 180) (size 1.13 1.13) (layers "F.Paste") (roundrect_rratio 0.2212389381))
+    (pad "" smd roundrect (at 0 0 180) (size 1.13 1.13) (layers "F.Paste") (roundrect_rratio 0.2212389381))
+    (pad "" smd roundrect (at 0 1.4 180) (size 1.13 1.13) (layers "F.Paste") (roundrect_rratio 0.2212389381))
+    (pad "" smd roundrect (at 1.4 -1.4 180) (size 1.13 1.13) (layers "F.Paste") (roundrect_rratio 0.2212389381))
+    (pad "" smd roundrect (at 1.4 0 180) (size 1.13 1.13) (layers "F.Paste") (roundrect_rratio 0.2212389381))
+    (pad "" smd roundrect (at 1.4 1.4 180) (size 1.13 1.13) (layers "F.Paste") (roundrect_rratio 0.2212389381))
     (pad "1" smd roundrect (at -2.95 -2.2 180) (size 0.85 0.2) (layers "F.Cu" "F.Paste" "F.Mask") (roundrect_rratio 0.25)
       (net 64 "unconnected-(U1-NC-Pad1)") (pinfunction "NC") (pintype "no_connect"))
@@
     (fp_line (start 3 2.5) (end -3 2.5)
       (stroke (width 0.1) (type solid)) (layer "F.Fab"))
-    (pad "" smd roundrect (at -0.85 -1.075) (size 1.37 1.73) (layers "F.Paste") (roundrect_rratio 0.182482))
-    (pad "" smd roundrect (at -0.85 1.075) (size 1.37 1.73) (layers "F.Paste") (roundrect_rratio 0.182482))
-    (pad "" smd roundrect (at 0.85 -1.075) (size 1.37 1.73) (layers "F.Paste") (roundrect_rratio 0.182482))
-    (pad "" smd roundrect (at 0.85 1.075) (size 1.37 1.73) (layers "F.Paste") (roundrect_rratio 0.182482))
+    (pad "" smd roundrect (at -0.85 -1.075) (size 1.37 1.73) (layers "F.Paste") (roundrect_rratio 0.1824817518))
+    (pad "" smd roundrect (at -0.85 1.075) (size 1.37 1.73) (layers "F.Paste") (roundrect_rratio 0.1824817518))
+    (pad "" smd roundrect (at 0.85 -1.075) (size 1.37 1.73) (layers "F.Paste") (roundrect_rratio 0.1824817518))
+    (pad "" smd roundrect (at 0.85 1.075) (size 1.37 1.73) (layers "F.Paste") (roundrect_rratio 0.1824817518))
     (pad "1" smd roundrect (at -2.7 -1.905) (size 0.75 0.5) (layers "F.Cu" "F.Paste" "F.Mask") (roundrect_rratio 0.25)
       (net 63 "QSPI_CS") (pinfunction "~{CS}") (pintype "input"))
@@
     (fp_line (start 1 0.625) (end 1 -0.625)
       (stroke (width 0.1) (type solid)) (layer "F.Fab"))
-    (pad "1" smd roundrect (at -0.8875 0) (size 1.125 1.05) (layers "F.Cu" "F.Paste" "F.Mask") (roundrect_rratio 0.238095)
+    (pad "1" smd roundrect (at -0.8875 0) (size 1.125 1.05) (layers "F.Cu" "F.Paste" "F.Mask") (roundrect_rratio 0.2380952381)
       (net 2 "+3V3") (pintype "passive"))
-    (pad "2" smd roundrect (at 0.8875 0) (size 1.125 1.05) (layers "F.Cu" "F.Paste" "F.Mask") (roundrect_rratio 0.238095)
+    (pad "2" smd roundrect (at 0.8875 0) (size 1.125 1.05) (layers "F.Cu" "F.Paste" "F.Mask") (roundrect_rratio 0.2380952381)
       (net 1 "GND") (pintype "passive"))
     (model "${KICAD6_3DMODEL_DIR}/Capacitor_Tantalum_SMD.3dshapes/CP_EIA-2012-15_AVX-P.wrl"
@@
     (fp_line (start 3.5 3.5) (end -3.5 3.5)
       (stroke (width 0.1) (type solid)) (layer "F.Fab"))
-    (pad "" smd roundrect (at -0.6375 -0.6375 90) (size 1.084435 1.084435) (layers "F.Paste") (roundrect_rratio 0.230535))
-    (pad "" smd roundrect (at -0.6375 0.6375 90) (size 1.084435 1.084435) (layers "F.Paste") (roundrect_rratio 0.230535))
-    (pad "" smd roundrect (at 0.6375 -0.6375 90) (size 1.084435 1.084435) (layers "F.Paste") (roundrect_rratio 0.230535))
-    (pad "" smd roundrect (at 0.6375 0.6375 90) (size 1.084435 1.084435) (layers "F.Paste") (roundrect_rratio 0.230535))
+    (pad "" smd roundrect (at -0.6375 -0.6375 90) (size 1.084435 1.084435) (layers "F.Paste") (roundrect_rratio 0.2305347946))
+    (pad "" smd roundrect (at -0.6375 0.6375 90) (size 1.084435 1.084435) (layers "F.Paste") (roundrect_rratio 0.2305347946))
+    (pad "" smd roundrect (at 0.6375 -0.6375 90) (size 1.084435 1.084435) (layers "F.Paste") (roundrect_rratio 0.2305347946))
+    (pad "" smd roundrect (at 0.6375 0.6375 90) (size 1.084435 1.084435) (layers "F.Paste") (roundrect_rratio 0.2305347946))
     (pad "1" smd roundrect (at -3.4375 -2.6 90) (size 0.875 0.2) (layers "F.Cu" "F.Paste" "F.Mask") (roundrect_rratio 0.25)
       (net 2 "+3V3") (pinfunction "IOVDD") (pintype "power_in"))
@@
     (property "ki_keywords" "capacitor cap")
     (attr smd)
-    (fp_text reference "C6" (at -1.4706 0 180) (layer "F.SilkS")
+    (fp_text reference "C6" (at -1.0896 1.0668 270) (layer "F.SilkS")
         (effects (font (size 1 1) (thickness 0.15)))
     )
@@
     (fp_line (start 1 0.625) (end 1 -0.625)
       (stroke (width 0.1) (type solid)) (layer "F.Fab"))
-    (pad "1" smd roundrect (at -0.8875 0 270) (size 1.125 1.05) (layers "F.Cu" "F.Paste" "F.Mask") (roundrect_rratio 0.238095)
+    (pad "1" smd roundrect (at -0.8875 0 270) (size 1.125 1.05) (layers "F.Cu" "F.Paste" "F.Mask") (roundrect_rratio 0.2380952381)
       (net 2 "+3V3") (pintype "passive"))
-    (pad "2" smd roundrect (at 0.8875 0 270) (size 1.125 1.05) (layers "F.Cu" "F.Paste" "F.Mask") (roundrect_rratio 0.238095)
+    (pad "2" smd roundrect (at 0.8875 0 270) (size 1.125 1.05) (layers "F.Cu" "F.Paste" "F.Mask") (roundrect_rratio 0.2380952381)
       (net 1 "GND") (pintype "passive"))
     (model "${KICAD6_3DMODEL_DIR}/Capacitor_Tantalum_SMD.3dshapes/CP_EIA-2012-15_AVX-P.wrl"
@@
   (gr_line (start 39.116 69.596) (end 39.116 68.5038)
     (stroke (width 0.15) (type default)) (layer "User.1"))
+  (gr_text "JLCJLCJLCJLC" (at 44.2976 50.3174) (layer "F.SilkS")
+    (effects (font (size 0.8 1) (thickness 0.15)) (justify left bottom))
+  )
   (segment (start 46.4058 61.976) (end 46.4058 61.5188) (width 0.381) (layer "F.Cu") (net 1))
   (segment (start 67.867 62.9176) (end 69.3166 61.468) (width 0.381) (layer "F.Cu") (net 1))

Commit message: tiling
Parts:
- removed the REF** at (80.9, 56.3)
- removed the REF** at (43.4, 55.2)
- added REF**: Fiducial_1mm_Mask2mm, Fiducial:Fiducial_1mm_Mask2mm, F.Cu at (43.4, 54.9)
- added REF**: Fiducial_1mm_Mask2mm, Fiducial:Fiducial_1mm_Mask2mm, F.Cu at (80.9, 56.2)
Other:
- board text removed: "JLCJLCJLCJLC"
Changed lines of the file:
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@@
     )
+  )
+  (footprint "Fiducial:Fiducial_1mm_Mask2mm" (layer "F.Cu")
+    (at 43.4086 54.9402)
+    (descr "Circular Fiducial, 1mm bare copper, 2mm soldermask opening (Level A)")
+    (tags "fiducial")
+    (attr smd)
+    (fp_text reference "REF**" (at 0 -2) (layer "F.SilkS") hide
+        (effects (font (size 1 1) (thickness 0.15)))
+    )
+    (fp_text value "Fiducial_1mm_Mask2mm" (at 0 2) (layer "F.Fab")
+        (effects (font (size 1 1) (thickness 0.15)))
+    )
+    (fp_text user "${REFERENCE}" (at 0 0) (layer "F.Fab")
+        (effects (font (size 0.4 0.4) (thickness 0.06)))
+    )
+    (fp_circle (center 0 0) (end 1.25 0)
+      (stroke (width 0.05) (type solid)) (fill none) (layer "F.CrtYd"))
+    (fp_circle (center 0 0) (end 1 0)
+      (stroke (width 0.1) (type solid)) (fill none) (layer "F.Fab"))
+    (pad "" smd circle (at 0 0) (size 1 1) (layers "F.Cu" "F.Mask")
+      (solder_mask_margin 0.5) (clearance 0.5))
   )
   (footprint "Frooastboard Footprints:PinHeader_1x12_P1.27mm_Vertical" (layer "F.Cu")
@@
       (rotate (xyz 0 0 0))
     )
-  )
-  (footprint "Fiducial:Fiducial_1mm_Mask2mm" (layer "F.Cu")
-    (at 80.9498 56.3118)
-    (descr "Circular Fiducial, 1mm bare copper, 2mm soldermask opening (Level A)")
-    (tags "fiducial")
-    (attr smd)
-    (fp_text reference "REF**" (at 0 -2) (layer "F.SilkS") hide
-        (effects (font (size 1 1) (thickness 0.15)))
-    )
-    (fp_text value "Fiducial_1mm_Mask2mm" (at 0 2) (layer "F.Fab")
-        (effects (font (size 1 1) (thickness 0.15)))
-    )
-    (fp_text user "${REFERENCE}" (at 0 0) (layer "F.Fab")
-        (effects (font (size 0.4 0.4) (thickness 0.06)))
-    )
-    (fp_circle (center 0 0) (end 1.25 0)
-      (stroke (width 0.05) (type solid)) (fill none) (layer "F.CrtYd"))
-    (fp_circle (center 0 0) (end 1 0)
-      (stroke (width 0.1) (type solid)) (fill none) (layer "F.Fab"))
-    (pad "" smd circle (at 0 0) (size 1 1) (layers "F.Cu" "F.Mask")
-      (solder_mask_margin 0.5) (clearance 0.5))
-  )
-  (footprint "Fiducial:Fiducial_1mm_Mask2mm" (layer "F.Cu")
-    (at 43.434 55.1688)
-    (descr "Circular Fiducial, 1mm bare copper, 2mm soldermask opening (Level A)")
-    (tags "fiducial")
-    (attr smd)
-    (fp_text reference "REF**" (at 0 -2) (layer "F.SilkS") hide
-        (effects (font (size 1 1) (thickness 0.15)))
-    )
-    (fp_text value "Fiducial_1mm_Mask2mm" (at 0 2) (layer "F.Fab")
-        (effects (font (size 1 1) (thickness 0.15)))
-    )
-    (fp_text user "${REFERENCE}" (at 0 0) (layer "F.Fab")
-        (effects (font (size 0.4 0.4) (thickness 0.06)))
-    )
-    (fp_circle (center 0 0) (end 1.25 0)
-      (stroke (width 0.05) (type solid)) (fill none) (layer "F.CrtYd"))
-    (fp_circle (center 0 0) (end 1 0)
-      (stroke (width 0.1) (type solid)) (fill none) (layer "F.Fab"))
-    (pad "" smd circle (at 0 0) (size 1 1) (layers "F.Cu" "F.Mask")
-      (solder_mask_margin 0.5) (clearance 0.5))
   )
   (footprint "Capacitor_SMD:C_0402_1005Metric" (layer "F.Cu")
@@
       (rotate (xyz 0 0 0))
     )
+  )
+  (footprint "Fiducial:Fiducial_1mm_Mask2mm" (layer "F.Cu")
+    (at 80.9498 56.2356)
+    (descr "Circular Fiducial, 1mm bare copper, 2mm soldermask opening (Level A)")
+    (tags "fiducial")
+    (attr smd)
+    (fp_text reference "REF**" (at 0 -2) (layer "F.SilkS") hide
+        (effects (font (size 1 1) (thickness 0.15)))
+    )
+    (fp_text value "Fiducial_1mm_Mask2mm" (at 0 2) (layer "F.Fab")
+        (effects (font (size 1 1) (thickness 0.15)))
+    )
+    (fp_text user "${REFERENCE}" (at 0 0) (layer "F.Fab")
+        (effects (font (size 0.4 0.4) (thickness 0.06)))
+    )
+    (fp_circle (center 0 0) (end 1.25 0)
+      (stroke (width 0.05) (type solid)) (fill none) (layer "F.CrtYd"))
+    (fp_circle (center 0 0) (end 1 0)
+      (stroke (width 0.1) (type solid)) (fill none) (layer "F.Fab"))
+    (pad "" smd circle (at 0 0) (size 1 1) (layers "F.Cu" "F.Mask")
+      (solder_mask_margin 0.5) (clearance 0.5))
   )
   (footprint "Connector_PinHeader_1.27mm:PinHeader_1x02_P1.27mm_Vertical" (layer "F.Cu")
@@
   (gr_line (start 39.116 69.596) (end 39.116 68.5038)
     (stroke (width 0.15) (type default)) (layer "User.1"))
-  (gr_text "JLCJLCJLCJLC" (at 44.2976 50.3174) (layer "F.SilkS")
-    (effects (font (size 0.8 1) (thickness 0.15)) (justify left bottom))
-  )
   (segment (start 46.4058 61.976) (end 46.4058 61.5188) (width 0.381) (layer "F.Cu") (net 1))
   (segment (start 67.867 62.9176) (end 69.3166 61.468) (width 0.381) (layer "F.Cu") (net 1))

Commit message: some stuff and caps lock
Parts:
- moved REF** 0.20 mm to (43.4, 55.1)
Changed lines of the file:
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@@
     (property "ki_keywords" "Adjustable Voltage Regulator 1A Positive")
     (attr smd)
-    (fp_text reference "U4" (at -0.1222 -1.7526) (layer "F.SilkS")
+    (fp_text reference "U4" (at 0.0302 1.5494) (layer "F.SilkS")
         (effects (font (size 1 1) (thickness 0.15)))
     )
@@
     (property "ki_keywords" "capacitor cap")
     (attr smd)
-    (fp_text reference "C5" (at -1.5468 0.9144) (layer "F.SilkS")
+    (fp_text reference "C5" (at -1.5468 0.508) (layer "F.SilkS")
         (effects (font (size 1 1) (thickness 0.15)))
     )
@@
     (property "ki_keywords" "R resistor")
     (attr smd)
-    (fp_text reference "R10" (at 0.7093 -1.524) (layer "F.SilkS")
+    (fp_text reference "R10" (at 0.7093 -1.397) (layer "F.SilkS")
         (effects (font (size 1 1) (thickness 0.15)))
     )
@@
   )
   (footprint "Fiducial:Fiducial_1mm_Mask2mm" (layer "F.Cu")
-    (at 43.4086 54.9402)
+    (at 43.4086 55.1434)
     (descr "Circular Fiducial, 1mm bare copper, 2mm soldermask opening (Level A)")
     (tags "fiducial")
@@
     (property "ki_keywords" "capacitor cap")
     (attr smd)
-    (fp_text reference "C15" (at -0.5614 -1.3462) (layer "F.SilkS")
+    (fp_text reference "C15" (at -0.0026 -1.1938) (layer "F.SilkS")
         (effects (font (size 1 1) (thickness 0.15)))
     )
@@
     (property "ki_keywords" "capacitor cap")
     (attr smd)
-    (fp_text reference "C11" (at -0.3784 -1.1176) (layer "F.SilkS")
+    (fp_text reference "C11" (at 0.155 -1.143) (layer "F.SilkS")
         (effects (font (size 1 1) (thickness 0.15)))
     )
@@
     (property "ki_keywords" "R resistor")
     (attr smd)
-    (fp_text reference "R9" (at -1.8308 0.0674) (layer "F.SilkS")
+    (fp_text reference "R9" (at 1.395 -0.5676 90) (layer "F.SilkS")
         (effects (font (size 1 1) (thickness 0.15)))
     )
@@
     (property "ki_keywords" "R resistor")
     (attr smd)
-    (fp_text reference "R8" (at 0.0234 1.1176) (layer "F.SilkS")
+    (fp_text reference "R8" (at 1.395 0.1778 90) (layer "F.SilkS")
         (effects (font (size 1 1) (thickness 0.15)))
     )
@@
     (property "ki_keywords" "capacitor cap")
     (attr smd)
-    (fp_text reference "C7" (at 1.8314 0.0254 90) (layer "F.SilkS")
+    (fp_text reference "C7" (at -1.5722 0.4572 180) (layer "F.SilkS")
         (effects (font (size 1 1) (thickness 0.15)))
     )
@@
     (property "ki_keywords" "capacitor cap")
     (attr smd)
-    (fp_text reference "C6" (at -1.0896 1.0668 270) (layer "F.SilkS")
+    (fp_text reference "C6" (at -1.0674 1.6674) (layer "F.SilkS")
         (effects (font (size 1 1) (thickness 0.15)))
     )
@@
     (property "ki_keywords" "connector")
     (attr through_hole)
-    (fp_text reference "J6" (at 1.4732 7.112 180) (layer "F.SilkS")
+    (fp_text reference "J6" (at 1.7272 5.1562 180) (layer "F.SilkS")
         (effects (font (size 1 1) (thickness 0.15)))
     )
@@
     (property "ki_keywords" "connector")
     (attr through_hole)
-    (fp_text reference "J7" (at 1.6256 -1.7018) (layer "F.SilkS")
-        (effects (font (size 1 1) (thickness 0.15)))
-    )
+    (fp_text reference "J7" (at 1.5748 -1.5748) (layer "F.SilkS")
+        (effects (font (size 1 1) (thickness 0.15)))
+    )

Commit message: stuff
Other:
- board text added: "JLCJLCJLCJLC"
Changed lines of the file:
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@@
   (gr_line (start 39.116 69.596) (end 39.116 68.5038)
     (stroke (width 0.15) (type default)) (layer "User.1"))
+  (gr_text "JLCJLCJLCJLC" (at 44.3484 50.292) (layer "F.SilkS")
+    (effects (font (size 0.8 0.8) (thickness 0.15)) (justify left bottom))
+  )
   (segment (start 46.4058 61.976) (end 46.4058 61.5188) (width 0.381) (layer "F.Cu") (net 1))
   (segment (start 67.867 62.9176) (end 69.3166 61.468) (width 0.381) (layer "F.Cu") (net 1))

Commit message: fix drc erc errors
Parts:
- removed REF** (x2): Fiducial_1mm_Mask2mm, Fiducial:Fiducial_1mm_Mask2mm
- added FID1: Fiducial, Fiducial:Fiducial_1mm_Mask2mm, F.Cu at (43.4, 55.2)
- added FID2: Fiducial, Fiducial:Fiducial_1mm_Mask2mm, F.Cu at (80.9, 56.2)
- H1: renamed from REF**; value 1U -> MountingHole
Connections:
- net +3V3 renamed +3.3V

Commit message: some stuff
Routing:
- net Net-(U1-~{SDB}): track 4.67 -> 5.17 mm
