File: Frooastboard Modular/Kicad Project/Frooastboard Modular.kicad_sch (KiCad schematic)
At the start: 40 parts, among them J1 Conn_01x16, J2 Conn_01x06, J3 Conn_01x06, J4 Conn_01x10, J5 Conn_01x12, J6 SW Interface, J7 Conn_01x04, U1 IS31FL3733-QF, U2 RP2040, U3 W25Q32JVZP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

Commit message: basic left side
Parts:
- R10: footprint Resistor_SMD:R_0402_1005Metric -> Resistor_SMD:R_0805_2012Metric
Changed lines of the file:
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@@
       (effects (font (size 1.27 1.27)))
     )
-    (property "Footprint" "Resistor_SMD:R_0402_1005Metric" (at 182.88 39.37 0)
+    (property "Footprint" "Resistor_SMD:R_0805_2012Metric" (at 182.88 39.37 0)
       (effects (font (size 1.27 1.27)) hide)
     )

Commit message: backup before differential
Connections:
- net DN: now also J7.2 (Pin_2), R8.2; no longer J7.4 (Pin_4), R9.2
- net DP: now also R9.2; no longer R8.2
- net GND: now also J7.4 (Pin_4); no longer J7.2 (Pin_2)
- net RP_D+: now also R9.1; no longer R8.1
- net RP_D-: now also R8.1; no longer R9.1
Other:
- moved on the sheet: R8, R9
Changed lines of the file:
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@@
     (stroke (width 0) (type default))
   )
+  (wire (pts (xy 186.69 135.89) (xy 186.69 138.43))
+    (stroke (width 0) (type default))
+  )
   (wire (pts (xy 68.58 267.97) (xy 66.04 267.97))
     (stroke (width 0) (type default))
@@
     (stroke (width 0) (type default))
   )
-  (wire (pts (xy 189.23 130.81) (xy 186.69 130.81))
-    (stroke (width 0) (type default))
-  )
   (wire (pts (xy 83.82 217.17) (xy 86.36 217.17))
     (stroke (width 0) (type default))
@@
     (stroke (width 0) (type default))
   )
-  (wire (pts (xy 184.15 133.35) (xy 189.23 133.35))
+  (wire (pts (xy 184.15 130.81) (xy 189.23 130.81))
     (stroke (width 0) (type default))
   )
@@
     (stroke (width 0) (type default))
   )
-  (wire (pts (xy 184.15 135.89) (xy 189.23 135.89))
+  (wire (pts (xy 184.15 133.35) (xy 189.23 133.35))
     (stroke (width 0) (type default))
   )
@@
     (stroke (width 0) (type default))
   )
-  (wire (pts (xy 176.53 135.89) (xy 179.07 135.89))
+  (wire (pts (xy 176.53 133.35) (xy 179.07 133.35))
     (stroke (width 0) (type default))
   )
@@
     (stroke (width 0) (type default))
   )
-  (wire (pts (xy 186.69 130.81) (xy 186.69 138.43))
-    (stroke (width 0) (type default))
-  )
   (wire (pts (xy 46.99 60.96) (xy 49.53 60.96))
     (stroke (width 0) (type default))
@@
     (stroke (width 0) (type default))
   )
-  (wire (pts (xy 176.53 133.35) (xy 179.07 133.35))
+  (wire (pts (xy 176.53 130.81) (xy 179.07 130.81))
     (stroke (width 0) (type default))
   )
@@
     (stroke (width 0) (type default))
   )
+  (wire (pts (xy 189.23 135.89) (xy 186.69 135.89))
+    (stroke (width 0) (type default))
+  )
   (wire (pts (xy 46.99 26.67) (xy 62.23 26.67))
     (stroke (width 0) (type default))
@@
     (stroke (width 0) (type default))
   )
-  (label "DP" (at 185.42 133.35 0) (fields_autoplaced)
+  (label "DN" (at 185.42 130.81 0) (fields_autoplaced)
     (effects (font (size 1.27 1.27)) (justify left bottom))
   )
-  (label "DN" (at 185.42 135.89 0) (fields_autoplaced)
+  (label "DP" (at 185.42 133.35 0) (fields_autoplaced)
     (effects (font (size 1.27 1.27)) (justify left bottom))
   )
@@
     )
   )
-  (global_label "RP_D-" (shape input) (at 176.53 135.89 180) (fields_autoplaced)
+  (global_label "RP_D-" (shape input) (at 176.53 130.81 180) (fields_autoplaced)
     (effects (font (size 1.27 1.27)) (justify right))
-    (property "Intersheetrefs" "${INTERSHEET_REFS}" (at 167.7669 135.8106 0)
+    (property "Intersheetrefs" "${INTERSHEET_REFS}" (at 167.7669 130.7306 0)
       (effects (font (size 1.27 1.27)) (justify right) hide)
     )
@@
     )
   )
-  (symbol (lib_id "Device:R_Small") (at 181.61 133.35 90) (unit 1)
+  (symbol (lib_id "Device:R_Small") (at 181.61 130.81 90) (unit 1)
     (in_bom yes) (on_board yes) (dnp no) (fields_autoplaced)
-    (property "Reference" "R8" (at 181.61 127 90)
+    (property "Reference" "R8" (at 181.61 124.46 90)
       (effects (font (size 1.27 1.27)))
     )
-    (property "Value" "27R" (at 181.61 129.54 90)
+    (property "Value" "27R" (at 181.61 127 90)
       (effects (font (size 1.27 1.27)))
     )
-    (property "Footprint" "Resistor_SMD:R_0402_1005Metric" (at 181.61 133.35 0)
+    (property "Footprint" "Resistor_SMD:R_0402_1005Metric" (at 181.61 130.81 0)
       (effects (font (size 1.27 1.27)) hide)
     )
-    (property "Datasheet" "~" (at 181.61 133.35 0)
+    (property "Datasheet" "~" (at 181.61 130.81 0)
       (effects (font (size 1.27 1.27)) hide)
     )
@@
     )
   )
-  (symbol (lib_id "Device:R_Small") (at 181.61 135.89 90) (unit 1)
+  (symbol (lib_id "Device:R_Small") (at 181.61 133.35 90) (unit 1)
     (in_bom yes) (on_board yes) (dnp no) (fields_autoplaced)
-    (property "Reference" "R9" (at 181.61 129.54 90)
+    (property "Reference" "R9" (at 181.61 127 90)
       (effects (font (size 1.27 1.27)))
     )
-    (property "Value" "27R" (at 181.61 132.08 90)
+    (property "Value" "27R" (at 181.61 129.54 90)
       (effects (font (size 1.27 1.27)))
     )
-    (property "Footprint" "Resistor_SMD:R_0402_1005Metric" (at 181.61 135.89 0)
+    (property "Footprint" "Resistor_SMD:R_0402_1005Metric" (at 181.61 133.35 0)
       (effects (font (size 1.27 1.27)) hide)
     )
-    (property "Datasheet" "~" (at 181.61 135.89 0)
+    (property "Datasheet" "~" (at 181.61 133.35 0)
       (effects (font (size 1.27 1.27)) hide)
     )

Commit message: some updates
Parts:
- removed J1: Conn_01x16, Frooastboard Footprints:PinHeader_1x16_P1.27mm_Vertical, symbol Connector_Generic:Conn_01x16
- added J1, J8: Conn_01x08, Frooastboard Footprints:PinHeader_1x08_P1.27mm_Vertical, symbol Connector_Generic:Conn_01x08
Connections:
- net at U1.16 (CS1): now also J8.1 (Pin_1)
- net at U1.17 (CS2): now also J8.2 (Pin_2)
- net at U1.18 (CS3): now also J8.3 (Pin_3)
- net at U1.19 (CS4): now also J8.4 (Pin_4)
- net at U1.21 (CS5): now also J8.5 (Pin_5)
- net at U1.22 (CS6): now also J8.6 (Pin_6)
- net at U1.23 (CS7): now also J8.7 (Pin_7)
- net at U1.24 (CS8): now also J8.8 (Pin_8)
- net at U1.25 (CS9): now also J1.1 (Pin_1)
- net at U1.26 (CS10): now also J1.2 (Pin_2)
- net at U1.27 (CS11): now also J1.3 (Pin_3)
- net at U1.28 (CS12): now also J1.4 (Pin_4)
- net at U1.30 (CS13): now also J1.5 (Pin_5)
- net at U1.31 (CS14): now also J1.6 (Pin_6)
- net at U1.32 (CS15): now also J1.7 (Pin_7)
- net at U1.33 (CS16): now also J1.8 (Pin_8)
Changed lines of the file:
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@@
     )
   )
-  (symbol (lib_id "Connector_Generic:Conn_01x16") (at 91.44 207.01 0) (unit 1)
-    (in_bom yes) (on_board yes) (dnp no) (fields_autoplaced)
-    (property "Reference" "J1" (at 93.98 207.0099 0)
-      (effects (font (size 1.27 1.27)) (justify left))
-    )
-    (property "Value" "Conn_01x16" (at 93.98 209.5499 0)
-      (effects (font (size 1.27 1.27)) (justify left))
-    )
-    (property "Footprint" "Frooastboard Footprints:PinHeader_1x16_P1.27mm_Vertical" (at 91.44 207.01 0)
-      (effects (font (size 1.27 1.27)) hide)
-    )
-    (property "Datasheet" "~" (at 91.44 207.01 0)
-      (effects (font (size 1.27 1.27)) hide)
-    )
-    (pin "1")
-    (pin "10")
-    (pin "11")
-    (pin "12")
-    (pin "13")
-    (pin "14")
-    (pin "15")
-    (pin "16")
+  (symbol (lib_id "Connector_Generic:Conn_01x08") (at 91.44 217.17 0) (unit 1)
+    (in_bom yes) (on_board yes) (dnp no) (fields_autoplaced)
+    (property "Reference" "J1" (at 93.98 217.17 0)
+      (effects (font (size 1.27 1.27)) (justify left))
+    )
+    (property "Value" "Conn_01x08" (at 93.98 219.71 0)
+      (effects (font (size 1.27 1.27)) (justify left))
+    )
+    (property "Footprint" "Frooastboard Footprints:PinHeader_1x08_P1.27mm_Vertical" (at 91.44 217.17 0)
+      (effects (font (size 1.27 1.27)) hide)
+    )
+    (property "Datasheet" "~" (at 91.44 217.17 0)
+      (effects (font (size 1.27 1.27)) hide)
+    )
+    (pin "1")
     (pin "2")
     (pin "3")
@@
     (pin "7")
     (pin "8")
-    (pin "9")
-    (instances
-      (project "Frooastboard Modular"
-        (path "/9ee55997-d93e-462c-b474-dae14d38ea26"
-          (reference "J1") (unit 1)
-        )
-      )
-      (project "Frooastboard Walnut Modular"
-        (path "/e63e39d7-6ac0-4ffd-8aa3-1841a4541b55"
-          (reference "J2") (unit 1)
-        )
-        (path "/e63e39d7-6ac0-4ffd-8aa3-1841a4541b55/eba7bed6-3b4a-4b7a-b4a2-784017f24fe8"
+    (instances
+      (project "Frooastboard Modular"
+        (path "/9ee55997-d93e-462c-b474-dae14d38ea26"
           (reference "J1") (unit 1)
         )
@@
         )
       )
+    )
+  )
+  (symbol (lib_id "Connector_Generic:Conn_01x08") (at 91.44 196.85 0) (unit 1)
+    (in_bom yes) (on_board yes) (dnp no) (fields_autoplaced)
+    (property "Reference" "J8" (at 93.98 196.85 0)
+      (effects (font (size 1.27 1.27)) (justify left))
+    )
+    (property "Value" "Conn_01x08" (at 93.98 199.39 0)
+      (effects (font (size 1.27 1.27)) (justify left))
+    )
+    (property "Footprint" "Frooastboard Footprints:PinHeader_1x08_P1.27mm_Vertical" (at 91.44 196.85 0)
+      (effects (font (size 1.27 1.27)) hide)
+    )
+    (property "Datasheet" "~" (at 91.44 196.85 0)
+      (effects (font (size 1.27 1.27)) hide)
+    )
+    (pin "1")
+    (pin "2")
+    (pin "3")
+    (pin "4")
+    (pin "5")
+    (pin "6")
+    (pin "7")
+    (pin "8")
+    (instances
+      (project "Frooastboard Modular"
+        (path "/9ee55997-d93e-462c-b474-dae14d38ea26"
+          (reference "J8") (unit 1)
+        )
+      )

Commit message: before moving stuff
Parts:
- added J9: Conn_01x04, Frooastboard Footprints:PinHeader_1x04_P1.27mm_Vertical, symbol Connector_Generic:Conn_01x04
Connections:
- net +3V3: now also J9.1 (Pin_1)
- net GND: now also J9.4 (Pin_4)
- net GPIO_1: now reaches U2.38 (GPIO26/ADC0)
- net GPIO_1: now also J9.2 (Pin_2)
- net GPIO_2: now reaches U2.39 (GPIO27/ADC1)
- net GPIO_2: now also J9.3 (Pin_3)
- no-connect marks 3 -> 6
Changed lines of the file:
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@@
   (junction (at 203.2 29.21) (diameter 0) (color 0 0 0 0)
   )
+  (no_connect (at 90.17 95.25))
   (no_connect (at 48.26 199.39))
-  (no_connect (at 90.17 109.22))
+  (no_connect (at 90.17 97.79))
+  (no_connect (at 90.17 100.33))
+  (no_connect (at 90.17 92.71))
   (no_connect (at 48.26 209.55))
   (wire (pts (xy 138.43 40.64) (xy 135.89 40.64))
@@
     (stroke (width 0) (type default))
   )
+  (wire (pts (xy 90.17 106.68) (xy 92.71 106.68))
+    (stroke (width 0) (type default))
+  )
   (wire (pts (xy 66.04 128.27) (xy 66.04 130.81))
     (stroke (width 0) (type default))
@@
     (stroke (width 0) (type default))
   )
+  (wire (pts (xy 90.17 109.22) (xy 92.71 109.22))
+    (stroke (width 0) (type default))
+  )
   (wire (pts (xy 261.62 36.83) (xy 261.62 39.37))
     (stroke (width 0) (type default))
@@
     (stroke (width 0) (type default))
   )
+  (wire (pts (xy 186.69 157.48) (xy 189.23 157.48))
+    (stroke (width 0) (type default))
+  )
   (wire (pts (xy 66.04 267.97) (xy 66.04 265.43))
     (stroke (width 0) (type default))
@@
     (stroke (width 0) (type default))
   )
+  (wire (pts (xy 186.69 160.02) (xy 189.23 160.02))
+    (stroke (width 0) (type default))
+  )
   (wire (pts (xy 123.825 193.04) (xy 133.985 193.04))
     (stroke (width 0) (type default))
@@
     (stroke (width 0) (type default))
   )
+  (wire (pts (xy 186.69 154.94) (xy 189.23 154.94))
+    (stroke (width 0) (type default))
+  )
   (wire (pts (xy 135.89 40.64) (xy 135.89 43.18))
     (stroke (width 0) (type default))
@@
     (stroke (width 0) (type default))
   )
+  (wire (pts (xy 186.69 152.4) (xy 189.23 152.4))
+    (stroke (width 0) (type default))
+  )
   (wire (pts (xy 261.62 39.37) (xy 264.16 39.37))
     (stroke (width 0) (type default))
@@
     )
   )
+  (global_label "GPIO_1" (shape input) (at 186.69 154.94 180) (fields_autoplaced)
+    (effects (font (size 1.27 1.27)) (justify right))
+    (property "Intersheetrefs" "${INTERSHEET_REFS}" (at 177.1318 154.94 0)
+      (effects (font (size 1.27 1.27)) (justify right) hide)
+    )
+  )
   (global_label "QSPI_SD0" (shape input) (at 46.99 104.14 180) (fields_autoplaced)
     (effects (font (size 1.27 1.27)) (justify right))
@@
     )
   )
+  (global_label "GPIO_1" (shape input) (at 92.71 106.68 0) (fields_autoplaced)
+    (effects (font (size 1.27 1.27)) (justify left))
+    (property "Intersheetrefs" "${INTERSHEET_REFS}" (at 102.2682 106.68 0)
+      (effects (font (size 1.27 1.27)) (justify left) hide)
+    )
+  )
   (global_label "SWDIO" (shape input) (at 46.99 93.98 180) (fields_autoplaced)
     (effects (font (size 1.27 1.27)) (justify right))
@@
     )
   )
+  (global_label "GPIO_2" (shape input) (at 92.71 109.22 0) (fields_autoplaced)
+    (effects (font (size 1.27 1.27)) (justify left))
+    (property "Intersheetrefs" "${INTERSHEET_REFS}" (at 102.2682 109.22 0)
+      (effects (font (size 1.27 1.27)) (justify left) hide)
+    )
+  )
   (global_label "QSPI_SD3" (shape input) (at 46.99 111.76 180) (fields_autoplaced)
     (effects (font (size 1.27 1.27)) (justify right))
@@
     )
   )
+  (global_label "GPIO_2" (shape input) (at 186.69 157.48 180) (fields_autoplaced)
+    (effects (font (size 1.27 1.27)) (justify right))
+    (property "Intersheetrefs" "${INTERSHEET_REFS}" (at 177.1318 157.48 0)
+      (effects (font (size 1.27 1.27)) (justify right) hide)
+    )
+  )
   (global_label "SDA" (shape input) (at 45.72 194.31 180) (fields_autoplaced)
     (effects (font (size 1.27 1.27)) (justify right))
@@
     )
   )
+  (symbol (lib_id "power:GND") (at 186.69 160.02 270) (unit 1)
+    (in_bom yes) (on_board yes) (dnp no) (fields_autoplaced)
+    (property "Reference" "#PWR032" (at 180.34 160.02 0)
+      (effects (font (size 1.27 1.27)) hide)
+    )
+    (property "Value" "GND" (at 182.88 160.0199 90)
+      (effects (font (size 1.27 1.27)) (justify right))
+    )
+    (property "Footprint" "" (at 186.69 160.02 0)
+      (effects (font (size 1.27 1.27)) hide)
+    )
+    (property "Datasheet" "" (at 186.69 160.02 0)
+      (effects (font (size 1.27 1.27)) hide)
+    )
+    (pin "1")
+    (instances
+      (project "Frooastboard Modular"
+        (path "/9ee55997-d93e-462c-b474-dae14d38ea26"
+          (reference "#PWR032") (unit 1)
+        )
+      )
+      (project "Frooastboard Walnut Modular"
+        (path "/e63e39d7-6ac0-4ffd-8aa3-1841a4541b55"
+          (reference "#PWR0120") (unit 1)
+        )
+        (path "/e63e39d7-6ac0-4ffd-8aa3-1841a4541b55/eba7bed6-3b4a-4b7a-b4a2-784017f24fe8"
+          (reference "#PWR020") (unit 1)
+        )
+      )
+    )
+  )
   (symbol (lib_id "Device:R_Small") (at 97.79 111.76 90) (unit 1)
     (in_bom yes) (on_board yes) (dnp no)
@@
     )
   )
+  (symbol (lib_id "Connector_Generic:Conn_01x04") (at 194.31 154.94 0) (unit 1)
+    (in_bom yes) (on_board yes) (dnp no) (fields_autoplaced)
+    (property "Reference" "J9" (at 196.85 154.94 0)
+      (effects (font (size 1.27 1.27)) (justify left))
+    )
+    (property "Value" "Conn_01x04" (at 196.85 157.48 0)
+      (effects (font (size 1.27 1.27)) (justify left))
+    )
+    (property "Footprint" "Frooastboard Footprints:PinHeader_1x04_P1.27mm_Vertical" (at 194.31 154.94 0)
+      (effects (font (size 1.27 1.27)) hide)
+    )
+    (property "Datasheet" "~" (at 194.31 154.94 0)
+      (effects (font (size 1.27 1.27)) hide)
+    )
+    (pin "1")
+    (pin "2")
+    (pin "3")
+    (pin "4")
+    (instances
+      (project "Frooastboard Modular"
+        (path "/9ee55997-d93e-462c-b474-dae14d38ea26"
+          (reference "J9") (unit 1)
+        )
+      )
+    )
+  )
   (symbol (lib_id "power:+3.3V") (at 109.855 180.34 0) (unit 1)
     (in_bom yes) (on_board yes) (dnp no) (fields_autoplaced)
@@
         )
       )
+    )
+  )
+  (symbol (lib_id "power:+3.3V") (at 186.69 152.4 90) (unit 1)
+    (in_bom yes) (on_board yes) (dnp no)
+    (property "Reference" "#PWR031" (at 190.5 152.4 0)
+      (effects (font (size 1.27 1.27)) hide)
+    )
+    (property "Value" "+3.3V" (at 177.8 152.4 90)
+      (effects (font (size 1.27 1.27)) (justify right))
+    )
+    (property "Footprint" "" (at 186.69 152.4 0)
+      (effects (font (size 1.27 1.27)) hide)
+    )
+    (property "Datasheet" "" (at 186.69 152.4 0)
+      (effects (font (size 1.27 1.27)) hide)
+    )
+    (pin "1")
+    (instances
+      (project "Frooastboard Modular"
+        (path "/9ee55997-d93e-462c-b474-dae14d38ea26"
+          (reference "#PWR031") (unit 1)
+        )
+      )
+      (project "Frooastboard Walnut Modular"
+        (path "/e63e39d7-6ac0-4ffd-8aa3-1841a4541b55"
+          (reference "#PWR0119") (unit 1)
+        )
+        (path "/e63e39d7-6ac0-4ffd-8aa3-1841a4541b55/eba7bed6-3b4a-4b7a-b4a2-784017f24fe8"
+          (reference "#PWR019") (unit 1)
+        )
+      )

Commit message: somewhat good
Connections:
- net +3V3: now also J9.4 (Pin_4); no longer J9.1 (Pin_1)
- net GND: now also J9.1 (Pin_1); no longer J9.4 (Pin_4)
- net GPIO_1: now also J9.3 (Pin_3); no longer J9.2 (Pin_2)
- net GPIO_2: now also J9.2 (Pin_2); no longer J9.3 (Pin_3)
Changed lines of the file:
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@@
     )
   )
-  (global_label "GPIO_1" (shape input) (at 186.69 154.94 180) (fields_autoplaced)
+  (global_label "GPIO_1" (shape input) (at 186.69 157.48 180) (fields_autoplaced)
     (effects (font (size 1.27 1.27)) (justify right))
-    (property "Intersheetrefs" "${INTERSHEET_REFS}" (at 177.1318 154.94 0)
+    (property "Intersheetrefs" "${INTERSHEET_REFS}" (at 177.1318 157.48 0)
       (effects (font (size 1.27 1.27)) (justify right) hide)
     )
@@
     )
   )
-  (global_label "GPIO_2" (shape input) (at 186.69 157.48 180) (fields_autoplaced)
+  (global_label "GPIO_2" (shape input) (at 186.69 154.94 180) (fields_autoplaced)
     (effects (font (size 1.27 1.27)) (justify right))
-    (property "Intersheetrefs" "${INTERSHEET_REFS}" (at 177.1318 157.48 0)
+    (property "Intersheetrefs" "${INTERSHEET_REFS}" (at 177.1318 154.94 0)
       (effects (font (size 1.27 1.27)) (justify right) hide)
     )
@@
     )
   )
-  (symbol (lib_id "power:GND") (at 186.69 160.02 270) (unit 1)
-    (in_bom yes) (on_board yes) (dnp no) (fields_autoplaced)
-    (property "Reference" "#PWR032" (at 180.34 160.02 0)
-      (effects (font (size 1.27 1.27)) hide)
-    )
-    (property "Value" "GND" (at 182.88 160.0199 90)
+  (symbol (lib_id "power:GND") (at 186.69 152.4 270) (unit 1)
+    (in_bom yes) (on_board yes) (dnp no) (fields_autoplaced)
+    (property "Reference" "#PWR032" (at 180.34 152.4 0)
+      (effects (font (size 1.27 1.27)) hide)
+    )
+    (property "Value" "GND" (at 182.88 152.3999 90)
       (effects (font (size 1.27 1.27)) (justify right))
     )
-    (property "Footprint" "" (at 186.69 160.02 0)
-      (effects (font (size 1.27 1.27)) hide)
-    )
-    (property "Datasheet" "" (at 186.69 160.02 0)
+    (property "Footprint" "" (at 186.69 152.4 0)
+      (effects (font (size 1.27 1.27)) hide)
+    )
+    (property "Datasheet" "" (at 186.69 152.4 0)
       (effects (font (size 1.27 1.27)) hide)
     )
@@
     )
   )
-  (symbol (lib_id "power:+3.3V") (at 186.69 152.4 90) (unit 1)
+  (symbol (lib_id "power:+3.3V") (at 186.69 160.02 90) (unit 1)
     (in_bom yes) (on_board yes) (dnp no)
-    (property "Reference" "#PWR031" (at 190.5 152.4 0)
-      (effects (font (size 1.27 1.27)) hide)
-    )
-    (property "Value" "+3.3V" (at 177.8 152.4 90)
+    (property "Reference" "#PWR031" (at 190.5 160.02 0)
+      (effects (font (size 1.27 1.27)) hide)
+    )
+    (property "Value" "+3.3V" (at 177.8 160.02 90)
       (effects (font (size 1.27 1.27)) (justify right))
     )
-    (property "Footprint" "" (at 186.69 152.4 0)
-      (effects (font (size 1.27 1.27)) hide)
-    )
-    (property "Datasheet" "" (at 186.69 152.4 0)
-      (effects (font (size 1.27 1.27)) hide)
-    )
+    (property "Footprint" "" (at 186.69 160.02 0)
+      (effects (font (size 1.27 1.27)) hide)
+    )
+    (property "Datasheet" "" (at 186.69 160.02 0)
+      (effects (font (size 1.27 1.27)) hide)
+    )
