File: Frooastboard Modular/Kicad Project/Frooastboard Modular.kicad_sch (KiCad schematic)
At the start: 42 parts, among them J1 Conn_01x08, J2 Conn_01x06, J3 Conn_01x06, J4 Conn_01x10, J5 Conn_01x12, J6 SW Interface, J7 Conn_01x04, J8 Conn_01x08, J9 Conn_01x04, U1 IS31FL3733-QF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

Commit message: some stuff
Connections:
- net SW1: now reaches J2.1 (Pin_1), U1.2 (SW1)
- net SW2: now reaches J2.2 (Pin_2), U1.3 (SW2)
- net SW3: now reaches J2.3 (Pin_3), U1.4 (SW3)
- net SW4: now reaches J2.4 (Pin_4), U1.6 (SW4)
- net SW5: now reaches J2.5 (Pin_5), U1.7 (SW5)
- net SW6: now reaches J2.6 (Pin_6), U1.8 (SW6)
- net SW7: now reaches J3.1 (Pin_1), U1.9 (SW7)
- net SW8: now reaches J3.2 (Pin_2), U1.10 (SW8)
- net SW9: now reaches J3.3 (Pin_3), U1.11 (SW9)
- net SW10: now reaches J3.4 (Pin_4), U1.13 (SW10)
- net SW11: now reaches J3.5 (Pin_5), U1.14 (SW11)
- net SW12: now reaches J3.6 (Pin_6), U1.15 (SW12)
- net CS1: now reaches J8.1 (Pin_1), U1.16 (CS1)
- net CS2: now reaches J8.2 (Pin_2), U1.17 (CS2)
- net CS3: now reaches J8.3 (Pin_3), U1.18 (CS3)
- net CS4: now reaches J8.4 (Pin_4), U1.19 (CS4)
- net CS5: now reaches J8.5 (Pin_5), U1.21 (CS5)
- net CS6: now reaches J8.6 (Pin_6), U1.22 (CS6)
- net CS7: now reaches J8.7 (Pin_7), U1.23 (CS7)
- net CS8: now reaches J8.8 (Pin_8), U1.24 (CS8)
- net CS9: now reaches J1.1 (Pin_1), U1.25 (CS9)
- net CS10: now reaches J1.2 (Pin_2), U1.26 (CS10)
- net CS11: now reaches J1.3 (Pin_3), U1.27 (CS11)
- net CS12: now reaches J1.4 (Pin_4), U1.28 (CS12)
- net CS13: now reaches J1.5 (Pin_5), U1.30 (CS13)
- net CS14: now reaches J1.6 (Pin_6), U1.31 (CS14)
- net CS15: now reaches J1.7 (Pin_7), U1.32 (CS15)
- net CS16: now reaches J1.8 (Pin_8), U1.33 (CS16)
Changed lines of the file:
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@@
     (stroke (width 0) (type default))
   )
+  (label "SW3" (at 83.82 237.49 0) (fields_autoplaced)
+    (effects (font (size 1.27 1.27)) (justify left bottom))
+  )
+  (label "CS8" (at 83.82 207.01 0) (fields_autoplaced)
+    (effects (font (size 1.27 1.27)) (justify left bottom))
+  )
+  (label "CS4" (at 83.82 196.85 0) (fields_autoplaced)
+    (effects (font (size 1.27 1.27)) (justify left bottom))
+  )
+  (label "SW5" (at 83.82 242.57 0) (fields_autoplaced)
+    (effects (font (size 1.27 1.27)) (justify left bottom))
+  )
+  (label "CS12" (at 83.82 217.17 0) (fields_autoplaced)
+    (effects (font (size 1.27 1.27)) (justify left bottom))
+  )
+  (label "SW2" (at 83.82 234.95 0) (fields_autoplaced)
+    (effects (font (size 1.27 1.27)) (justify left bottom))
+  )
+  (label "CS6" (at 83.82 201.93 0) (fields_autoplaced)
+    (effects (font (size 1.27 1.27)) (justify left bottom))
+  )
+  (label "SW12" (at 83.82 260.35 0) (fields_autoplaced)
+    (effects (font (size 1.27 1.27)) (justify left bottom))
+  )
+  (label "SW8" (at 83.82 250.19 0) (fields_autoplaced)
+    (effects (font (size 1.27 1.27)) (justify left bottom))
+  )
+  (label "SW6" (at 83.82 245.11 0) (fields_autoplaced)
+    (effects (font (size 1.27 1.27)) (justify left bottom))
+  )
+  (label "SW7" (at 83.82 247.65 0) (fields_autoplaced)
+    (effects (font (size 1.27 1.27)) (justify left bottom))
+  )
   (label "DN" (at 185.42 130.81 0) (fields_autoplaced)
+    (effects (font (size 1.27 1.27)) (justify left bottom))
+  )
+  (label "SW1" (at 83.82 232.41 0) (fields_autoplaced)
     (effects (font (size 1.27 1.27)) (justify left bottom))
   )
@@
     (effects (font (size 1.27 1.27)) (justify left bottom))
   )
+  (label "CS5" (at 83.82 199.39 0) (fields_autoplaced)
+    (effects (font (size 1.27 1.27)) (justify left bottom))
+  )
+  (label "SW4" (at 83.82 240.03 0) (fields_autoplaced)
+    (effects (font (size 1.27 1.27)) (justify left bottom))
+  )
   (label "QSPI_CS_TP" (at 175.26 39.37 0) (fields_autoplaced)
     (effects (font (size 1.27 1.27)) (justify left bottom))
   )
+  (label "CS10" (at 83.82 212.09 0) (fields_autoplaced)
+    (effects (font (size 1.27 1.27)) (justify left bottom))
+  )
+  (label "CS13" (at 83.82 219.71 0) (fields_autoplaced)
+    (effects (font (size 1.27 1.27)) (justify left bottom))
+  )
+  (label "CS9" (at 83.82 209.55 0) (fields_autoplaced)
+    (effects (font (size 1.27 1.27)) (justify left bottom))
+  )
+  (label "CS16" (at 83.82 227.33 0) (fields_autoplaced)
+    (effects (font (size 1.27 1.27)) (justify left bottom))
+  )
+  (label "CS14" (at 83.82 222.25 0) (fields_autoplaced)
+    (effects (font (size 1.27 1.27)) (justify left bottom))
+  )
+  (label "CS11" (at 83.82 214.63 0) (fields_autoplaced)
+    (effects (font (size 1.27 1.27)) (justify left bottom))
+  )
+  (label "CS2" (at 83.82 191.77 0) (fields_autoplaced)
+    (effects (font (size 1.27 1.27)) (justify left bottom))
+  )
+  (label "SW10" (at 83.82 255.27 0) (fields_autoplaced)
+    (effects (font (size 1.27 1.27)) (justify left bottom))
+  )
+  (label "CS3" (at 83.82 194.31 0) (fields_autoplaced)
+    (effects (font (size 1.27 1.27)) (justify left bottom))
+  )
+  (label "CS7" (at 83.82 204.47 0) (fields_autoplaced)
+    (effects (font (size 1.27 1.27)) (justify left bottom))
+  )
+  (label "SW11" (at 83.82 257.81 0) (fields_autoplaced)
+    (effects (font (size 1.27 1.27)) (justify left bottom))
+  )
+  (label "CS1" (at 83.82 189.23 0) (fields_autoplaced)
+    (effects (font (size 1.27 1.27)) (justify left bottom))
+  )
+  (label "CS15" (at 83.82 224.79 0) (fields_autoplaced)
+    (effects (font (size 1.27 1.27)) (justify left bottom))
+  )
+  (label "SW9" (at 83.82 252.73 0) (fields_autoplaced)
+    (effects (font (size 1.27 1.27)) (justify left bottom))
+  )

Commit message: do some stuff
Parts:
- removed J9: Conn_01x04, Frooastboard Footprints:PinHeader_1x04_P1.27mm_Vertical, symbol Connector_Generic:Conn_01x04
- added J10: Conn_01x02, Frooastboard Footprints:PinHeader_1x02_P1.27mm_Vertical, symbol Connector_Generic:Conn_01x02
- added J9: Conn_01x05, Frooastboard Footprints:PinHeader_1x05_P1.27mm_Vertical, symbol Connector_Generic:Conn_01x05
Connections:
- net +3V3: now also J10.2 (Pin_2), J9.4 (Pin_4)
- net +5V: now also J9.5 (Pin_5)
- net GND: now also J10.1 (Pin_1), J9.1 (Pin_1)
- net GPIO_1: now also J9.3 (Pin_3)
- net GPIO_2: now also J9.2 (Pin_2)
Changed lines of the file:
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@@
+    (stroke (width 0) (type default))
+  )
+  (wire (pts (xy 186.69 162.56) (xy 189.23 162.56))
     (stroke (width 0) (type default))
   )
@@
     (stroke (width 0) (type default))
   )
+  (wire (pts (xy 186.69 173.99) (xy 189.23 173.99))
+    (stroke (width 0) (type default))
+  )
   (wire (pts (xy 48.26 214.63) (xy 45.72 214.63))
     (stroke (width 0) (type default))
@@
   )
   (wire (pts (xy 90.17 72.39) (xy 92.71 72.39))
+    (stroke (width 0) (type default))
+  )
+  (wire (pts (xy 186.69 171.45) (xy 189.23 171.45))
     (stroke (width 0) (type default))
   )
@@
     )
   )
+  (symbol (lib_id "Connector_Generic:Conn_01x05") (at 194.31 157.48 0) (unit 1)
+    (in_bom yes) (on_board yes) (dnp no) (fields_autoplaced)
+    (property "Reference" "J9" (at 196.85 156.21 0)
+      (effects (font (size 1.27 1.27)) (justify left))
+    )
+    (property "Value" "Conn_01x05" (at 196.85 158.75 0)
+      (effects (font (size 1.27 1.27)) (justify left))
+    )
+    (property "Footprint" "Frooastboard Footprints:PinHeader_1x05_P1.27mm_Vertical" (at 194.31 157.48 0)
+      (effects (font (size 1.27 1.27)) hide)
+    )
+    (property "Datasheet" "~" (at 194.31 157.48 0)
+      (effects (font (size 1.27 1.27)) hide)
+    )
+    (pin "1")
+    (pin "2")
+    (pin "3")
+    (pin "4")
+    (pin "5")
+    (instances
+      (project "Frooastboard Modular"
+        (path "/9ee55997-d93e-462c-b474-dae14d38ea26"
+          (reference "J9") (unit 1)
+        )
+      )
+    )
+  )
   (symbol (lib_id "Device:C_Small") (at 187.96 82.55 0) (unit 1)
     (in_bom yes) (on_board yes) (dnp no) (fields_autoplaced)
@@
     )
   )
+  (symbol (lib_id "Connector_Generic:Conn_01x02") (at 194.31 171.45 0) (unit 1)
+    (in_bom yes) (on_board yes) (dnp no) (fields_autoplaced)
+    (property "Reference" "J10" (at 196.85 171.45 0)
+      (effects (font (size 1.27 1.27)) (justify left))
+    )
+    (property "Value" "Conn_01x02" (at 196.85 173.99 0)
+      (effects (font (size 1.27 1.27)) (justify left))
+    )
+    (property "Footprint" "Frooastboard Footprints:PinHeader_1x02_P1.27mm_Vertical" (at 194.31 171.45 0)
+      (effects (font (size 1.27 1.27)) hide)
+    )
+    (property "Datasheet" "~" (at 194.31 171.45 0)
+      (effects (font (size 1.27 1.27)) hide)
+    )
+    (pin "1")
+    (pin "2")
+    (instances
+      (project "Frooastboard Modular"
+        (path "/9ee55997-d93e-462c-b474-dae14d38ea26"
+          (reference "J10") (unit 1)
+        )
+      )
+    )
+  )
   (symbol (lib_id "Device:R_Small") (at 182.88 39.37 90) (unit 1)
     (in_bom yes) (on_board yes) (dnp no) (fields_autoplaced)
@@
     )
   )
-  (symbol (lib_id "Connector_Generic:Conn_01x04") (at 194.31 154.94 0) (unit 1)
-    (in_bom yes) (on_board yes) (dnp no) (fields_autoplaced)
-    (property "Reference" "J9" (at 196.85 154.94 0)
-      (effects (font (size 1.27 1.27)) (justify left))
-    )
-    (property "Value" "Conn_01x04" (at 196.85 157.48 0)
-      (effects (font (size 1.27 1.27)) (justify left))
-    )
-    (property "Footprint" "Frooastboard Footprints:PinHeader_1x04_P1.27mm_Vertical" (at 194.31 154.94 0)
-      (effects (font (size 1.27 1.27)) hide)
-    )
-    (property "Datasheet" "~" (at 194.31 154.94 0)
-      (effects (font (size 1.27 1.27)) hide)
-    )
-    (pin "1")
-    (pin "2")
-    (pin "3")
-    (pin "4")
-    (instances
-      (project "Frooastboard Modular"
-        (path "/9ee55997-d93e-462c-b474-dae14d38ea26"
-          (reference "J9") (unit 1)
+  (symbol (lib_id "power:+3.3V") (at 186.69 173.99 90) (unit 1)
+    (in_bom yes) (on_board yes) (dnp no)
+    (property "Reference" "#PWR035" (at 190.5 173.99 0)
+      (effects (font (size 1.27 1.27)) hide)
+    )
+    (property "Value" "+3.3V" (at 177.8 173.99 90)
+      (effects (font (size 1.27 1.27)) (justify right))
+    )
+    (property "Footprint" "" (at 186.69 173.99 0)
+      (effects (font (size 1.27 1.27)) hide)
+    )
+    (property "Datasheet" "" (at 186.69 173.99 0)
+      (effects (font (size 1.27 1.27)) hide)
+    )
+    (pin "1")
+    (instances
+      (project "Frooastboard Modular"
+        (path "/9ee55997-d93e-462c-b474-dae14d38ea26"
+          (reference "#PWR035") (unit 1)
+        )
+      )
+      (project "Frooastboard Walnut Modular"
+        (path "/e63e39d7-6ac0-4ffd-8aa3-1841a4541b55"
+          (reference "#PWR0119") (unit 1)
+        )
+        (path "/e63e39d7-6ac0-4ffd-8aa3-1841a4541b55/eba7bed6-3b4a-4b7a-b4a2-784017f24fe8"
+          (reference "#PWR019") (unit 1)
+        )
+      )
+    )
+  )
+  (symbol (lib_id "power:GND") (at 186.69 171.45 270) (unit 1)
+    (in_bom yes) (on_board yes) (dnp no) (fields_autoplaced)
+    (property "Reference" "#PWR034" (at 180.34 171.45 0)
+      (effects (font (size 1.27 1.27)) hide)
+    )
+    (property "Value" "GND" (at 182.88 171.4499 90)
+      (effects (font (size 1.27 1.27)) (justify right))
+    )
+    (property "Footprint" "" (at 186.69 171.45 0)
+      (effects (font (size 1.27 1.27)) hide)
+    )
+    (property "Datasheet" "" (at 186.69 171.45 0)
+      (effects (font (size 1.27 1.27)) hide)
+    )
+    (pin "1")
+    (instances
+      (project "Frooastboard Modular"
+        (path "/9ee55997-d93e-462c-b474-dae14d38ea26"
+          (reference "#PWR034") (unit 1)
+        )
+      )
+      (project "Frooastboard Walnut Modular"
+        (path "/e63e39d7-6ac0-4ffd-8aa3-1841a4541b55"
+          (reference "#PWR0120") (unit 1)
+        )
+        (path "/e63e39d7-6ac0-4ffd-8aa3-1841a4541b55/eba7bed6-3b4a-4b7a-b4a2-784017f24fe8"
+          (reference "#PWR020") (unit 1)
         )
       )
@@
         )
       )
+    )
+  )
+  (symbol (lib_name "+5V_1") (lib_id "power:+5V") (at 186.69 162.56 90) (unit 1)
+    (in_bom yes) (on_board yes) (dnp no) (fields_autoplaced)
+    (property "Reference" "#PWR033" (at 190.5 162.56 0)
+      (effects (font (size 1.27 1.27)) hide)
+    )
+    (property "Value" "+5V" (at 182.88 162.56 90)
+      (effects (font (size 1.27 1.27)) (justify left))
+    )
+    (property "Footprint" "" (at 186.69 162.56 0)
+      (effects (font (size 1.27 1.27)) hide)
+    )
+    (property "Datasheet" "" (at 186.69 162.56 0)
+      (effects (font (size 1.27 1.27)) hide)
+    )
+    (pin "1")
+    (instances
+      (project "Frooastboard Modular"
+        (path "/9ee55997-d93e-462c-b474-dae14d38ea26"
+          (reference "#PWR033") (unit 1)
+        )
+      )

Commit message: fix drc erc errors
Parts:
- added FID1, FID2: Fiducial, Fiducial:Fiducial_1mm_Mask2mm, symbol Mechanical:Fiducial
- added H1: MountingHole, Frooastboard Footprints:Two_Key_Holes, symbol Mechanical:MountingHole
- J6: symbol Connector:Conn_01x05_Male -> Connector:Conn_01x05_Pin
Connections:
- net +3V3 renamed +3.3V
Other:
- moved on the sheet: C1, C14, C2, C3, C4, R10, TP1, U3
