File: Frooastboard A600/Kicad Project/Frooastboard A600.kicad_pcb (KiCad board)
At the start: 2 copper layers, 319.1 x 128.6 mm, 207 parts, among them J1 PS2_5V, J3 SW Interface, J8 USB, Q1 BSS138, Q2 BSS138, U2 RP2040, U3 W25Q32JVZP, U4 LM317L_SOT-89, Y1 12MHz

Commit message: Add Ground Plane
Routing:
- net GND: track 728.7 -> 733.1 mm, vias 22 -> 32
- added copper zone on B.Cu, net GND
- added copper zone on F.Cu, net GND
Changed lines of the file:
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@@
 			(svgprecision 4)
 			(plotframeref no)
-			(viasonmask yes)
+			(viasonmask no)
 			(mode 1)
 			(useauxorigin no)
@@
 	)
 	(segment
+		(start 280.30375 30.95625)
+		(end 281.78125 30.95625)
+		(width 0.381)
+		(layer "F.Cu")
+		(net 2)
+	)
+	(segment
 		(start 302.1 32.4)
 		(end 302.1 31.6)
@@
 	)
 	(segment
+		(start 278.26 33)
+		(end 280.30375 30.95625)
+		(width 0.381)
+		(layer "F.Cu")
+		(net 2)
+	)
+	(segment
 		(start 307.8 14.7)
 		(end 221.3 14.7)
@@
 	)
 	(via
+		(at 282.575 41.275)
+		(size 0.56)
+		(drill 0.3)
+		(layers "F.Cu" "B.Cu")
+		(free yes)
+		(net 2)
+	)
+	(via
 		(at 301.8 30.2625)
 		(size 0.6)
@@
 	)
 	(via
+		(at 309.5625 41.275)
+		(size 0.56)
+		(drill 0.3)
+		(layers "F.Cu" "B.Cu")
+		(free yes)
+		(net 2)
+	)
+	(via
 		(at 305.810571 37.089429)
 		(size 0.6)
@@
 	)
 	(via
+		(at 311.94375 25.4)
+		(size 0.56)
+		(drill 0.3)
+		(layers "F.Cu" "B.Cu")
+		(free yes)
+		(net 2)
+	)
+	(via
 		(at 301.6 37.1)
 		(size 0.6)
@@
 	)
 	(via
+		(at 281.78125 30.95625)
+		(size 0.6)
+		(drill 0.35)
+		(layers "F.Cu" "B.Cu")
+		(net 2)
+	)
+	(via
+		(at 309.5625 38.1)
+		(size 0.56)
+		(drill 0.3)
+		(layers "F.Cu" "B.Cu")
+		(free yes)
+		(net 2)
+	)
+	(via
+		(at 299.24375 23.8125)
+		(size 0.56)
+		(drill 0.3)
+		(layers "F.Cu" "B.Cu")
+		(free yes)
+		(net 2)
+	)
+	(via
 		(at 295.7 28.3)
 		(size 0.6)
@@
 	)
 	(via
+		(at 312.7375 37.30625)
+		(size 0.56)
+		(drill 0.3)
+		(layers "F.Cu" "B.Cu")
+		(free yes)
+		(net 2)
+	)
+	(via
 		(at 296.4 41.3)
 		(size 0.6)
@@
 	)
 	(via
+		(at 282.575 26.9875)
+		(size 0.56)
+		(drill 0.3)
+		(layers "F.Cu" "B.Cu")
+		(free yes)
+		(net 2)
+	)
+	(via
 		(at 302.1 32.4)
 		(size 0.6)
@@
 	)
 	(via
+		(at 295.5 44.4)
+		(size 0.56)
+		(drill 0.3)
+		(layers "F.Cu" "B.Cu")
+		(free yes)
+		(net 2)
+	)
+	(via
 		(at 287.1 37.2)
 		(size 0.6)
@@
 	)
 	(via
+		(at 275.43125 38.1)
+		(size 0.56)
+		(drill 0.3)
+		(layers "F.Cu" "B.Cu")
+		(free yes)
+		(net 2)
+	)
+	(via
 		(at 308.1 37.1)
 		(size 0.6)
@@
 		(net 140)
 	)
+	(zone
+		(net 2)
+		(net_name "GND")
+		(layers "F&B.Cu")
+		(hatch edge 0.5)
+		(priority 4)
+		(connect_pads
+			(clearance 0.2)
+		)
+		(min_thickness 0.2)
+		(filled_areas_thickness no)
+		(fill yes
+			(thermal_gap 0.5)
+			(thermal_bridge_width 0.5)
+		)
+		(polygon
+			(pts
+				(xy 307.18125 26.9875) (xy 318.29375 26.9875) (xy 318.29375 34.925) (xy 307.18125 34.925)
+			)
+		)
+	)
+	(zone
+		(net 2)
+		(net_name "GND")
+		(layers "F&B.Cu")
+		(hatch edge 0.5)
+		(priority 2)
+		(connect_pads
+			(clearance 0.2)
+		)
+		(min_thickness 0.2)
+		(filled_areas_thickness no)
+		(fill yes
+			(thermal_gap 0.5)
+			(thermal_bridge_width 0.5)
+		)
+		(polygon
+			(pts
+				(xy 266.7 26.19375) (xy 284.1625 26.19375) (xy 284.1625 35.71875) (xy 266.7 35.71875)
+			)
+		)
+	)
+	(zone
+		(net 2)
+		(net_name "GND")
+		(layers "F&B.Cu")
+		(hatch edge 0.5)
+		(priority 1)
+		(connect_pads
+			(clearance 0.2)
+		)
+		(min_thickness 0.2)
+		(filled_areas_thickness no)
+		(fill yes
+			(thermal_gap 0.5)
+			(thermal_bridge_width 0.5)
+		)
+		(polygon
+			(pts
+				(xy 179.3875 14.2875) (xy 188.9125 14.2875) (xy 188.9125 38.89375) (xy 179.3875 38.89375)
+			)
+		)
+	)
+	(zone
+		(net 2)
+		(net_name "GND")
+		(layers "F&B.Cu")
+		(hatch edge 0.5)
+		(priority 3)
+		(connect_pads
+			(clearance 0.2)
+		)
+		(min_thickness 0.2)
+		(filled_areas_thickness no)
+		(fill yes
+			(thermal_gap 0.5)
+			(thermal_bridge_width 0.5)
+		)
+		(polygon
+			(pts
+				(xy 325.4375 55.5625) (xy 338.1375 55.5625) (xy 338.1375 64.29375) (xy 325.4375 64.29375)
+			)
+		)
+	)
+	(zone
+		(net 2)
+		(net_name "GND")
+		(layers "F&B.Cu")
+		(hatch edge 0.5)
+		(connect_pads yes
+			(clearance 0.2)
+		)
+		(min_thickness 0.2)
+		(filled_areas_thickness no)
+		(fill yes
+			(thermal_gap 0.5)
+			(thermal_bridge_width 0.5)
+		)
+		(polygon
+			(pts
+				(xy 25.4 12.7) (xy 342.9 12.7) (xy 342.9 139.7) (xy 25.4 139.7)
+			)
+		)
+	)
 )

Commit message: bug fixes
Parts:
- MX30: footprint MX_Solderable:MX-Solderable-8U -> MX_Solderable:MX-Solderable-7U
- MX52: footprint MX_Solderable:MX-Solderable-1U -> MX_Solderable:MX-Solderable-1.25U
- moved D35 19.1 mm to (242.9, 122.2)
- moved MX41 19.1 mm to (234.2, 128.6)
- moved MX52 19.0 mm to (255.6, 128.6)
- moved D44 19.0 mm to (264.3, 122.2)
- moved D25 9.53 mm to (164.3, 122.2)
- moved MX30 9.53 mm to (155.6, 128.6)
- moved USB1 2.95 mm to (184.2, 12.0)
- moved R11 2.40 mm to (182.0, 22.6)
- moved R12 1.71 mm to (186.2, 23.4), turned to -90 degrees
- moved R13 1.20 mm to (190.2, 25.3)
- moved D16 0.86 mm to (331.8, 90.5)
- moved R1 0.86 mm to (336.3, 90.4)
Connections:
- USB1 pad 5: RP_D+ -> RP_D-
- USB1 pad 6: RP_D- -> RP_D+
- USB1 pad 7: RP_D+ -> RP_D-
- USB1 pad 8: RP_D- -> RP_D+
Routing:
- net col4: track 496.7 -> 513.4 mm
- net col3: track 487.9 -> 501.8 mm
- net GND: track 733.1 -> 745.3 mm
- net col2: track 573.8 -> 564.3 mm
- net +5V: track 193.6 -> 197.1 mm
- net RP_D-: track 161.1 -> 159.5 mm
- net Net-(D16-A): track 102.4 -> 101.1 mm
- net Net-(C18-Pad1): track 1.64 -> 2.84 mm
- net Net-(USB1-CC1): track 1.93 -> 2.90 mm
- net RP_D+: track 160.7 -> 160.2 mm
- net Net-(USB1-CC2): track 2.35 -> 2.90 mm

Commit message: update afa24 pos
Parts:
- moved FPC2 76.1 mm to (260.2, 33.4)
Routing:
- net GND: track 745.3 -> 770.5 mm, vias 32 -> 36
- net +5V: track 197.1 -> 209.3 mm
- net RP_D-: track 159.5 -> 162.1 mm, vias 6 -> 4
- net RP_D+: track 160.2 -> 162.8 mm, vias 6 -> 4
- net CapsLock: track 288.5 -> 287.2 mm
- net row1: track 146.5 -> 147.3 mm

Commit message: move ralt
Parts:
- moved MX52 2.38 mm to (258.0, 128.6)
- moved D44 2.38 mm to (266.7, 122.2)
Routing:
- net col4: track 513.4 -> 511.0 mm
Changed lines of the file:
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@@
 	(footprint "MX_Solderable:MX-Solderable-1.25U"
 		(layer "F.Cu")
-		(at 255.5875 128.5875)
+		(at 257.96875 128.5875)
 		(property "Reference" "MX52"
 			(at 0 3.175 0)
@@
 	(footprint "Diode_SMD:D_0805_2012Metric"
 		(layer "B.Cu")
-		(at 264.31875 122.2375 -90)
+		(at 266.7 122.2375 -90)
 		(descr "Diode SMD 0805 (2012 Metric), square (rectangular) end terminal, IPC_7351 nominal, (Body size source: https://docs.google.com/spreadsheets/d/1BsfQQcO9C6DZCsRaXUlFlo91Tg2WpOkGARC1WS5S8t0/edit?usp=sharing), generated with kicad-footprint-generator")
 		(tags "diode")
@@
 	)
 	(segment
-		(start 264.31875 123.175)
-		(end 261.762 123.175)
+		(start 266.7 123.175)
+		(end 264.14325 123.175)
 		(width 0.2)
 		(layer "B.Cu")
@@
 	)
 	(segment
-		(start 261.762 123.175)
-		(end 261.4295 123.5075)
+		(start 264.14325 123.175)
+		(end 263.81075 123.5075)
 		(width 0.2)
 		(layer "B.Cu")
@@
 	)
 	(segment
-		(start 258.1275 123.5075)
-		(end 261.4295 123.5075)
+		(start 260.50875 123.5075)
+		(end 263.81075 123.5075)
 		(width 0.2)
 		(layer "B.Cu")
@@
 	)
 	(segment
+		(start 277.01875 118.26875)
+		(end 277.01875 107.15625)
+		(width 0.2)
+		(layer "F.Cu")
+		(net 132)
+	)
+	(segment
 		(start 134.14375 40.74425)
 		(end 134.1 40.788)
@@
 	)
 	(segment
-		(start 277.01875 115.09375)
-		(end 277.01875 107.15625)
+		(start 255.5875 119.0625)
+		(end 276.225 119.0625)
 		(width 0.2)
 		(layer "F.Cu")
@@
 	)
 	(segment
-		(start 277.01875 115.09375)
-		(end 277.01875 118.26875)
-		(width 0.2)
-		(layer "F.Cu")
-		(net 132)
-	)
-	(segment
 		(start 265.1125 50.00625)
 		(end 265.1125 43.65625)
@@
 	)
 	(segment
-		(start 251.8 120.46875)
-		(end 251.8 123.4)
-		(width 0.2)
-		(layer "F.Cu")
-		(net 132)
-	)
-	(segment
 		(start 265.1125 54.76875)
 		(end 265.1125 53.975)
@@
 	)
 	(segment
-		(start 276.225 119.0625)
-		(end 253.20625 119.0625)
-		(width 0.2)
-		(layer "F.Cu")
-		(net 132)
-	)
-	(segment
 		(start 122.2375 72.23125)
 		(end 122.2375 69.05625)
@@
 	)
 	(segment
-		(start 252.4125 119.85625)
-		(end 251.8 120.46875)
-		(width 0.2)
-		(layer "F.Cu")
-		(net 132)
-	)
-	(segment
 		(start 117.475 107.15625)
 		(end 117.475 101.6)
@@
 	)
 	(segment
-		(start 277.01875 118.26875)
-		(end 276.225 119.0625)
-		(width 0.2)
-		(layer "F.Cu")
-		(net 132)
-	)
-	(segment
 		(start 117.475 101.6)
 		(end 107.95 92.075)
@@
 	)
 	(segment
-		(start 253.20625 119.0625)
-		(end 252.4125 119.85625)
-		(width 0.2)
-		(layer "F.Cu")
-		(net 132)
-	)
-	(segment
 		(start 134.14375 40.48125)
 		(end 134.14375 40.74425)
@@
 	)
 	(segment
+		(start 254.18125 123.4)
+		(end 254.18125 120.46875)
+		(width 0.2)
+		(layer "F.Cu")
+		(net 132)
+	)
+	(segment
 		(start 112.7125 50.00625)
 		(end 112.7125 43.65625)
@@
 		(net 132)
 	)
+	(segment
+		(start 276.225 119.0625)
+		(end 277.01875 118.26875)
+		(width 0.2)
+		(layer "F.Cu")
+		(net 132)
+	)
+	(segment
+		(start 254.18125 120.46875)
+		(end 255.5875 119.0625)
+		(width 0.2)
+		(layer "F.Cu")
+		(net 132)
+	)
 	(via
 		(at 117.475 107.15625)
@@
 	)
 	(via
-		(at 251.8 123.4)
+		(at 254.18125 123.4)
 		(size 0.56)
 		(drill 0.3)
@@
 	)
 	(segment
-		(start 251.7775 123.4225)
-		(end 251.7775 126.0475)
+		(start 254.15875 123.4225)
+		(end 254.15875 126.0475)
+		(width 0.2)
+		(layer "B.Cu")
+		(net 132)
+	)
+	(segment
+		(start 254.15875 123.4225)
+		(end 254.18125 123.4)
 		(width 0.2)
 		(layer "B.Cu")
@@
 		(width 0.2)
 		(layer "B.Cu")
-		(net 132)
-	)
-	(segment
-		(start 251.8 123.4)
-		(end 251.7775 123.4225)
-		(width 0.2)
-		(layer "B.Cu")
