File: Frooastboard A600/Kicad Project/Frooastboard A600.kicad_pcb (KiCad board)
At the start: 2 copper layers, 319.1 x 128.6 mm, 207 parts, among them J1 PS2_5V, J3 SW Interface, J8 USB, Q1 BSS138, Q2 BSS138, U2 RP2040, U3 W25Q32JVZP, U4 LM317L_SOT-89, Y1 12MHz

Commit message: cutout
Parts:
- removed D16: ST_LED2, Frooastboard Footprints:LED_RGB_SMD_6028_Reverse
- removed D26: ST_LED1, Frooastboard Footprints:LED_RGB_SMD_6028_Reverse
- removed D6: ST_LED3, Frooastboard Footprints:LED_RGB_SMD_6028_Reverse
- removed R1, R15, R3: 1k, Resistor_SMD:R_0805_2012Metric
Routing:
- net Net-(D6-A): track 119.2 -> 59.6 mm, vias 5 -> 4
- net GND: track 742.1 -> 688.3 mm, vias 47 -> 44
- net Net-(D16-A): track 101.1 -> 61.6 mm, vias 5 -> 4
- net Net-(D26-A): track 84.6 -> 63.5 mm, vias 5 -> 4
- net Net-(D16-K): track 2.66 -> 0.00 mm
- net Net-(D6-K): track 2.65 -> 0.00 mm
- net Net-(D26-K): track 2.60 -> 0.00 mm
Other:
- outline, holes or cut-outs redrawn

Commit message: plate and afa01
Parts:
- D1, D10, D100, D101, D102, D103, D104, D105, D106, D107, D11, D12, D13, D14, D15, D17, D18, D19, D2, D20, D21, D22, D23, D24, D25, D27, D28, D29, D3, D30, D31, D32, D33, D34, D35, D36, D37, D38, D39, D4, D40, D41, D42, D43, D44, D45, D46, D47, D48, D49, D5, D50, D51, D52, D54, D55, D56, D58, D59, D60, D61, D63, D67, D68, D69, D7, D70, D72, D8, D9, D92, D93, D94, D95, D96, D97, D98, D99: footprint Diode_SMD:D_0805_2012Metric -> Diode_SMD:D_SOD-323
- FPC1, FPC2, FPC4: footprint AFA24-SXXFIA-HF:FPC-SMD_4P-P1.00_AFA24-S04FIA-HF -> AFA01-SXXFCX-00:FPC-SMD_4P-P1.00_AFA01-S04FCC-00

Commit message: move resistor for easy led access
also move to linux
Parts:
- moved R16 6.02 mm to (60.3, 99.2), turned to 180 degrees
Routing:
- net GND: track 688.3 -> 681.6 mm
- net Net-(D53-K): track 2.64 -> 6.50 mm
